File: 05_PCB/_DEV_EC11_button_breakout/EC11BREAKOUT.kicad_sch (KiCad schematic)
At the start: 19 parts, among them J1 Conn_01x04_Pin, J2 Conn_01x04_Pin, SW1 EC11_Rotary_Encoder, SW2 SW_Push_LED, U1 74HC14

Commit message: added all datasheets
Other:
- note added: "KNOB_A, KNOB_B, KNOB_SW, SW -> GPIO Inputs on the MCP23017 LED from the 74HCT595"
- company: (none) -> CAPSTONE
- title: (none) -> EC11 and pushbutton hardware debounce
Changed lines of the file:
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@@
 	(generator_version "10.0")
 	(paper "A4")
+	(title_block
+		(title "EC11 and pushbutton hardware debounce")
+		(date "2026-08-04")
+		(company "CAPSTONE")
+		(comment 1 "Engineer: Skylar Denno")
+	)
+	(text "KNOB_A, KNOB_B, KNOB_SW, SW -> GPIO Inputs on the MCP23017\nLED from the 74HCT595\n"
+		(exclude_from_sim no)
+		(at 219.202 149.352 0)
+		(effects
+			(font
+				(size 2.032 2.032)
+			)
+		)
+	)
 	(junction
 		(at 54.61 68.58)
