File: 06_PCB/led_ring/led_ring_rev1_KICAD/led_ring_rev1.kicad_sch (KiCad schematic)
At the start: 104 parts, among them J1 DATA, J2 POW, U1 74HCT595PW, U2 74HCT595PW, U3 74HCT595PW, U4 74HCT595PW

Commit message: more stuff
Parts:
- C1, C2, C3, C4: value 1u -> 100n; LCSC C14445 -> C1525
- C5: LCSC C15525 -> C386033
- R1, R10, R11, R12, R13, R14, R15, R16, R17, R18, R19, R2, R20, R21, R22, R23, R24, R25, R26, R27, R28, R29, R3, R30, R31, R32, R4, R5, R6, R7, R8, R9: value 470 -> 560; LCSC C295802 -> C295808
