File: 06_PCB/CHANNEL_STRIP_LL/CHANNEL_STRIP_LL.kicad_sch (KiCad schematic)
At the start: 172 parts, among them J1 Conn_01x04_Socket, J10 Conn_01x04_Socket, J11 Conn_01x04_Socket, J12 Conn_01x04_Socket, J13 Conn_01x04_Socket, J14 Conn_01x04_Socket, J15 Conn_01x04_Socket, J16 Conn_01x04_Socket, J17 Conn_01x04_Socket, J18 Conn_01x04_Socket, J19 Conn_01x04_Socket, J2 Conn_01x04_Socket, J20 Conn_01x04_Socket, J21 Conn_01x04_Socket, J22 Conn_01x04_Socket, J23 Conn_01x04_Socket, J24 Conn_01x04_Socket, J25 Conn_01x04_Socket, J26 Conn_01x04_Socket, J27 Conn_01x04_Socket, J28 Conn_01x04_Socket, J29 Conn_01x04_Socket, J3 Conn_01x04_Socket, J30 Conn_01x04_Socket, J31 Conn_01x04_Socket, J32 Conn_01x04_Socket, J33 Conn_01x04_Socket, J34 Conn_01x04_Socket, J35 Conn_01x04_Socket, J36 Conn_01x04_Socket, J37 Conn_01x04_Socket, J38 Conn_01x04_Socket, J39 Conn_01x04_Socket, J4 Conn_01x04_Socket, J40 Conn_01x04_Socket, J41 Conn_01x04_Socket, J42 Conn_01x04_Socket, J43 Conn_01x04_Socket, J44 Conn_01x04_Socket, J45 Conn_01x04_Socket, J46 Conn_01x04_Socket, J47 Conn_01x04_Socket, J48 Conn_01x04_Socket, J49 Conn_01x04_Socket, J5 Conn_01x04_Socket, J50 Conn_01x04_Socket, J51 Conn_01x04_Socket, J52 Conn_01x04_Socket, J53 Conn_01x04_Socket, J54 Conn_01x04_Socket, J55 Conn_01x04_Socket, J56 Conn_01x04_Socket, J57 Conn_01x04_Socket, J58 Conn_01x04_Socket, J59 Conn_01x04_Socket, J6 Conn_01x04_Socket, J60 Conn_01x04_Socket, J61 Conn_01x04_Socket, J62 Conn_01x04_Socket, J63 Conn_01x04_Socket, J64 Conn_01x04_Socket, J65 Conn_01x04_Socket, J66 Conn_01x04_Socket, J67 Conn_01x04_Socket, J68 Conn_01x04_Socket, J69 Conn_01x04_Socket, J7 Conn_01x04_Socket, J70 Conn_01x04_Socket, J71 Conn_01x04_Socket, J72 Conn_01x04_Socket, J73 Conn_01x04_Socket, J74 Conn_01x04_Socket, J75 Conn_01x04_Socket, J76 Conn_01x04_Socket, J77 Conn_01x04_Socket, J78 Conn_01x04_Socket, J79 Conn_01x04_Socket, J8 Conn_01x04_Socket, J80 Conn_01x04_Socket, J9 Conn_01x04_Socket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

Commit message: stuff and things idk
Parts:
- removed C1, C11, C13, C15, C17, C19, C21, C23, C25, C27, C29, C3, C31, C33, C35, C37, C39, C41, C43, C45, C47, C49, C5, C51, C53, C55, C57, C59, C61, C63, C65, C67, C69, C7, C71, C73, C75, C77, C79, C9: 10u, Capacitor_SMD:C_0603_1608Metric, symbol Device:C
- removed C10, C12, C14, C16, C18, C2, C20, C22, C24, C26, C28, C30, C32, C34, C36, C38, C4, C40, C42, C44, C46, C48, C50, C52, C54, C56, C58, C6, C60, C62, C64, C66, C68, C70, C72, C74, C76, C78, C8, C80: 100n, Capacitor_SMD:C_0402_1005Metric, symbol Device:C
