File: 06_PCB/PSU/PSU_KICAD/PSU.kicad_pcb (KiCad board)
At the start: 4 copper layers, 190 x 160 mm, 98 parts, among them J10 SMPS_IN, J11 D/C_CAP3, J12 D/C_CAP2, J13 D/C_CAP1, J2 OUT_ANLG, J3 MAINS_IN, J4 T1_PRI, J5 T1_SEC, J6 GND_LIFT, J7 FAN1_12V, J8 FAN2_12V, J9 OUT_DIGI, U1 LM317AT/NOPB, U2 LM337T/NOPB, U3 LD1117V33C, U5 3V3 URB2403LD-20WR3, U6 MeanWell NID-100-5, U7 12V URB2412LD-50WR3

Commit message: fixed some dum dum stuff on the psu lol
Connections:
- C16 pad 2: Net-(J10-Pin_2) -> Net-(D10-K)
- C17 pad 2: Net-(J10-Pin_2) -> Net-(D10-K)
- C18 pad 2: Net-(C18-Pad2) -> Net-(D10-K)
- C19 pad 2: Net-(C18-Pad2) -> Net-(D10-K)
- C20 pad 2: Net-(C20-Pad2) -> Net-(D10-K)
- C21 pad 2: Net-(C20-Pad2) -> Net-(D10-K)
- D5 pad 3: Net-(D5--) -> Net-(D5-Pad3)
- J10 pad 2: Net-(J10-Pin_2) -> Net-(D10-K)
- TR2 pad 5: Net-(D5--) -> Net-(D5-Pad3)
- TR2 pad 7: Net-(D5--) -> Net-(D5-Pad3)
Routing:
- net Net-(D5-Pad3): track 0.00 -> 37.9 mm
- net Net-(D10-K): track 393.0 -> 429.5 mm
- net Net-(J10-Pin_2): track 24.2 -> 0.00 mm
- net Net-(C18-Pad2): track 12.3 -> 0.00 mm
- net Net-(C20-Pad2): track 11.7 -> 0.00 mm
Changed lines of the file:
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@@
 			(layers "*.Cu" "*.Mask")
 			(remove_unused_layers no)
-			(net "Net-(J10-Pin_2)")
+			(net "Net-(D10-K)")
 			(pintype "passive")
 		)
@@
 			(layers "*.Cu" "*.Mask")
 			(remove_unused_layers no)
-			(net "Net-(D5--)")
+			(net "Net-(D5-Pad3)")
 			(pinfunction "5_5")
 			(pintype "passive")
@@
 			(layers "*.Cu" "*.Mask")
 			(remove_unused_layers no)
-			(net "Net-(D5--)")
+			(net "Net-(D5-Pad3)")
 			(pinfunction "7_7")
 			(pintype "passive")
@@
 			(layers "*.Cu" "*.Mask")
 			(remove_unused_layers no)
-			(net "Net-(C18-Pad2)")
+			(net "Net-(D10-K)")
 			(pintype "passive")
 		)
@@
 			(layers "*.Cu" "*.Mask")
 			(remove_unused_layers no)
-			(net "Net-(D5--)")
+			(net "Net-(D5-Pad3)")
 			(pintype "passive")
 		)
@@
 			(layers "*.Cu" "*.Mask")
 			(remove_unused_layers no)
-			(net "Net-(J10-Pin_2)")
+			(net "Net-(D10-K)")
 			(pinfunction "Pin_2_2")
 			(pintype "passive")
@@
 			(layers "*.Cu" "*.Mask")
 			(remove_unused_layers no)
-			(net "Net-(C20-Pad2)")
+			(net "Net-(D10-K)")
 			(pintype "passive")
 		)
@@
 			(layers "*.Cu" "*.Mask")
 			(remove_unused_layers no)
-			(net "Net-(J10-Pin_2)")
+			(net "Net-(D10-K)")
 			(pintype "passive")
 		)
@@
 			(layers "*.Cu" "*.Mask")
 			(remove_unused_layers no)
-			(net "Net-(C20-Pad2)")
+			(net "Net-(D10-K)")
 			(pintype "passive")
 		)
@@
 			(layers "*.Cu" "*.Mask")
 			(remove_unused_layers no)
-			(net "Net-(C18-Pad2)")
+			(net "Net-(D10-K)")
 			(pintype "passive")
 		)
@@
 	)
 	(segment
+		(start 160.104773 168.865)
+		(end 155.965 168.865)
+		(width 1)
+		(layer "B.Cu")
+		(net "Net-(D1-A)")
+	)
+	(segment
+		(start 174.835633 183.451024)
+		(end 190.011261 168.275396)
+		(width 1)
+		(layer "B.Cu")
+		(net "Net-(D1-A)")
+	)
+	(segment
+		(start 174.835633 183.59586)
+		(end 160.104773 168.865)
+		(width 1)
+		(layer "B.Cu")
+		(net "Net-(D1-A)")
+	)
+	(segment
+		(start 177.844134 175.5)
+		(end 188.059978 175.5)
+		(width 1)
+		(layer "F.Cu")
+		(net "Net-(D2-A)")
+	)
+	(segment
+		(start 169.58 183.62)
+		(end 169.095 184.105)
+		(width 1)
+		(layer "F.Cu")
+		(net "Net-(D2-A)")
+	)
+	(segment
+		(start 169.724134 183.62)
+		(end 169.58 183.62)
+		(width 1)
+		(layer "F.Cu")
+		(net "Net-(D2-A)")
+	)
+	(segment
+		(start 169.724134 183.62)
+		(end 177.844134 175.5)
+		(width 1)
+		(layer "F.Cu")
+		(net "Net-(D2-A)")
+	)
+	(segment
+		(start 188.059978 175.5)
+		(end 195.179978 168.38)
+		(width 1)
+		(layer "F.Cu")
+		(net "Net-(D2-A)")
+	)
+	(segment
+		(start 169.095 184.105)
+		(end 155.965 184.105)
+		(width 1)
+		(layer "F.Cu")
+		(net "Net-(D2-A)")
+	)
+	(segment
 		(start 316.57358 96.320318)
 		(end 321.82358 101.570318)
@@
 		(width 2.5)
 		(layer "F.Cu")
-		(net "Net-(J10-Pin_2)")
+		(net "Net-(D10-K)")
 	)
 	(segment
@@
 		(width 1.7)
 		(layer "F.Cu")
-		(net "Net-(J10-Pin_2)")
-	)
-	(segment
-		(start 316 93.114416)
-		(end 316 100.746738)
-		(width 2.5)
-		(layer "F.Cu")
-		(net "Net-(J10-Pin_2)")
-	)
-	(segment
-		(start 318.685028 90.320318)
-		(end 322.930618 86.074728)
-		(width 2.5)
-		(layer "F.Cu")
-		(net "Net-(J10-Pin_2)")
-	)
-	(segment
-		(start 313.205902 90.320318)
-		(end 318.685028 90.320318)
-		(width 2.5)
-		(layer "F.Cu")
-		(net "Net-(J10-Pin_2)")
+		(net "Net-(D10-K)")
 	)
 	(segment
@@
 	)
 	(segment
+		(start 316 93.114416)
+		(end 316 100.746738)
+		(width 2.5)
+		(layer "F.Cu")
+		(net "Net-(D10-K)")
+	)
+	(segment
+		(start 318.685028 90.320318)
+		(end 322.930618 86.074728)
+		(width 2.5)
+		(layer "F.Cu")
+		(net "Net-(D10-K)")
+	)
+	(segment
+		(start 279.029861 202.937995)
+		(end 276.779862 205.187994)
+		(width 2.5)
+		(layer "F.Cu")
+		(net "Net-(D10-K)")
+	)
+	(segment
 		(start 262 90.5)
 		(end 268.1 90.5)
@@
 	)
 	(segment
+		(start 313.205902 90.320318)
+		(end 318.685028 90.320318)
+		(width 2.5)
+		(layer "F.Cu")
+		(net "Net-(D10-K)")
+	)
+	(segment
+		(start 279.029861 193.820318)
+		(end 279.029861 202.937995)
+		(width 2.5)
+		(layer "F.Cu")
+		(net "Net-(D10-K)")
+	)
+	(segment
 		(start 262 103.5)
 		(end 262 90.5)
@@
 	)
 	(segment
-		(start 177.844134 175.5)
-		(end 188.059978 175.5)
-		(width 1)
-		(layer "F.Cu")
-		(net "Net-(D2-A)")
-	)
-	(segment
-		(start 169.58 183.62)
-		(end 169.095 184.105)
-		(width 1)
-		(layer "F.Cu")
-		(net "Net-(D2-A)")
-	)
-	(segment
-		(start 169.724134 183.62)
-		(end 169.58 183.62)
-		(width 1)
-		(layer "F.Cu")
-		(net "Net-(D2-A)")
-	)
-	(segment
-		(start 169.724134 183.62)
-		(end 177.844134 175.5)
-		(width 1)
-		(layer "F.Cu")
-		(net "Net-(D2-A)")
-	)
-	(segment
-		(start 188.059978 175.5)
-		(end 195.179978 168.38)
-		(width 1)
-		(layer "F.Cu")
-		(net "Net-(D2-A)")
-	)
-	(segment
-		(start 169.095 184.105)
-		(end 155.965 184.105)
-		(width 1)
-		(layer "F.Cu")
-		(net "Net-(D2-A)")
-	)
-	(segment
 		(start 232.29 83)
 		(end 230.29 85)
@@
 	)
 	(segment
-		(start 222 211)
-		(end 212.640124 211)
+		(start 212.521889 210.881765)
+		(end 221.881765 210.881765)
 		(width 0.8)
 		(layer "F.Cu")
@@
 	)
 	(segment
-		(start 212.521889 210.881765)
-		(end 212.521889 220.881765)
+		(start 221.881765 210.881765)
+		(end 222 211)
+		(width 0.8)
+		(layer "F.Cu")
+		(net "Net-(D5-Pad2)")
+	)
+	(segment
+		(start 212.521889 220.881765)
+		(end 212.521889 210.881765)
 		(width 0.8)
 		(layer "F.Cu")
@@
 	)
 	(segment
-		(start 279.029861 202.937995)
-		(end 276.779862 205.187994)
-		(width 2.5)
-		(layer "F.Cu")
-		(net "Net-(C18-Pad2)")
-	)
-	(segment
-		(start 279.029861 193.820318)
-		(end 279.029861 202.937995)
-		(width 2.5)
-		(layer "F.Cu")
-		(net "Net-(C18-Pad2)")
-	)
-	(segment
 		(start 163.76 109.435)
 		(end 189.265515 134.940515)
@@
 	)
 	(segment
+		(start 232 228)
+		(end 232.000001 231.5375)
+		(width 0.8)
+		(layer "F.Cu")
+		(net "Net-(D11-K)")
+	)
+	(segment
 		(start 297.995902 232.120318)
 		(end 297.995902 228.602819)
@@
 	)
 	(segment
-		(start 278.779861 163.246358)
-		(end 276.455902 165.570317)
-		(width 2.5)
-		(layer "F.Cu")
-		(net "Net-(C20-Pad2)")
-	)
-	(segment
-		(start 278.779861 154.820318)
-		(end 278.779861 163.246358)
-		(width 2.5)
-		(layer "F.Cu")
-		(net "Net-(C20-Pad2)")
-	)
-	(segment
-		(start 160.104773 168.865)
-		(end 155.965 168.865)
-		(width 1)
-		(layer "B.Cu")
-		(net "Net-(D1-A)")
-	)
-	(segment
-		(start 174.835633 183.451024)
-		(end 190.011261 168.275396)
-		(width 1)
-		(layer "B.Cu")
-		(net "Net-(D1-A)")
-	)
-	(segment
-		(start 174.835633 183.59586)
-		(end 160.104773 168.865)
-		(width 1)
-		(layer "B.Cu")
-		(net "Net-(D1-A)")
-	)
-	(segment
 		(start 225.84 194.16)
 		(end 229 191)
@@
 	)
 	(segment
-		(start 232 228)
-		(end 232.000001 231.5375)
+		(start 212.521889 227.978111)
+		(end 222 218.5)
 		(width 0.8)
 		(layer "F.Cu")
-		(net "Net-(D11-K)")
+		(net "Net-(D5-Pad3)")
+	)
+	(segment
+		(start 212.521889 230.881765)
+		(end 212.521889 227.978111)
+		(width 0.8)
+		(layer "F.Cu")
+		(net "Net-(D5-Pad3)")
+	)
+	(segment
+		(start 217.59589 214.09589)
+		(end 217.59589 205.955766)
+		(width 0.8)
+		(layer "B.Cu")
+		(net "Net-(D5-Pad3)")
+	)
+	(segment
+		(start 217.59589 205.955766)
+		(end 212.521889 200.881765)
+		(width 0.8)
+		(layer "B.Cu")
+		(net "Net-(D5-Pad3)")
+	)
+	(segment
+		(start 222 218.5)
+		(end 217.59589 214.09589)
+		(width 0.8)
+		(layer "B.Cu")
+		(net "Net-(D5-Pad3)")
 	)
 	(zone
@@
 		(hatch edge 0.5)
 		(priority 1)
-		(connect_pads yes
+		(connect_pads
 			(clearance 0.5)
 		)

Commit message: upload proposal
Parts:
- removed the C16 at (313.2, 85.3)
- removed the C17 at (321.8, 101.6)
- removed J11: D/C_CAP3, Connector_PinHeader_2.54mm:PinHeader_1x02_P2.54mm_Vertical
- removed J12: D/C_CAP2, Connector_PinHeader_2.54mm:PinHeader_1x02_P2.54mm_Vertical
- removed J13: D/C_CAP1, Connector_PinHeader_2.54mm:PinHeader_1x02_P2.54mm_Vertical
- removed the L1 at (301.5, 100.3)
- removed the R1 at (156.8, 108.0)
- removed the R15 at (302.0, 87.0)
- removed R16: 0.33R, Resistor_THT:R_Axial_DIN0207_L6.3mm_D2.5mm_P10.16mm_Horizontal
- removed the R3 at (222.0, 173.8)
- R2: value 220 -> 56k; footprint Resistor_THT:R_Axial_DIN0414_L11.9mm_D4.5mm_P20.32mm_Horizontal -> Resistor_SMD:R_1206_3216Metric
- U2: renamed from U5; footprint Converter_DCDC:Converter_DCDC_XP_POWER_JTDxxxxxxx_THT -> My Footprints:urb 50w dc-dc
- moved R2 124.5 mm to (307.3, 92.0)
- moved D1 87.2 mm to (262.0, 142.5)
- moved C6 87.0 mm to (233.6, 213.3)
- moved C5 86.9 mm to (233.4, 192.0)
- moved C7 86.8 mm to (162.5, 145.8), turned to 0 degrees
- moved C4 82.2 mm to (162.5, 118.7), turned to 0 degrees
- moved C3 70.9 mm to (233.4, 168.9), turned to 0 degrees
- moved C2 69.9 mm to (219.6, 168.9)
- moved C1 60.2 mm to (262.2, 152.5)
- moved R1 60.2 mm to (262.2, 158.5)
- moved C10 57.1 mm to (191.6, 131.5), turned to -90 degrees
- moved C15 48.4 mm to (246.4, 154.4)
- moved C8 40.0 mm to (205.4, 95.6), turned to 180 degrees
- moved C16 32.0 mm to (199.5, 108.2)
- moved D9 28.4 mm to (183.9, 110.5)
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- renumbered C15 to C1, C13 to C10, C18 to C11, C20 to C12, C22 to C13, C7 to C14, C8 to C15, C14 to C16, C19 to C17, C21 to C18, C23 to C19, C1 to C2, C9 to C20, C10 to C21, C11 to C4, C2 to C5, C4 to C6, C12 to C7, C5 to C8, C6 to C9, D6 to D1, D1 to D2, D2 to D3, D3 to D4, D4 to D5, D5 to D6, J9 to J10, J3 to J2, J4 to J3, J10 to J4, J2 to J8, J8 to J9, L2 to L1, L3 to L2, L4 to L3, R4 to R1, R9 to R10, R10 to R11, R11 to R12, R12 to R13, R13 to R14, R14 to R15, R5 to R3, R6 to R4, R7 to R5, R8 to R6, R17 to R7, R18 to R8, R19 to R9, U6 to U3, U7 to U4, U1 to U5, U2 to U6, U3 to U7
Connections:
- C1 pad 1: Net-(D5--) -> Net-(D10-K)
- C1 pad 2: Net-(D10-K) -> Net-(D1-+)
- C10 pad 2: Net-(D5--) -> Net-(D10-K)
- C12 pad 1: Net-(U5-Enable) -> Net-(C12-Pad1)
- C13 pad 1: Net-(J7-Pin_2) -> Net-(U4-+VOUT)
- C14 pad 2: Net-(D5--) -> Net-(D10-K)
- C15 pad 1: Net-(D5--) -> Net-(D10-K)
- C16 pad 2: Net-(D5--) -> Net-(D10-K)
- C2 pad 1: Net-(D1-K) -> Net-(D2-K)
- C2 pad 2: Net-(D5--) -> Net-(D10-K)
- C20 pad 2: Net-(D5--) -> Net-(D10-K)
- C21 pad 1: Net-(D5--) -> Net-(D10-K)
- C3 pad 1: Net-(D1-K) -> Net-(D10-K)
- C3 pad 2: Net-(D5--) -> Net-(D4-A)
- C4 pad 2: Net-(D5--) -> Net-(D10-K)
- C5 pad 1: Net-(D5--) -> Net-(D2-K)
- C5 pad 2: Net-(D3-A) (its old number) -> Net-(D10-K)
- C6 pad 1: Net-(D5--) -> Net-(D10-K)
- C6 pad 2: Net-(D3-A) (its old number) -> Net-(D4-A)
- C7 pad 2: Net-(D5--) -> Net-(D10-K)
- C8 pad 2: Net-(D5--) -> Net-(D10-K)
- C9 pad 1: Net-(D5--) -> Net-(D10-K)
- D1 pad 1: Net-(D10-K) -> Net-(D1-+)
- D1 pad 2: Net-(D5--) -> Net-(D10-K)
- D1 pad 3: Net-(D5--) -> Net-(D10-K)
- D1 pad 4: Net-(D10-K) -> Net-(D1-+)
- D11 pad 1: Net-(D11-K) -> Net-(D10-K)
- D11 pad 2: Net-(D10-K) -> Net-(D11-A)
- D12 pad 1: Net-(D10-K) -> Net-(D12-K)
- D12 pad 2: Net-(D12-A) -> Net-(D10-K)
- D2 pad 1: Net-(D1-K) -> Net-(D2-K)
- D3 pad 1: Net-(D1-K) -> Net-(D2-K)
- D4 pad 2: Net-(D3-A) (its old number) -> Net-(D4-A)
- D5 pad 2: Net-(D3-A) (its old number) -> Net-(D4-A)
- D6 pad 4: Net-(D5--) -> Net-(D10-K)
- D7 pad 1: Net-(D1-K) -> Net-(D2-K)
- D8 pad 2: Net-(D3-A) (its old number) -> Net-(D4-A)
- H1 pad 1: Net-(D10-K) -> Net-(D1-+)
- J4 pad 1: Net-(J10-Pin_1) -> Net-(J4-Pin_1)
- J5 pad 2: Net-(D5--) -> Net-(D10-K)
- J5 pad 3: Net-(D5--) -> Net-(D10-K)
- J6 pad 1: Net-(D10-K) -> Net-(D1-+)
- J6 pad 2: Net-(D10-K) -> Net-(D1-+)
- J6 pad 3: Net-(D5--) -> Net-(D10-K)
- J7 pad 2: Net-(J7-Pin_2) -> /+10V_MOTORS
- J8 pad 1: /+18V -> /-18V
- J8 pad 2: Net-(D5--) -> Net-(D10-K)
- J8 pad 3: /-18V -> /+18V
- J9 pad 2: Net-(J7-Pin_2) -> /+10V_MOTORS
- L2 pad 1: Net-(U5-Enable) -> Net-(C12-Pad1)
- L3 pad 1: Net-(J7-Pin_2) -> Net-(U4-+VOUT)
- R1 pad 1: Net-(D10-K) -> Net-(D1-+)
- R1 pad 2: Net-(D5--) -> Net-(D10-K)
- R11 pad 2: Net-(D11-K) -> Net-(D12-K)
- R12 pad 2: Net-(D12-A) -> Net-(D11-A)
- R2 pad 1: Net-(J12-Pin_2) -> Net-(U4-Trim)
- R2 pad 2: Net-(D3-A) (its old number) -> Net-(U4-+VOUT)
- R3 pad 2: Net-(D5--) -> Net-(D10-K)
- R4 pad 1: Net-(D5--) -> Net-(D10-K)
- U2 pad 1: Net-(U5-Enable) -> unconnected-(U2-Enable-Pad1)
- U2 pad 3: Net-(U5-Vin) -> Net-(J4-Pin_1)
- U2 pad 5: unconnected-(U5-Trim-Pad5) -> Net-(D10-K)
- U2 pad 6: Net-(D10-K) -> unconnected-(U2-Trim-Pad6)
- U3 pad 1: Net-(U5-Enable) -> Net-(C12-Pad1)
- U3 pad 10: Net-(U5-Vin) -> Net-(J4-Pin_1)
- U3 pad 2: Net-(U5-Enable) -> Net-(C12-Pad1)
- U3 pad 3: Net-(U5-Enable) -> Net-(C12-Pad1)
- U3 pad 4: Net-(U5-Enable) -> Net-(C12-Pad1)
- U3 pad 9: Net-(U5-Vin) -> Net-(J4-Pin_1)
- U4 pad 1: Net-(U5-Enable) -> unconnected-(U4-Enable-Pad1)
- U4 pad 3: Net-(U5-Vin) -> Net-(J4-Pin_1)
- U4 pad 4: Net-(J7-Pin_2) -> Net-(U4-+VOUT)
- U4 pad 6: Net-(U7-Trim) -> Net-(U4-Trim)
- U5 pad 3: Net-(D1-K) -> Net-(D2-K)
- U6 pad 2: Net-(D3-A) (its old number) -> Net-(D4-A)
- U7 pad 1: Net-(D5--) -> Net-(D10-K)
Routing:
- net Net-(D10-K): track 429.5 -> 0.00 mm, vias 3 -> 0
- net /-18V: track 305.5 -> 0.90 mm, vias 1 -> 0
- net /+18V: track 225.4 -> 0.00 mm, vias 1 -> 0
- net /+3V3_REF: track 212.3 -> 0.00 mm
- net /+5V_LEDS: track 199.6 -> 0.00 mm
- net /+10V_MOTORS: track 186.7 -> 0.00 mm
- net /+3V3_LOGIC: track 184.8 -> 0.00 mm
- net Net-(J7-Pin_2): track 157.2 -> 0.00 mm
- net Net-(U5-Enable): track 144.9 -> 0.00 mm
- net Net-(D3-A) (its old number): track 137.4 -> 0.00 mm
- net Net-(D1-K): track 123.5 -> 0.00 mm, vias 1 -> 0
- net Net-(D6-+): track 114.9 -> 0.00 mm
- net Net-(U5-Vin): track 108.0 -> 0.00 mm
- net Net-(D6-Pad3): track 37.9 -> 0.00 mm
- net Net-(J10-Pin_1): track 33.1 -> 0.00 mm
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- removed copper zone on B.Cu, net Net-(D5--)
- removed copper zone on F.Cu, net Net-(D5--)
- removed copper zone on In1.Cu, net Net-(D5--)
- removed copper zone on In2.Cu, net Net-(D5--)
Other:
- board text added: "10v 5V 3V3 GND"
- board text added: "3V3 Ref +16V GND -16V"
- board text added: "Rev 2"
- board text removed: "3V3 Ref -16V GND +16V"
- board text removed: "GND 3V3 Logic 5V LEDs 10V Motors"
- board text removed: "Rev 0.2"

Commit message: stuff and things idk
Parts:
- removed the R2 at (307.3, 92.0)
- added C16: 1000u, Capacitor_THT:CP_Radial_D12.5mm_P5.00mm, F.Cu at (313.2, 85.3)
- added C17: 470u, Capacitor_THT:CP_Radial_D10.0mm_P5.00mm, F.Cu at (321.8, 101.6)
- added L1: 4.7u, Inductor_SMD:L_Vishay_IHLP-5050, F.Cu at (301.5, 100.3)
- added R15: 56k, Resistor_SMD:R_1206_3216Metric, F.Cu at (302.0, 87.0)
- added R16: 0.33R, Resistor_THT:R_Axial_DIN0207_L6.3mm_D2.5mm_P10.16mm_Horizontal, F.Cu at (311.2, 106.5)
- U5: renamed from U2; footprint My Footprints:urb 50w dc-dc -> Converter_DCDC:Converter_DCDC_XP_POWER_JTDxxxxxxx_THT
- moved C11 107.0 mm to (238.5, 194.0)
- moved C12 102.8 mm to (238.6, 214.9)
- moved C3 63.9 mm to (174.0, 145.2), turned to 180 degrees
- moved C1 63.9 mm to (174.0, 124.0)
- moved C14 54.7 mm to (254.0, 112.3)
- moved HS3 54.4 mm to (246.0, 110.0)
- moved U3 54.4 mm to (241.8, 107.5)
- moved D9 54.4 mm to (238.3, 110.9)
- moved C13 54.4 mm to (246.0, 131.8)
- moved C4 43.9 mm to (245.5, 171.0), turned to 180 degrees
- moved C2 29.3 mm to (213.0, 171.0)
- moved C8 26.3 mm to (220.1, 154.2)
- moved C7 26.2 mm to (193.0, 131.8)
- moved C9 26.1 mm to (204.0, 118.0)
- moved C10 26.0 mm to (210.0, 118.0)
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- renumbered C2 to C1, C21 to C10, C4 to C11, C7 to C12, C10 to C13, C16 to C14, C1 to C15, C11 to C18, C17 to C19, C5 to C2, C12 to C20, C18 to C21, C13 to C22, C19 to C23, C6 to C4, C8 to C5, C9 to C6, C14 to C7, C15 to C8, C20 to C9, D2 to D1, D3 to D2, D4 to D3, D5 to D4, D6 to D5, D1 to D6, J4 to J10, J8 to J2, J2 to J3, J3 to J4, J9 to J8, J10 to J9, L1 to L2, L2 to L3, L3 to L4, R7 to R1, R11 to R10, R12 to R11, R13 to R12, R14 to R13, R15 to R14, R8 to R2, R9 to R3, R1 to R4, R3 to R5, R4 to R6, R5 to R7, R6 to R8, R10 to R9, U5 to U1, U6 to U2, U7 to U3, U3 to U6, U4 to U7
Connections:
- C1 pad 1: Net-(D2-K) -> Net-(D1-K)
- C2 pad 1: Net-(D2-K) -> Net-(D10-K)
- C2 pad 2: Net-(D10-K) -> Net-(D3-A)
- C22 pad 1: Net-(U4-+VOUT) -> Net-(J7-Pin_2)
- C3 pad 1: Net-(D10-K) -> Net-(D1-K)
- C3 pad 2: Net-(D4-A) -> Net-(D10-K)
- C4 pad 2: Net-(D4-A) -> Net-(D3-A)
- D1 pad 1: Net-(D2-K) -> Net-(D1-K)
- D11 pad 1: Net-(D10-K) -> Net-(D11-K)
- D11 pad 2: Net-(D11-A) -> Net-(D10-K)
- D12 pad 1: Net-(D12-K) -> Net-(D10-K)
- D12 pad 2: Net-(D10-K) -> Net-(D12-A)
- D2 pad 1: Net-(D2-K) -> Net-(D1-K)
- D3 pad 2: Net-(D4-A) -> Net-(D3-A)
- D4 pad 2: Net-(D4-A) -> Net-(D3-A)
- D7 pad 1: Net-(D2-K) -> Net-(D1-K)
- D8 pad 2: Net-(D4-A) -> Net-(D3-A)
- J10 pad 1: Net-(J4-Pin_1) (its old number) -> Net-(J10-Pin_1)
- J2 pad 1: /-18V -> /+3V3_REF
- J2 pad 2: Net-(D10-K) -> /-18V
- J2 pad 3: /+18V -> Net-(D10-K)
- J2 pad 4: /+3V3_REF -> /+18V
- J7 pad 2: /+10V_MOTORS -> Net-(J7-Pin_2)
- J8 pad 2: /+10V_MOTORS -> Net-(J7-Pin_2)
- L4 pad 1: Net-(U4-+VOUT) -> Net-(J7-Pin_2)
- R10 pad 2: Net-(D12-K) -> Net-(D11-K)
- R11 pad 2: Net-(D11-A) -> Net-(D12-A)
- U1 pad 3: Net-(D2-K) -> Net-(D1-K)
- U2 pad 2: Net-(D4-A) -> Net-(D3-A)
- U5 pad 3: Net-(J4-Pin_1) (its old number) -> Net-(U5-Vin)
- U5 pad 5: Net-(D10-K) -> unconnected-(U5-Trim-Pad5)
- U5 pad 6: unconnected-(U2-Trim-Pad6) -> Net-(D10-K)
- U6 pad 10: Net-(J4-Pin_1) (its old number) -> Net-(U5-Vin)
- U6 pad 9: Net-(J4-Pin_1) (its old number) -> Net-(U5-Vin)
- U7 pad 3: Net-(J4-Pin_1) (its old number) -> Net-(U5-Vin)
- U7 pad 4: Net-(U4-+VOUT) -> Net-(J7-Pin_2)
Routing:
- net /+3V3_REF: track 0.00 -> 228.7 mm
- net /-18V: track 0.90 -> 228.1 mm
- net /+18V: track 0.00 -> 217.7 mm
- net /+5V_LEDS: track 0.00 -> 199.6 mm
- net /+10V_MOTORS: track 0.00 -> 188.3 mm
- net /+3V3_LOGIC: track 0.00 -> 183.7 mm
- net Net-(J7-Pin_2): track 0.00 -> 157.2 mm
- net Net-(D5-+): track 0.00 -> 126.9 mm
- net Net-(D3-A): track 0.00 -> 125.9 mm
- net Net-(U5-Vin): track 0.00 -> 111.2 mm
- net Net-(C20-Pad1): track 0.00 -> 103.3 mm
- net Net-(D6-+): track 0.00 -> 73.2 mm
- net Net-(D1-K): track 0.00 -> 69.2 mm
- net Net-(D10-K): track 0.00 -> 54.9 mm, vias 0 -> 230
- net Net-(U2-ADJ): track 0.00 -> 46.1 mm
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Other:
- board text added: "10V 5V 3V3 GND"
- board text added: "3V3 Ref -16V GND +16V"
- board text added: "REV 1"
- board text added: "SKD ANALOG"
- board text removed: "10v 5V 3V3 GND"
- board text removed: "3V3 Ref +16V GND -16V"
- board text removed: "NEU EECE"
- board text removed: "NORTHEASTERN EECE"
- board text removed: "Rev 2"
