File: 06_PCB/PSU/PSU_KICAD/PSU.kicad_sch (KiCad schematic)
At the start: 92 parts, among them J1 IEC_60320_C14_Receptacle, J10 SMPS_IN, J11 D/C_CAP3, J12 D/C_CAP2, J13 D/C_CAP1, J2 OUT_ANLG, J3 MAINS_IN, J4 T1_PRI, J5 T1_SEC, J6 GND_LIFT, J7 FAN1_12V, J8 FAN2_12V, J9 OUT_DIGI, M1 Fan, M2 Fan, SW1 POWER, U1 LM317AT/NOPB, U2 LM337T/NOPB, U3 LD1117V33C, U4 MeanWell RS-100-15, U5 3V3 URB2403LD-20WR3, U6 MeanWell NID-100-5, U7 12V URB2412LD-50WR3

Commit message: fixed some dum dum stuff on the psu lol
Connections:
- net at C20.2, C21.2: now also C15.2, C16.2, C17.2, C18.2, C19.2, C22.2, C23.2, D10.1 (K), D11.2 (A), D12.1 (K), D13.1 (K), D14.1 (K), D15.1 (K), D6.1 (+), D6.4 (-), H1.1, J1.3 (PE), J10.2 (Pin_2), J6.1 (Pin_1), J6.2 (Pin_2), J7.1 (Pin_1), J8.1 (Pin_1), J9.1 (Pin_1), R4.1, U5.2 (GND), U5.6 (GND), U6.5 (GND), U6.6 (GND), U6.7 (GND), U6.8 (GND), U7.2 (GND), U7.5 (GND)
- net at C1.2, C10.1, C11.2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: no longer D5.3, TR2.5, TR2.7
- new net: D5.3, TR2.5, TR2.7
Changed lines of the file:
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@@
 	)
 	(junction
-		(at 212.09 53.34)
+		(at 284.48 151.13)
 		(diameter 0)
 		(color 0 0 0 0)
 	)
 	(junction
-		(at 283.21 120.65)
+		(at 212.09 53.34)
 		(diameter 0)
 		(color 0 0 0 0)
 	)
 	(junction
-		(at 200.66 116.84)
+		(at 283.21 120.65)
 		(diameter 0)
 		(color 0 0 0 0)
@@
 	)
 	(junction
-		(at 212.09 116.84)
-		(diameter 0)
-		(color 0 0 0 0)
-	)
-	(junction
 		(at 321.31 53.34)
 		(diameter 0)
@@
 	)
 	(junction
+		(at 184.15 191.77)
+		(diameter 0)
+		(color 0 0 0 0)
+	)
+	(junction
 		(at 114.3 58.42)
 		(diameter 0)
@@
 	)
 	(junction
+		(at 200.66 116.84)
+		(diameter 0)
+		(color 0 0 0 0)
+	)
+	(junction
 		(at 245.11 53.34)
 		(diameter 0)
@@
 	)
 	(junction
+		(at 290.83 151.13)
+		(diameter 0)
+		(color 0 0 0 0)
+	)
+	(junction
 		(at 121.92 58.42)
 		(diameter 0)
@@
 	)
 	(junction
+		(at 325.12 191.77)
+		(diameter 0)
+		(color 0 0 0 0)
+	)
+	(junction
 		(at 252.73 191.77)
 		(diameter 0)
@@
 	)
 	(junction
+		(at 325.12 167.64)
+		(diameter 0)
+		(color 0 0 0 0)
+	)
+	(junction
 		(at 245.11 100.33)
 		(diameter 0)
@@
 	(wire
 		(pts
-			(xy 97.79 191.77) (xy 226.06 191.77)
+			(xy 97.79 191.77) (xy 184.15 191.77)
 		)
 		(stroke
@@
 	(wire
 		(pts
+			(xy 325.12 167.64) (xy 318.77 167.64)
+		)
+		(stroke
+			(width 0)
+			(type default)
+		)
+	)
+	(wire
+		(pts
 			(xy 270.51 80.01) (xy 279.4 80.01)
 		)
@@
 	(wire
 		(pts
+			(xy 184.15 191.77) (xy 226.06 191.77)
+		)
+		(stroke
+			(width 0)
+			(type default)
+		)
+	)
+	(wire
+		(pts
 			(xy 184.15 138.43) (xy 186.69 138.43)
 		)
@@
 	(wire
 		(pts
+			(xy 184.15 156.21) (xy 184.15 191.77)
+		)
+		(stroke
+			(width 0)
+			(type default)
+		)
+	)
+	(wire
+		(pts
 			(xy 270.51 26.67) (xy 270.51 36.83)
 		)
@@
 	(wire
 		(pts
+			(xy 200.66 116.84) (xy 219.71 116.84)
+		)
+		(stroke
+			(width 0)
+			(type default)
+		)
+	)
+	(wire
+		(pts
 			(xy 184.15 147.32) (xy 184.15 139.7)
 		)
@@
 	(wire
 		(pts
+			(xy 325.12 191.77) (xy 331.47 191.77)
+		)
+		(stroke
+			(width 0)
+			(type default)
+		)
+	)
+	(wire
+		(pts
 			(xy 209.55 46.99) (xy 210.82 46.99)
 		)
@@
 	(wire
 		(pts
+			(xy 284.48 151.13) (xy 290.83 151.13)
+		)
+		(stroke
+			(width 0)
+			(type default)
+		)
+	)
+	(wire
+		(pts
 			(xy 308.61 113.03) (xy 308.61 120.65)
 		)
@@
 	(wire
 		(pts
-			(xy 212.09 120.65) (xy 212.09 116.84)
+			(xy 212.09 110.49) (xy 212.09 120.65)
 		)
 		(stroke
@@
 	(wire
 		(pts
-			(xy 331.47 167.64) (xy 318.77 167.64)
+			(xy 331.47 167.64) (xy 325.12 167.64)
 		)
 		(stroke
@@
 	(wire
 		(pts
-			(xy 318.77 191.77) (xy 331.47 191.77)
+			(xy 318.77 191.77) (xy 325.12 191.77)
 		)
 		(stroke
@@
 	(wire
 		(pts
-			(xy 200.66 116.84) (xy 212.09 116.84)
-		)
-		(stroke
-			(width 0)
-			(type default)
-		)
-	)
-	(wire
-		(pts
 			(xy 318.77 158.75) (xy 318.77 154.94)
 		)
@@
 	(wire
 		(pts
-			(xy 212.09 110.49) (xy 212.09 116.84)
-		)
-		(stroke
-			(width 0)
-			(type default)
-		)
-	)
-	(wire
-		(pts
 			(xy 270.51 69.85) (xy 270.51 80.01)
 		)
@@
 	(wire
 		(pts
-			(xy 284.48 143.51) (xy 284.48 171.45)
+			(xy 284.48 143.51) (xy 284.48 151.13)
 		)
 		(stroke
@@
 	(wire
 		(pts
+			(xy 325.12 167.64) (xy 325.12 191.77)
+		)
+		(stroke
+			(width 0)
+			(type default)
+		)
+	)
+	(wire
+		(pts
 			(xy 386.08 104.14) (xy 386.08 95.25)
 		)
@@
 	(wire
 		(pts
+			(xy 284.48 151.13) (xy 284.48 171.45)
+		)
+		(stroke
+			(width 0)
+			(type default)
+		)
+	)
+	(wire
+		(pts
 			(xy 349.25 77.47) (xy 349.25 106.68)
 		)
@@
 		)
 		(stroke
-			(width 0)
-			(type default)
-		)
-	)
-	(wire
-		(pts
-			(xy 212.09 116.84) (xy 219.71 116.84)
-		)
-		(stroke

Commit message: upload proposal
Parts:
- removed C16: 1000u, Capacitor_THT:CP_Radial_D12.5mm_P5.00mm, symbol Device:C_Polarized
- removed C17: 470u, Capacitor_THT:CP_Radial_D10.0mm_P5.00mm, symbol Device:C_Polarized
- removed J11: D/C_CAP3, Connector_PinHeader_2.54mm:PinHeader_1x02_P2.54mm_Vertical, symbol Connector:Conn_01x02_Pin
- removed J12: D/C_CAP2, Connector_PinHeader_2.54mm:PinHeader_1x02_P2.54mm_Vertical, symbol Connector:Conn_01x02_Pin
- removed J13: D/C_CAP1, Connector_PinHeader_2.54mm:PinHeader_1x02_P2.54mm_Vertical, symbol Connector:Conn_01x02_Pin
- removed J8: FAN2_12V, Connector_PinHeader_2.54mm:PinHeader_1x02_P2.54mm_Vertical, symbol Connector:Conn_01x02_Pin
- removed L1: 4.7u, Inductor_SMD:L_Vishay_IHLP-5050, symbol Device:L
- removed R1, R2, R3: 220, Resistor_THT:R_Axial_DIN0414_L11.9mm_D4.5mm_P20.32mm_Horizontal, symbol Device:R_US
- removed R16: 0.33R, Resistor_THT:R_Axial_DIN0207_L6.3mm_D2.5mm_P10.16mm_Horizontal, symbol Device:R_US
- added J9: FAN2_12V, Connector_PinHeader_2.54mm:PinHeader_1x02_P2.54mm_Vertical, symbol Connector:Conn_01x02_Pin
- U1: renamed from U4; footprint (none) -> Converter_ACDC:Converter_ACDC_MeanWell_IRM-60-xx_THT
- U2: renamed from U5; footprint Converter_DCDC:Converter_DCDC_XP_POWER_JTDxxxxxxx_THT -> My Footprints:urb 50w dc-dc
- renumbered C15 to C1, C13 to C10, C18 to C11, C20 to C12, C22 to C13, C7 to C14, C8 to C15, C14 to C16, C19 to C17, C21 to C18, C23 to C19, C1 to C2, C9 to C20, C10 to C21, C2 to C3, C11 to C4, C3 to C5, C4 to C6, C12 to C7, C5 to C8, C6 to C9, D6 to D1, D12 to D11, D11 to D12, D1 to D2, D2 to D3, D3 to D4, D4 to D5, D5 to D6, J9 to J10, J3 to J2, J4 to J3, J10 to J4, J2 to J8, L2 to L1, L3 to L2, L4 to L3, R4 to R1, R9 to R10, R10 to R11, R11 to R12, R12 to R13, R13 to R14, R14 to R15, R15 to R2, R5 to R3, R6 to R4, R7 to R5, R8 to R6, R17 to R7, R18 to R8, R19 to R9, U6 to U3, U7 to U4, U1 to U5, U2 to U6, U3 to U7
Connections:
- net +10V_MOTORS: now also J7.2 (Pin_2), J9.2 (Pin_2)
- net +18V: now also J8.3 (Pin_3); no longer J8.1 (Pin_1)
- net -18V: now also J8.1 (Pin_1); no longer J8.3 (Pin_3)
- net at C11.2, C12.2, C13.2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: now also C1.1, C10.2, C14.2, C15.1, C16.2, C2.2, C20.2, C21.1, C3.1, C4.2, C5.2, C6.1, C7.2, C8.2, C9.1, D1.2, D1.3, D6.4 (-), J5.2 (Pin_2), J5.3 (Pin_3), J6.3 (Pin_3), J8.2 (Pin_2), R1.2, R3.2, R4.1, U2.5 (GND), U7.1 (GND), J9.1 (Pin_1); no longer C1.2, D1.1 (+), D1.4 (-), H1.1, J1.3 (PE), J6.1 (Pin_1), J6.2 (Pin_2), R1.1, U2.6 (GND)
- net at J4.1 (Pin_1): now also U2.3 (Vin), U3.10 (Vin), U3.9 (Vin), U4.3 (Vin)
- net at C13.1, L3.1, R2.2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: no longer J7.2 (Pin_2)
- net at C12.1, L2.1, U3.1 (Vout)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: no longer U2.1 (Enable), U4.1 (Enable)
- new net: C1.2, D1.1 (+), D1.4 (-), H1.1, J1.3 (PE), J6.1 (Pin_1), J6.2 (Pin_2), R1.1
Other:
- note added: "COMPONENT NOTES: For all other resistors, use 1/4W. All resistors are metal film, 1% or better tolerance. All screw terminals (J2, J3, J4. J5, J9, J10) are the Phoenix Contact MKDS 1,5 series, 5.08mm pin pitch. Pin headers (J6, J7, J8, J11, J12, J13) are standard 2.54mm pin pitch male pin headers. Regulators (U1, U2, U3) are all TO-220 3 pin package. Heatsinks used are Same Sky Devices HSE-B20254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"
- note removed: "COMPONENT NOTES: R1, R2, R3, (discharges big filter caps) use 2W at least Resistors. For all other resistors, use 1/4W. All resistors are metal film, 1% or better tolerance. All screw terminals (J2, J3, J4. J5, J9, J10) are the Phoenix Contact MKDS 1,5 series, 5.08mm pin pitch. Pin headers (J6, J7, J8, J11, J12, J13) are standard 2.54mm pin pitch male pin headers. Regulators (U1, U2, U3) are all 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"
- moved on the sheet: C11, C12, C13, C17, C18, C19, C2, C3, C4, C5, C6, C7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

Commit message: stuff and things idk
Parts:
- removed J9: FAN2_12V, Connector_PinHeader_2.54mm:PinHeader_1x02_P2.54mm_Vertical, symbol Connector:Conn_01x02_Pin
- added C16: 1000u, Capacitor_THT:CP_Radial_D12.5mm_P5.00mm, symbol Device:C_Polarized
- added C17: 470u, Capacitor_THT:CP_Radial_D10.0mm_P5.00mm, symbol Device:C_Polarized
- added J8: FAN2_12V, Connector_PinHeader_2.54mm:PinHeader_1x02_P2.54mm_Vertical, symbol Connector:Conn_01x02_Pin
- added L1: 4.7u, Inductor_SMD:L_Vishay_IHLP-5050, symbol Device:L
- added R16: 0.33R, Resistor_THT:R_Axial_DIN0207_L6.3mm_D2.5mm_P10.16mm_Horizontal, symbol Device:R_US
- U4: renamed from U1; footprint Converter_ACDC:Converter_ACDC_MeanWell_IRM-60-xx_THT -> (none)
- U5: renamed from U2; footprint My Footprints:urb 50w dc-dc -> Converter_DCDC:Converter_DCDC_XP_POWER_JTDxxxxxxx_THT
- renumbered C2 to C1, C21 to C10, C4 to C11, C7 to C12, C10 to C13, C16 to C14, C1 to C15, C11 to C18, C17 to C19, C3 to C2, C12 to C20, C18 to C21, C13 to C22, C19 to C23, C5 to C3, C6 to C4, C8 to C5, C9 to C6, C14 to C7, C15 to C8, C20 to C9, D2 to D1, D12 to D11, D11 to D12, D3 to D2, D4 to D3, D5 to D4, D6 to D5, D1 to D6, J4 to J10, J8 to J2, J2 to J3, J3 to J4, J10 to J9, L1 to L2, L2 to L3, L3 to L4, R7 to R1, R11 to R10, R12 to R11, R13 to R12, R14 to R13, R15 to R14, R2 to R15, R8 to R2, R9 to R3, R1 to R4, R3 to R5, R4 to R6, R5 to R7, R6 to R8, R10 to R9, U5 to U1, U6 to U2, U7 to U3, U3 to U6, U4 to U7
Connections:
- net +10V_MOTORS: no longer J7.2 (Pin_2)
- net +18V: now also J2.4 (Pin_4); no longer J2.3 (Pin_3)
- net +3V3_REF: now also J2.1 (Pin_1); no longer J2.4 (Pin_4)
- net -18V: now also J2.2 (Pin_2); no longer J2.1 (Pin_1)
- net at C1.2, C10.1, C11.2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: now also J2.3 (Pin_3), U5.6 (GND), C16.2, C17.2, J8.1 (Pin_1); no longer J2.2 (Pin_2), U5.5 (GND)
- net at U5.3 (Vin), U6.10 (Vin), U6.9 (Vin)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: now also L1.2, R16.1; no longer J10.1 (Pin_1)
- net at C22.1, L4.1, R15.2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: now also J7.2 (Pin_2), J8.2 (Pin_2)
- new net: C16.1, J10.1 (Pin_1), L1.1
- new net: C17.1, R16.2
Other:
- note added: "+5Vrms"
- note added: "COMPONENT NOTES: R1, R2, R3, (discharges big filter caps) use 2W at least Resistors. For all other resistors, use 1/4W. All resistors are metal film, 1% or better tolerance. All screw terminals (J2, J3, J4. J5, J9, J10) are the Phoenix Contact MKDS 1,5 series, 5.08mm pin pitch. Pin headers (J6, J7, J8, J11, J12, J13) are standard 2.54mm pin pitch male pin headers. Regulators (U1, U2, U3) are all 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"
- note added: "~+7V DC"
- note removed: "+7Vrms"
- note removed: "COMPONENT NOTES: For all other resistors, use 1/4W. All resistors are metal film, 1% or better tolerance. All screw terminals (J2, J3, J4. J5, J9, J10) are the Phoenix Contact MKDS 1,5 series, 5.08mm pin pitch. Pin headers (J6, J7, J8, J11, J12, J13) are standard 2.54mm pin pitch male pin headers. Regulators (U1, U2, U3) are all TO-220 3 pin package. Heatsinks used are Same Sky Devices HSE-B20254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"
- note removed: "~+10V DC"
- moved on the sheet: C1, C11, C12, C18, C19, C2, C20, C21, C22, C23, J10, J2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
