File: PCB_CAD/DEV_BOARDS/_DEV_EC11_button_breakout/_restore_backup_2026-08-24T17-16-47-379/EC11BREAKOUT.kicad_pcb (KiCad board)
At the start: 4 copper layers, 33 x 35.6 mm, 19 parts, among them J1 Conn_01x04_Pin, J2 Conn_01x04_Pin, SW1 EC11_Rotary_Encoder, SW2 SW_Push_LED, U1 74HC14

Commit message: temporary so i can compare with other branch
Routing:
- net +3V3: track 0.00 -> 30.3 mm
- net Net-(D1-A): track 0.00 -> 28.1 mm
- net Net-(SW1-Pin_5): track 0.00 -> 27.9 mm, vias 0 -> 1
- net Net-(SW1-Pin_3): track 0.00 -> 26.0 mm
- net Net-(SW1-Pin_1): track 0.00 -> 22.5 mm
- net KNOB_SW: track 0.00 -> 19.1 mm, vias 0 -> 1
- net Net-(C3-Pad1): track 0.00 -> 18.9 mm
- net SW: track 0.00 -> 13.9 mm, vias 0 -> 1
- net Net-(SW2-A): track 0.00 -> 12.1 mm
- net GND: track 0.00 -> 11.6 mm, vias 0 -> 2
- net Net-(D1-K): track 0.00 -> 11.1 mm
- net KNOB_A: track 0.00 -> 10.5 mm, vias 0 -> 1
- net Net-(C2-Pad1): track 0.00 -> 10.0 mm
- net KNOB_B: track 0.00 -> 10.0 mm, vias 0 -> 1
- net Net-(C4-Pad1): track 0.00 -> 5.73 mm
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