File: PCB_CAD/DEV_BOARDS/_DEV_EC11_button_breakout/_restore_backup_2026-08-24T17-16-47-379/EC11BREAKOUT.kicad_sch (KiCad schematic)
At the start: 19 parts, among them J1 Conn_01x04_Pin, J2 Conn_01x04_Pin, SW1 EC11_Rotary_Encoder, SW2 SW_Push_LED, U1 74HC14

Commit message: temporary so i can compare with other branch
Changed lines of the file:
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@@
 		(property "Reference" "SW2"
 			(at 73.66 124.46 0)
-			(hide yes)
 			(show_name no)
 			(do_not_autoplace no)
@@
 		(property "Value" "GND"
 			(at 105.41 149.86 0)
-			(hide yes)
 			(show_name no)
 			(do_not_autoplace no)
@@
 		(property "Value" "GND"
 			(at 99.06 86.106 0)
-			(hide yes)
 			(show_name no)
 			(do_not_autoplace no)
@@
 		(property "Value" "GND"
 			(at 52.07 86.106 0)
-			(hide yes)
 			(show_name no)
 			(do_not_autoplace no)
@@
 		(property "Reference" "U1"
 			(at 115.57 116.84 0)
-			(hide yes)
 			(show_name no)
 			(do_not_autoplace no)
@@
 		(property "Value" "74HC14"
 			(at 115.57 119.38 0)
-			(hide yes)
 			(show_name no)
 			(do_not_autoplace no)
@@
 		(property "LCSC" "C5605"
 			(at 115.57 125.73 0)
-			(hide yes)
 			(show_name no)
 			(do_not_autoplace no)
@@
 		(property "Reference" "U1"
 			(at 46.99 57.15 0)
-			(hide yes)
 			(show_name no)
 			(do_not_autoplace no)
@@
 		(property "Value" "74HC14"
 			(at 46.99 59.69 0)
-			(hide yes)
 			(show_name no)
 			(do_not_autoplace no)
@@
 		(property "LCSC" "C5605"
 			(at 46.99 62.23 0)
-			(hide yes)
 			(show_name no)
 			(do_not_autoplace no)
@@
 		(property "Value" "GND"
 			(at 131.064 88.646 0)
-			(hide yes)
 			(show_name no)
 			(do_not_autoplace no)
@@
 		(property "Reference" "U1"
 			(at 141.986 58.674 0)
-			(hide yes)
 			(show_name no)
 			(do_not_autoplace no)
@@
 		(property "Value" "74HC14"
 			(at 145.034 60.706 0)
-			(hide yes)
 			(show_name no)
 			(do_not_autoplace no)
@@
 		(property "LCSC" "C5605"
 			(at 140.97 63.5 0)
-			(hide yes)
 			(show_name no)
 			(do_not_autoplace no)
@@
 		(property "Reference" "U1"
 			(at 144.78 76.2 0)
-			(hide yes)
 			(show_name no)
 			(do_not_autoplace no)
@@
 		(property "Value" "74HC14"
 			(at 143.002 77.978 0)
-			(hide yes)
 			(show_name no)
 			(do_not_autoplace no)
@@
 		(property "LCSC" "C5605"
 			(at 140.97 73.66 0)
-			(hide yes)
 			(show_name no)
 			(do_not_autoplace no)
@@
 		(property "Value" "GND"
 			(at 78.74 86.106 0)
-			(hide yes)
 			(show_name no)
 			(do_not_autoplace no)
@@
 		(property "Reference" "SW1"
 			(at 87.63 59.69 0)
-			(hide yes)
 			(show_name no)
 			(do_not_autoplace no)
@@
 		(property "Value" "GND"
 			(at 58.42 149.86 0)
-			(hide yes)
-			(show_name no)
-			(do_not_autoplace no)
+			(show_name no)
+			(do_not_autoplace no)
