File: PCB_CAD/DEV_BOARDS/FullChanDevBoard/FullChanDevBoard.kicad_pcb (KiCad board)
At the start: 4 copper layers, 200 x 300 mm, 318 parts, among them J1 I2C_0x20, J10 Conn_01x04_Socket, J11 Conn_01x04_Socket, J12 Conn_01x04_Socket, J13 Conn_01x04_Socket, J14 Conn_01x04_Socket, J15 Conn_01x04_Socket, J16 Conn_01x04_Socket, J17 Conn_01x04_Socket, J18 Conn_01x04_Socket, J19 Conn_01x04_Socket, J2 I2C_0x21, J20 Conn_01x04_Socket, J21 Conn_01x04_Socket, J22 Conn_01x04_Socket, J23 Conn_01x04_Socket, J24 Conn_01x04_Socket, J25 Conn_01x04_Socket, J26 Conn_01x04_Socket, J27 Conn_01x04_Socket, J28 Conn_01x04_Socket, J29 SPI_MASTER, J3 I2C_0x22, J30 DISP1, J31 DISP2, J32 DISP3, J33 DISP4, J34 USART2, J35 SWD_PGM, J36 0x20_A, J37 0x20_B, J38 0x21_A, J39 0x21_B, J4 I2C_0x60, J40 0x22_A, J41 0x22_B, J42 0x60_L, J43 0x60_R, J44 0x61_L, J45 0x61_R, J46 0x62_L, J47 0x62_R, J48 0x63_L, J49 0x63_R, J5 I2C_0x61, J50 0x64_L, J51 0x64_R, J52 EXT_POW_IN, J53 DC_10V, J54 CV1, J55 CV2, J56 PSU_IN_DIGI, J57 BANANA_3V3, J58 BANANA_5V, J59 BANANA_10V, J6 I2C_0x62, J60 BANANA_GND, J61 10V_SRC, J62 JUMPER_STORE, J7 I2C_0x63, J8 I2C_0x64, J9 Conn_01x04_Socket, SW1 K0, SW10 K5, SW11 B0, SW12 B1A, SW13 B1B, SW14 B1C, SW15 B2A, SW16 B2B, SW17 B2C, SW18 B3A, SW19 B3B, SW2 K1A, SW20 B3C, SW21 B4A, SW22 B4B, SW23 RESET, SW3 K1B, SW4 K2A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

Commit message: chonker dev board
Parts:
- added C100: 470u, Capacitor_SMD:CP_Elec_8x6.9, F.Cu at (60.8, 207.0)
- added C101: 10u, Capacitor_SMD:C_0805_2012Metric, F.Cu at (58.6, 230.9)
- added C102: 10u, Capacitor_SMD:C_0805_2012Metric, F.Cu at (215.5, 116.7)
- added C103: 100n, Capacitor_SMD:C_0603_1608Metric, F.Cu at (217.5, 113.7)
- added C104: 10u, Capacitor_SMD:C_0805_2012Metric, F.Cu at (240.4, 60.1)
- added C105: 100n, Capacitor_SMD:C_0603_1608Metric, F.Cu at (240.5, 54.5)
- added C106: 10u, Capacitor_SMD:C_0805_2012Metric, F.Cu at (240.1, 80.1)
- added C107: 100n, Capacitor_SMD:C_0603_1608Metric, F.Cu at (240.6, 73.7)
- added C108: 10u, Capacitor_SMD:C_0805_2012Metric, F.Cu at (240.1, 99.5)
- added C109: 100n, Capacitor_SMD:C_0603_1608Metric, F.Cu at (241.0, 92.8)
- added C110: 10u, Capacitor_SMD:C_0805_2012Metric, F.Cu at (240.0, 117.9)
- added C111: 100n, Capacitor_SMD:C_0603_1608Metric, F.Cu at (240.6, 112.4)
- added C46: 100n, Capacitor_SMD:C_0603_1608Metric, F.Cu at (58.4, 233.1)
- added C47: 100n, Capacitor_SMD:C_0603_1608Metric, F.Cu at (62.8, 192.6)
- added C48: 20p, Capacitor_SMD:C_0603_1608Metric, F.Cu at (71.5, 192.8)
- added D19: LED, LED_THT:LED_Rectangular_W3.9mm_H1.8mm, F.Cu at (98.6, 82.3)
- added D20: LED, LED_THT:LED_Rectangular_W3.9mm_H1.8mm, F.Cu at (98.6, 74.5)
- added D21: LED, LED_THT:LED_Rectangular_W3.9mm_H1.8mm, F.Cu at (98.6, 67.0)
- added G***: LOGO, LOGO, F.Cu at (204.6, 61.9)
- added G***: LOGO, LOGO, F.Cu at (212.3, 62.3)
- added J63: AUDIO_SWITCHES, Connector_PinHeader_2.54mm:PinHeader_1x08_P2.54mm_Vertical, F.Cu at (210.2, 100.4)
- added J64: Conn_01x02_Pin, Connector_PinHeader_2.54mm:PinHeader_1x02_P2.54mm_Vertical, F.Cu at (226.1, 132.0)
- added J65: SPI_3, Connector_PinHeader_2.54mm:PinHeader_1x07_P2.54mm_Vertical, F.Cu at (248.0, 163.4)
- added Q1: 2N7002, Package_TO_SOT_SMD:SOT-23, F.Cu at (236.8, 62.3)
- added R105: 10k, Resistor_SMD:R_0603_1608Metric, F.Cu at (53.6, 231.7)
- added R106: 10k, Resistor_SMD:R_0603_1608Metric, F.Cu at (53.6, 235.1)
- added R107: 10k, Resistor_SMD:R_0603_1608Metric, F.Cu at (53.7, 238.4)
- added R108: 68, Resistor_SMD:R_1206_3216Metric, F.Cu at (99.5, 89.8)
- added R109: 220, Resistor_SMD:R_1206_3216Metric, F.Cu at (99.5, 93.1)
- added R110: 470, Resistor_SMD:R_1206_3216Metric, F.Cu at (99.5, 96.4)
- added R111: 22, Resistor_THT:R_Axial_DIN0207_L6.3mm_D2.5mm_P10.16mm_Horizontal, F.Cu at (113.4, 171.4)
- added R112: 390, Resistor_SMD:R_1206_3216Metric, F.Cu at (240.3, 57.0)
- added R113: 390, Resistor_SMD:R_1206_3216Metric, F.Cu at (240.1, 76.9)
- added R114: 390, Resistor_SMD:R_1206_3216Metric, F.Cu at (240.0, 96.4)
- added R115: 390, Resistor_SMD:R_1206_3216Metric, F.Cu at (239.9, 115.0)
- added R116: 47k, Resistor_SMD:R_0603_1608Metric, F.Cu at (231.9, 62.8)
- added R117: 47k, Resistor_SMD:R_0603_1608Metric, F.Cu at (231.9, 64.7)
- added R118: 68, Resistor_SMD:R_1206_3216Metric, F.Cu at (232.2, 60.4)
- added R119: 10k, Resistor_SMD:R_0603_1608Metric, F.Cu at (239.5, 103.9)
- added R120: 10k, Resistor_SMD:R_0603_1608Metric, F.Cu at (239.4, 84.9)
- added R121: 10k, Resistor_SMD:R_0603_1608Metric, F.Cu at (239.5, 65.8)
- added R122: 10k, Resistor_SMD:R_0603_1608Metric, F.Cu at (239.5, 46.4)
- added REF**: LayerMarker_4_6.35x2.54mm_TextH1mm_P1.27mm_BottomMirrored, Symbol:LayerMarker_4_6.35x2.54mm_TextH1mm_P1.27mm_BottomMirrored, F.Cu at (242.4, 337.8)
- J29: footprint Connector_PinHeader_2.54mm:PinHeader_1x04_P2.54mm_Vertical -> Connector_PinHeader_2.54mm:PinHeader_1x06_P2.54mm_Vertical
- J35: footprint Connector_PinHeader_2.54mm:PinHeader_1x04_P2.54mm_Vertical -> My Footprints:FTSH-107-01-L-DV-K-TR
- moved U3 76.9 mm to (56.6, 226.9)
- moved J34 39.4 mm to (241.6, 126.1)
- moved C87 28.0 mm to (179.3, 227.3)
- moved C90 28.0 mm to (179.3, 223.0)
- moved C86 28.0 mm to (179.3, 225.1)
- moved C88 28.0 mm to (179.3, 229.4)
- moved C89 28.0 mm to (179.3, 221.1)
- moved U2 23.6 mm to (67.8, 193.7)
- moved J29 20.6 mm to (241.5, 145.4)
- moved U4 20.5 mm to (223.6, 111.4)
- moved J35 17.0 mm to (241.6, 176.7), turned to 90 degrees
- moved C94 2.77 mm to (202.5, 219.1)
- moved C95 2.77 mm to (200.7, 219.2)
- moved X1 2.68 mm to (175.4, 204.6)
- moved C83 2.68 mm to (183.4, 205.3)
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Connections:
- C80 pad 2: Net-(U1-PG10) -> NRST
- F1 pad 1: unconnected-(F1-Pin_1-Pad1) -> +3V3
- F1 pad 2: unconnected-(F1-Pin_2-Pad2) -> Fader_ADC
- F1 pad 3: unconnected-(F1-Pin_3-Pad3) -> GND
- F1 pad A: unconnected-(F1-Pin_5-PadA) -> Net-(F1-Pin_5)
- F1 pad B: unconnected-(F1-Pin_6-PadB) -> Net-(F1-Pin_6)
- F1 pad T: unconnected-(F1-Pin_4-PadT) -> Net-(F1-Pin_4)
- J29 pad 1: unconnected-(J29-Pin_1-Pad1) -> +3V3
- J29 pad 2: unconnected-(J29-Pin_2-Pad2) -> MASTER_CK
- J29 pad 3: unconnected-(J29-Pin_3-Pad3) -> MASTER_MOSI
- J29 pad 4: unconnected-(J29-Pin_4-Pad4) -> MASTER_MISO
- J30 pad 1: unconnected-(J30-Pin_1-Pad1) -> Net-(J30-Pin_1)
- J30 pad 10: unconnected-(J30-Pin_10-Pad10) -> GND
- J30 pad 11: unconnected-(J30-Pin_11-Pad11) -> GND
- J30 pad 12: unconnected-(J30-Pin_12-Pad12) -> GND
- J30 pad 13: unconnected-(J30-Pin_13-Pad13) -> GND
- J30 pad 14: unconnected-(J30-Pin_14-Pad14) -> GND
- J30 pad 15: unconnected-(J30-Pin_15-Pad15) -> GND
- J30 pad 16: unconnected-(J30-Pin_16-Pad16) -> DISP1_DC
- J30 pad 17: unconnected-(J30-Pin_17-Pad17) -> DISP_CK
- J30 pad 18: unconnected-(J30-Pin_18-Pad18) -> DISP1_CS
- J30 pad 2: unconnected-(J30-Pin_2-Pad2) -> DISP_BL-
- J30 pad 20: unconnected-(J30-Pin_20-Pad20) -> +3V3
- J30 pad 21: unconnected-(J30-Pin_21-Pad21) -> DISP_MOSI
- J30 pad 22: unconnected-(J30-Pin_22-Pad22) -> GND
- J30 pad 3: unconnected-(J30-Pin_3-Pad3) -> +3V3
- J30 pad 4: unconnected-(J30-Pin_4-Pad4) -> +3V3
- J30 pad 5: unconnected-(J30-Pin_5-Pad5) -> GND
- J30 pad 6: unconnected-(J30-Pin_6-Pad6) -> +3V3
- J30 pad 7: unconnected-(J30-Pin_7-Pad7) -> GND
- J30 pad 8: unconnected-(J30-Pin_8-Pad8) -> GND
- J30 pad 9: unconnected-(J30-Pin_9-Pad9) -> GND
- J30 pad MP: (no net) -> GND
- J31 pad 1: unconnected-(J31-Pin_1-Pad1) -> Net-(J31-Pin_1)
- J31 pad 10: unconnected-(J31-Pin_10-Pad10) -> GND
- J31 pad 11: unconnected-(J31-Pin_11-Pad11) -> GND
- J31 pad 12: unconnected-(J31-Pin_12-Pad12) -> GND
- J31 pad 13: unconnected-(J31-Pin_13-Pad13) -> GND
- J31 pad 14: unconnected-(J31-Pin_14-Pad14) -> GND
- J31 pad 15: unconnected-(J31-Pin_15-Pad15) -> GND
- J31 pad 16: unconnected-(J31-Pin_16-Pad16) -> DISP2_DC
- J31 pad 17: unconnected-(J31-Pin_17-Pad17) -> DISP_CK
- J31 pad 18: unconnected-(J31-Pin_18-Pad18) -> DISP2_CS
- J31 pad 2: unconnected-(J31-Pin_2-Pad2) -> DISP_BL-
- J31 pad 20: unconnected-(J31-Pin_20-Pad20) -> +3V3
- J31 pad 21: unconnected-(J31-Pin_21-Pad21) -> DISP_MOSI
- J31 pad 22: unconnected-(J31-Pin_22-Pad22) -> GND
- J31 pad 3: unconnected-(J31-Pin_3-Pad3) -> +3V3
- J31 pad 4: unconnected-(J31-Pin_4-Pad4) -> +3V3
- J31 pad 5: unconnected-(J31-Pin_5-Pad5) -> GND
- J31 pad 6: unconnected-(J31-Pin_6-Pad6) -> +3V3
- J31 pad 7: unconnected-(J31-Pin_7-Pad7) -> GND
- J31 pad 8: unconnected-(J31-Pin_8-Pad8) -> GND
- J31 pad 9: unconnected-(J31-Pin_9-Pad9) -> GND
- J31 pad MP: (no net) -> GND
- J32 pad 1: unconnected-(J32-Pin_1-Pad1) -> Net-(J32-Pin_1)
- J32 pad 10: unconnected-(J32-Pin_10-Pad10) -> GND
- J32 pad 11: unconnected-(J32-Pin_11-Pad11) -> GND
- J32 pad 12: unconnected-(J32-Pin_12-Pad12) -> GND
- J32 pad 13: unconnected-(J32-Pin_13-Pad13) -> GND
- J32 pad 14: unconnected-(J32-Pin_14-Pad14) -> GND
- J32 pad 15: unconnected-(J32-Pin_15-Pad15) -> GND
- J32 pad 16: unconnected-(J32-Pin_16-Pad16) -> DISP3_DC
- J32 pad 17: unconnected-(J32-Pin_17-Pad17) -> DISP_CK
- J32 pad 18: unconnected-(J32-Pin_18-Pad18) -> DISP3_CS
- J32 pad 2: unconnected-(J32-Pin_2-Pad2) -> DISP_BL-
- J32 pad 20: unconnected-(J32-Pin_20-Pad20) -> +3V3
- J32 pad 21: unconnected-(J32-Pin_21-Pad21) -> DISP_MOSI
- J32 pad 22: unconnected-(J32-Pin_22-Pad22) -> GND
- J32 pad 3: unconnected-(J32-Pin_3-Pad3) -> +3V3
- J32 pad 4: unconnected-(J32-Pin_4-Pad4) -> +3V3
- J32 pad 5: unconnected-(J32-Pin_5-Pad5) -> GND
- J32 pad 6: unconnected-(J32-Pin_6-Pad6) -> +3V3
- J32 pad 7: unconnected-(J32-Pin_7-Pad7) -> GND
- J32 pad 8: unconnected-(J32-Pin_8-Pad8) -> GND
- J32 pad 9: unconnected-(J32-Pin_9-Pad9) -> GND
- J32 pad MP: (no net) -> GND
- J33 pad 1: unconnected-(J33-Pin_1-Pad1) -> Net-(J33-Pin_1)
- J33 pad 10: unconnected-(J33-Pin_10-Pad10) -> GND
- J33 pad 11: unconnected-(J33-Pin_11-Pad11) -> GND
- J33 pad 12: unconnected-(J33-Pin_12-Pad12) -> GND
- J33 pad 13: unconnected-(J33-Pin_13-Pad13) -> GND
- J33 pad 14: unconnected-(J33-Pin_14-Pad14) -> GND
- J33 pad 15: unconnected-(J33-Pin_15-Pad15) -> GND
- J33 pad 16: unconnected-(J33-Pin_16-Pad16) -> DISP4_DC
- J33 pad 17: unconnected-(J33-Pin_17-Pad17) -> DISP_CK
- J33 pad 18: unconnected-(J33-Pin_18-Pad18) -> DISP4_CS
- J33 pad 2: unconnected-(J33-Pin_2-Pad2) -> DISP_BL-
- J33 pad 20: unconnected-(J33-Pin_20-Pad20) -> +3V3
- J33 pad 21: unconnected-(J33-Pin_21-Pad21) -> DISP_MOSI
- J33 pad 22: unconnected-(J33-Pin_22-Pad22) -> GND
- J33 pad 3: unconnected-(J33-Pin_3-Pad3) -> +3V3
- J33 pad 4: unconnected-(J33-Pin_4-Pad4) -> +3V3
- J33 pad 5: unconnected-(J33-Pin_5-Pad5) -> GND
- J33 pad 6: unconnected-(J33-Pin_6-Pad6) -> +3V3
- J33 pad 7: unconnected-(J33-Pin_7-Pad7) -> GND
- J33 pad 8: unconnected-(J33-Pin_8-Pad8) -> GND
- J33 pad 9: unconnected-(J33-Pin_9-Pad9) -> GND
- J33 pad MP: (no net) -> GND
- J34 pad 1: unconnected-(J34-Pin_1-Pad1) -> GND
- J34 pad 4: unconnected-(J34-Pin_4-Pad4) -> USART2_TX
- J34 pad 5: unconnected-(J34-Pin_5-Pad5) -> USART2_RX
- J35 pad 3: unconnected-(J35-Pin_3-Pad3) -> +3V3
- J35 pad 4: unconnected-(J35-Pin_4-Pad4) -> SWDIO
- J42 pad 5: unconnected-(J42-Pin_5-Pad5) -> LDAC1
- J44 pad 5: unconnected-(J44-Pin_5-Pad5) -> LDAC2
- J46 pad 5: unconnected-(J46-Pin_5-Pad5) -> LDAC3
- J48 pad 5: unconnected-(J48-Pin_5-Pad5) -> LDAC4
- J50 pad 5: unconnected-(J50-Pin_5-Pad5) -> LDAC5
- SW23 pad 2: Net-(U1-PG10) -> NRST
- U1 pad 23: unconnected-(U1-PC5-Pad23) -> MCP23S17_CS
- U1 pad 52: unconnected-(U1-PC10-Pad52) -> SPI3_CLK
- U1 pad 53: unconnected-(U1-PC11-Pad53) -> SPI3_MISO
- U1 pad 54: unconnected-(U1-PC12-Pad54) -> SPI3_MOSI
- U1 pad 59: unconnected-(U1-PB6-Pad59) -> SPI3_CS1
- U1 pad 60: unconnected-(U1-PB7-Pad60) -> SPI3_CS0
- U1 pad 7: Net-(U1-PG10) -> NRST
- U2 pad 2: unconnected-(U2-VSS-Pad2) -> GND
- U2 pad 3: unconnected-(U2-I-Pad3) -> Net-(F1-Pin_4)
- U2 pad 4: unconnected-(U2-AHLB-Pad4) -> GND
- U2 pad 5: unconnected-(U2-VDD-Pad5) -> +3V3
- U2 pad 6: unconnected-(U2-TOG-Pad6) -> GND
- U3 pad 1: Net-(U3-GND-Pad1) -> GND
- U3 pad 2: unconnected-(U3-IN2-Pad2) -> Fader_M1
- U3 pad 3: unconnected-(U3-IN1-Pad3) -> Fader_M2
- U3 pad 4: unconnected-(U3-ILIM-Pad4) -> Net-(U3-ILIM)
- U3 pad 5: unconnected-(U3-VM-Pad5) -> +10V
- U3 pad 6: unconnected-(U3-OUT1-Pad6) -> Net-(F1-Pin_6)
- U3 pad 7: Net-(U3-GND-Pad1) -> GND
- U3 pad 8: unconnected-(U3-OUT2-Pad8) -> Net-(F1-Pin_5)
- U3 pad 9: Net-(U3-GND-Pad1) -> GND
- U4 pad 1: unconnected-(U4-GPB0-Pad1) -> Net-(J63-Pin_1)
- U4 pad 10: unconnected-(U4-V_{SS}-Pad10) -> GND
- U4 pad 11: unconnected-(U4-~{CS}-Pad11) -> MCP23S17_CS
- U4 pad 12: unconnected-(U4-SCK-Pad12) -> DISP_CK
- U4 pad 13: unconnected-(U4-SI-Pad13) -> DISP_MOSI
- U4 pad 15: unconnected-(U4-A0-Pad15) -> GND
- U4 pad 16: unconnected-(U4-A1-Pad16) -> GND
- U4 pad 17: unconnected-(U4-A2-Pad17) -> GND
- U4 pad 18: unconnected-(U4-~{RESET}-Pad18) -> +3V3
- U4 pad 2: unconnected-(U4-GPB1-Pad2) -> Net-(J63-Pin_2)
- U4 pad 21: unconnected-(U4-GPA0-Pad21) -> DISP4_DC
- U4 pad 22: unconnected-(U4-GPA1-Pad22) -> DISP4_CS
- U4 pad 23: unconnected-(U4-GPA2-Pad23) -> DISP3_DC
- U4 pad 24: unconnected-(U4-GPA3-Pad24) -> DISP3_CS
- U4 pad 25: unconnected-(U4-GPA4-Pad25) -> DISP2_DC
- U4 pad 26: unconnected-(U4-GPA5-Pad26) -> DISP2_CS
- U4 pad 27: unconnected-(U4-GPA6-Pad27) -> DISP1_DC
- U4 pad 28: unconnected-(U4-GPA7-Pad28) -> DISP1_CS
- U4 pad 3: unconnected-(U4-GPB2-Pad3) -> Net-(J63-Pin_3)
- U4 pad 4: unconnected-(U4-GPB3-Pad4) -> Net-(J63-Pin_4)
- U4 pad 5: unconnected-(U4-GPB4-Pad5) -> Net-(J63-Pin_5)
- U4 pad 6: unconnected-(U4-GPB5-Pad6) -> Net-(J63-Pin_6)
- U4 pad 7: unconnected-(U4-GPB6-Pad7) -> Net-(J63-Pin_7)
- U4 pad 8: unconnected-(U4-GPB7-Pad8) -> Net-(J63-Pin_8)
- U4 pad 9: unconnected-(U4-V_{DD}-Pad9) -> +3V3
- U6 pad 14: Net-(U5-QH') -> Net-(U6-SER)
- U7 pad 1: unconnected-(U7-QB-Pad1) -> LDAC4
- U7 pad 15: unconnected-(U7-QA-Pad15) -> LDAC5
- U7 pad 2: unconnected-(U7-QC-Pad2) -> LDAC3
- U7 pad 3: unconnected-(U7-QD-Pad3) -> LDAC2
- U7 pad 4: unconnected-(U7-QE-Pad4) -> LDAC1
Routing:
- net +3V3: track 1134.4 -> 2281.7 mm, vias 22 -> 54
- net Fader_M1: track 0.00 -> 462.6 mm, vias 0 -> 2
- net Fader_M2: track 0.00 -> 455.6 mm, vias 0 -> 2
- net +5V: track 548.3 -> 886.6 mm, vias 3 -> 15
- net Fader_ADC: track 0.00 -> 335.8 mm, vias 0 -> 1
- net Net-(J27-Pin_1): track 0.00 -> 313.9 mm, vias 0 -> 10
- net DISP_MOSI: track 0.00 -> 252.9 mm, vias 0 -> 7
- net DISP_CK: track 0.00 -> 242.1 mm, vias 0 -> 7
- net DISP_PWM: track 0.00 -> 199.6 mm, vias 0 -> 2
- net LED_LAT: track 355.2 -> 536.8 mm, vias 0 -> 8
- net LED_DATA: track 0.00 -> 181.3 mm, vias 0 -> 4
- net +10V: track 114.2 -> 287.9 mm, vias 1 -> 3
- net LED_OE: track 349.3 -> 515.0 mm, vias 0 -> 7
- net USART2_TX: track 0.00 -> 160.8 mm, vias 0 -> 5
- net B2C_LED: track 0.00 -> 157.1 mm, vias 0 -> 4
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- added copper zone on B.Cu, net GND
- added copper zone on F.Cu, net GND
Other:
- board text added: "8"
- board text added: "BLK BRO RED ORA YEL GRN"
- board text added: "CONTROL VOLTAGE OUTPUTS"
- board text added: "DISP CONTROL PINS"
- board text added: "DISPLAY CONNECTORS"
- board text added: "DISP_MOSI DISP_CLK"
- board text added: "DO NOT PLACE ON A METAL SURFACE!!"
- board text added: "DRV8871 MOTOR DRIVER"
- board text added: "Darya Petrova Evan Forcucci Xinhao Chen Luke Garrity Daniel Salas"
- board text added: "EVALUATION HEADERS"
- board text added: "FULL CHANNEL STRIP EVALUATION BOARD"
- board text added: "GND CS[1] CS[0] MOSI MISO CLK VCC"
- board text added: "GND X X UART_TX UART_RX X"
- board text added: "LED DRIVER 74HCT959"
- board text added: "LINUX ls -l /dev/serial/by-id/ picocom -b 115200 /dev/ttyACM0 STM32_Programmer_CLI -c port=SWD mode=UR reset=SWrst freq=480 \ -w path/to/project/build/Debug/BucketController.elf -rst -run MAC - THRU USB HUB ls /dev/cu.* picocom -b 115200 /dev/cu.usbserial-XXXX STM32_Programmer_CLI -c port=SWD mode=UR reset=SWrst freq=480 \ -w path/to/project/build/Debug/BucketController.elf -rst -run WINDOWS POWE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"
- board text added: "MCP23S17"
- board text added: "MCP4728 ADDR PROGRAMMER"
- board text added: "PIN_NAME............PIN_NUM..DESC............... _________________________________________________ I2C1_CLK............PB8......Channel 1 Chips I2C1_DATA...........PB9...... I2C2_CLK............PA9......Channel 2 Chips I2C2_DATA...........PA8...... I2C3_CLK............PC8......Channel 3 Chips I2C3_DATA...........PB5...... I2C4_CLK............PC6......Channel 4 Chips I2C4_DATA...........PC7...... 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"
- board text added: "REV 0"
- board text added: "SKYLAR DENNO"
- board text added: "SPI MASTER"
- board text added: "SPI3"
- board text added: "STLINK-V3"
- board text added: "SWITCHES CV"
- board text added: "TTP223-BA6 TOUCH SENSOR"
- board text added: "UART DEBUG"
- board text added: "VCC CLK MOSI MISO CHSEL GND"
- board text added: "docs.skylar.lgbt"
