File: PCB_CAD/00 Development Boards/Digital System Dev/disps.kicad_sch (KiCad schematic)
At the start: 21 parts, among them J17 DISP0, J18 DISP1, J19 DISP2, J20 DISP3, Q1 2N7002

Commit message: working on the digital systems dev board project
Parts:
- removed C34: 10u, Capacitor_SMD:C_0805_2012Metric, symbol Device:C
- added C47, C49: 10u, Capacitor_SMD:C_1206_3216Metric, symbol Device:C
- C35, C36, C37, C38, C44, C45, C46, C48: LCSC C57112 -> C1590
Connections:
- net +3V3: now also C47.1, C49.1
- net GND: now also C47.2, C49.2
Other:
- note added: "BULK DECOUPLING"
- note added: "Local Decoupling"
- company: (none) -> EECE CAPSTONE
- moved on the sheet: C35, C36, C37, C38, C44, C45, C46, C48
