File: PCB_CAD/00 Development Boards/Digital System Dev/Digital System Dev.kicad_sch (KiCad schematic)
At the start: 37 parts, among them J1 STLINK, J10 F2_LOGIC, J13 F3_LOGIC, J2 FADER_POW, J24 I2C_SEL_CLK, J25 I2C_SEL_SDA, J3 F0_LOGIC, J30 I2C, J31 CTRL_POW_SR, J4 FADER_POS, J5 LED_SEL, J6 F1_LOGIC, J7 SPI_MASTER, SW1 RESET, U1 STM32G474VETx, U5 MCP4728, X1 HSE_24

Commit message: working on the digital systems dev board project
Parts:
- added C10, C11, C12, C13, C14, C15, C8, C9: 100n, Capacitor_SMD:C_0603_1608Metric, symbol Device:C
- added C60, C61: 10u, Capacitor_SMD:C_1206_3216Metric, symbol Device:C
- C3, C5, C7: LCSC C57112 -> C1590
- C4, C6: LCSC C57112 -> C1592
Connections:
- net +3V3: now also C10.1, C11.1, C12.1, C13.1, C14.1, C15.1, C60.1, C61.1, C8.1, C9.1
- net GND: now also C10.2, C11.2, C12.2, C13.2, C14.2, C15.2, C60.2, C61.2, C8.2, C9.2
Other:
- note added: "BULK DECOUPLING"
- note added: "LOCAL AT PIN DECOUPLING"
- title: (none) -> DIGITAL SYSTEMS DEV BOARD

Commit message: pushing for catching the team up later
Parts:
- C39: footprint Capacitor_SMD:C_0402_1005Metric -> Capacitor_SMD:C_0603_1608Metric; LCSC C1525 -> C1590
Changed lines of the file:
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@@
 			)
 		)
-		(property "Footprint" "Capacitor_SMD:C_0402_1005Metric"
+		(property "Footprint" "Capacitor_SMD:C_0603_1608Metric"
 			(at 192.8728 171.9212 0)
 			(hide yes)
@@
 			)
 		)
-		(property "LCSC" "C1525"
+		(property "LCSC" "C1590"
 			(at 191.9076 168.1112 0)
 			(hide yes)
