File: PCB_CAD/00 Development Boards/Digital System Dev/ctrls_leds.kicad_sch (KiCad schematic)
At the start: 47 parts, among them J101 Conn_01x04_Socket, J102 Conn_01x04_Socket, J103 Conn_01x04_Socket, J104 Conn_01x04_Socket, SW101 B2A, SW102 B2B, SW103 B2C, SW104 K1A, SW105 K1B, U101 74HCT595, U102 MCP23017x-x-SS

Commit message: working on the digital systems dev board project
Parts:
- added C50, C51: 10u, Capacitor_SMD:C_1206_3216Metric, symbol Device:C
- C110, C117, C123: LCSC C57112 -> C1590
Connections:
- net +3V3: now also C50.1, C51.1
- net GND: now also C50.2, C51.2
Other:
- note added: "LED DRIVER"
- note added: "MCP23017 GPIO"
- note added: "ONBOARD CONTROLS + HARDWARE DEBOUNCE"
- note removed: "ONBOARD CONTROLS"
- company: (none) -> EECE CAPSTONE
- moved on the sheet: C110, C123, J101, J102, J103, J104, U101, U102

Commit message: pushing for catching the team up later
Parts:
- C101, C102, C103: LCSC C15849 -> C1592
Changed lines of the file:
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@@
 			)
 		)
-		(property "LCSC" "C15849"
+		(property "LCSC" "C1592"
 			(at 232.41 83.82 0)
 			(hide yes)
@@
 			)
 		)
-		(property "LCSC" "C15849"
+		(property "LCSC" "C1592"
 			(at 87.63 83.82 0)
 			(hide yes)
@@
 			)
 		)
-		(property "LCSC" "C15849"
+		(property "LCSC" "C1592"
 			(at 160.02 83.82 0)
 			(hide yes)
