File: PCB_CAD/Development Boards/Digital System Dev/cv_sw.kicad_sch (KiCad schematic)
At the start: 30 parts, among them J26 CV_SW_1, J27 CV_SW_2, J28 CV_SW_4, J29 CV_SW_3, U28 74HC595, U29 74HC595, U30 74HC595, U31 74HC595, U32 74HC595, U33 74HC595, U34 74HC595, U35 74HC595, U36 74HC595, U37 74HC595, U38 74HC595, U39 74HC595

Commit message: pcb for displays
Parts:
- added C100, C101, C102, C103, C104, C105, C106, C107, C108, C109, C110, C111, C112, C113, C114, C115, C116, C117, C118, C119, C120, C121, C122, C123, C124, C125, C126, C127, C128, C129, C130, C131, C132, C133, C134, C135, C136, C137, C138, C139, C140, C141, C142, C143, C144, C145, C146, C147, C148, C149, C150, C151, C152, C153, C154, C155, C156, C157, C158, C159, C160, C161, C162, C163, C164, C165, C166, C167, C168, C169, C74, C75, C76, C77, C78, C79, C80, C81, C82, C83, C84, C85, C86, C87, C88, C89, C90, C91, C92, C93, C94, C95, C96, C97, C98, C99: 100n, Capacitor_SMD:C_0603_1608Metric, symbol Device:C_Small
- added C170, C171, C172, C173, C174, C175, C176, C177, C178, C179, C180, C181: 100n, Capacitor_SMD:C_0603_1608Metric, symbol Device:C
Connections:
- net +3V3: now also C170.1, C171.1, C172.1, C173.1, C174.1, C175.1, C176.1, C177.1, C178.1, C179.1, C180.1, C181.1
- net 1_1: now also C121.1
- net 1_10: now also C126.1
- net 1_11: now also C116.1
- net 1_12: now also C127.1
- net 1_13: now also C133.1
- net 1_14: now also C110.1
- net 1_15: now also C132.1
- net 1_16: now also C111.1
- net 1_17: now also C131.1
- net 1_18: now also C112.1
- net 1_19: now also C130.1
- net 1_2: now also C122.1
- net 1_20: now also C113.1
- net 1_21: now also C129.1
- net 1_22: now also C114.1
- net 1_23: now also C128.1
- net 1_24: now also C115.1
- net 1_3: now also C120.1
- net 1_4: now also C123.1
- net 1_5: now also C119.1
- net 1_6: now also C124.1
- net 1_7: now also C118.1
- net 1_8: now also C125.1
- net 1_9: now also C117.1
- net 2_1: now also C97.1
- net 2_10: now also C150.1
- net 2_11: now also C92.1
- net 2_12: now also C151.1
- net 2_13: now also C157.1
- net 2_14: now also C86.1
- net 2_15: now also C156.1
- net 2_16: now also C87.1
- net 2_17: now also C155.1
- net 2_18: now also C88.1
- net 2_19: now also C154.1
- net 2_2: now also C146.1
- net 2_20: now also C89.1
- net 2_21: now also C153.1
- net 2_22: now also C90.1
- net 2_23: now also C152.1
- net 2_24: now also C91.1
- net 2_3: now also C96.1
- net 2_4: now also C147.1
- net 2_5: now also C95.1
- net 2_6: now also C148.1
- net 2_7: now also C94.1
- net 2_8: now also C149.1
- net 2_9: now also C93.1
- net 3_1: now also C109.1
- net 3_10: now also C138.1
- net 3_11: now also C104.1
- net 3_12: now also C139.1
- net 3_13: now also C145.1
- net 3_14: now also C98.1
- net 3_15: now also C144.1
- net 3_16: now also C99.1
- net 3_17: now also C143.1
- net 3_18: now also C100.1
- net 3_19: now also C142.1
- net 3_2: now also C134.1
- net 3_20: now also C101.1
- net 3_21: now also C141.1
- net 3_22: now also C102.1
- net 3_23: now also C140.1
- net 3_24: now also C103.1
- net 3_3: now also C108.1
- net 3_4: now also C135.1
- net 3_5: now also C107.1
- net 3_6: now also C136.1
- net 3_7: now also C106.1
- net 3_8: now also C137.1
- net 3_9: now also C105.1
- net 4_1: now also C79.1
- net 4_10: now also C168.1
- net 4_11: now also C74.1
- net 4_12: now also C169.1
- net 4_13: now also C163.1
- net 4_14: now also C85.1
- net 4_15: now also C162.1
- net 4_16: now also C84.1
- net 4_17: now also C161.1
- net 4_18: now also C83.1
- net 4_19: now also C160.1
- net 4_2: now also C164.1
- net 4_20: now also C82.1
- net 4_21: now also C159.1
- net 4_22: now also C81.1
- net 4_23: now also C158.1
- net 4_24: now also C80.1
- net 4_3: now also C78.1
- net 4_4: now also C165.1
- net 4_5: now also C77.1
- net 4_6: now also C166.1
- net 4_7: now also C76.1
- net 4_8: now also C167.1
- net 4_9: now also C75.1
- net GND: now also C100.2, C101.2, C102.2, C103.2, C104.2, C105.2, C106.2, C107.2, C108.2, C109.2, C110.2, C111.2, C112.2, C113.2, C114.2, C115.2, C116.2, C117.2, C118.2, C119.2, C120.2, C121.2, C122.2, C123.2, C124.2, C125.2, C126.2, C127.2, C128.2, C129.2, C130.2, C131.2, C132.2, C133.2, C134.2, C135.2, C136.2, C137.2, C138.2, C139.2, C140.2, C141.2, C142.2, C143.2, C144.2, C145.2, C146.2, C147.2, C148.2, C149.2, C150.2, C151.2, C152.2, C153.2, C154.2, C155.2, C156.2, C157.2, C158.2, C159.2, C160.2, C161.2, C162.2, C163.2, C164.2, C165.2, C166.2, C167.2, C168.2, C169.2, C170.2, C171.2, C172.2, C173.2, C174.2, C175.2, C176.2, C177.2, C178.2, C179.2, C180.2, C181.2, C74.2, C75.2, C76.2, C77.2, C78.2, C79.2, C80.2, C81.2, C82.2, C83.2, C84.2, C85.2, C86.2, C87.2, C88.2, C89.2, C90.2, C91.2, C92.2, C93.2, C94.2, C95.2, C96.2, C97.2, C98.2, C99.2
Other:
- moved on the sheet: C41, C42, J26, J27, J28, J29
