File: PCB_CAD/Development Boards/Digital System Dev/power.kicad_sch (KiCad schematic)
At the start: 50 parts, among them J15 DC_10V, J8 EXT_POW_IN, U4 TPS54302DDCT, U6 TPS54302DDCT

Commit message: pcb for displays
Parts:
- removed C16, C17, C18, C21, C31, C33: 20p, Capacitor_SMD:C_0603_1608Metric, symbol Device:C_Small
- removed C24, C27: 1u, Capacitor_SMD:C_0603_1608Metric, symbol Device:C
- removed C28, C32: 33u, Capacitor_SMD:CP_Elec_6.3x5.4, symbol Device:C_Polarized
- removed C40, C53, C56: 100n, Capacitor_SMD:C_0603_1608Metric, symbol Device:C
- removed C52, C54, C55, C57: 10u, Capacitor_SMD:C_1206_3216Metric, symbol Device:C
- removed C58, C59: 100n, Capacitor_SMD:C_0603_1608Metric, symbol Device:C_Small
- removed D3: LED, LED_SMD:LED_0603_1608Metric, symbol Device:LED
- removed D6: 2N5062, Package_TO_SOT_THT:TO-92, symbol Device:Q_SCR_KGA
- removed DZ3: BZG04-12, PCM_4ms_Diode:D_DO-214AC_SMA, symbol PCM_Diode_Zener_AKL:D_Zener_Generic
- removed J15: DC_10V, Connector_BarrelJack:BarrelJack_Horizontal, symbol Connector:Jack-DC
- removed L1, L2: 6.8u, Inductor_SMD:L_1210_3225Metric, symbol Device:L_Small
- removed R23: 1k, Resistor_SMD:R_0603_1608Metric, symbol Device:R_US
- removed R24: 12k, Resistor_SMD:R_0603_1608Metric, symbol Device:R_US
- removed R3: 22.1k, Resistor_SMD:R_0805_2012Metric, symbol Device:R_Small_US
- removed R4, R6: 100k, symbol Device:R_Small_US
- removed R5: 13.5k, Resistor_SMD:R_0603_1608Metric, symbol Device:R_Small_US
- removed TP11: TestPoint_Probe, TestPoint:TestPoint_Keystone_5019_Miniature, symbol Connector:TestPoint_Probe
- removed U4, U6: TPS54302DDCT, Package_TO_SOT_SMD:SOT-23-6, symbol Regulator_Switching:TPS54302
Connections:
- net +10V is gone; now on net GND: J8.3 (Pin_3)
- no-connect marks 2 -> 0
Other:
- note removed: "3V3 RAIL CONVERTER REGULATOR"
- note removed: "5V RAIL CONVERTER REGULATOR"

Commit message: digital dev (or maybe final) board
Parts:
- removed C22, C29: 100n, Capacitor_SMD:C_0603_1608Metric, symbol Device:C
- removed D1, D2: LED, LED_SMD:LED_0603_1608Metric, symbol Device:LED
- removed D4, D5: 2N5062, Package_TO_SOT_THT:TO-92, symbol Device:Q_SCR_KGA
- removed DZ1: MMSZ5227B, Diode_SMD:D_SOD-123, symbol PCM_Diode_Zener_AKL:D_Zener_Generic
- removed DZ2: MMSZ5233BT1G, Diode_SMD:D_SOD-123, symbol PCM_Diode_Zener_AKL:D_Zener_Generic
- removed J8: EXT_POW_IN, Connector_PinHeader_2.54mm:PinHeader_1x04_P2.54mm_Vertical, symbol Connector:Conn_01x04_Pin
- removed R15, R22: 1k, Resistor_SMD:R_0603_1608Metric, symbol Device:R_US
- removed R16: 680, Resistor_SMD:R_0603_1608Metric, symbol Device:R_US
- removed R17: 3.3k, Resistor_SMD:R_0603_1608Metric, symbol Device:R_US
- removed TP10, TP19, TP9: TestPoint_Probe, TestPoint:TestPoint_Keystone_5019_Miniature, symbol Connector:TestPoint_Probe
Other:
- note removed: "LED INDICATORS"
- note removed: "OVERVOLT PROTECTION"
- note removed: "POWER INPUT"
