File: PCB_CAD/PAN_FADER/PAN_FADER.kicad_pcb (KiCad board)
At the start: 4 copper layers, 36 x 110 mm, 87 parts, among them J1 COMP_CV, J2 CV_FROM_DAC, J3 POWER, J4 INTERNAL_AUDIO_CONN, J5 TO_INSERT_MATRIX, U1 THAT2180A, U2 OPA1679, U3 OPA1637, U4 TL074, U5 THAT2180A, U7 OPA1637, U8 ADR5041, U9 ADG1436

Commit message: fader/pan analog board
Parts:
- added REF**: Screw_Generic_2.0x3.0mm_SilkScreen, Symbol:Screw_Generic_2.0x3.0mm_SilkScreen, F.Cu at (102.5, 99.2)
- added REF**: LayerMarker_4_6.35x2.54mm_TextH1mm_P1.27mm_BottomMirrored, Symbol:LayerMarker_4_6.35x2.54mm_TextH1mm_P1.27mm_BottomMirrored, F.Cu at (104.0, 111.0)
- added REF**: Screw_Generic_2.0x3.0mm_SilkScreen, Symbol:Screw_Generic_2.0x3.0mm_SilkScreen, F.Cu at (134.2, 52.5)
- H1, H2: footprint MountingHole:MountingHole_3.2mm_M3_DIN965_Pad_TopBottom -> MountingHole:MountingHole_2.2mm_M2
- U3, U7: footprint Package_SO:VSSOP-8_3x3mm_P0.65mm -> Package_SO:Texas_S-PDSO-G8_3x3mm_P0.65mm
Routing:
- net GND: vias 41 -> 100
Other:
- board text added: "+15V GND -15V"
- board text added: "1"
- board text added: "AUD PRE AUD IN GND MIXBUS R- MIXBUS R+ MIXBUS L- MIXBUS L+"
- board text added: "AUDIO I/O"
- board text added: "COMP CV"
- board text added: "COMP NO"
- board text added: "CTRL Vs"
- board text added: "Channel Output VCA Card"
- board text added: "GND LCV:PRE LCV:INS CV:R_GAIN CV:L_GAIN"
- board text added: "INSERT"
- board text added: "POWER"
- board text added: "RTN SEND GND"
- board text added: "S.E.D. REV 0 2026 RoHS"
- board text removed: "S.E.D. REV 0 2026"
