File: PCB_CAD/BUCKET_CONTROLS/bucket_controls.kicad_pcb (KiCad board)
At the start: 4 copper layers, 146 x 380 mm, 924 parts, among them J1 Pow, J10 Data, J101 Pow, J102 Data, J103 Pow, J104 Data, J105 Pow, J106 Data, J107 Pow, J108 Data, J109 Pow, J11 Pow, J110 Data, J111 Pow, J112 Data, J113 Pow, J114 Data, J115 Pow, J116 Data, J117 Pow, J118 Data, J119 Pow, J12 Data, J120 Data, J13 Pow, J14 Data, J15 Pow, J16 Data, J17 Pow, J18 Data, J19 Pow, J2 Data, J20 Data, J201 Pow, J202 Data, J203 Pow, J204 Data, J205 Pow, J206 Data, J207 Pow, J208 Data, J209 Pow, J21 DISP0, J210 Data, J211 Pow, J212 Data, J213 Pow, J214 Data, J215 Pow, J216 Data, J217 Pow, J218 Data, J219 Pow, J22 DISP1, J220 Data, J23 DISP2, J24 DISP3, J25 DISP0A, J26 DISP1A, J27 DISP2A, J28 DISP3A, J3 Pow, J301 Pow, J302 Data, J303 Pow, J304 Data, J305 Pow, J306 Data, J307 Pow, J308 Data, J309 Pow, J310 Data, J311 Pow, J312 Data, J313 Pow, J314 Data, J315 Pow, J316 Data, J317 Pow, J318 Data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

Commit message: more pcbs
Parts:
- removed C131, C132, C133, C134, C135, C136, C137, C138, C139, C140, C141, C142, C231, C232, C233, C234, C235, C236, C237, C238, C239, C240, C241, C242, C331, C332, C333, C334, C335, C336, C337, C338, C339, C340, C341, C342: 1u, Capacitor_SMD:C_0603_1608Metric
- removed D101, D105, D106, D107, D111, D112, D113, D114, D115, D116, D117, D118, D201, D205, D206, D207, D211, D212, D213, D214, D215, D216, D217, D218, D301, D305, D306, D307, D311, D312, D313, D314, D315, D316, D317, D318: 1N4148, Diode_SMD:D_SOD-323
- removed D102, D103, D104, D108, D109, D110, D119, D120, D202, D203, D204, D208, D209, D210, D219, D220, D302, D303, D304, D308, D309, D310, D319, D320: LED, LED_THT:LED_D3.0mm_FlatTop
- removed R161, R167, R168, R169, R176, R177, R178, R185, R186, R187, R194, R195, R261, R267, R268, R269, R276, R277, R278, R285, R286, R287, R294, R295, R361, R367, R368, R369, R376, R377, R378, R385, R386, R387, R394, R395: 47k, Resistor_SMD:R_0603_1608Metric
- removed R162, R170, R171, R172, R179, R180, R181, R188, R189, R190, R196, R197, R262, R270, R271, R272, R279, R280, R281, R288, R289, R290, R296, R297, R362, R370, R371, R372, R379, R380, R381, R388, R389, R390, R396, R397: 15k, Resistor_SMD:R_0603_1608Metric
- removed R163, R164, R165, R166, R173, R174, R175, R182, R183, R184, R191, R192, R193, R198, R199, R263, R264, R265, R266, R273, R274, R275, R282, R283, R284, R291, R292, R293, R298, R299, R363, R364, R365, R366, R373, R374, R375, R382, R383, R384, R391, R392, R393, R398, R399: 330, Resistor_SMD:R_0603_1608Metric
- removed SW111: C1_B0, My Footprints:CFPB-1CC-4W6
- removed SW112: C1_B1, My Footprints:TL2201EEZB
- removed SW113: C1_B2, My Footprints:TL2201EEZB
- removed SW114: C1_B3, My Footprints:TL2201EEZB
- removed SW115: C1_B4, My Footprints:CFPB-1CC-4W6
- removed SW116: C1_B5, My Footprints:CFPB-1CC-4W6
- removed SW117: C1_B6, My Footprints:CFPB-1CC-4W6
- removed SW118: C1_B7, My Footprints:CFPB-1CC-4W6
- removed SW119: C1_B8, My Footprints:CFPB-1CC-4W6
- removed SW120: C1_B9, My Footprints:CFPB-1CC-4W6
- removed SW121: C1_B10, My Footprints:TL2201EEZB
- removed SW122: C1_B11, My Footprints:TL2201EEZB
- removed SW211: C2_B0, My Footprints:CFPB-1CC-4W6
- removed SW212: C2_B1, My Footprints:TL2201EEZB
- removed SW213: C2_B2, My Footprints:TL2201EEZB
- removed SW214: C2_B3, My Footprints:TL2201EEZB
- removed SW215: C2_B4, My Footprints:CFPB-1CC-4W6
- removed SW216: C2_B5, My Footprints:CFPB-1CC-4W6
- removed SW217: C2_B6, My Footprints:CFPB-1CC-4W6
- removed SW218: C2_B7, My Footprints:CFPB-1CC-4W6
- removed SW219: C2_B8, My Footprints:CFPB-1CC-4W6
- removed SW220: C2_B9, My Footprints:CFPB-1CC-4W6
- removed SW221: C2_B10, My Footprints:TL2201EEZB
- removed SW222: C2_B11, My Footprints:TL2201EEZB
- removed SW311: C3_B0, My Footprints:CFPB-1CC-4W6
- removed SW312: C3_B1, My Footprints:TL2201EEZB
- removed SW313: C3_B2, My Footprints:TL2201EEZB
- removed SW314: C3_B3, My Footprints:TL2201EEZB
- removed SW315: C3_B4, My Footprints:CFPB-1CC-4W6
- removed SW316: C3_B5, My Footprints:CFPB-1CC-4W6
- removed SW317: C3_B6, My Footprints:CFPB-1CC-4W6
- removed SW318: C3_B7, My Footprints:CFPB-1CC-4W6
- removed SW319: C3_B8, My Footprints:CFPB-1CC-4W6
- removed SW320: C3_B9, My Footprints:CFPB-1CC-4W6
- removed SW321: C3_B10, My Footprints:TL2201EEZB
- removed SW322: C3_B11, My Footprints:TL2201EEZB
- moved C100 258.7 mm to (740.7, -99.9)
- moved C143 258.7 mm to (707.3, -101.8)
- moved C144 258.7 mm to (707.3, -99.9)
- moved C43 258.7 mm to (698.1, -132.3)
- moved C49 258.7 mm to (698.1, -124.8)
- moved C50 258.7 mm to (709.6, -126.7)
- moved C53 258.7 mm to (702.1, -132.3)
- moved C58 258.7 mm to (712.5, -126.7)
- moved C59 258.7 mm to (734.9, -103.8)
- moved C60 258.7 mm to (734.9, -101.8)
- moved C61 258.7 mm to (734.9, -99.9)
- moved C62 258.7 mm to (701.6, -103.8)
- moved C63 258.7 mm to (701.6, -101.8)
- moved C64 258.7 mm to (701.6, -99.9)
- moved C71 258.7 mm to (737.8, -103.8)
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Routing:
- added copper zone on In2.Cu, net GND
- removed copper zone on In2.Cu, net +5V
Other:
- board size 146 x 380 mm -> 146 x 320 mm
