File: PCB_CAD/BUCKET_CONTROLS/gpio1.kicad_sch (KiCad schematic)
At the start: 16 parts, among them U12 MCP23017_I2C2_0x20, U13 MCP23017_I2C2_0x21, U14 MCP23017_I2C2_0x22

Commit message: pcb controls
Parts:
- U12, U13, U14: footprint Package_SO:SSOP-28_5.3x10.2mm_P0.65mm -> Package_DFN_QFN:QFN-28-1EP_6x6mm_P0.65mm_EP4.25x4.25mm; symbol Interface_Expansion:MCP23017x-x-SS -> Interface_Expansion:MCP23017x-x-ML; LCSC C558584 -> C629439
Connections:
- net +3V3: now also U12.5 (V_{DD}), U13.11 (A0), U13.5 (V_{DD}), U14.12 (A1), U14.5 (V_{DD}); no longer U12.9 (V_{DD}), U13.15 (A0), U13.9 (V_{DD}), U14.16 (A1), U14.9 (V_{DD})
- net C1_B0: now also U14.19 (GPA2); no longer U14.23 (GPA2)
- net C1_B1: now also U14.20 (GPA3); no longer U14.24 (GPA3)
- net C1_B10: now also U14.2 (GPB5); no longer U14.6 (GPB5)
- net C1_B11: now also U14.3 (GPB6); no longer U14.7 (GPB6)
- net C1_B2: now also U14.21 (GPA4); no longer U14.25 (GPA4)
- net C1_B3: now also U14.22 (GPA5); no longer U14.26 (GPA5)
- net C1_B4: now also U14.23 (GPA6); no longer U14.27 (GPA6)
- net C1_B5: now also U14.25 (GPB0); no longer U14.1 (GPB0)
- net C1_B6: now also U14.26 (GPB1); no longer U14.2 (GPB1)
- net C1_B7: now also U14.27 (GPB2); no longer U14.3 (GPB2)
- net C1_B8: now also U14.28 (GPB3); no longer U14.4 (GPB3)
- net C1_B9: now also U14.1 (GPB4); no longer U14.5 (GPB4)
- net C1_K0_A: now also U12.17 (GPA0); no longer U12.21 (GPA0)
- net C1_K0_B: now also U12.25 (GPB0); no longer U12.1 (GPB0)
- net C1_K0_Push: now also U12.22 (GPA5); no longer U12.26 (GPA5)
- net C1_K1_A: now also U12.18 (GPA1); no longer U12.22 (GPA1)
- net C1_K1_B: now also U12.26 (GPB1); no longer U12.2 (GPB1)
- net C1_K1_Push: now also U12.23 (GPA6); no longer U12.27 (GPA6)
- net C1_K2_A: now also U12.19 (GPA2); no longer U12.23 (GPA2)
- net C1_K2_B: now also U12.27 (GPB2); no longer U12.3 (GPB2)
- net C1_K2_Push: now also U12.2 (GPB5); no longer U12.6 (GPB5)
- net C1_K3_A: now also U12.20 (GPA3); no longer U12.24 (GPA3)
- net C1_K3_B: now also U12.28 (GPB3); no longer U12.4 (GPB3)
- net C1_K3_Push: now also U12.3 (GPB6); no longer U12.7 (GPB6)
- net C1_K4_A: now also U12.21 (GPA4); no longer U12.25 (GPA4)
- net C1_K4_B: now also U12.1 (GPB4); no longer U12.5 (GPB4)
- net C1_K4_Push: now also U13.22 (GPA5); no longer U13.26 (GPA5)
- net C1_K5_A: now also U13.17 (GPA0); no longer U13.21 (GPA0)
- net C1_K5_B: now also U13.25 (GPB0); no longer U13.1 (GPB0)
- net C1_K5_Push: now also U13.23 (GPA6); no longer U13.27 (GPA6)
- net C1_K6_A: now also U13.18 (GPA1); no longer U13.22 (GPA1)
- net C1_K6_B: now also U13.26 (GPB1); no longer U13.2 (GPB1)
- net C1_K6_Push: now also U13.2 (GPB5); no longer U13.6 (GPB5)
- net C1_K7_A: now also U13.19 (GPA2); no longer U13.23 (GPA2)
- net C1_K7_B: now also U13.27 (GPB2); no longer U13.3 (GPB2)
- net C1_K7_Push: now also U13.3 (GPB6); no longer U13.7 (GPB6)
- net C1_K8_A: now also U13.20 (GPA3); no longer U13.24 (GPA3)
- net C1_K8_B: now also U13.28 (GPB3); no longer U13.4 (GPB3)
- net C1_K8_Push: now also U14.17 (GPA0); no longer U14.21 (GPA0)
- net C1_K9_A: now also U13.21 (GPA4); no longer U13.25 (GPA4)
- net C1_K9_B: now also U13.1 (GPB4); no longer U13.5 (GPB4)
- net C1_K9_Push: now also U14.18 (GPA1); no longer U14.22 (GPA1)
- net I2C2_CLK: now also U12.8 (SCK), U13.8 (SCK), U14.8 (SCK); no longer U12.12 (SCK), U13.12 (SCK), U14.12 (SCK)
- net I2C2_SDA: now also U12.9 (SDA), U13.9 (SDA), U14.9 (SDA); no longer U12.13 (SDA), U13.13 (SDA), U14.13 (SDA)
- net at C74.1, R400.2: now also U12.14 (~{RESET}); no longer U12.18 (~{RESET})
- net at C76.1, R402.2: now also U14.14 (~{RESET}); no longer U14.18 (~{RESET})
- net at C75.1, R401.2: now also U13.14 (~{RESET}); no longer U13.18 (~{RESET})
- net at U14.11 (A0): now also U14.13 (A2), U14.6 (V_{SS})
- net at U12.11 (A0): now also U12.12 (A1), U12.13 (A2), U12.6 (V_{SS})
- new net: U13.12 (A1), U13.13 (A2), U13.6 (V_{SS})
- now unconnected: U12.10 (V_{SS}), U12.15 (A0), U12.16 (A1), U13.10 (V_{SS}), U13.16 (A1), U14.10 (V_{SS}), U14.15 (A0)
Changed lines of the file:
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@@
 	)
 	(symbol
-		(lib_id "Interface_Expansion:MCP23017x-x-SS")
+		(lib_id "Interface_Expansion:MCP23017x-x-ML")
 		(at 193.04 77.47 0)
 		(unit 1)
@@
 			)
 		)
-		(property "Footprint" "Package_SO:SSOP-28_5.3x10.2mm_P0.65mm"
+		(property "Footprint" "Package_DFN_QFN:QFN-28-1EP_6x6mm_P0.65mm_EP4.25x4.25mm"
 			(at 198.12 102.87 0)
 			(hide yes)
@@
 			)
 		)
-		(property "Description" "16-bit I/O expander, I2C, interrupts, w pull-ups, SSOP-28"
+		(property "Description" "16-bit I/O expander, I2C, interrupts, w pull-ups, GPA7/GPB7 output only (https://microchip.my.site.com/s/article/GPA7---GPB7-Cannot-Be-Used-as-Inputs-In-MCP23017), QFN-28"
 			(at 193.04 77.47 0)
 			(hide yes)
@@
 			)
 		)
-		(property "LCSC" "C558584"
+		(property "LCSC" "C629439"
 			(at 193.04 77.47 0)
 			(hide yes)
@@
 		)
 		(pin "25"
+		)
+		(pin "29"
 		)
 		(instances
@@
 	)
 	(symbol
-		(lib_id "Interface_Expansion:MCP23017x-x-SS")
+		(lib_id "Interface_Expansion:MCP23017x-x-ML")
 		(at 88.9 77.47 0)
 		(unit 1)
@@
 			)
 		)
-		(property "Footprint" "Package_SO:SSOP-28_5.3x10.2mm_P0.65mm"
+		(property "Footprint" "Package_DFN_QFN:QFN-28-1EP_6x6mm_P0.65mm_EP4.25x4.25mm"
 			(at 93.98 102.87 0)
 			(hide yes)
@@
 			)
 		)
-		(property "Description" "16-bit I/O expander, I2C, interrupts, w pull-ups, SSOP-28"
+		(property "Description" "16-bit I/O expander, I2C, interrupts, w pull-ups, GPA7/GPB7 output only (https://microchip.my.site.com/s/article/GPA7---GPB7-Cannot-Be-Used-as-Inputs-In-MCP23017), QFN-28"
 			(at 88.9 77.47 0)
 			(hide yes)
@@
 			)
 		)
-		(property "LCSC" "C558584"
+		(property "LCSC" "C629439"
 			(at 88.9 77.47 0)
 			(hide yes)
@@
 		)
 		(pin "28"
+		)
+		(pin "29"
 		)
 		(instances
@@
 	)
 	(symbol
-		(lib_id "Interface_Expansion:MCP23017x-x-SS")
+		(lib_id "Interface_Expansion:MCP23017x-x-ML")
 		(at 140.97 77.47 0)
 		(unit 1)
@@
 			)
 		)
-		(property "Footprint" "Package_SO:SSOP-28_5.3x10.2mm_P0.65mm"
+		(property "Footprint" "Package_DFN_QFN:QFN-28-1EP_6x6mm_P0.65mm_EP4.25x4.25mm"
 			(at 146.05 102.87 0)
 			(hide yes)
@@
 			)
 		)
-		(property "Description" "16-bit I/O expander, I2C, interrupts, w pull-ups, SSOP-28"
+		(property "Description" "16-bit I/O expander, I2C, interrupts, w pull-ups, GPA7/GPB7 output only (https://microchip.my.site.com/s/article/GPA7---GPB7-Cannot-Be-Used-as-Inputs-In-MCP23017), QFN-28"
 			(at 140.97 77.47 0)
 			(hide yes)
@@
 			)
 		)
-		(property "LCSC" "C558584"
+		(property "LCSC" "C629439"
 			(at 140.97 77.47 0)
 			(hide yes)
@@
 		(pin "26"
 		)
-		(instances
+		(pin "29"
+		)
+		(instances

Commit message: save pcb progress lol
Parts:
- removed C143, C144, C96: 100n, Capacitor_SMD:C_0402_1005Metric, symbol Device:C
Connections:
- net GND: now also U12.11 (A0), U12.12 (A1), U12.13 (A2), U12.29 (EP), U12.6 (V_{SS}), U13.12 (A1), U13.13 (A2), U13.29 (EP), U13.6 (V_{SS}), U14.11 (A0), U14.13 (A2), U14.29 (EP), U14.6 (V_{SS})

Commit message: pcb routing all day
Connections:
- net C1_B4: now also U14.26 (GPB1); no longer U14.23 (GPA6)
- net C1_B6: now also U14.23 (GPA6); no longer U14.26 (GPB1)
- net C1_B10 renamed btnA_1
- net C1_B11 renamed btnB_1
Changed lines of the file:
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@@
 	(global_label "C1_B4"
 		(shape input)
-		(at 205.74 72.39 0)
-		(fields_autoplaced yes)
-		(effects
-			(font
-				(size 1.27 1.27)
-			)
-			(justify left)
-		)
-		(property "Intersheetrefs" "${INTERSHEET_REFS}"
-			(at 214.6518 72.39 0)
+		(at 205.74 82.55 0)
+		(fields_autoplaced yes)
+		(effects
+			(font
+				(size 1.27 1.27)
+			)
+			(justify left)
+		)
+		(property "Intersheetrefs" "${INTERSHEET_REFS}"
+			(at 214.6518 82.55 0)
 			(hide yes)
 			(show_name no)
@@
 		)
 	)
-	(global_label "C1_B11"
-		(shape input)
-		(at 205.74 95.25 0)
-		(fields_autoplaced yes)
-		(effects
-			(font
-				(size 1.27 1.27)
-			)
-			(justify left)
-		)
-		(property "Intersheetrefs" "${INTERSHEET_REFS}"
-			(at 215.8613 95.25 0)
+	(global_label "btnA_1"
+		(shape output)
+		(at 205.74 92.71 0)
+		(fields_autoplaced yes)
+		(effects
+			(font
+				(size 1.27 1.27)
+				(color 255 255 255 1)
+			)
+			(justify left)
+		)
+		(property "Intersheetrefs" "${INTERSHEET_REFS}"
+			(at 215.0146 92.71 0)
 			(hide yes)
 			(show_name no)
@@
 		)
 	)
-	(global_label "C1_B10"
-		(shape input)
-		(at 205.74 92.71 0)
-		(fields_autoplaced yes)
-		(effects
-			(font
-				(size 1.27 1.27)
-			)
-			(justify left)
-		)
-		(property "Intersheetrefs" "${INTERSHEET_REFS}"
-			(at 215.8613 92.71 0)
+	(global_label "btnB_1"
+		(shape output)
+		(at 205.74 95.25 0)
+		(fields_autoplaced yes)
+		(effects
+			(font
+				(size 1.27 1.27)
+				(color 255 255 255 1)
+			)
+			(justify left)
+		)
+		(property "Intersheetrefs" "${INTERSHEET_REFS}"
+			(at 215.196 95.25 0)
 			(hide yes)
 			(show_name no)
@@
 	(global_label "C1_B6"
 		(shape input)
-		(at 205.74 82.55 0)
-		(fields_autoplaced yes)
-		(effects
-			(font
-				(size 1.27 1.27)
-			)
-			(justify left)
-		)
-		(property "Intersheetrefs" "${INTERSHEET_REFS}"
-			(at 214.6518 82.55 0)
-			(hide yes)
-			(show_name no)
+		(at 205.74 72.39 0)
+		(fields_autoplaced yes)
+		(effects
+			(font
+				(size 1.27 1.27)
+			)
+			(justify left)
+		)
+		(property "Intersheetrefs" "${INTERSHEET_REFS}"
+			(at 214.6518 72.39 0)
+			(hide yes)
+			(show_name no)
