File: PCB_CAD/BUCKET_CONTROLS/gpio3.kicad_sch (KiCad schematic)
At the start: 16 parts, among them U16 MCP23017_I2C4_0x20, U18 MCP23017_I2C4_0x21, U20 MCP23017_I2C4_0x22

Commit message: pcb controls
Parts:
- U16, U18, U20: footprint Package_SO:SSOP-28_5.3x10.2mm_P0.65mm -> Package_DFN_QFN:QFN-28-1EP_6x6mm_P0.65mm_EP4.25x4.25mm; symbol Interface_Expansion:MCP23017x-x-SS -> Interface_Expansion:MCP23017x-x-ML; LCSC C558584 -> C629439
Connections:
- net +3V3: now also U16.5 (V_{DD}), U18.11 (A0), U18.5 (V_{DD}), U20.12 (A1), U20.5 (V_{DD}); no longer U16.9 (V_{DD}), U18.15 (A0), U18.9 (V_{DD}), U20.16 (A1), U20.9 (V_{DD})
- net C3_B0: now also U20.19 (GPA2); no longer U20.23 (GPA2)
- net C3_B1: now also U20.20 (GPA3); no longer U20.24 (GPA3)
- net C3_B10: now also U20.2 (GPB5); no longer U20.6 (GPB5)
- net C3_B11: now also U20.3 (GPB6); no longer U20.7 (GPB6)
- net C3_B2: now also U20.21 (GPA4); no longer U20.25 (GPA4)
- net C3_B3: now also U20.22 (GPA5); no longer U20.26 (GPA5)
- net C3_B4: now also U20.23 (GPA6); no longer U20.27 (GPA6)
- net C3_B5: now also U20.25 (GPB0); no longer U20.1 (GPB0)
- net C3_B6: now also U20.26 (GPB1); no longer U20.2 (GPB1)
- net C3_B7: now also U20.27 (GPB2); no longer U20.3 (GPB2)
- net C3_B8: now also U20.28 (GPB3); no longer U20.4 (GPB3)
- net C3_B9: now also U20.1 (GPB4); no longer U20.5 (GPB4)
- net C3_K0_A: now also U16.17 (GPA0); no longer U16.21 (GPA0)
- net C3_K0_B: now also U16.25 (GPB0); no longer U16.1 (GPB0)
- net C3_K0_Push: now also U16.22 (GPA5); no longer U16.26 (GPA5)
- net C3_K1_A: now also U16.18 (GPA1); no longer U16.22 (GPA1)
- net C3_K1_B: now also U16.26 (GPB1); no longer U16.2 (GPB1)
- net C3_K1_Push: now also U16.23 (GPA6); no longer U16.27 (GPA6)
- net C3_K2_A: now also U16.19 (GPA2); no longer U16.23 (GPA2)
- net C3_K2_B: now also U16.27 (GPB2); no longer U16.3 (GPB2)
- net C3_K2_Push: now also U16.2 (GPB5); no longer U16.6 (GPB5)
- net C3_K3_A: now also U16.20 (GPA3); no longer U16.24 (GPA3)
- net C3_K3_B: now also U16.28 (GPB3); no longer U16.4 (GPB3)
- net C3_K3_Push: now also U16.3 (GPB6); no longer U16.7 (GPB6)
- net C3_K4_A: now also U16.21 (GPA4); no longer U16.25 (GPA4)
- net C3_K4_B: now also U16.1 (GPB4); no longer U16.5 (GPB4)
- net C3_K4_Push: now also U18.22 (GPA5); no longer U18.26 (GPA5)
- net C3_K5_A: now also U18.17 (GPA0); no longer U18.21 (GPA0)
- net C3_K5_B: now also U18.25 (GPB0); no longer U18.1 (GPB0)
- net C3_K5_Push: now also U18.23 (GPA6); no longer U18.27 (GPA6)
- net C3_K6_A: now also U18.18 (GPA1); no longer U18.22 (GPA1)
- net C3_K6_B: now also U18.26 (GPB1); no longer U18.2 (GPB1)
- net C3_K6_Push: now also U18.2 (GPB5); no longer U18.6 (GPB5)
- net C3_K7_A: now also U18.19 (GPA2); no longer U18.23 (GPA2)
- net C3_K7_B: now also U18.27 (GPB2); no longer U18.3 (GPB2)
- net C3_K7_Push: now also U18.3 (GPB6); no longer U18.7 (GPB6)
- net C3_K8_A: now also U18.20 (GPA3); no longer U18.24 (GPA3)
- net C3_K8_B: now also U18.28 (GPB3); no longer U18.4 (GPB3)
- net C3_K8_Push: now also U20.17 (GPA0); no longer U20.21 (GPA0)
- net C3_K9_A: now also U18.21 (GPA4); no longer U18.25 (GPA4)
- net C3_K9_B: now also U18.1 (GPB4); no longer U18.5 (GPB4)
- net C3_K9_Push: now also U20.18 (GPA1); no longer U20.22 (GPA1)
- net I2C4_CLK: now also U16.8 (SCK), U18.8 (SCK), U20.8 (SCK); no longer U16.12 (SCK), U18.12 (SCK), U20.12 (SCK)
- net I2C4_SDA: now also U16.9 (SDA), U18.9 (SDA), U20.9 (SDA); no longer U16.13 (SDA), U18.13 (SDA), U20.13 (SDA)
- net at C82.1, R408.2: now also U20.14 (~{RESET}); no longer U20.18 (~{RESET})
- net at C81.1, R407.2: now also U18.14 (~{RESET}); no longer U18.18 (~{RESET})
- net at U20.11 (A0): now also U20.13 (A2), U20.6 (V_{SS})
- net at U16.11 (A0): now also U16.12 (A1), U16.13 (A2), U16.6 (V_{SS})
- net at U16.14 (~{RESET}): now also C80.1, R406.2
- new net: U18.12 (A1), U18.13 (A2), U18.6 (V_{SS})
- now unconnected: U16.10 (V_{SS}), U16.15 (A0), U16.16 (A1), U18.10 (V_{SS}), U18.16 (A1), U20.10 (V_{SS}), U20.15 (A0)
Changed lines of the file:
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@@
 	)
 	(symbol
-		(lib_id "Interface_Expansion:MCP23017x-x-SS")
+		(lib_id "Interface_Expansion:MCP23017x-x-ML")
 		(at 184.15 85.09 0)
 		(unit 1)
@@
 			)
 		)
-		(property "Footprint" "Package_SO:SSOP-28_5.3x10.2mm_P0.65mm"
+		(property "Footprint" "Package_DFN_QFN:QFN-28-1EP_6x6mm_P0.65mm_EP4.25x4.25mm"
 			(at 189.23 110.49 0)
 			(hide yes)
@@
 			)
 		)
-		(property "Description" "16-bit I/O expander, I2C, interrupts, w pull-ups, SSOP-28"
+		(property "Description" "16-bit I/O expander, I2C, interrupts, w pull-ups, GPA7/GPB7 output only (https://microchip.my.site.com/s/article/GPA7---GPB7-Cannot-Be-Used-as-Inputs-In-MCP23017), QFN-28"
 			(at 184.15 85.09 0)
 			(hide yes)
@@
 			)
 		)
-		(property "LCSC" "C558584"
+		(property "LCSC" "C629439"
 			(at 184.15 85.09 0)
 			(hide yes)
@@
 		)
 		(pin "28"
+		)
+		(pin "29"
 		)
 		(instances
@@
 	)
 	(symbol
-		(lib_id "Interface_Expansion:MCP23017x-x-SS")
+		(lib_id "Interface_Expansion:MCP23017x-x-ML")
 		(at 80.01 85.09 0)
 		(unit 1)
@@
 			)
 		)
-		(property "Footprint" "Package_SO:SSOP-28_5.3x10.2mm_P0.65mm"
+		(property "Footprint" "Package_DFN_QFN:QFN-28-1EP_6x6mm_P0.65mm_EP4.25x4.25mm"
 			(at 85.09 110.49 0)
 			(hide yes)
@@
 			)
 		)
-		(property "Description" "16-bit I/O expander, I2C, interrupts, w pull-ups, SSOP-28"
+		(property "Description" "16-bit I/O expander, I2C, interrupts, w pull-ups, GPA7/GPB7 output only (https://microchip.my.site.com/s/article/GPA7---GPB7-Cannot-Be-Used-as-Inputs-In-MCP23017), QFN-28"
 			(at 80.01 85.09 0)
 			(hide yes)
@@
 			)
 		)
-		(property "LCSC" "C558584"
+		(property "LCSC" "C629439"
 			(at 80.01 85.09 0)
 			(hide yes)
@@
 		)
 		(pin "25"
+		)
+		(pin "29"
 		)
 		(instances
@@
 	)
 	(symbol
-		(lib_id "Interface_Expansion:MCP23017x-x-SS")
+		(lib_id "Interface_Expansion:MCP23017x-x-ML")
 		(at 132.08 85.09 0)
 		(unit 1)
@@
 			)
 		)
-		(property "Footprint" "Package_SO:SSOP-28_5.3x10.2mm_P0.65mm"
+		(property "Footprint" "Package_DFN_QFN:QFN-28-1EP_6x6mm_P0.65mm_EP4.25x4.25mm"
 			(at 137.16 110.49 0)
 			(hide yes)
@@
 			)
 		)
-		(property "Description" "16-bit I/O expander, I2C, interrupts, w pull-ups, SSOP-28"
+		(property "Description" "16-bit I/O expander, I2C, interrupts, w pull-ups, GPA7/GPB7 output only (https://microchip.my.site.com/s/article/GPA7---GPB7-Cannot-Be-Used-as-Inputs-In-MCP23017), QFN-28"
 			(at 132.08 85.09 0)
 			(hide yes)
@@
 			)
 		)
-		(property "LCSC" "C558584"
+		(property "LCSC" "C629439"
 			(at 132.08 85.09 0)
 			(hide yes)
@@
 		(pin "28"
 		)
+		(pin "29"
+		)
 		(instances

Commit message: save pcb progress lol
Parts:
- removed C147, C148, C98: 100n, Capacitor_SMD:C_0402_1005Metric, symbol Device:C
Connections:
- net GND: now also U16.11 (A0), U16.12 (A1), U16.13 (A2), U16.29 (EP), U16.6 (V_{SS}), U18.12 (A1), U18.13 (A2), U18.29 (EP), U18.6 (V_{SS}), U20.11 (A0), U20.13 (A2), U20.29 (EP), U20.6 (V_{SS})

Commit message: pcb routing all day
Connections:
- net C3_B4: now also U20.26 (GPB1); no longer U20.23 (GPA6)
- net C3_B6: now also U20.23 (GPA6); no longer U20.26 (GPB1)
- net C3_B10 renamed btnA_3
- net C3_B11 renamed btnB_3
Changed lines of the file:
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@@
 	(global_label "C3_B6"
 		(shape input)
-		(at 196.85 90.17 0)
-		(fields_autoplaced yes)
-		(effects
-			(font
-				(size 1.27 1.27)
-			)
-			(justify left)
-		)
-		(property "Intersheetrefs" "${INTERSHEET_REFS}"
-			(at 205.7618 90.17 0)
+		(at 196.85 80.01 0)
+		(fields_autoplaced yes)
+		(effects
+			(font
+				(size 1.27 1.27)
+			)
+			(justify left)
+		)
+		(property "Intersheetrefs" "${INTERSHEET_REFS}"
+			(at 205.7618 80.01 0)
 			(hide yes)
 			(show_name no)
@@
 		)
 	)
-	(global_label "C3_B10"
-		(shape input)
-		(at 196.85 100.33 0)
-		(fields_autoplaced yes)
-		(effects
-			(font
-				(size 1.27 1.27)
-			)
-			(justify left)
-		)
-		(property "Intersheetrefs" "${INTERSHEET_REFS}"
-			(at 206.9713 100.33 0)
-			(hide yes)
-			(show_name no)
-			(do_not_autoplace no)
-			(effects
-				(font
-					(size 1.27 1.27)
-				)
-				(justify left)
-			)
-		)
-	)
 	(global_label "C3_K1_Push"
 		(shape input)
@@
 		(property "Intersheetrefs" "${INTERSHEET_REFS}"
 			(at 103.8594 87.63 0)
+			(hide yes)
+			(show_name no)
+			(do_not_autoplace no)
+			(effects
+				(font
+					(size 1.27 1.27)
+				)
+				(justify left)
+			)
+		)
+	)
+	(global_label "btnB_3"
+		(shape output)
+		(at 196.85 102.87 0)
+		(fields_autoplaced yes)
+		(effects
+			(font
+				(size 1.27 1.27)
+				(color 255 255 255 1)
+			)
+			(justify left)
+		)
+		(property "Intersheetrefs" "${INTERSHEET_REFS}"
+			(at 206.306 102.87 0)
 			(hide yes)
 			(show_name no)
@@
 	(global_label "C3_B4"
 		(shape input)
-		(at 196.85 80.01 0)
-		(fields_autoplaced yes)
-		(effects
-			(font
-				(size 1.27 1.27)
-			)
-			(justify left)
-		)
-		(property "Intersheetrefs" "${INTERSHEET_REFS}"
-			(at 205.7618 80.01 0)
+		(at 196.85 90.17 0)
+		(fields_autoplaced yes)
+		(effects
+			(font
+				(size 1.27 1.27)
+			)
+			(justify left)
+		)
+		(property "Intersheetrefs" "${INTERSHEET_REFS}"
+			(at 205.7618 90.17 0)
 			(hide yes)
 			(show_name no)
@@
 		)
 	)
-	(global_label "C3_B11"
-		(shape input)
-		(at 196.85 102.87 0)
-		(fields_autoplaced yes)
-		(effects
-			(font
-				(size 1.27 1.27)
-			)
-			(justify left)
-		)
-		(property "Intersheetrefs" "${INTERSHEET_REFS}"
-			(at 206.9713 102.87 0)
-			(hide yes)
-			(show_name no)
+	(global_label "btnA_3"
+		(shape output)
+		(at 196.85 100.33 0)
+		(fields_autoplaced yes)
+		(effects
+			(font
+				(size 1.27 1.27)
+				(color 255 255 255 1)
+			)
+			(justify left)
+		)
+		(property "Intersheetrefs" "${INTERSHEET_REFS}"
+			(at 206.1246 100.33 0)
+			(hide yes)
+			(show_name no)
