File: PCB_CAD/BUCKET_CONTROLS/encoders_debounce.kicad_sch (KiCad schematic)
At the start: 100 parts, among them SW1 C0_K0, SW10 C0_K9, SW2 C0_K1, SW3 C0_K2, SW4 C0_K3, SW5 C0_K4, SW6 C0_K5, SW7 C0_K6, SW8 C0_K7, SW9 C0_K8

Commit message: saving progress on controls pcb
Parts:
- C1, C10, C11, C12, C13, C14, C15, C16, C17, C18, C19, C2, C20, C21, C22, C23, C24, C25, C26, C27, C28, C29, C3, C30, C4, C5, C6, C7, C8, C9: footprint Capacitor_SMD:C_0603_1608Metric -> Capacitor_SMD:C_0402_1005Metric; LCSC C57112 -> C1524
- SW1, SW10, SW2, SW3, SW4, SW5, SW6, SW7, SW8, SW9: LCSC dnp -> manual
Other:
- note added: "FX KNOB 1A"
- note added: "FX KNOB 1B"
- note added: "FX KNOB 2A"
- note added: "FX KNOB 2B"
- note added: "FX KNOB 3A"
- note added: "FX KNOB 3B"
- note added: "FX KNOB 4A"
- note added: "FX KNOB 4B"
- note added: "INPUT GAIN"
- note added: "PAN"

Commit message: pcb controls
Parts:
- SW1, SW10, SW2, SW3, SW4, SW5, SW6, SW7, SW8, SW9: footprint My Footprints:EC11J0924411 -> My Footprints:EC11_miniboard_castellated; LCSC manual -> dnp
Changed lines of the file:
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@@
 			)
 		)
-		(property "Footprint" "My Footprints:EC11J0924411"
+		(property "Footprint" "My Footprints:EC11_miniboard_castellated"
 			(at 81.28 96.52 0)
 			(hide yes)
@@
 			)
 		)
-		(property "LCSC" "manual"
+		(property "LCSC" "dnp"
 			(at 81.28 96.52 0)
 			(hide yes)
@@
 			)
 		)
-		(property "Footprint" "My Footprints:EC11J0924411"
+		(property "Footprint" "My Footprints:EC11_miniboard_castellated"
 			(at 81.28 248.92 0)
 			(hide yes)
@@
 			)
 		)
-		(property "LCSC" "manual"
+		(property "LCSC" "dnp"
 			(at 81.28 248.92 0)
 			(hide yes)
@@
 			)
 		)
-		(property "Footprint" "My Footprints:EC11J0924411"
+		(property "Footprint" "My Footprints:EC11_miniboard_castellated"
 			(at 81.28 198.12 0)
 			(hide yes)
@@
 			)
 		)
-		(property "LCSC" "manual"
+		(property "LCSC" "dnp"
 			(at 81.28 198.12 0)
 			(hide yes)
@@
 			)
 		)
-		(property "Footprint" "My Footprints:EC11J0924411"
+		(property "Footprint" "My Footprints:EC11_miniboard_castellated"
 			(at 201.93 96.52 0)
 			(hide yes)
@@
 			)
 		)
-		(property "LCSC" "manual"
+		(property "LCSC" "dnp"
 			(at 201.93 96.52 0)
 			(hide yes)
@@
 			)
 		)
-		(property "Footprint" "My Footprints:EC11J0924411"
+		(property "Footprint" "My Footprints:EC11_miniboard_castellated"
 			(at 81.28 45.72 0)
 			(hide yes)
@@
 			)
 		)
-		(property "LCSC" "manual"
+		(property "LCSC" "dnp"
 			(at 81.28 45.72 0)
 			(hide yes)
@@
 			)
 		)
-		(property "Footprint" "My Footprints:EC11J0924411"
+		(property "Footprint" "My Footprints:EC11_miniboard_castellated"
 			(at 201.93 45.72 0)
 			(hide yes)
@@
 			)
 		)
-		(property "LCSC" "manual"
+		(property "LCSC" "dnp"
 			(at 201.93 45.72 0)
 			(hide yes)
@@
 			)
 		)
-		(property "Footprint" "My Footprints:EC11J0924411"
+		(property "Footprint" "My Footprints:EC11_miniboard_castellated"
 			(at 81.28 147.32 0)
 			(hide yes)
@@
 			)
 		)
-		(property "LCSC" "manual"
+		(property "LCSC" "dnp"
 			(at 81.28 147.32 0)
 			(hide yes)
@@
 			)
 		)
-		(property "Footprint" "My Footprints:EC11J0924411"
+		(property "Footprint" "My Footprints:EC11_miniboard_castellated"
 			(at 201.93 198.12 0)
 			(hide yes)
@@
 			)
 		)
-		(property "LCSC" "manual"
+		(property "LCSC" "dnp"
 			(at 201.93 198.12 0)
 			(hide yes)
@@
 			)
 		)
-		(property "Footprint" "My Footprints:EC11J0924411"
+		(property "Footprint" "My Footprints:EC11_miniboard_castellated"
 			(at 201.93 147.32 0)
 			(hide yes)
@@
 			)
 		)
-		(property "LCSC" "manual"
+		(property "LCSC" "dnp"
 			(at 201.93 147.32 0)
 			(hide yes)
@@
 			)
 		)
-		(property "Footprint" "My Footprints:EC11J0924411"
+		(property "Footprint" "My Footprints:EC11_miniboard_castellated"
 			(at 201.93 248.92 0)
 			(hide yes)
@@
 			)
 		)
-		(property "LCSC" "manual"
+		(property "LCSC" "dnp"
 			(at 201.93 248.92 0)
 			(hide yes)

Commit message: pcb
Parts:
- SW1, SW10, SW2, SW3, SW4, SW5, SW6, SW7, SW8, SW9: symbol My Symbols:EC11_Rotary_Encoder -> My Symbols:EC11_Rotary_Encoder_Board
Connections:
- net GND: no longer SW1.C (Pin_2), SW1.D (Pin_4), SW10.C (Pin_2), SW10.D (Pin_4), SW2.C (Pin_2), SW2.D (Pin_4), SW3.C (Pin_2), SW3.D (Pin_4), SW4.C (Pin_2), SW4.D (Pin_4), SW5.C (Pin_2), SW5.D (Pin_4), SW6.C (Pin_2), SW6.D (Pin_4), SW7.C (Pin_2), SW7.D (Pin_4), SW8.C (Pin_2), SW8.D (Pin_4), SW9.C (Pin_2), SW9.D (Pin_4)
Changed lines of the file:
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@@
 	)
 	(symbol
-		(lib_id "My Symbols:EC11_Rotary_Encoder")
+		(lib_id "My Symbols:EC11_Rotary_Encoder_Board")
 		(at 81.28 96.52 180)
 		(unit 1)
@@
 			)
 		)
-		(pin "D"
-		)
-		(pin "C"
-		)
 		(pin "G"
 		)
@@
 	)
 	(symbol
-		(lib_id "My Symbols:EC11_Rotary_Encoder")
+		(lib_id "My Symbols:EC11_Rotary_Encoder_Board")
 		(at 81.28 248.92 180)
 		(unit 1)
@@
 			)
 		)
-		(pin "D"
-		)
-		(pin "C"
-		)
 		(pin "G"
 		)
@@
 	)
 	(symbol
-		(lib_id "My Symbols:EC11_Rotary_Encoder")
+		(lib_id "My Symbols:EC11_Rotary_Encoder_Board")
 		(at 81.28 198.12 180)
 		(unit 1)
@@
 			)
 		)
-		(pin "D"
-		)
-		(pin "C"
-		)
 		(pin "G"
 		)
@@
 	)
 	(symbol
-		(lib_id "My Symbols:EC11_Rotary_Encoder")
+		(lib_id "My Symbols:EC11_Rotary_Encoder_Board")
 		(at 201.93 96.52 180)
 		(unit 1)
@@
 			)
 		)
-		(pin "D"
-		)
-		(pin "C"
-		)
 		(pin "G"
 		)
@@
 	)
 	(symbol
-		(lib_id "My Symbols:EC11_Rotary_Encoder")
+		(lib_id "My Symbols:EC11_Rotary_Encoder_Board")
 		(at 81.28 45.72 180)
 		(unit 1)
@@
 			)
 		)
-		(pin "D"
-		)
-		(pin "C"
-		)
 		(pin "G"
 		)
@@
 	)
 	(symbol
-		(lib_id "My Symbols:EC11_Rotary_Encoder")
+		(lib_id "My Symbols:EC11_Rotary_Encoder_Board")
 		(at 201.93 45.72 180)
 		(unit 1)
@@
 			)
 		)
-		(pin "D"
-		)
-		(pin "C"
-		)
 		(pin "G"
 		)
@@
 	)
 	(symbol
-		(lib_id "My Symbols:EC11_Rotary_Encoder")
+		(lib_id "My Symbols:EC11_Rotary_Encoder_Board")
 		(at 81.28 147.32 180)
 		(unit 1)
@@
 			)
 		)
-		(pin "D"
-		)
-		(pin "C"
-		)
 		(pin "G"
 		)
@@
 	)
 	(symbol
-		(lib_id "My Symbols:EC11_Rotary_Encoder")
+		(lib_id "My Symbols:EC11_Rotary_Encoder_Board")
 		(at 201.93 198.12 180)
 		(unit 1)
@@
 			)
 		)
-		(pin "D"
-		)
-		(pin "C"
-		)
 		(pin "G"
 		)
@@
 	)
 	(symbol
-		(lib_id "My Symbols:EC11_Rotary_Encoder")
+		(lib_id "My Symbols:EC11_Rotary_Encoder_Board")
 		(at 201.93 147.32 180)
 		(unit 1)
@@
 			)
 		)
-		(pin "D"
-		)
-		(pin "C"
-		)
 		(pin "G"
 		)
@@
 	)
 	(symbol
-		(lib_id "My Symbols:EC11_Rotary_Encoder")
+		(lib_id "My Symbols:EC11_Rotary_Encoder_Board")
 		(at 201.93 248.92 180)
 		(unit 1)
@@
 			)
 		)
-		(pin "D"
-		)
-		(pin "C"
-		)
 		(pin "G"
