File: PCB_CAD/BUCKET_CONTROLS/encoders_debounce_1.kicad_sch (KiCad schematic)
At the start: 100 parts, among them SW101 C1_K0, SW102 C1_K1, SW103 C1_K2, SW104 C1_K3, SW105 C1_K4, SW106 C1_K5, SW107 C1_K6, SW108 C1_K7, SW109 C1_K8, SW110 C1_K9

Commit message: saving progress on controls pcb
Parts:
- C101, C102, C103, C104, C105, C106, C107, C108, C109, C110, C111, C112, C113, C114, C115, C116, C117, C118, C119, C120, C121, C122, C123, C124, C125, C126, C127, C128, C129, C130: footprint Capacitor_SMD:C_0603_1608Metric -> Capacitor_SMD:C_0402_1005Metric; LCSC C57112 -> C1524
- SW101, SW102, SW103, SW104, SW105, SW106, SW107, SW108, SW109, SW110: LCSC dnp -> manual
Other:
- note added: "FX KNOB 1A"
- note added: "FX KNOB 1B"
- note added: "FX KNOB 2A"
- note added: "FX KNOB 2B"
- note added: "FX KNOB 3A"
- note added: "FX KNOB 3B"
- note added: "FX KNOB 4A"
- note added: "FX KNOB 4B"
- note added: "INPUT GAIN"
- note added: "PAN"

Commit message: pcb controls
Parts:
- SW101, SW102, SW103, SW104, SW105, SW106, SW107, SW108, SW109, SW110: footprint My Footprints:EC11J0924411 -> My Footprints:EC11_miniboard_castellated; LCSC manual -> dnp
Changed lines of the file:
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@@
 			)
 		)
-		(property "Footprint" "My Footprints:EC11J0924411"
+		(property "Footprint" "My Footprints:EC11_miniboard_castellated"
 			(at 81.28 147.32 0)
 			(hide yes)
@@
 			)
 		)
-		(property "LCSC" "manual"
+		(property "LCSC" "dnp"
 			(at 81.28 147.32 0)
 			(hide yes)
@@
 			)
 		)
-		(property "Footprint" "My Footprints:EC11J0924411"
+		(property "Footprint" "My Footprints:EC11_miniboard_castellated"
 			(at 81.28 45.72 0)
 			(hide yes)
@@
 			)
 		)
-		(property "LCSC" "manual"
+		(property "LCSC" "dnp"
 			(at 81.28 45.72 0)
 			(hide yes)
@@
 			)
 		)
-		(property "Footprint" "My Footprints:EC11J0924411"
+		(property "Footprint" "My Footprints:EC11_miniboard_castellated"
 			(at 81.28 96.52 0)
 			(hide yes)
@@
 			)
 		)
-		(property "LCSC" "manual"
+		(property "LCSC" "dnp"
 			(at 81.28 96.52 0)
 			(hide yes)
@@
 			)
 		)
-		(property "Footprint" "My Footprints:EC11J0924411"
+		(property "Footprint" "My Footprints:EC11_miniboard_castellated"
 			(at 201.93 147.32 0)
 			(hide yes)
@@
 			)
 		)
-		(property "LCSC" "manual"
+		(property "LCSC" "dnp"
 			(at 201.93 147.32 0)
 			(hide yes)
@@
 			)
 		)
-		(property "Footprint" "My Footprints:EC11J0924411"
+		(property "Footprint" "My Footprints:EC11_miniboard_castellated"
 			(at 201.93 96.52 0)
 			(hide yes)
@@
 			)
 		)
-		(property "LCSC" "manual"
+		(property "LCSC" "dnp"
 			(at 201.93 96.52 0)
 			(hide yes)
@@
 			)
 		)
-		(property "Footprint" "My Footprints:EC11J0924411"
+		(property "Footprint" "My Footprints:EC11_miniboard_castellated"
 			(at 201.93 248.92 0)
 			(hide yes)
@@
 			)
 		)
-		(property "LCSC" "manual"
+		(property "LCSC" "dnp"
 			(at 201.93 248.92 0)
 			(hide yes)
@@
 			)
 		)
-		(property "Footprint" "My Footprints:EC11J0924411"
+		(property "Footprint" "My Footprints:EC11_miniboard_castellated"
 			(at 201.93 45.72 0)
 			(hide yes)
@@
 			)
 		)
-		(property "LCSC" "manual"
+		(property "LCSC" "dnp"
 			(at 201.93 45.72 0)
 			(hide yes)
@@
 			)
 		)
-		(property "Footprint" "My Footprints:EC11J0924411"
+		(property "Footprint" "My Footprints:EC11_miniboard_castellated"
 			(at 81.28 198.12 0)
 			(hide yes)
@@
 			)
 		)
-		(property "LCSC" "manual"
+		(property "LCSC" "dnp"
 			(at 81.28 198.12 0)
 			(hide yes)
@@
 			)
 		)
-		(property "Footprint" "My Footprints:EC11J0924411"
+		(property "Footprint" "My Footprints:EC11_miniboard_castellated"
 			(at 201.93 198.12 0)
 			(hide yes)
@@
 			)
 		)
-		(property "LCSC" "manual"
+		(property "LCSC" "dnp"
 			(at 201.93 198.12 0)
 			(hide yes)
@@
 			)
 		)
-		(property "Footprint" "My Footprints:EC11J0924411"
+		(property "Footprint" "My Footprints:EC11_miniboard_castellated"
 			(at 81.28 248.92 0)
 			(hide yes)
@@
 			)
 		)
-		(property "LCSC" "manual"
+		(property "LCSC" "dnp"
 			(at 81.28 248.92 0)
 			(hide yes)

Commit message: pcb
Parts:
- SW101, SW102, SW103, SW104, SW105, SW106, SW107, SW108, SW109, SW110: symbol My Symbols:EC11_Rotary_Encoder -> My Symbols:EC11_Rotary_Encoder_Board
Connections:
- net GND: no longer SW101.C (Pin_2), SW101.D (Pin_4), SW102.C (Pin_2), SW102.D (Pin_4), SW103.C (Pin_2), SW103.D (Pin_4), SW104.C (Pin_2), SW104.D (Pin_4), SW105.C (Pin_2), SW105.D (Pin_4), SW106.C (Pin_2), SW106.D (Pin_4), SW107.C (Pin_2), SW107.D (Pin_4), SW108.C (Pin_2), SW108.D (Pin_4), SW109.C (Pin_2), SW109.D (Pin_4), SW110.C (Pin_2), SW110.D (Pin_4)
Changed lines of the file:
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@@
 	)
 	(symbol
-		(lib_id "My Symbols:EC11_Rotary_Encoder")
+		(lib_id "My Symbols:EC11_Rotary_Encoder_Board")
 		(at 81.28 147.32 180)
 		(unit 1)
@@
 			)
 		)
-		(pin "D"
-		)
-		(pin "C"
-		)
 		(pin "G"
 		)
@@
 	)
 	(symbol
-		(lib_id "My Symbols:EC11_Rotary_Encoder")
+		(lib_id "My Symbols:EC11_Rotary_Encoder_Board")
 		(at 81.28 45.72 180)
 		(unit 1)
@@
 			)
 		)
-		(pin "D"
-		)
-		(pin "C"
-		)
 		(pin "G"
 		)
@@
 	)
 	(symbol
-		(lib_id "My Symbols:EC11_Rotary_Encoder")
+		(lib_id "My Symbols:EC11_Rotary_Encoder_Board")
 		(at 81.28 96.52 180)
 		(unit 1)
@@
 			)
 		)
-		(pin "D"
-		)
-		(pin "C"
-		)
 		(pin "G"
 		)
@@
 	)
 	(symbol
-		(lib_id "My Symbols:EC11_Rotary_Encoder")
+		(lib_id "My Symbols:EC11_Rotary_Encoder_Board")
 		(at 201.93 147.32 180)
 		(unit 1)
@@
 			)
 		)
-		(pin "D"
-		)
-		(pin "C"
-		)
 		(pin "G"
 		)
@@
 	)
 	(symbol
-		(lib_id "My Symbols:EC11_Rotary_Encoder")
+		(lib_id "My Symbols:EC11_Rotary_Encoder_Board")
 		(at 201.93 96.52 180)
 		(unit 1)
@@
 			)
 		)
-		(pin "D"
-		)
-		(pin "C"
-		)
 		(pin "G"
 		)
@@
 	)
 	(symbol
-		(lib_id "My Symbols:EC11_Rotary_Encoder")
+		(lib_id "My Symbols:EC11_Rotary_Encoder_Board")
 		(at 201.93 248.92 180)
 		(unit 1)
@@
 			)
 		)
-		(pin "D"
-		)
-		(pin "C"
-		)
 		(pin "G"
 		)
@@
 	)
 	(symbol
-		(lib_id "My Symbols:EC11_Rotary_Encoder")
+		(lib_id "My Symbols:EC11_Rotary_Encoder_Board")
 		(at 201.93 45.72 180)
 		(unit 1)
@@
 			)
 		)
-		(pin "D"
-		)
-		(pin "C"
-		)
 		(pin "G"
 		)
@@
 	)
 	(symbol
-		(lib_id "My Symbols:EC11_Rotary_Encoder")
+		(lib_id "My Symbols:EC11_Rotary_Encoder_Board")
 		(at 81.28 198.12 180)
 		(unit 1)
@@
 			)
 		)
-		(pin "D"
-		)
-		(pin "C"
-		)
 		(pin "G"
 		)
@@
 	)
 	(symbol
-		(lib_id "My Symbols:EC11_Rotary_Encoder")
+		(lib_id "My Symbols:EC11_Rotary_Encoder_Board")
 		(at 201.93 198.12 180)
 		(unit 1)
@@
 			)
 		)
-		(pin "D"
-		)
-		(pin "C"
-		)
 		(pin "G"
 		)
@@
 	)
 	(symbol
-		(lib_id "My Symbols:EC11_Rotary_Encoder")
+		(lib_id "My Symbols:EC11_Rotary_Encoder_Board")
 		(at 81.28 248.92 180)
 		(unit 1)
@@
 			)
 		)
-		(pin "D"
-		)
-		(pin "C"
-		)
 		(pin "G"
