File: PCB_CAD/BUCKET_CONTROLS/encoders_debounce_2.kicad_sch (KiCad schematic)
At the start: 100 parts, among them SW201 C2_K0, SW202 C2_K1, SW203 C2_K2, SW204 C2_K3, SW205 C2_K4, SW206 C2_K5, SW207 C2_K6, SW208 C2_K7, SW209 C2_K8, SW210 C2_K9

Commit message: saving progress on controls pcb
Parts:
- C201, C202, C203, C204, C205, C206, C207, C208, C209, C210, C211, C212, C213, C214, C215, C216, C217, C218, C219, C220, C221, C222, C223, C224, C225, C226, C227, C228, C229, C230: footprint Capacitor_SMD:C_0603_1608Metric -> Capacitor_SMD:C_0402_1005Metric; LCSC C57112 -> C1524
- SW201, SW202, SW203, SW204, SW205, SW206, SW207, SW208, SW209, SW210: LCSC dnp -> manual
Other:
- note added: "FX KNOB 1A"
- note added: "FX KNOB 1B"
- note added: "FX KNOB 2A"
- note added: "FX KNOB 2B"
- note added: "FX KNOB 3A"
- note added: "FX KNOB 3B"
- note added: "FX KNOB 4A"
- note added: "FX KNOB 4B"
- note added: "INPUT GAIN"
- note added: "PAN"

Commit message: pcb controls
Parts:
- SW201, SW202, SW203, SW204, SW205, SW206, SW207, SW208, SW209, SW210: footprint My Footprints:EC11J0924411 -> My Footprints:EC11_miniboard_castellated; LCSC manual -> dnp
Changed lines of the file:
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@@
 			)
 		)
-		(property "Footprint" "My Footprints:EC11J0924411"
+		(property "Footprint" "My Footprints:EC11_miniboard_castellated"
 			(at 81.28 147.32 0)
 			(hide yes)
@@
 			)
 		)
-		(property "LCSC" "manual"
+		(property "LCSC" "dnp"
 			(at 81.28 147.32 0)
 			(hide yes)
@@
 			)
 		)
-		(property "Footprint" "My Footprints:EC11J0924411"
+		(property "Footprint" "My Footprints:EC11_miniboard_castellated"
 			(at 201.93 248.92 0)
 			(hide yes)
@@
 			)
 		)
-		(property "LCSC" "manual"
+		(property "LCSC" "dnp"
 			(at 201.93 248.92 0)
 			(hide yes)
@@
 			)
 		)
-		(property "Footprint" "My Footprints:EC11J0924411"
+		(property "Footprint" "My Footprints:EC11_miniboard_castellated"
 			(at 201.93 96.52 0)
 			(hide yes)
@@
 			)
 		)
-		(property "LCSC" "manual"
+		(property "LCSC" "dnp"
 			(at 201.93 96.52 0)
 			(hide yes)
@@
 			)
 		)
-		(property "Footprint" "My Footprints:EC11J0924411"
+		(property "Footprint" "My Footprints:EC11_miniboard_castellated"
 			(at 81.28 96.52 0)
 			(hide yes)
@@
 			)
 		)
-		(property "LCSC" "manual"
+		(property "LCSC" "dnp"
 			(at 81.28 96.52 0)
 			(hide yes)
@@
 			)
 		)
-		(property "Footprint" "My Footprints:EC11J0924411"
+		(property "Footprint" "My Footprints:EC11_miniboard_castellated"
 			(at 201.93 147.32 0)
 			(hide yes)
@@
 			)
 		)
-		(property "LCSC" "manual"
+		(property "LCSC" "dnp"
 			(at 201.93 147.32 0)
 			(hide yes)
@@
 			)
 		)
-		(property "Footprint" "My Footprints:EC11J0924411"
+		(property "Footprint" "My Footprints:EC11_miniboard_castellated"
 			(at 81.28 198.12 0)
 			(hide yes)
@@
 			)
 		)
-		(property "LCSC" "manual"
+		(property "LCSC" "dnp"
 			(at 81.28 198.12 0)
 			(hide yes)
@@
 			)
 		)
-		(property "Footprint" "My Footprints:EC11J0924411"
+		(property "Footprint" "My Footprints:EC11_miniboard_castellated"
 			(at 201.93 45.72 0)
 			(hide yes)
@@
 			)
 		)
-		(property "LCSC" "manual"
+		(property "LCSC" "dnp"
 			(at 201.93 45.72 0)
 			(hide yes)
@@
 			)
 		)
-		(property "Footprint" "My Footprints:EC11J0924411"
+		(property "Footprint" "My Footprints:EC11_miniboard_castellated"
 			(at 201.93 198.12 0)
 			(hide yes)
@@
 			)
 		)
-		(property "LCSC" "manual"
+		(property "LCSC" "dnp"
 			(at 201.93 198.12 0)
 			(hide yes)
@@
 			)
 		)
-		(property "Footprint" "My Footprints:EC11J0924411"
+		(property "Footprint" "My Footprints:EC11_miniboard_castellated"
 			(at 81.28 45.72 0)
 			(hide yes)
@@
 			)
 		)
-		(property "LCSC" "manual"
+		(property "LCSC" "dnp"
 			(at 81.28 45.72 0)
 			(hide yes)
@@
 			)
 		)
-		(property "Footprint" "My Footprints:EC11J0924411"
+		(property "Footprint" "My Footprints:EC11_miniboard_castellated"
 			(at 81.28 248.92 0)
 			(hide yes)
@@
 			)
 		)
-		(property "LCSC" "manual"
+		(property "LCSC" "dnp"
 			(at 81.28 248.92 0)
 			(hide yes)

Commit message: pcb
Parts:
- SW201, SW202, SW203, SW204, SW205, SW206, SW207, SW208, SW209, SW210: symbol My Symbols:EC11_Rotary_Encoder -> My Symbols:EC11_Rotary_Encoder_Board
Connections:
- net GND: no longer SW201.C (Pin_2), SW201.D (Pin_4), SW202.C (Pin_2), SW202.D (Pin_4), SW203.C (Pin_2), SW203.D (Pin_4), SW204.C (Pin_2), SW204.D (Pin_4), SW205.C (Pin_2), SW205.D (Pin_4), SW206.C (Pin_2), SW206.D (Pin_4), SW207.C (Pin_2), SW207.D (Pin_4), SW208.C (Pin_2), SW208.D (Pin_4), SW209.C (Pin_2), SW209.D (Pin_4), SW210.C (Pin_2), SW210.D (Pin_4)
Changed lines of the file:
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@@
 	)
 	(symbol
-		(lib_id "My Symbols:EC11_Rotary_Encoder")
+		(lib_id "My Symbols:EC11_Rotary_Encoder_Board")
 		(at 81.28 147.32 180)
 		(unit 1)
@@
 			)
 		)
-		(pin "D"
-		)
-		(pin "C"
-		)
 		(pin "G"
 		)
@@
 	)
 	(symbol
-		(lib_id "My Symbols:EC11_Rotary_Encoder")
+		(lib_id "My Symbols:EC11_Rotary_Encoder_Board")
 		(at 201.93 248.92 180)
 		(unit 1)
@@
 			)
 		)
-		(pin "D"
-		)
-		(pin "C"
-		)
 		(pin "G"
 		)
@@
 	)
 	(symbol
-		(lib_id "My Symbols:EC11_Rotary_Encoder")
+		(lib_id "My Symbols:EC11_Rotary_Encoder_Board")
 		(at 201.93 96.52 180)
 		(unit 1)
@@
 			)
 		)
-		(pin "D"
-		)
-		(pin "C"
-		)
 		(pin "G"
 		)
@@
 	)
 	(symbol
-		(lib_id "My Symbols:EC11_Rotary_Encoder")
+		(lib_id "My Symbols:EC11_Rotary_Encoder_Board")
 		(at 81.28 96.52 180)
 		(unit 1)
@@
 			)
 		)
-		(pin "D"
-		)
-		(pin "C"
-		)
 		(pin "G"
 		)
@@
 	)
 	(symbol
-		(lib_id "My Symbols:EC11_Rotary_Encoder")
+		(lib_id "My Symbols:EC11_Rotary_Encoder_Board")
 		(at 201.93 147.32 180)
 		(unit 1)
@@
 			)
 		)
-		(pin "D"
-		)
-		(pin "C"
-		)
 		(pin "G"
 		)
@@
 	)
 	(symbol
-		(lib_id "My Symbols:EC11_Rotary_Encoder")
+		(lib_id "My Symbols:EC11_Rotary_Encoder_Board")
 		(at 81.28 198.12 180)
 		(unit 1)
@@
 			)
 		)
-		(pin "D"
-		)
-		(pin "C"
-		)
 		(pin "G"
 		)
@@
 	)
 	(symbol
-		(lib_id "My Symbols:EC11_Rotary_Encoder")
+		(lib_id "My Symbols:EC11_Rotary_Encoder_Board")
 		(at 201.93 45.72 180)
 		(unit 1)
@@
 			)
 		)
-		(pin "D"
-		)
-		(pin "C"
-		)
 		(pin "G"
 		)
@@
 	)
 	(symbol
-		(lib_id "My Symbols:EC11_Rotary_Encoder")
+		(lib_id "My Symbols:EC11_Rotary_Encoder_Board")
 		(at 201.93 198.12 180)
 		(unit 1)
@@
 			)
 		)
-		(pin "D"
-		)
-		(pin "C"
-		)
 		(pin "G"
 		)
@@
 	)
 	(symbol
-		(lib_id "My Symbols:EC11_Rotary_Encoder")
+		(lib_id "My Symbols:EC11_Rotary_Encoder_Board")
 		(at 81.28 45.72 180)
 		(unit 1)
@@
 			)
 		)
-		(pin "D"
-		)
-		(pin "C"
-		)
 		(pin "G"
 		)
@@
 	)
 	(symbol
-		(lib_id "My Symbols:EC11_Rotary_Encoder")
+		(lib_id "My Symbols:EC11_Rotary_Encoder_Board")
 		(at 81.28 248.92 180)
 		(unit 1)
@@
 			)
 		)
-		(pin "D"
-		)
-		(pin "C"
-		)
 		(pin "G"
