File: PCB_CAD/BUCKET_CONTROLS/encoders_debounce_3.kicad_sch (KiCad schematic)
At the start: 100 parts, among them SW301 C3_K0, SW302 C3_K1, SW303 C3_K2, SW304 C3_K3, SW305 C3_K4, SW306 C3_K5, SW307 C3_K6, SW308 C3_K7, SW309 C3_K8, SW310 C3_K9

Commit message: saving progress on controls pcb
Parts:
- C301, C302, C303, C304, C305, C306, C307, C308, C309, C310, C311, C312, C313, C314, C315, C316, C317, C318, C319, C320, C321, C322, C323, C324, C325, C326, C327, C328, C329, C330: footprint Capacitor_SMD:C_0603_1608Metric -> Capacitor_SMD:C_0402_1005Metric; LCSC C57112 -> C1524
- SW301, SW302, SW303, SW304, SW305, SW306, SW307, SW308, SW309, SW310: LCSC dnp -> manual
Other:
- note added: "FX KNOB 1A"
- note added: "FX KNOB 1B"
- note added: "FX KNOB 2A"
- note added: "FX KNOB 2B"
- note added: "FX KNOB 3A"
- note added: "FX KNOB 3B"
- note added: "FX KNOB 4A"
- note added: "FX KNOB 4B"
- note added: "INPUT GAIN"
- note added: "PAN"

Commit message: pcb controls
Parts:
- SW301, SW302, SW303, SW304, SW305, SW306, SW307, SW308, SW309, SW310: footprint My Footprints:EC11J0924411 -> My Footprints:EC11_miniboard_castellated; LCSC manual -> dnp
Changed lines of the file:
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@@
 			)
 		)
-		(property "Footprint" "My Footprints:EC11J0924411"
+		(property "Footprint" "My Footprints:EC11_miniboard_castellated"
 			(at 81.28 96.52 0)
 			(hide yes)
@@
 			)
 		)
-		(property "LCSC" "manual"
+		(property "LCSC" "dnp"
 			(at 81.28 96.52 0)
 			(hide yes)
@@
 			)
 		)
-		(property "Footprint" "My Footprints:EC11J0924411"
+		(property "Footprint" "My Footprints:EC11_miniboard_castellated"
 			(at 81.28 248.92 0)
 			(hide yes)
@@
 			)
 		)
-		(property "LCSC" "manual"
+		(property "LCSC" "dnp"
 			(at 81.28 248.92 0)
 			(hide yes)
@@
 			)
 		)
-		(property "Footprint" "My Footprints:EC11J0924411"
+		(property "Footprint" "My Footprints:EC11_miniboard_castellated"
 			(at 201.93 45.72 0)
 			(hide yes)
@@
 			)
 		)
-		(property "LCSC" "manual"
+		(property "LCSC" "dnp"
 			(at 201.93 45.72 0)
 			(hide yes)
@@
 			)
 		)
-		(property "Footprint" "My Footprints:EC11J0924411"
+		(property "Footprint" "My Footprints:EC11_miniboard_castellated"
 			(at 201.93 198.12 0)
 			(hide yes)
@@
 			)
 		)
-		(property "LCSC" "manual"
+		(property "LCSC" "dnp"
 			(at 201.93 198.12 0)
 			(hide yes)
@@
 			)
 		)
-		(property "Footprint" "My Footprints:EC11J0924411"
+		(property "Footprint" "My Footprints:EC11_miniboard_castellated"
 			(at 201.93 248.92 0)
 			(hide yes)
@@
 			)
 		)
-		(property "LCSC" "manual"
+		(property "LCSC" "dnp"
 			(at 201.93 248.92 0)
 			(hide yes)
@@
 			)
 		)
-		(property "Footprint" "My Footprints:EC11J0924411"
+		(property "Footprint" "My Footprints:EC11_miniboard_castellated"
 			(at 81.28 147.32 0)
 			(hide yes)
@@
 			)
 		)
-		(property "LCSC" "manual"
+		(property "LCSC" "dnp"
 			(at 81.28 147.32 0)
 			(hide yes)
@@
 			)
 		)
-		(property "Footprint" "My Footprints:EC11J0924411"
+		(property "Footprint" "My Footprints:EC11_miniboard_castellated"
 			(at 201.93 96.52 0)
 			(hide yes)
@@
 			)
 		)
-		(property "LCSC" "manual"
+		(property "LCSC" "dnp"
 			(at 201.93 96.52 0)
 			(hide yes)
@@
 			)
 		)
-		(property "Footprint" "My Footprints:EC11J0924411"
+		(property "Footprint" "My Footprints:EC11_miniboard_castellated"
 			(at 81.28 198.12 0)
 			(hide yes)
@@
 			)
 		)
-		(property "LCSC" "manual"
+		(property "LCSC" "dnp"
 			(at 81.28 198.12 0)
 			(hide yes)
@@
 			)
 		)
-		(property "Footprint" "My Footprints:EC11J0924411"
+		(property "Footprint" "My Footprints:EC11_miniboard_castellated"
 			(at 81.28 45.72 0)
 			(hide yes)
@@
 			)
 		)
-		(property "LCSC" "manual"
+		(property "LCSC" "dnp"
 			(at 81.28 45.72 0)
 			(hide yes)
@@
 			)
 		)
-		(property "Footprint" "My Footprints:EC11J0924411"
+		(property "Footprint" "My Footprints:EC11_miniboard_castellated"
 			(at 201.93 147.32 0)
 			(hide yes)
@@
 			)
 		)
-		(property "LCSC" "manual"
+		(property "LCSC" "dnp"
 			(at 201.93 147.32 0)
 			(hide yes)

Commit message: pcb
Parts:
- SW301, SW302, SW303, SW304, SW305, SW306, SW307, SW308, SW309, SW310: symbol My Symbols:EC11_Rotary_Encoder -> My Symbols:EC11_Rotary_Encoder_Board
Connections:
- net GND: no longer SW301.C (Pin_2), SW301.D (Pin_4), SW302.C (Pin_2), SW302.D (Pin_4), SW303.C (Pin_2), SW303.D (Pin_4), SW304.C (Pin_2), SW304.D (Pin_4), SW305.C (Pin_2), SW305.D (Pin_4), SW306.C (Pin_2), SW306.D (Pin_4), SW307.C (Pin_2), SW307.D (Pin_4), SW308.C (Pin_2), SW308.D (Pin_4), SW309.C (Pin_2), SW309.D (Pin_4), SW310.C (Pin_2), SW310.D (Pin_4)
Changed lines of the file:
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@@
 	)
 	(symbol
-		(lib_id "My Symbols:EC11_Rotary_Encoder")
+		(lib_id "My Symbols:EC11_Rotary_Encoder_Board")
 		(at 81.28 96.52 180)
 		(unit 1)
@@
 			)
 		)
-		(pin "D"
-		)
-		(pin "C"
-		)
 		(pin "G"
 		)
@@
 	)
 	(symbol
-		(lib_id "My Symbols:EC11_Rotary_Encoder")
+		(lib_id "My Symbols:EC11_Rotary_Encoder_Board")
 		(at 81.28 248.92 180)
 		(unit 1)
@@
 			)
 		)
-		(pin "D"
-		)
-		(pin "C"
-		)
 		(pin "G"
 		)
@@
 	)
 	(symbol
-		(lib_id "My Symbols:EC11_Rotary_Encoder")
+		(lib_id "My Symbols:EC11_Rotary_Encoder_Board")
 		(at 201.93 45.72 180)
 		(unit 1)
@@
 			)
 		)
-		(pin "D"
-		)
-		(pin "C"
-		)
 		(pin "G"
 		)
@@
 	)
 	(symbol
-		(lib_id "My Symbols:EC11_Rotary_Encoder")
+		(lib_id "My Symbols:EC11_Rotary_Encoder_Board")
 		(at 201.93 198.12 180)
 		(unit 1)
@@
 			)
 		)
-		(pin "D"
-		)
-		(pin "C"
-		)
 		(pin "G"
 		)
@@
 	)
 	(symbol
-		(lib_id "My Symbols:EC11_Rotary_Encoder")
+		(lib_id "My Symbols:EC11_Rotary_Encoder_Board")
 		(at 201.93 248.92 180)
 		(unit 1)
@@
 			)
 		)
-		(pin "D"
-		)
-		(pin "C"
-		)
 		(pin "G"
 		)
@@
 	)
 	(symbol
-		(lib_id "My Symbols:EC11_Rotary_Encoder")
+		(lib_id "My Symbols:EC11_Rotary_Encoder_Board")
 		(at 81.28 147.32 180)
 		(unit 1)
@@
 			)
 		)
-		(pin "D"
-		)
-		(pin "C"
-		)
 		(pin "G"
 		)
@@
 	)
 	(symbol
-		(lib_id "My Symbols:EC11_Rotary_Encoder")
+		(lib_id "My Symbols:EC11_Rotary_Encoder_Board")
 		(at 201.93 96.52 180)
 		(unit 1)
@@
 			)
 		)
-		(pin "D"
-		)
-		(pin "C"
-		)
 		(pin "G"
 		)
@@
 	)
 	(symbol
-		(lib_id "My Symbols:EC11_Rotary_Encoder")
+		(lib_id "My Symbols:EC11_Rotary_Encoder_Board")
 		(at 81.28 198.12 180)
 		(unit 1)
@@
 			)
 		)
-		(pin "D"
-		)
-		(pin "C"
-		)
 		(pin "G"
 		)
@@
 	)
 	(symbol
-		(lib_id "My Symbols:EC11_Rotary_Encoder")
+		(lib_id "My Symbols:EC11_Rotary_Encoder_Board")
 		(at 81.28 45.72 180)
 		(unit 1)
@@
 			)
 		)
-		(pin "D"
-		)
-		(pin "C"
-		)
 		(pin "G"
 		)
@@
 	)
 	(symbol
-		(lib_id "My Symbols:EC11_Rotary_Encoder")
+		(lib_id "My Symbols:EC11_Rotary_Encoder_Board")
 		(at 201.93 147.32 180)
 		(unit 1)
@@
 			)
 		)
-		(pin "D"
-		)
-		(pin "C"
-		)
 		(pin "G"
