File: PCB_CAD/BUCKET_CONTROLS/screws.kicad_sch (KiCad schematic)
At the start: 22 parts

Commit message: save pcb progress lol
Parts:
- removed H5: dac1, My Footprints:SMTSO-M3-3ET, symbol Mechanical:MountingHole_Pad
- removed H6: dac2, My Footprints:SMTSO-M3-3ET, symbol Mechanical:MountingHole_Pad
- removed H7: dac3, My Footprints:SMTSO-M3-3ET, symbol Mechanical:MountingHole_Pad
- removed H8: dac4, My Footprints:SMTSO-M3-3ET, symbol Mechanical:MountingHole_Pad
- H10: value MCP23017_2 -> dac2
- H11: value MCP23017_3 -> dac3
- H13: value MCP23017_4 -> dac4
- H9: value MCP23017_1 -> dac1
Connections:
- no-connect marks 12 -> 8

Commit message: pcb
Parts:
- H1, H10, H11, H13, H2, H3, H4, H9: symbol Mechanical:MountingHole_Pad -> Mechanical:MountingHole
Connections:
- no-connect marks 8 -> 0
Changed lines of the file:
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@@
 		(comment 3 "S.E.D.")
-	)
-	(no_connect
-		(at 213.36 68.58)
-	)
-	(no_connect
-		(at 195.58 68.58)
-	)
-	(no_connect
-		(at 177.8 54.61)
-	)
-	(no_connect
-		(at 195.58 54.61)
-	)
-	(no_connect
-		(at 213.36 54.61)
-	)
-	(no_connect
-		(at 177.8 68.58)
-	)
-	(no_connect
-		(at 160.02 68.58)
-	)
-	(no_connect
-		(at 160.02 54.61)
 	)
 	(symbol
@@
 	)
 	(symbol
-		(lib_id "Mechanical:MountingHole_Pad")
+		(lib_id "Mechanical:MountingHole")
 		(at 177.8 66.04 0)
 		(unit 1)
@@
 		(fields_autoplaced yes)
 		(property "Reference" "H2"
-			(at 180.34 63.4999 0)
+			(at 180.34 64.7699 0)
 			(show_name no)
 			(do_not_autoplace no)
@@
 		)
 		(property "Value" "logic_board2"
-			(at 180.34 66.0399 0)
+			(at 180.34 67.3099 0)
 			(show_name no)
 			(do_not_autoplace no)
@@
 			)
 		)
-		(property "Description" "Mounting Hole with connection"
+		(property "Description" "Mounting Hole without connection"
 			(at 177.8 66.04 0)
 			(hide yes)
@@
 			)
 		)
-		(pin "1"
-		)
 		(instances
 			(project "bucket_controls"
@@
 	)
 	(symbol
-		(lib_id "Mechanical:MountingHole_Pad")
+		(lib_id "Mechanical:MountingHole")
 		(at 160.02 66.04 0)
 		(unit 1)
@@
 		(fields_autoplaced yes)
 		(property "Reference" "H1"
-			(at 162.56 63.4999 0)
+			(at 162.56 64.7699 0)
 			(show_name no)
 			(do_not_autoplace no)
@@
 		)
 		(property "Value" "logic_board1"
-			(at 162.56 66.0399 0)
+			(at 162.56 67.3099 0)
 			(show_name no)
 			(do_not_autoplace no)
@@
 			)
 		)
-		(property "Description" "Mounting Hole with connection"
+		(property "Description" "Mounting Hole without connection"
 			(at 160.02 66.04 0)
 			(hide yes)
@@
 			)
 		)
-		(pin "1"
-		)
 		(instances
 			(project "bucket_controls"
@@
 	)
 	(symbol
-		(lib_id "Mechanical:MountingHole_Pad")
+		(lib_id "Mechanical:MountingHole")
 		(at 213.36 52.07 0)
 		(unit 1)
@@
 		(fields_autoplaced yes)
 		(property "Reference" "H13"
-			(at 215.9 49.5299 0)
+			(at 215.9 50.7999 0)
 			(show_name no)
 			(do_not_autoplace no)
@@
 		)
 		(property "Value" "dac4"
-			(at 215.9 52.0699 0)
+			(at 215.9 53.3399 0)
 			(show_name no)
 			(do_not_autoplace no)
@@
 			)
 		)
-		(property "Description" "Mounting Hole with connection"
+		(property "Description" "Mounting Hole without connection"
 			(at 213.36 52.07 0)
 			(hide yes)
@@
 			)
 		)
-		(pin "1"
-		)
 		(instances
 			(project "bucket_controls"
@@
 	)
 	(symbol
-		(lib_id "Mechanical:MountingHole_Pad")
+		(lib_id "Mechanical:MountingHole")
 		(at 177.8 52.07 0)
 		(unit 1)
@@
 		(fields_autoplaced yes)
 		(property "Reference" "H10"
-			(at 180.34 49.5299 0)
+			(at 180.34 50.7999 0)
 			(show_name no)
 			(do_not_autoplace no)
@@
 		)
 		(property "Value" "dac2"
-			(at 180.34 52.0699 0)
+			(at 180.34 53.3399 0)
 			(show_name no)
 			(do_not_autoplace no)
@@
 			)
 		)
-		(property "Description" "Mounting Hole with connection"
+		(property "Description" "Mounting Hole without connection"
 			(at 177.8 52.07 0)
 			(hide yes)
@@
 			)
 		)
-		(pin "1"
-		)
 		(instances
 			(project "bucket_controls"
@@
 	)
 	(symbol
-		(lib_id "Mechanical:MountingHole_Pad")
+		(lib_id "Mechanical:MountingHole")
 		(at 195.58 66.04 0)
 		(unit 1)
@@
 		(fields_autoplaced yes)
 		(property "Reference" "H3"
-			(at 198.12 63.4999 0)
+			(at 198.12 64.7699 0)
 			(show_name no)
 			(do_not_autoplace no)
@@
 		)
 		(property "Value" "logic_board3"
-			(at 198.12 66.0399 0)
+			(at 198.12 67.3099 0)
 			(show_name no)
 			(do_not_autoplace no)
@@
 			)
 		)
-		(property "Description" "Mounting Hole with connection"
+		(property "Description" "Mounting Hole without connection"
 			(at 195.58 66.04 0)
 			(hide yes)
@@
 			)
 		)
-		(pin "1"
-		)
 		(instances
 			(project "bucket_controls"
@@
 	)
 	(symbol
-		(lib_id "Mechanical:MountingHole_Pad")
+		(lib_id "Mechanical:MountingHole")
 		(at 213.36 66.04 0)
 		(unit 1)
@@
 		(fields_autoplaced yes)
 		(property "Reference" "H4"
-			(at 215.9 63.4999 0)
+			(at 215.9 64.7699 0)
 			(show_name no)
 			(do_not_autoplace no)
@@
 		)
 		(property "Value" "logic_board4"
-			(at 215.9 66.0399 0)
+			(at 215.9 67.3099 0)
 			(show_name no)
 			(do_not_autoplace no)
@@
 			)
 		)
-		(property "Description" "Mounting Hole with connection"
+		(property "Description" "Mounting Hole without connection"
 			(at 213.36 66.04 0)
 			(hide yes)
@@
 			)
 		)
-		(pin "1"
-		)
 		(instances
 			(project "bucket_controls"
@@
 	)
 	(symbol
-		(lib_id "Mechanical:MountingHole_Pad")
+		(lib_id "Mechanical:MountingHole")
 		(at 195.58 52.07 0)
 		(unit 1)
@@
 		(fields_autoplaced yes)
 		(property "Reference" "H11"
-			(at 198.12 49.5299 0)
+			(at 198.12 50.7999 0)
 			(show_name no)
 			(do_not_autoplace no)
@@
 		)
 		(property "Value" "dac3"
-			(at 198.12 52.0699 0)
+			(at 198.12 53.3399 0)
 			(show_name no)
 			(do_not_autoplace no)
@@
 			)
 		)
-		(property "Description" "Mounting Hole with connection"
+		(property "Description" "Mounting Hole without connection"
 			(at 195.58 52.07 0)
 			(hide yes)
@@
 			)
 		)
-		(pin "1"
-		)
 		(instances
 			(project "bucket_controls"
@@
 	)
 	(symbol
-		(lib_id "Mechanical:MountingHole_Pad")
+		(lib_id "Mechanical:MountingHole")
 		(at 160.02 52.07 0)
 		(unit 1)
@@
 		(fields_autoplaced yes)
 		(property "Reference" "H9"
-			(at 162.56 49.5299 0)
+			(at 162.56 50.7999 0)
 			(show_name no)
 			(do_not_autoplace no)
@@
 		)
 		(property "Value" "dac1"
-			(at 162.56 52.0699 0)
+			(at 162.56 53.3399 0)
 			(show_name no)
 			(do_not_autoplace no)
@@
 			)
 		)
-		(property "Description" "Mounting Hole with connection"
+		(property "Description" "Mounting Hole without connection"
 			(at 160.02 52.07 0)
 			(hide yes)
@@
 			)
 		)
-		(pin "1"
-		)
-		(instances
+		(instances
