File: PCB_CAD/BUCKET_CONTROLS/btns0.kicad_sch (KiCad schematic)
At the start: 83 parts, among them SW11 C0_B0, SW12 C0_B1, SW13 C0_B2, SW14 C0_B3, SW15 C0_B4, SW16 C0_B5, SW17 C0_B6, SW18 C0_B7, SW19 C0_B8, SW20 C0_B9, SW21 C0_B10, SW22 C0_B11

Commit message: pcb controls
Parts:
- C41, C42, D17, D18, R94, R95, R96, R97, R98, R99: now not fitted
- D10, D2, D3, D4, D8, D9, SW12, SW13, SW14: LCSC manual -> dnp
- D19, D20, SW21, SW22: LCSC manual -> dnp; now not fitted
- SW11, SW15, SW16, SW17, SW18, SW19, SW20: footprint My Footprints:CFPB-1CC-4W6 -> My Footprints:CFPB-1CC-4W6_LOWPROF; LCSC manual -> dnp
Changed lines of the file:
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@@
 		(exclude_from_sim no)
 		(in_bom yes)
-		(on_board yes)
+		(on_board no)
 		(in_pos_files yes)
-		(dnp no)
+		(dnp yes)
 		(fields_autoplaced yes)
 		(property "Reference" "#PWR0177"
@@
 		(exclude_from_sim no)
 		(in_bom yes)
-		(on_board yes)
+		(on_board no)
 		(in_pos_files yes)
-		(dnp no)
+		(dnp yes)
 		(fields_autoplaced yes)
 		(property "Reference" "#PWR0181"
@@
 		(exclude_from_sim no)
 		(in_bom yes)
-		(on_board yes)
+		(on_board no)
 		(in_pos_files yes)
-		(dnp no)
+		(dnp yes)
 		(fields_autoplaced yes)
 		(property "Reference" "SW22"
@@
 			)
 		)
-		(property "LCSC" "manual"
+		(property "LCSC" "dnp"
 			(at 171.45 245.11 0)
 			(hide yes)
@@
 		(exclude_from_sim no)
 		(in_bom yes)
-		(on_board yes)
+		(on_board no)
 		(in_pos_files yes)
-		(dnp no)
+		(dnp yes)
 		(fields_autoplaced yes)
 		(property "Reference" "#PWR0179"
@@
 		(exclude_from_sim no)
 		(in_bom yes)
-		(on_board yes)
+		(on_board no)
 		(in_pos_files yes)
-		(dnp no)
+		(dnp yes)
 		(property "Reference" "R98"
 			(at 121.92 265.43 90)
@@
 			)
 		)
-		(property "Footprint" "My Footprints:CFPB-1CC-4W6"
+		(property "Footprint" "My Footprints:CFPB-1CC-4W6_LOWPROF"
 			(at 44.45 148.59 0)
 			(hide yes)
@@
 			)
 		)
-		(property "LCSC" "manual"
+		(property "LCSC" "dnp"
 			(at 44.45 156.21 0)
 			(hide yes)
@@
 			)
 		)
-		(property "LCSC" "manual"
+		(property "LCSC" "dnp"
 			(at 196.85 48.26 0)
 			(hide yes)
@@
 		(exclude_from_sim no)
 		(in_bom yes)
-		(on_board yes)
+		(on_board no)
 		(in_pos_files yes)
-		(dnp no)
+		(dnp yes)
 		(property "Reference" "R97"
 			(at 188.976 252.222 90)
@@
 			)
 		)
-		(property "Footprint" "My Footprints:CFPB-1CC-4W6"
+		(property "Footprint" "My Footprints:CFPB-1CC-4W6_LOWPROF"
 			(at 44.45 199.39 0)
 			(hide yes)
@@
 			)
 		)
-		(property "LCSC" "manual"
+		(property "LCSC" "dnp"
 			(at 44.45 207.01 0)
 			(hide yes)
@@
 			)
 		)
-		(property "Footprint" "My Footprints:CFPB-1CC-4W6"
+		(property "Footprint" "My Footprints:CFPB-1CC-4W6_LOWPROF"
 			(at 171.45 148.59 0)
 			(hide yes)
@@
 			)
 		)
-		(property "LCSC" "manual"
+		(property "LCSC" "dnp"
 			(at 171.45 156.21 0)
 			(hide yes)
@@
 		(exclude_from_sim no)
 		(in_bom yes)
-		(on_board yes)
+		(on_board no)
 		(in_pos_files yes)
-		(dnp no)
+		(dnp yes)
 		(fields_autoplaced yes)
 		(property "Reference" "C41"
@@
 			)
 		)
-		(property "Footprint" "My Footprints:CFPB-1CC-4W6"
+		(property "Footprint" "My Footprints:CFPB-1CC-4W6_LOWPROF"
 			(at 107.95 199.39 0)
 			(hide yes)
@@
 			)
 		)
-		(property "LCSC" "manual"
+		(property "LCSC" "dnp"
 			(at 107.95 207.01 0)
 			(hide yes)
@@
 			)
 		)
-		(property "LCSC" "manual"
+		(property "LCSC" "dnp"
 			(at 171.45 91.44 0)
 			(hide yes)
@@
 		(exclude_from_sim no)
 		(in_bom yes)
-		(on_board yes)
+		(on_board no)
 		(in_pos_files yes)
-		(dnp no)
+		(dnp yes)
 		(fields_autoplaced yes)
 		(property "Reference" "#PWR0184"
@@
 			)
 		)
-		(property "LCSC" "manual"
+		(property "LCSC" "dnp"
 			(at 48.26 109.22 0)
 			(hide yes)
@@
 		(exclude_from_sim no)
 		(in_bom yes)
-		(on_board yes)
+		(on_board no)
 		(in_pos_files yes)
-		(dnp no)
+		(dnp yes)
 		(property "Reference" "R99"
 			(at 185.42 265.43 90)
@@
 			)
 		)
-		(property "LCSC" "manual"
+		(property "LCSC" "dnp"
 			(at 114.3 48.26 0)
 			(hide yes)
@@
 		(exclude_from_sim no)
 		(in_bom yes)
-		(on_board yes)
+		(on_board no)
 		(in_pos_files yes)
-		(dnp no)
+		(dnp yes)
 		(fields_autoplaced yes)
 		(property "Reference" "C42"
@@
 			)
 		)
-		(property "Footprint" "My Footprints:CFPB-1CC-4W6"
+		(property "Footprint" "My Footprints:CFPB-1CC-4W6_LOWPROF"
 			(at 44.45 45.72 0)
 			(hide yes)
@@
 			)
 		)
-		(property "LCSC" "manual"
+		(property "LCSC" "dnp"
 			(at 44.45 53.34 0)
 			(hide yes)
@@
 			)
 		)
-		(property "LCSC" "manual"
+		(property "LCSC" "dnp"
 			(at 107.95 91.44 0)
 			(hide yes)
@@
 			)
 		)
-		(property "LCSC" "manual"
+		(property "LCSC" "dnp"
 			(at 44.45 91.44 0)
 			(hide yes)
@@
 		(exclude_from_sim no)
 		(in_bom yes)
-		(on_board yes)
+		(on_board no)
 		(in_pos_files yes)
-		(dnp no)
+		(dnp yes)
 		(fields_autoplaced yes)
 		(property "Reference" "D19"
@@
 			)
 		)
-		(property "LCSC" "manual"
+		(property "LCSC" "dnp"
 			(at 111.76 262.89 0)
 			(hide yes)
@@
 		(exclude_from_sim no)
 		(in_bom yes)
-		(on_board yes)
+		(on_board no)
 		(in_pos_files yes)
-		(dnp no)
+		(dnp yes)
 		(property "Reference" "D17"
 			(at 128.016 237.236 0)
@@
 		(exclude_from_sim no)
 		(in_bom yes)
-		(on_board yes)
+		(on_board no)
 		(in_pos_files yes)
-		(dnp no)
+		(dnp yes)
 		(fields_autoplaced yes)
 		(property "Reference" "#PWR0183"
@@
 		(exclude_from_sim no)
 		(in_bom yes)
-		(on_board yes)
+		(on_board no)
 		(in_pos_files yes)
-		(dnp no)
+		(dnp yes)
 		(fields_autoplaced yes)
 		(property "Reference" "SW21"
@@
 			)
 		)
-		(property "LCSC" "manual"
+		(property "LCSC" "dnp"
 			(at 107.95 245.11 0)
 			(hide yes)
@@
 			)
 		)
-		(property "LCSC" "manual"
+		(property "LCSC" "dnp"
 			(at 175.26 109.22 0)
 			(hide yes)
@@
 		(exclude_from_sim no)
 		(in_bom yes)
-		(on_board yes)
+		(on_board no)
 		(in_pos_files yes)
-		(dnp no)
+		(dnp yes)
 		(property "Reference" "D18"
 			(at 191.516 237.236 0)
@@
 		(exclude_from_sim no)
 		(in_bom yes)
-		(on_board yes)
+		(on_board no)
 		(in_pos_files yes)
-		(dnp no)
+		(dnp yes)
 		(fields_autoplaced yes)
 		(property "Reference" "D20"
@@
 			)
 		)
-		(property "LCSC" "manual"
+		(property "LCSC" "dnp"
 			(at 175.26 262.89 0)
 			(hide yes)
@@
 			)
 		)
-		(property "LCSC" "manual"
+		(property "LCSC" "dnp"
 			(at 156.21 48.26 0)
 			(hide yes)
@@
 		(exclude_from_sim no)
 		(in_bom yes)
-		(on_board yes)
+		(on_board no)
 		(in_pos_files yes)
-		(dnp no)
+		(dnp yes)
 		(fields_autoplaced yes)
 		(property "Reference" "#PWR0180"
@@
 		(exclude_from_sim no)
 		(in_bom yes)
-		(on_board yes)
+		(on_board no)
 		(in_pos_files yes)
-		(dnp no)
+		(dnp yes)
 		(property "Reference" "R95"
 			(at 179.324 235.458 0)
@@
 		(exclude_from_sim no)
 		(in_bom yes)
-		(on_board yes)
+		(on_board no)
 		(in_pos_files yes)
-		(dnp no)
+		(dnp yes)
 		(property "Reference" "R96"
 			(at 125.476 252.222 90)
@@
 		(exclude_from_sim no)
 		(in_bom yes)
-		(on_board yes)
+		(on_board no)
 		(in_pos_files yes)
-		(dnp no)
+		(dnp yes)
 		(fields_autoplaced yes)
 		(property "Reference" "#PWR0178"
@@
 		(exclude_from_sim no)
 		(in_bom yes)
-		(on_board yes)
+		(on_board no)
 		(in_pos_files yes)
-		(dnp no)
+		(dnp yes)
 		(fields_autoplaced yes)
 		(property "Reference" "#PWR0182"
@@
 			)
 		)
-		(property "Footprint" "My Footprints:CFPB-1CC-4W6"
+		(property "Footprint" "My Footprints:CFPB-1CC-4W6_LOWPROF"
 			(at 107.95 148.59 0)
 			(hide yes)
@@
 			)
 		)
-		(property "LCSC" "manual"
+		(property "LCSC" "dnp"
 			(at 107.95 156.21 0)
 			(hide yes)
@@
 			)
 		)
-		(property "LCSC" "manual"
+		(property "LCSC" "dnp"
 			(at 111.76 109.22 0)
 			(hide yes)
@@
 			)
 		)
-		(property "Footprint" "My Footprints:CFPB-1CC-4W6"
+		(property "Footprint" "My Footprints:CFPB-1CC-4W6_LOWPROF"
 			(at 171.45 199.39 0)
 			(hide yes)
@@
 			)
 		)
-		(property "LCSC" "manual"
+		(property "LCSC" "dnp"
 			(at 171.45 207.01 0)
 			(hide yes)
@@
 		(exclude_from_sim no)
 		(in_bom yes)
-		(on_board yes)
+		(on_board no)
 		(in_pos_files yes)
-		(dnp no)
+		(dnp yes)
 		(property "Reference" "R94"
 			(at 115.824 235.458 0)

Commit message: ctrls board rev 0 done & sent to fab
Parts:
- R63, R64, R65, R73, R74, R75: value 330 -> 6.8k; LCSC C23138 -> C23212
- R66, R82, R83, R84, R91, R92, R93, R98, R99: value 330 -> 470; LCSC C23138 -> C25241
Changed lines of the file:
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@@
 			)
 		)
-		(property "Value" "330"
+		(property "Value" "470"
 			(at 117.856 158.75 90)
 			(show_name no)
@@
 			)
 		)
-		(property "LCSC" "C23138"
+		(property "LCSC" "C25241"
 			(at 120.65 156.21 90)
 			(hide yes)
@@
 			)
 		)
-		(property "Value" "330"
+		(property "Value" "470"
 			(at 54.356 158.75 90)
 			(show_name no)
@@
 			)
 		)
-		(property "LCSC" "C23138"
+		(property "LCSC" "C25241"
 			(at 57.15 156.21 90)
 			(hide yes)
@@
 			)
 		)
-		(property "Value" "330"
+		(property "Value" "470"
 			(at 116.586 265.43 90)
 			(show_name no)
@@
 			)
 		)
-		(property "LCSC" "C23138"
+		(property "LCSC" "C25241"
 			(at 119.38 262.89 90)
 			(hide yes)
@@
 			)
 		)
-		(property "Value" "330"
+		(property "Value" "470"
 			(at 181.356 209.55 90)
 			(show_name no)
@@
 			)
 		)
-		(property "LCSC" "C23138"
+		(property "LCSC" "C25241"
 			(at 184.15 207.01 90)
 			(hide yes)
@@
 			)
 		)
-		(property "Value" "330"
+		(property "Value" "6.8k"
 			(at 201.676 50.8 90)
 			(show_name no)
@@
 			)
 		)
-		(property "LCSC" "C23138"
+		(property "LCSC" "C23212"
 			(at 204.47 48.26 90)
 			(hide yes)
@@
 			)
 		)
-		(property "Value" "330"
+		(property "Value" "470"
 			(at 54.356 209.55 90)
 			(show_name no)
@@
 			)
 		)
-		(property "LCSC" "C23138"
+		(property "LCSC" "C25241"
 			(at 57.15 207.01 90)
 			(hide yes)
@@
 			)
 		)
-		(property "Value" "330"
+		(property "Value" "470"
 			(at 180.086 265.43 90)
 			(show_name no)
@@
 			)
 		)
-		(property "LCSC" "C23138"
+		(property "LCSC" "C25241"
 			(at 182.88 262.89 90)
 			(hide yes)
@@
 			)
 		)
-		(property "Value" "330"
+		(property "Value" "6.8k"
 			(at 119.126 50.8 90)
 			(show_name no)
@@
 			)
 		)
-		(property "LCSC" "C23138"
+		(property "LCSC" "C23212"
 			(at 121.92 48.26 90)
 			(hide yes)
@@
 			)
 		)
-		(property "Value" "330"
+		(property "Value" "470"
 			(at 181.356 158.75 90)
 			(show_name no)
@@
 			)
 		)
-		(property "LCSC" "C23138"
+		(property "LCSC" "C25241"
 			(at 184.15 156.21 90)
 			(hide yes)
@@
 			)
 		)
-		(property "Value" "330"
+		(property "Value" "6.8k"
 			(at 53.086 111.76 90)
 			(show_name no)
@@
 			)
 		)
-		(property "LCSC" "C23138"
+		(property "LCSC" "C23212"
 			(at 55.88 109.22 90)
 			(hide yes)
@@
 			)
 		)
-		(property "Value" "330"
+		(property "Value" "6.8k"
 			(at 161.036 50.8 90)
 			(show_name no)
@@
 			)
 		)
-		(property "LCSC" "C23138"
+		(property "LCSC" "C23212"
 			(at 163.83 48.26 90)
 			(hide yes)
@@
 			)
 		)
-		(property "Value" "330"
+		(property "Value" "470"
 			(at 54.356 55.88 90)
 			(show_name no)
@@
 			)
 		)
-		(property "LCSC" "C23138"
+		(property "LCSC" "C25241"
 			(at 57.15 53.34 90)
 			(hide yes)
@@
 			)
 		)
-		(property "Value" "330"
+		(property "Value" "6.8k"
 			(at 116.586 111.76 90)
 			(show_name no)
@@
 			)
 		)
-		(property "LCSC" "C23138"
+		(property "LCSC" "C23212"
 			(at 119.38 109.22 90)
 			(hide yes)
@@
 			)
 		)
-		(property "Value" "330"
+		(property "Value" "6.8k"
 			(at 180.086 111.76 90)
 			(show_name no)
@@
 			)
 		)
-		(property "LCSC" "C23138"
+		(property "LCSC" "C23212"
 			(at 182.88 109.22 90)
 			(hide yes)
@@
 			)
 		)
-		(property "Value" "330"
+		(property "Value" "470"
 			(at 117.856 209.55 90)
 			(show_name no)
@@
 			)
 		)
-		(property "LCSC" "C23138"
+		(property "LCSC" "C25241"
 			(at 120.65 207.01 90)
 			(hide yes)
