File: PCB_CAD/BUCKET_CONTROLS/btns1.kicad_sch (KiCad schematic)
At the start: 83 parts, among them SW11 C0_B0, SW12 C0_B1, SW13 C0_B2, SW14 C0_B3, SW15 C0_B4, SW16 C0_B5, SW17 C0_B6, SW18 C0_B7, SW19 C0_B8, SW20 C0_B9, SW21 C0_B10, SW22 C0_B11

Commit message: saving progress on controls pcb
Parts:
- removed C31, C32, C33, C34, C35, C36, C37, C38, C39, C40, C41, C42: 1u, Capacitor_SMD:C_0603_1608Metric, symbol Device:C
- removed D1, D11, D12, D13, D14, D15, D16, D17, D18, D5, D6, D7: 1N4148, Diode_SMD:D_SOD-323, symbol Device:D
- removed D10, D19, D2, D20, D3, D4, D8, D9: LED, LED_THT:LED_D3.0mm_FlatTop, symbol Device:LED
- removed R61, R67, R68, R69, R76, R77, R78, R85, R86, R87, R94, R95: 47k, Resistor_SMD:R_0603_1608Metric, symbol Device:R_US
- removed R62, R70, R71, R72, R79, R80, R81, R88, R89, R90, R96, R97: 15k, Resistor_SMD:R_0603_1608Metric, symbol Device:R_US
- removed R63, R64, R65, R66, R73, R74, R75, R82, R83, R84, R91, R92, R93, R98, R99: 330, Resistor_SMD:R_0603_1608Metric, symbol Device:R_US
- removed SW11: C0_B0, My Footprints:CFPB-1CC-4W6, symbol Switch:SW_Push_LED
- removed SW12: C0_B1, My Footprints:TL2201EEZB, symbol Switch:SW_Push_DPDT
- removed SW13: C0_B2, My Footprints:TL2201EEZB, symbol Switch:SW_Push_DPDT
- removed SW14: C0_B3, My Footprints:TL2201EEZB, symbol Switch:SW_Push_DPDT
- removed SW15: C0_B4, My Footprints:CFPB-1CC-4W6, symbol Switch:SW_Push_LED
- removed SW16: C0_B5, My Footprints:CFPB-1CC-4W6, symbol Switch:SW_Push_LED
- removed SW17: C0_B6, My Footprints:CFPB-1CC-4W6, symbol Switch:SW_Push_LED
- removed SW18: C0_B7, My Footprints:CFPB-1CC-4W6, symbol Switch:SW_Push_LED
- removed SW19: C0_B8, My Footprints:CFPB-1CC-4W6, symbol Switch:SW_Push_LED
- removed SW20: C0_B9, My Footprints:CFPB-1CC-4W6, symbol Switch:SW_Push_LED
- removed SW21: C0_B10, My Footprints:TL2201EEZB, symbol Switch:SW_Push_DPDT
- removed SW22: C0_B11, My Footprints:TL2201EEZB, symbol Switch:SW_Push_DPDT
- added C131, C132, C133, C134, C135, C136, C137, C138, C139, C140, C141, C142: 1u, Capacitor_SMD:C_0603_1608Metric, symbol Device:C
- added D101, D105, D106, D107, D111, D112, D113, D114, D115, D116, D117, D118: 1N4148, Diode_SMD:D_SOD-323, symbol Device:D
- added D102, D103, D104, D108, D109, D110, D119, D120: LED, LED_THT:LED_D3.0mm_FlatTop, symbol Device:LED
- added R161, R167, R168, R169, R176, R177, R178, R185, R186, R187, R194, R195: 47k, Resistor_SMD:R_0603_1608Metric, symbol Device:R_US
- added R162, R170, R171, R172, R179, R180, R181, R188, R189, R190, R196, R197: 15k, Resistor_SMD:R_0603_1608Metric, symbol Device:R_US
- added R163, R164, R165, R166, R173, R174, R175, R182, R183, R184, R191, R192, R193, R198, R199: 330, Resistor_SMD:R_0603_1608Metric, symbol Device:R_US
- added SW111: C1_B0, My Footprints:CFPB-1CC-4W6, symbol Switch:SW_Push_LED
- added SW112: C1_B1, My Footprints:TL2201EEZB, symbol Switch:SW_Push_DPDT
- added SW113: C1_B2, My Footprints:TL2201EEZB, symbol Switch:SW_Push_DPDT
- added SW114: C1_B3, My Footprints:TL2201EEZB, symbol Switch:SW_Push_DPDT
- added SW115: C1_B4, My Footprints:CFPB-1CC-4W6, symbol Switch:SW_Push_LED
- added SW116: C1_B5, My Footprints:CFPB-1CC-4W6, symbol Switch:SW_Push_LED
- added SW117: C1_B6, My Footprints:CFPB-1CC-4W6, symbol Switch:SW_Push_LED
- added SW118: C1_B7, My Footprints:CFPB-1CC-4W6, symbol Switch:SW_Push_LED
- added SW119: C1_B8, My Footprints:CFPB-1CC-4W6, symbol Switch:SW_Push_LED
- added SW120: C1_B9, My Footprints:CFPB-1CC-4W6, symbol Switch:SW_Push_LED
- added SW121: C1_B10, My Footprints:TL2201EEZB, symbol Switch:SW_Push_DPDT
- added SW122: C1_B11, My Footprints:TL2201EEZB, symbol Switch:SW_Push_DPDT
Connections:
- net +3V3: now also R161.1, R167.1, R168.1, R169.1, R176.1, R177.1, R178.1, R185.1, R186.1, R187.1, R194.1, R195.1
- net GND: now also C131.2, C132.2, C133.2, C134.2, C135.2, C136.2, C137.2, C138.2, C139.2, C140.2, C141.2, C142.2, D102.1 (K), D103.1 (K), D104.1 (K), D108.1 (K), D109.1 (K), D110.1 (K), D119.1 (K), D120.1 (K), SW111.1, SW111.4 (K), SW112.2 (B), SW113.2 (B), SW114.2 (B), SW115.1, SW115.4 (K), SW116.1, SW116.4 (K), SW117.1, SW117.4 (K), SW118.1, SW118.4 (K), SW119.1, SW119.4 (K), SW120.1, SW120.4 (K), SW121.2 (B), SW122.2 (B)
- new net: D101.2 (A), R161.2, R162.1, SW111.2
- new net: D102.2 (A), R163.1
- new net: D105.2 (A), R167.2, R170.1, SW112.3 (C)
- new net: D115.2 (A), R186.2, R189.1, SW119.2
- new net: D113.2 (A), R178.2, R181.1, SW117.2
- new net: D108.2 (A), R173.1
- new net: R184.1, SW117.3 (A)
- new net: D109.2 (A), R174.1
- new net: D114.2 (A), R185.2, R188.1, SW118.2
- new net: D116.2 (A), R187.2, R190.1, SW120.2
- new net: R193.1, SW120.3 (A)
- new net: D104.2 (A), R165.1
- new net: D118.2 (A), R195.2, R197.1, SW122.3 (C)
- new net: D111.2 (A), R176.2, R179.1, SW115.2
- new net: D119.2 (A), R198.1
- new net: D106.2 (A), R168.2, R171.1, SW113.3 (C)
- new net: D112.2 (A), R177.2, R180.1, SW116.2
- new net: D110.2 (A), R175.1
- new net: D117.2 (A), R194.2, R196.1, SW121.3 (C)
- new net: R191.1, SW118.3 (A)
- new net: R182.1, SW115.3 (A)
- new net: R166.1, SW111.3 (A)
- new net: D107.2 (A), R169.2, R172.1, SW114.3 (C)
- new net: D103.2 (A), R164.1
- new net: R183.1, SW116.3 (A)
- new net: R192.1, SW119.3 (A)
- new net: D120.2 (A), R199.1
- new net C1_B0: C131.1, D101.1 (K), R162.2
- new net C1_B0_L: R166.2
- new net C1_B0_LA: R163.2
- new net C1_B0_LB: R164.2
- new net C1_B0_LC: R165.2
- new net C1_B1: C132.1, D105.1 (K), R170.2
- new net C1_B10: C141.1, D117.1 (K), R196.2
- new net C1_B10_L: R198.2
- new net C1_B11: C142.1, D118.1 (K), R197.2
- new net C1_B11_L: R199.2
- new net C1_B1_L: R173.2
- new net C1_B2: C133.1, D106.1 (K), R171.2
- new net C1_B2_L: R174.2
- new net C1_B3: C134.1, D107.1 (K), R172.2
- new net C1_B3_L: R175.2
- new net C1_B4: C135.1, D111.1 (K), R179.2
- new net C1_B4_L: R182.2
- new net C1_B5: C136.1, D112.1 (K), R180.2
- new net C1_B5_L: R183.2
- new net C1_B6: C137.1, D113.1 (K), R181.2
- new net C1_B6_L: R184.2
- new net C1_B7: C138.1, D114.1 (K), R188.2
- new net C1_B7_L: R191.2
- new net C1_B8: C139.1, D115.1 (K), R189.2
- new net C1_B8_L: R192.2
- new net C1_B9: C140.1, D116.1 (K), R190.2
- new net C1_B9_L: R193.2

Commit message: pcb controls
Parts:
- C141, C142, D117, D118, R194, R195, R196, R197, R198, R199: now not fitted
- D102, D103, D104, D108, D109, D110, SW112, SW113, SW114: LCSC manual -> dnp
- D119, D120, SW121, SW122: LCSC manual -> dnp; now not fitted
- SW111, SW115, SW116, SW117, SW118, SW119, SW120: footprint My Footprints:CFPB-1CC-4W6 -> My Footprints:CFPB-1CC-4W6_LOWPROF; LCSC manual -> dnp
Changed lines of the file:
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@@
 		(exclude_from_sim no)
 		(in_bom yes)
-		(on_board yes)
+		(on_board no)
 		(in_pos_files yes)
-		(dnp no)
+		(dnp yes)
 		(fields_autoplaced yes)
 		(property "Reference" "#PWR0292"
@@
 			)
 		)
-		(property "LCSC" "manual"
+		(property "LCSC" "dnp"
 			(at 114.3 48.26 0)
 			(hide yes)
@@
 			)
 		)
-		(property "LCSC" "manual"
+		(property "LCSC" "dnp"
 			(at 44.45 91.44 0)
 			(hide yes)
@@
 			)
 		)
-		(property "Footprint" "My Footprints:CFPB-1CC-4W6"
+		(property "Footprint" "My Footprints:CFPB-1CC-4W6_LOWPROF"
 			(at 171.45 148.59 0)
 			(hide yes)
@@
 			)
 		)
-		(property "LCSC" "manual"
+		(property "LCSC" "dnp"
 			(at 171.45 156.21 0)
 			(hide yes)
@@
 		(exclude_from_sim no)
 		(in_bom yes)
-		(on_board yes)
+		(on_board no)
 		(in_pos_files yes)
-		(dnp no)
+		(dnp yes)
 		(fields_autoplaced yes)
 		(property "Reference" "C142"
@@
 			)
 		)
-		(property "Footprint" "My Footprints:CFPB-1CC-4W6"
+		(property "Footprint" "My Footprints:CFPB-1CC-4W6_LOWPROF"
 			(at 171.45 199.39 0)
 			(hide yes)
@@
 			)
 		)
-		(property "LCSC" "manual"
+		(property "LCSC" "dnp"
 			(at 171.45 207.01 0)
 			(hide yes)
@@
 			)
 		)
-		(property "LCSC" "manual"
+		(property "LCSC" "dnp"
 			(at 196.85 48.26 0)
 			(hide yes)
@@
 		(exclude_from_sim no)
 		(in_bom yes)
-		(on_board yes)
+		(on_board no)
 		(in_pos_files yes)
-		(dnp no)
+		(dnp yes)
 		(property "Reference" "R197"
 			(at 188.976 252.222 90)
@@
 		(exclude_from_sim no)
 		(in_bom yes)
-		(on_board yes)
+		(on_board no)
 		(in_pos_files yes)
-		(dnp no)
+		(dnp yes)
 		(fields_autoplaced yes)
 		(property "Reference" "#PWR0297"
@@
 		(exclude_from_sim no)
 		(in_bom yes)
-		(on_board yes)
+		(on_board no)
 		(in_pos_files yes)
-		(dnp no)
+		(dnp yes)
 		(fields_autoplaced yes)
 		(property "Reference" "#PWR0294"
@@
 		(exclude_from_sim no)
 		(in_bom yes)
-		(on_board yes)
+		(on_board no)
 		(in_pos_files yes)
-		(dnp no)
+		(dnp yes)
 		(fields_autoplaced yes)
 		(property "Reference" "#PWR0293"
@@
 		(exclude_from_sim no)
 		(in_bom yes)
-		(on_board yes)
+		(on_board no)
 		(in_pos_files yes)
-		(dnp no)
+		(dnp yes)
 		(fields_autoplaced yes)
 		(property "Reference" "D119"
@@
 			)
 		)
-		(property "LCSC" "manual"
+		(property "LCSC" "dnp"
 			(at 111.76 262.89 0)
 			(hide yes)
@@
 			)
 		)
-		(property "LCSC" "manual"
+		(property "LCSC" "dnp"
 			(at 111.76 109.22 0)
 			(hide yes)
@@
 		(exclude_from_sim no)
 		(in_bom yes)
-		(on_board yes)
+		(on_board no)
 		(in_pos_files yes)
-		(dnp no)
+		(dnp yes)
 		(fields_autoplaced yes)
 		(property "Reference" "C141"
@@
 		(exclude_from_sim no)
 		(in_bom yes)
-		(on_board yes)
+		(on_board no)
 		(in_pos_files yes)
-		(dnp no)
+		(dnp yes)
 		(fields_autoplaced yes)
 		(property "Reference" "#PWR0296"
@@
 		(exclude_from_sim no)
 		(in_bom yes)
-		(on_board yes)
+		(on_board no)
 		(in_pos_files yes)
-		(dnp no)
+		(dnp yes)
 		(property "Reference" "R194"
 			(at 115.824 235.458 0)
@@
 			)
 		)
-		(property "LCSC" "manual"
+		(property "LCSC" "dnp"
 			(at 48.26 109.22 0)
 			(hide yes)
@@
 		(exclude_from_sim no)
 		(in_bom yes)
-		(on_board yes)
+		(on_board no)
 		(in_pos_files yes)
-		(dnp no)
+		(dnp yes)
 		(property "Reference" "D118"
 			(at 191.516 237.236 0)
@@
 		(exclude_from_sim no)
 		(in_bom yes)
-		(on_board yes)
+		(on_board no)
 		(in_pos_files yes)
-		(dnp no)
+		(dnp yes)
 		(fields_autoplaced yes)
 		(property "Reference" "#PWR0291"
@@
 			)
 		)
-		(property "Footprint" "My Footprints:CFPB-1CC-4W6"
+		(property "Footprint" "My Footprints:CFPB-1CC-4W6_LOWPROF"
 			(at 44.45 45.72 0)
 			(hide yes)
@@
 			)
 		)
-		(property "LCSC" "manual"
+		(property "LCSC" "dnp"
 			(at 44.45 53.34 0)
 			(hide yes)
@@
 		(exclude_from_sim no)
 		(in_bom yes)
-		(on_board yes)
+		(on_board no)
 		(in_pos_files yes)
-		(dnp no)
+		(dnp yes)
 		(fields_autoplaced yes)
 		(property "Reference" "#PWR0298"
@@
 		(exclude_from_sim no)
 		(in_bom yes)
-		(on_board yes)
+		(on_board no)
 		(in_pos_files yes)
-		(dnp no)
+		(dnp yes)
 		(property "Reference" "D117"
 			(at 128.016 237.236 0)
@@
 			)
 		)
-		(property "LCSC" "manual"
+		(property "LCSC" "dnp"
 			(at 156.21 48.26 0)
 			(hide yes)
@@
 		(exclude_from_sim no)
 		(in_bom yes)
-		(on_board yes)
+		(on_board no)
 		(in_pos_files yes)
-		(dnp no)
+		(dnp yes)
 		(property "Reference" "R198"
 			(at 121.92 265.43 90)
@@
 			)
 		)
-		(property "LCSC" "manual"
+		(property "LCSC" "dnp"
 			(at 175.26 109.22 0)
 			(hide yes)
@@
 		(exclude_from_sim no)
 		(in_bom yes)
-		(on_board yes)
+		(on_board no)
 		(in_pos_files yes)
-		(dnp no)
+		(dnp yes)
 		(fields_autoplaced yes)
 		(property "Reference" "SW122"
@@
 			)
 		)
-		(property "LCSC" "manual"
+		(property "LCSC" "dnp"
 			(at 171.45 245.11 0)
 			(hide yes)
@@
 			)
 		)
-		(property "LCSC" "manual"
+		(property "LCSC" "dnp"
 			(at 171.45 91.44 0)
 			(hide yes)
@@
 			)
 		)
-		(property "Footprint" "My Footprints:CFPB-1CC-4W6"
+		(property "Footprint" "My Footprints:CFPB-1CC-4W6_LOWPROF"
 			(at 44.45 148.59 0)
 			(hide yes)
@@
 			)
 		)
-		(property "LCSC" "manual"
+		(property "LCSC" "dnp"
 			(at 44.45 156.21 0)
 			(hide yes)
@@
 			)
 		)
-		(property "LCSC" "manual"
+		(property "LCSC" "dnp"
 			(at 107.95 91.44 0)
 			(hide yes)
@@
 		(exclude_from_sim no)
 		(in_bom yes)
-		(on_board yes)
+		(on_board no)
 		(in_pos_files yes)
-		(dnp no)
+		(dnp yes)
 		(fields_autoplaced yes)
 		(property "Reference" "#PWR0295"
@@
 			)
 		)
-		(property "Footprint" "My Footprints:CFPB-1CC-4W6"
+		(property "Footprint" "My Footprints:CFPB-1CC-4W6_LOWPROF"
 			(at 107.95 148.59 0)
 			(hide yes)
@@
 			)
 		)
-		(property "LCSC" "manual"
+		(property "LCSC" "dnp"
 			(at 107.95 156.21 0)
 			(hide yes)
@@
 			)
 		)
-		(property "Footprint" "My Footprints:CFPB-1CC-4W6"
+		(property "Footprint" "My Footprints:CFPB-1CC-4W6_LOWPROF"
 			(at 44.45 199.39 0)
 			(hide yes)
@@
 			)
 		)
-		(property "LCSC" "manual"
+		(property "LCSC" "dnp"
 			(at 44.45 207.01 0)
 			(hide yes)
@@
 		(exclude_from_sim no)
 		(in_bom yes)
-		(on_board yes)
+		(on_board no)
 		(in_pos_files yes)
-		(dnp no)
+		(dnp yes)
 		(property "Reference" "R199"
 			(at 185.42 265.43 90)
@@
 		(exclude_from_sim no)
 		(in_bom yes)
-		(on_board yes)
+		(on_board no)
 		(in_pos_files yes)
-		(dnp no)
+		(dnp yes)
 		(fields_autoplaced yes)
 		(property "Reference" "D120"
@@
 			)
 		)
-		(property "LCSC" "manual"
+		(property "LCSC" "dnp"
 			(at 175.26 262.89 0)
 			(hide yes)
@@
 		(exclude_from_sim no)
 		(in_bom yes)
-		(on_board yes)
+		(on_board no)
 		(in_pos_files yes)
-		(dnp no)
+		(dnp yes)
 		(property "Reference" "R195"
 			(at 179.324 235.458 0)
@@
 		(exclude_from_sim no)
 		(in_bom yes)
-		(on_board yes)
+		(on_board no)
 		(in_pos_files yes)
-		(dnp no)
+		(dnp yes)
 		(fields_autoplaced yes)
 		(property "Reference" "SW121"
@@
 			)
 		)
-		(property "LCSC" "manual"
+		(property "LCSC" "dnp"
 			(at 107.95 245.11 0)
 			(hide yes)
@@
 			)
 		)
-		(property "Footprint" "My Footprints:CFPB-1CC-4W6"
+		(property "Footprint" "My Footprints:CFPB-1CC-4W6_LOWPROF"
 			(at 107.95 199.39 0)
 			(hide yes)
@@
 			)
 		)
-		(property "LCSC" "manual"
+		(property "LCSC" "dnp"
 			(at 107.95 207.01 0)
 			(hide yes)
@@
 		(exclude_from_sim no)
 		(in_bom yes)
-		(on_board yes)
+		(on_board no)
 		(in_pos_files yes)
-		(dnp no)
+		(dnp yes)
 		(property "Reference" "R196"
 			(at 125.476 252.222 90)

Commit message: ctrls board rev 0 done & sent to fab
Parts:
- R163, R164, R165, R173, R174, R175: value 330 -> 6.8k; LCSC C23138 -> C23212
- R166, R182, R183, R184, R191, R192, R193, R198, R199: value 330 -> 470; LCSC C23138 -> C25241
Changed lines of the file:
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@@
 			)
 		)
-		(property "Value" "330"
+		(property "Value" "6.8k"
 			(at 53.086 111.76 90)
 			(show_name no)
@@
 			)
 		)
-		(property "LCSC" "C23138"
+		(property "LCSC" "C23212"
 			(at 55.88 109.22 90)
 			(hide yes)
@@
 			)
 		)
-		(property "Value" "330"
+		(property "Value" "6.8k"
 			(at 116.586 111.76 90)
 			(show_name no)
@@
 			)
 		)
-		(property "LCSC" "C23138"
+		(property "LCSC" "C23212"
 			(at 119.38 109.22 90)
 			(hide yes)
@@
 			)
 		)
-		(property "Value" "330"
+		(property "Value" "6.8k"
 			(at 180.086 111.76 90)
 			(show_name no)
@@
 			)
 		)
-		(property "LCSC" "C23138"
+		(property "LCSC" "C23212"
 			(at 182.88 109.22 90)
 			(hide yes)
@@
 			)
 		)
-		(property "Value" "330"
+		(property "Value" "470"
 			(at 54.356 209.55 90)
 			(show_name no)
@@
 			)
 		)
-		(property "LCSC" "C23138"
+		(property "LCSC" "C25241"
 			(at 57.15 207.01 90)
 			(hide yes)
@@
 			)
 		)
-		(property "Value" "330"
+		(property "Value" "470"
 			(at 54.356 158.75 90)
 			(show_name no)
@@
 			)
 		)
-		(property "LCSC" "C23138"
+		(property "LCSC" "C25241"
 			(at 57.15 156.21 90)
 			(hide yes)
@@
 			)
 		)
-		(property "Value" "330"
+		(property "Value" "6.8k"
 			(at 119.126 50.8 90)
 			(show_name no)
@@
 			)
 		)
-		(property "LCSC" "C23138"
+		(property "LCSC" "C23212"
 			(at 121.92 48.26 90)
 			(hide yes)
@@
 			)
 		)
-		(property "Value" "330"
+		(property "Value" "470"
 			(at 181.356 158.75 90)
 			(show_name no)
@@
 			)
 		)
-		(property "LCSC" "C23138"
+		(property "LCSC" "C25241"
 			(at 184.15 156.21 90)
 			(hide yes)
@@
 			)
 		)
-		(property "Value" "330"
+		(property "Value" "6.8k"
 			(at 201.676 50.8 90)
 			(show_name no)
@@
 			)
 		)
-		(property "LCSC" "C23138"
+		(property "LCSC" "C23212"
 			(at 204.47 48.26 90)
 			(hide yes)
@@
 			)
 		)
-		(property "Value" "330"
+		(property "Value" "470"
 			(at 116.586 265.43 90)
 			(show_name no)
@@
 			)
 		)
-		(property "LCSC" "C23138"
+		(property "LCSC" "C25241"
 			(at 119.38 262.89 90)
 			(hide yes)
@@
 			)
 		)
-		(property "Value" "330"
+		(property "Value" "6.8k"
 			(at 161.036 50.8 90)
 			(show_name no)
@@
 			)
 		)
-		(property "LCSC" "C23138"
+		(property "LCSC" "C23212"
 			(at 163.83 48.26 90)
 			(hide yes)
@@
 			)
 		)
-		(property "Value" "330"
+		(property "Value" "470"
 			(at 181.356 209.55 90)
 			(show_name no)
@@
 			)
 		)
-		(property "LCSC" "C23138"
+		(property "LCSC" "C25241"
 			(at 184.15 207.01 90)
 			(hide yes)
@@
 			)
 		)
-		(property "Value" "330"
+		(property "Value" "470"
 			(at 117.856 209.55 90)
 			(show_name no)
@@
 			)
 		)
-		(property "LCSC" "C23138"
+		(property "LCSC" "C25241"
 			(at 120.65 207.01 90)
 			(hide yes)
@@
 			)
 		)
-		(property "Value" "330"
+		(property "Value" "470"
 			(at 180.086 265.43 90)
 			(show_name no)
@@
 			)
 		)
-		(property "LCSC" "C23138"
+		(property "LCSC" "C25241"
 			(at 182.88 262.89 90)
 			(hide yes)
@@
 			)
 		)
-		(property "Value" "330"
+		(property "Value" "470"
 			(at 54.356 55.88 90)
 			(show_name no)
@@
 			)
 		)
-		(property "LCSC" "C23138"
+		(property "LCSC" "C25241"
 			(at 57.15 53.34 90)
 			(hide yes)
@@
 			)
 		)
-		(property "Value" "330"
+		(property "Value" "470"
 			(at 117.856 158.75 90)
 			(show_name no)
@@
 			)
 		)
-		(property "LCSC" "C23138"
+		(property "LCSC" "C25241"
 			(at 120.65 156.21 90)
 			(hide yes)
