File: PCB_CAD/BUCKET_CONTROLS/btns2.kicad_sch (KiCad schematic)
At the start: 83 parts, among them SW11 C0_B0, SW12 C0_B1, SW13 C0_B2, SW14 C0_B3, SW15 C0_B4, SW16 C0_B5, SW17 C0_B6, SW18 C0_B7, SW19 C0_B8, SW20 C0_B9, SW21 C0_B10, SW22 C0_B11

Commit message: saving progress on controls pcb
Parts:
- removed C31, C32, C33, C34, C35, C36, C37, C38, C39, C40, C41, C42: 1u, Capacitor_SMD:C_0603_1608Metric, symbol Device:C
- removed D1, D11, D12, D13, D14, D15, D16, D17, D18, D5, D6, D7: 1N4148, Diode_SMD:D_SOD-323, symbol Device:D
- removed D10, D19, D2, D20, D3, D4, D8, D9: LED, LED_THT:LED_D3.0mm_FlatTop, symbol Device:LED
- removed R61, R67, R68, R69, R76, R77, R78, R85, R86, R87, R94, R95: 47k, Resistor_SMD:R_0603_1608Metric, symbol Device:R_US
- removed R62, R70, R71, R72, R79, R80, R81, R88, R89, R90, R96, R97: 15k, Resistor_SMD:R_0603_1608Metric, symbol Device:R_US
- removed R63, R64, R65, R66, R73, R74, R75, R82, R83, R84, R91, R92, R93, R98, R99: 330, Resistor_SMD:R_0603_1608Metric, symbol Device:R_US
- removed SW11: C0_B0, My Footprints:CFPB-1CC-4W6, symbol Switch:SW_Push_LED
- removed SW12: C0_B1, My Footprints:TL2201EEZB, symbol Switch:SW_Push_DPDT
- removed SW13: C0_B2, My Footprints:TL2201EEZB, symbol Switch:SW_Push_DPDT
- removed SW14: C0_B3, My Footprints:TL2201EEZB, symbol Switch:SW_Push_DPDT
- removed SW15: C0_B4, My Footprints:CFPB-1CC-4W6, symbol Switch:SW_Push_LED
- removed SW16: C0_B5, My Footprints:CFPB-1CC-4W6, symbol Switch:SW_Push_LED
- removed SW17: C0_B6, My Footprints:CFPB-1CC-4W6, symbol Switch:SW_Push_LED
- removed SW18: C0_B7, My Footprints:CFPB-1CC-4W6, symbol Switch:SW_Push_LED
- removed SW19: C0_B8, My Footprints:CFPB-1CC-4W6, symbol Switch:SW_Push_LED
- removed SW20: C0_B9, My Footprints:CFPB-1CC-4W6, symbol Switch:SW_Push_LED
- removed SW21: C0_B10, My Footprints:TL2201EEZB, symbol Switch:SW_Push_DPDT
- removed SW22: C0_B11, My Footprints:TL2201EEZB, symbol Switch:SW_Push_DPDT
- added C231, C232, C233, C234, C235, C236, C237, C238, C239, C240, C241, C242: 1u, Capacitor_SMD:C_0603_1608Metric, symbol Device:C
- added D201, D205, D206, D207, D211, D212, D213, D214, D215, D216, D217, D218: 1N4148, Diode_SMD:D_SOD-323, symbol Device:D
- added D202, D203, D204, D208, D209, D210, D219, D220: LED, LED_THT:LED_D3.0mm_FlatTop, symbol Device:LED
- added R261, R267, R268, R269, R276, R277, R278, R285, R286, R287, R294, R295: 47k, Resistor_SMD:R_0603_1608Metric, symbol Device:R_US
- added R262, R270, R271, R272, R279, R280, R281, R288, R289, R290, R296, R297: 15k, Resistor_SMD:R_0603_1608Metric, symbol Device:R_US
- added R263, R264, R265, R266, R273, R274, R275, R282, R283, R284, R291, R292, R293, R298, R299: 330, Resistor_SMD:R_0603_1608Metric, symbol Device:R_US
- added SW211: C2_B0, My Footprints:CFPB-1CC-4W6, symbol Switch:SW_Push_LED
- added SW212: C2_B1, My Footprints:TL2201EEZB, symbol Switch:SW_Push_DPDT
- added SW213: C2_B2, My Footprints:TL2201EEZB, symbol Switch:SW_Push_DPDT
- added SW214: C2_B3, My Footprints:TL2201EEZB, symbol Switch:SW_Push_DPDT
- added SW215: C2_B4, My Footprints:CFPB-1CC-4W6, symbol Switch:SW_Push_LED
- added SW216: C2_B5, My Footprints:CFPB-1CC-4W6, symbol Switch:SW_Push_LED
- added SW217: C2_B6, My Footprints:CFPB-1CC-4W6, symbol Switch:SW_Push_LED
- added SW218: C2_B7, My Footprints:CFPB-1CC-4W6, symbol Switch:SW_Push_LED
- added SW219: C2_B8, My Footprints:CFPB-1CC-4W6, symbol Switch:SW_Push_LED
- added SW220: C2_B9, My Footprints:CFPB-1CC-4W6, symbol Switch:SW_Push_LED
- added SW221: C2_B10, My Footprints:TL2201EEZB, symbol Switch:SW_Push_DPDT
- added SW222: C2_B11, My Footprints:TL2201EEZB, symbol Switch:SW_Push_DPDT
Connections:
- net +3V3: now also R261.1, R267.1, R268.1, R269.1, R276.1, R277.1, R278.1, R285.1, R286.1, R287.1, R294.1, R295.1
- net GND: now also C231.2, C232.2, C233.2, C234.2, C235.2, C236.2, C237.2, C238.2, C239.2, C240.2, C241.2, C242.2, D202.1 (K), D203.1 (K), D204.1 (K), D208.1 (K), D209.1 (K), D210.1 (K), D219.1 (K), D220.1 (K), SW211.1, SW211.4 (K), SW212.2 (B), SW213.2 (B), SW214.2 (B), SW215.1, SW215.4 (K), SW216.1, SW216.4 (K), SW217.1, SW217.4 (K), SW218.1, SW218.4 (K), SW219.1, SW219.4 (K), SW220.1, SW220.4 (K), SW221.2 (B), SW222.2 (B)
- new net: D207.2 (A), R269.2, R272.1, SW214.3 (C)
- new net: D217.2 (A), R294.2, R296.1, SW221.3 (C)
- new net: D212.2 (A), R277.2, R280.1, SW216.2
- new net: R283.1, SW216.3 (A)
- new net: D220.2 (A), R299.1
- new net: D208.2 (A), R273.1
- new net: D219.2 (A), R298.1
- new net: D203.2 (A), R264.1
- new net: D213.2 (A), R278.2, R281.1, SW217.2
- new net: D201.2 (A), R261.2, R262.1, SW211.2
- new net: D215.2 (A), R286.2, R289.1, SW219.2
- new net: D205.2 (A), R267.2, R270.1, SW212.3 (C)
- new net: D204.2 (A), R265.1
- new net: D202.2 (A), R263.1
- new net: D216.2 (A), R287.2, R290.1, SW220.2
- new net: R293.1, SW220.3 (A)
- new net: D214.2 (A), R285.2, R288.1, SW218.2
- new net: R291.1, SW218.3 (A)
- new net: D206.2 (A), R268.2, R271.1, SW213.3 (C)
- new net: D211.2 (A), R276.2, R279.1, SW215.2
- new net: R292.1, SW219.3 (A)
- new net: R284.1, SW217.3 (A)
- new net: R282.1, SW215.3 (A)
- new net: R266.1, SW211.3 (A)
- new net: D218.2 (A), R295.2, R297.1, SW222.3 (C)
- new net: D210.2 (A), R275.1
- new net: D209.2 (A), R274.1
- new net C2_B0: C231.1, D201.1 (K), R262.2
- new net C2_B0_L: R266.2
- new net C2_B0_LA: R263.2
- new net C2_B0_LB: R264.2
- new net C2_B0_LC: R265.2
- new net C2_B1: C232.1, D205.1 (K), R270.2
- new net C2_B10: C241.1, D217.1 (K), R296.2
- new net C2_B10_L: R298.2
- new net C2_B11: C242.1, D218.1 (K), R297.2
- new net C2_B11_L: R299.2
- new net C2_B1_L: R273.2
- new net C2_B2: C233.1, D206.1 (K), R271.2
- new net C2_B2_L: R274.2
- new net C2_B3: C234.1, D207.1 (K), R272.2
- new net C2_B3_L: R275.2
- new net C2_B4: C235.1, D211.1 (K), R279.2
- new net C2_B4_L: R282.2
- new net C2_B5: C236.1, D212.1 (K), R280.2
- new net C2_B5_L: R283.2
- new net C2_B6: C237.1, D213.1 (K), R281.2
- new net C2_B6_L: R284.2
- new net C2_B7: C238.1, D214.1 (K), R288.2
- new net C2_B7_L: R291.2
- new net C2_B8: C239.1, D215.1 (K), R289.2
- new net C2_B8_L: R292.2
- new net C2_B9: C240.1, D216.1 (K), R290.2
- new net C2_B9_L: R293.2

Commit message: pcb controls
Parts:
- C241, C242, D217, D218, R294, R295, R296, R297, R298, R299: now not fitted
- D202, D203, D204, D208, D209, D210, SW212, SW213, SW214: LCSC manual -> dnp
- D219, D220, SW221, SW222: LCSC manual -> dnp; now not fitted
- SW211, SW215, SW216, SW217, SW218, SW219, SW220: footprint My Footprints:CFPB-1CC-4W6 -> My Footprints:CFPB-1CC-4W6_LOWPROF; LCSC manual -> dnp
Changed lines of the file:
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@@
 		(exclude_from_sim no)
 		(in_bom yes)
-		(on_board yes)
+		(on_board no)
 		(in_pos_files yes)
-		(dnp no)
+		(dnp yes)
 		(property "Reference" "R294"
 			(at 115.824 235.458 0)
@@
 		(exclude_from_sim no)
 		(in_bom yes)
-		(on_board yes)
+		(on_board no)
 		(in_pos_files yes)
-		(dnp no)
+		(dnp yes)
 		(fields_autoplaced yes)
 		(property "Reference" "#PWR0446"
@@
 			)
 		)
-		(property "LCSC" "manual"
+		(property "LCSC" "dnp"
 			(at 171.45 91.44 0)
 			(hide yes)
@@
 			)
 		)
-		(property "Footprint" "My Footprints:CFPB-1CC-4W6"
+		(property "Footprint" "My Footprints:CFPB-1CC-4W6_LOWPROF"
 			(at 107.95 148.59 0)
 			(hide yes)
@@
 			)
 		)
-		(property "LCSC" "manual"
+		(property "LCSC" "dnp"
 			(at 107.95 156.21 0)
 			(hide yes)
@@
 		(exclude_from_sim no)
 		(in_bom yes)
-		(on_board yes)
+		(on_board no)
 		(in_pos_files yes)
-		(dnp no)
+		(dnp yes)
 		(property "Reference" "R299"
 			(at 185.42 265.43 90)
@@
 		(exclude_from_sim no)
 		(in_bom yes)
-		(on_board yes)
+		(on_board no)
 		(in_pos_files yes)
-		(dnp no)
+		(dnp yes)
 		(property "Reference" "R298"
 			(at 121.92 265.43 90)
@@
 			)
 		)
-		(property "LCSC" "manual"
+		(property "LCSC" "dnp"
 			(at 156.21 48.26 0)
 			(hide yes)
@@
 			)
 		)
-		(property "LCSC" "manual"
+		(property "LCSC" "dnp"
 			(at 44.45 91.44 0)
 			(hide yes)
@@
 		(exclude_from_sim no)
 		(in_bom yes)
-		(on_board yes)
+		(on_board no)
 		(in_pos_files yes)
-		(dnp no)
+		(dnp yes)
 		(property "Reference" "R296"
 			(at 125.476 252.222 90)
@@
 			)
 		)
-		(property "Footprint" "My Footprints:CFPB-1CC-4W6"
+		(property "Footprint" "My Footprints:CFPB-1CC-4W6_LOWPROF"
 			(at 44.45 199.39 0)
 			(hide yes)
@@
 			)
 		)
-		(property "LCSC" "manual"
+		(property "LCSC" "dnp"
 			(at 44.45 207.01 0)
 			(hide yes)
@@
 		(exclude_from_sim no)
 		(in_bom yes)
-		(on_board yes)
+		(on_board no)
 		(in_pos_files yes)
-		(dnp no)
+		(dnp yes)
 		(fields_autoplaced yes)
 		(property "Reference" "#PWR0452"
@@
 			)
 		)
-		(property "LCSC" "manual"
+		(property "LCSC" "dnp"
 			(at 196.85 48.26 0)
 			(hide yes)
@@
 			)
 		)
-		(property "LCSC" "manual"
+		(property "LCSC" "dnp"
 			(at 114.3 48.26 0)
 			(hide yes)
@@
 		(exclude_from_sim no)
 		(in_bom yes)
-		(on_board yes)
+		(on_board no)
 		(in_pos_files yes)
-		(dnp no)
+		(dnp yes)
 		(fields_autoplaced yes)
 		(property "Reference" "D220"
@@
 			)
 		)
-		(property "LCSC" "manual"
+		(property "LCSC" "dnp"
 			(at 175.26 262.89 0)
 			(hide yes)
@@
 		(exclude_from_sim no)
 		(in_bom yes)
-		(on_board yes)
+		(on_board no)
 		(in_pos_files yes)
-		(dnp no)
+		(dnp yes)
 		(fields_autoplaced yes)
 		(property "Reference" "#PWR0449"
@@
 			)
 		)
-		(property "LCSC" "manual"
+		(property "LCSC" "dnp"
 			(at 107.95 91.44 0)
 			(hide yes)
@@
 			)
 		)
-		(property "Footprint" "My Footprints:CFPB-1CC-4W6"
+		(property "Footprint" "My Footprints:CFPB-1CC-4W6_LOWPROF"
 			(at 44.45 148.59 0)
 			(hide yes)
@@
 			)
 		)
-		(property "LCSC" "manual"
+		(property "LCSC" "dnp"
 			(at 44.45 156.21 0)
 			(hide yes)
@@
 			)
 		)
-		(property "Footprint" "My Footprints:CFPB-1CC-4W6"
+		(property "Footprint" "My Footprints:CFPB-1CC-4W6_LOWPROF"
 			(at 107.95 199.39 0)
 			(hide yes)
@@
 			)
 		)
-		(property "LCSC" "manual"
+		(property "LCSC" "dnp"
 			(at 107.95 207.01 0)
 			(hide yes)
@@
 			)
 		)
-		(property "Footprint" "My Footprints:CFPB-1CC-4W6"
+		(property "Footprint" "My Footprints:CFPB-1CC-4W6_LOWPROF"
 			(at 44.45 45.72 0)
 			(hide yes)
@@
 			)
 		)
-		(property "LCSC" "manual"
+		(property "LCSC" "dnp"
 			(at 44.45 53.34 0)
 			(hide yes)
@@
 		(exclude_from_sim no)
 		(in_bom yes)
-		(on_board yes)
+		(on_board no)
 		(in_pos_files yes)
-		(dnp no)
+		(dnp yes)
 		(fields_autoplaced yes)
 		(property "Reference" "C241"
@@
 		(exclude_from_sim no)
 		(in_bom yes)
-		(on_board yes)
+		(on_board no)
 		(in_pos_files yes)
-		(dnp no)
+		(dnp yes)
 		(fields_autoplaced yes)
 		(property "Reference" "#PWR0450"
@@
 		(exclude_from_sim no)
 		(in_bom yes)
-		(on_board yes)
+		(on_board no)
 		(in_pos_files yes)
-		(dnp no)
+		(dnp yes)
 		(property "Reference" "R297"
 			(at 188.976 252.222 90)
@@
 		(exclude_from_sim no)
 		(in_bom yes)
-		(on_board yes)
+		(on_board no)
 		(in_pos_files yes)
-		(dnp no)
+		(dnp yes)
 		(fields_autoplaced yes)
 		(property "Reference" "#PWR0445"
@@
 		(exclude_from_sim no)
 		(in_bom yes)
-		(on_board yes)
+		(on_board no)
 		(in_pos_files yes)
-		(dnp no)
+		(dnp yes)
 		(property "Reference" "D217"
 			(at 128.016 237.236 0)
@@
 		(exclude_from_sim no)
 		(in_bom yes)
-		(on_board yes)
+		(on_board no)
 		(in_pos_files yes)
-		(dnp no)
+		(dnp yes)
 		(fields_autoplaced yes)
 		(property "Reference" "SW222"
@@
 			)
 		)
-		(property "LCSC" "manual"
+		(property "LCSC" "dnp"
 			(at 171.45 245.11 0)
 			(hide yes)
@@
 		(exclude_from_sim no)
 		(in_bom yes)
-		(on_board yes)
+		(on_board no)
 		(in_pos_files yes)
-		(dnp no)
+		(dnp yes)
 		(fields_autoplaced yes)
 		(property "Reference" "#PWR0451"
@@
 		(exclude_from_sim no)
 		(in_bom yes)
-		(on_board yes)
+		(on_board no)
 		(in_pos_files yes)
-		(dnp no)
+		(dnp yes)
 		(fields_autoplaced yes)
 		(property "Reference" "SW221"
@@
 			)
 		)
-		(property "LCSC" "manual"
+		(property "LCSC" "dnp"
 			(at 107.95 245.11 0)
 			(hide yes)
@@
 			)
 		)
-		(property "Footprint" "My Footprints:CFPB-1CC-4W6"
+		(property "Footprint" "My Footprints:CFPB-1CC-4W6_LOWPROF"
 			(at 171.45 199.39 0)
 			(hide yes)
@@
 			)
 		)
-		(property "LCSC" "manual"
+		(property "LCSC" "dnp"
 			(at 171.45 207.01 0)
 			(hide yes)
@@
 		(exclude_from_sim no)
 		(in_bom yes)
-		(on_board yes)
+		(on_board no)
 		(in_pos_files yes)
-		(dnp no)
+		(dnp yes)
 		(fields_autoplaced yes)
 		(property "Reference" "#PWR0447"
@@
 		(exclude_from_sim no)
 		(in_bom yes)
-		(on_board yes)
+		(on_board no)
 		(in_pos_files yes)
-		(dnp no)
+		(dnp yes)
 		(property "Reference" "R295"
 			(at 179.324 235.458 0)
@@
 		(exclude_from_sim no)
 		(in_bom yes)
-		(on_board yes)
+		(on_board no)
 		(in_pos_files yes)
-		(dnp no)
+		(dnp yes)
 		(fields_autoplaced yes)
 		(property "Reference" "D219"
@@
 			)
 		)
-		(property "LCSC" "manual"
+		(property "LCSC" "dnp"
 			(at 111.76 262.89 0)
 			(hide yes)
@@
 			)
 		)
-		(property "LCSC" "manual"
+		(property "LCSC" "dnp"
 			(at 111.76 109.22 0)
 			(hide yes)
@@
 		(exclude_from_sim no)
 		(in_bom yes)
-		(on_board yes)
+		(on_board no)
 		(in_pos_files yes)
-		(dnp no)
+		(dnp yes)
 		(fields_autoplaced yes)
 		(property "Reference" "#PWR0448"
@@
 		(exclude_from_sim no)
 		(in_bom yes)
-		(on_board yes)
+		(on_board no)
 		(in_pos_files yes)
-		(dnp no)
+		(dnp yes)
 		(fields_autoplaced yes)
 		(property "Reference" "C242"
@@
 			)
 		)
-		(property "Footprint" "My Footprints:CFPB-1CC-4W6"
+		(property "Footprint" "My Footprints:CFPB-1CC-4W6_LOWPROF"
 			(at 171.45 148.59 0)
 			(hide yes)
@@
 			)
 		)
-		(property "LCSC" "manual"
+		(property "LCSC" "dnp"
 			(at 171.45 156.21 0)
 			(hide yes)
@@
 			)
 		)
-		(property "LCSC" "manual"
+		(property "LCSC" "dnp"
 			(at 175.26 109.22 0)
 			(hide yes)
@@
 		(exclude_from_sim no)
 		(in_bom yes)
-		(on_board yes)
+		(on_board no)
 		(in_pos_files yes)
-		(dnp no)
+		(dnp yes)
 		(property "Reference" "D218"
 			(at 191.516 237.236 0)
@@
 			)
 		)
-		(property "LCSC" "manual"
+		(property "LCSC" "dnp"
 			(at 48.26 109.22 0)
 			(hide yes)

Commit message: ctrls board rev 0 done & sent to fab
Parts:
- R263, R264, R265, R273, R274, R275: value 330 -> 6.8k; LCSC C23138 -> C23212
- R266, R282, R283, R284, R291, R292, R293, R298, R299: value 330 -> 470; LCSC C23138 -> C25241
Changed lines of the file:
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@@
 			)
 		)
-		(property "Value" "330"
+		(property "Value" "470"
 			(at 180.086 265.43 90)
 			(show_name no)
@@
 			)
 		)
-		(property "LCSC" "C23138"
+		(property "LCSC" "C25241"
 			(at 182.88 262.89 90)
 			(hide yes)
@@
 			)
 		)
-		(property "Value" "330"
+		(property "Value" "6.8k"
 			(at 53.086 111.76 90)
 			(show_name no)
@@
 			)
 		)
-		(property "LCSC" "C23138"
+		(property "LCSC" "C23212"
 			(at 55.88 109.22 90)
 			(hide yes)
@@
 			)
 		)
-		(property "Value" "330"
+		(property "Value" "470"
 			(at 116.586 265.43 90)
 			(show_name no)
@@
 			)
 		)
-		(property "LCSC" "C23138"
+		(property "LCSC" "C25241"
 			(at 119.38 262.89 90)
 			(hide yes)
@@
 			)
 		)
-		(property "Value" "330"
+		(property "Value" "6.8k"
 			(at 201.676 50.8 90)
 			(show_name no)
@@
 			)
 		)
-		(property "LCSC" "C23138"
+		(property "LCSC" "C23212"
 			(at 204.47 48.26 90)
 			(hide yes)
@@
 			)
 		)
-		(property "Value" "330"
+		(property "Value" "6.8k"
 			(at 119.126 50.8 90)
 			(show_name no)
@@
 			)
 		)
-		(property "LCSC" "C23138"
+		(property "LCSC" "C23212"
 			(at 121.92 48.26 90)
 			(hide yes)
@@
 			)
 		)
-		(property "Value" "330"
+		(property "Value" "470"
 			(at 181.356 209.55 90)
 			(show_name no)
@@
 			)
 		)
-		(property "LCSC" "C23138"
+		(property "LCSC" "C25241"
 			(at 184.15 207.01 90)
 			(hide yes)
@@
 			)
 		)
-		(property "Value" "330"
+		(property "Value" "470"
 			(at 54.356 209.55 90)
 			(show_name no)
@@
 			)
 		)
-		(property "LCSC" "C23138"
+		(property "LCSC" "C25241"
 			(at 57.15 207.01 90)
 			(hide yes)
@@
 			)
 		)
-		(property "Value" "330"
+		(property "Value" "470"
 			(at 117.856 209.55 90)
 			(show_name no)
@@
 			)
 		)
-		(property "LCSC" "C23138"
+		(property "LCSC" "C25241"
 			(at 120.65 207.01 90)
 			(hide yes)
@@
 			)
 		)
-		(property "Value" "330"
+		(property "Value" "470"
 			(at 181.356 158.75 90)
 			(show_name no)
@@
 			)
 		)
-		(property "LCSC" "C23138"
+		(property "LCSC" "C25241"
 			(at 184.15 156.21 90)
 			(hide yes)
@@
 			)
 		)
-		(property "Value" "330"
+		(property "Value" "470"
 			(at 54.356 55.88 90)
 			(show_name no)
@@
 			)
 		)
-		(property "LCSC" "C23138"
+		(property "LCSC" "C25241"
 			(at 57.15 53.34 90)
 			(hide yes)
@@
 			)
 		)
-		(property "Value" "330"
+		(property "Value" "470"
 			(at 117.856 158.75 90)
 			(show_name no)
@@
 			)
 		)
-		(property "LCSC" "C23138"
+		(property "LCSC" "C25241"
 			(at 120.65 156.21 90)
 			(hide yes)
@@
 			)
 		)
-		(property "Value" "330"
+		(property "Value" "470"
 			(at 54.356 158.75 90)
 			(show_name no)
@@
 			)
 		)
-		(property "LCSC" "C23138"
+		(property "LCSC" "C25241"
 			(at 57.15 156.21 90)
 			(hide yes)
@@
 			)
 		)
-		(property "Value" "330"
+		(property "Value" "6.8k"
 			(at 161.036 50.8 90)
 			(show_name no)
@@
 			)
 		)
-		(property "LCSC" "C23138"
+		(property "LCSC" "C23212"
 			(at 163.83 48.26 90)
 			(hide yes)
@@
 			)
 		)
-		(property "Value" "330"
+		(property "Value" "6.8k"
 			(at 180.086 111.76 90)
 			(show_name no)
@@
 			)
 		)
-		(property "LCSC" "C23138"
+		(property "LCSC" "C23212"
 			(at 182.88 109.22 90)
 			(hide yes)
@@
 			)
 		)
-		(property "Value" "330"
+		(property "Value" "6.8k"
 			(at 116.586 111.76 90)
 			(show_name no)
@@
 			)
 		)
-		(property "LCSC" "C23138"
+		(property "LCSC" "C23212"
 			(at 119.38 109.22 90)
 			(hide yes)
