File: PCB_CAD/BUCKET_CONTROLS/btns3.kicad_sch (KiCad schematic)
At the start: 83 parts, among them SW11 C0_B0, SW12 C0_B1, SW13 C0_B2, SW14 C0_B3, SW15 C0_B4, SW16 C0_B5, SW17 C0_B6, SW18 C0_B7, SW19 C0_B8, SW20 C0_B9, SW21 C0_B10, SW22 C0_B11

Commit message: saving progress on controls pcb
Parts:
- removed C31, C32, C33, C34, C35, C36, C37, C38, C39, C40, C41, C42: 1u, Capacitor_SMD:C_0603_1608Metric, symbol Device:C
- removed D1, D11, D12, D13, D14, D15, D16, D17, D18, D5, D6, D7: 1N4148, Diode_SMD:D_SOD-323, symbol Device:D
- removed D10, D19, D2, D20, D3, D4, D8, D9: LED, LED_THT:LED_D3.0mm_FlatTop, symbol Device:LED
- removed R61, R67, R68, R69, R76, R77, R78, R85, R86, R87, R94, R95: 47k, Resistor_SMD:R_0603_1608Metric, symbol Device:R_US
- removed R62, R70, R71, R72, R79, R80, R81, R88, R89, R90, R96, R97: 15k, Resistor_SMD:R_0603_1608Metric, symbol Device:R_US
- removed R63, R64, R65, R66, R73, R74, R75, R82, R83, R84, R91, R92, R93, R98, R99: 330, Resistor_SMD:R_0603_1608Metric, symbol Device:R_US
- removed SW11: C0_B0, My Footprints:CFPB-1CC-4W6, symbol Switch:SW_Push_LED
- removed SW12: C0_B1, My Footprints:TL2201EEZB, symbol Switch:SW_Push_DPDT
- removed SW13: C0_B2, My Footprints:TL2201EEZB, symbol Switch:SW_Push_DPDT
- removed SW14: C0_B3, My Footprints:TL2201EEZB, symbol Switch:SW_Push_DPDT
- removed SW15: C0_B4, My Footprints:CFPB-1CC-4W6, symbol Switch:SW_Push_LED
- removed SW16: C0_B5, My Footprints:CFPB-1CC-4W6, symbol Switch:SW_Push_LED
- removed SW17: C0_B6, My Footprints:CFPB-1CC-4W6, symbol Switch:SW_Push_LED
- removed SW18: C0_B7, My Footprints:CFPB-1CC-4W6, symbol Switch:SW_Push_LED
- removed SW19: C0_B8, My Footprints:CFPB-1CC-4W6, symbol Switch:SW_Push_LED
- removed SW20: C0_B9, My Footprints:CFPB-1CC-4W6, symbol Switch:SW_Push_LED
- removed SW21: C0_B10, My Footprints:TL2201EEZB, symbol Switch:SW_Push_DPDT
- removed SW22: C0_B11, My Footprints:TL2201EEZB, symbol Switch:SW_Push_DPDT
- added C331, C332, C333, C334, C335, C336, C337, C338, C339, C340, C341, C342: 1u, Capacitor_SMD:C_0603_1608Metric, symbol Device:C
- added D301, D305, D306, D307, D311, D312, D313, D314, D315, D316, D317, D318: 1N4148, Diode_SMD:D_SOD-323, symbol Device:D
- added D302, D303, D304, D308, D309, D310, D319, D320: LED, LED_THT:LED_D3.0mm_FlatTop, symbol Device:LED
- added R361, R367, R368, R369, R376, R377, R378, R385, R386, R387, R394, R395: 47k, Resistor_SMD:R_0603_1608Metric, symbol Device:R_US
- added R362, R370, R371, R372, R379, R380, R381, R388, R389, R390, R396, R397: 15k, Resistor_SMD:R_0603_1608Metric, symbol Device:R_US
- added R363, R364, R365, R366, R373, R374, R375, R382, R383, R384, R391, R392, R393, R398, R399: 330, Resistor_SMD:R_0603_1608Metric, symbol Device:R_US
- added SW311: C3_B0, My Footprints:CFPB-1CC-4W6, symbol Switch:SW_Push_LED
- added SW312: C3_B1, My Footprints:TL2201EEZB, symbol Switch:SW_Push_DPDT
- added SW313: C3_B2, My Footprints:TL2201EEZB, symbol Switch:SW_Push_DPDT
- added SW314: C3_B3, My Footprints:TL2201EEZB, symbol Switch:SW_Push_DPDT
- added SW315: C3_B4, My Footprints:CFPB-1CC-4W6, symbol Switch:SW_Push_LED
- added SW316: C3_B5, My Footprints:CFPB-1CC-4W6, symbol Switch:SW_Push_LED
- added SW317: C3_B6, My Footprints:CFPB-1CC-4W6, symbol Switch:SW_Push_LED
- added SW318: C3_B7, My Footprints:CFPB-1CC-4W6, symbol Switch:SW_Push_LED
- added SW319: C3_B8, My Footprints:CFPB-1CC-4W6, symbol Switch:SW_Push_LED
- added SW320: C3_B9, My Footprints:CFPB-1CC-4W6, symbol Switch:SW_Push_LED
- added SW321: C3_B10, My Footprints:TL2201EEZB, symbol Switch:SW_Push_DPDT
- added SW322: C3_B11, My Footprints:TL2201EEZB, symbol Switch:SW_Push_DPDT
Connections:
- net +3V3: now also R361.1, R367.1, R368.1, R369.1, R376.1, R377.1, R378.1, R385.1, R386.1, R387.1, R394.1, R395.1
- net GND: now also C331.2, C332.2, C333.2, C334.2, C335.2, C336.2, C337.2, C338.2, C339.2, C340.2, C341.2, C342.2, D302.1 (K), D303.1 (K), D304.1 (K), D308.1 (K), D309.1 (K), D310.1 (K), D319.1 (K), D320.1 (K), SW311.1, SW311.4 (K), SW312.2 (B), SW313.2 (B), SW314.2 (B), SW315.1, SW315.4 (K), SW316.1, SW316.4 (K), SW317.1, SW317.4 (K), SW318.1, SW318.4 (K), SW319.1, SW319.4 (K), SW320.1, SW320.4 (K), SW321.2 (B), SW322.2 (B)
- new net: D314.2 (A), R385.2, R388.1, SW318.2
- new net: D315.2 (A), R386.2, R389.1, SW319.2
- new net: D307.2 (A), R369.2, R372.1, SW314.3 (C)
- new net: D320.2 (A), R399.1
- new net: D318.2 (A), R395.2, R397.1, SW322.3 (C)
- new net: D312.2 (A), R377.2, R380.1, SW316.2
- new net: R383.1, SW316.3 (A)
- new net: D317.2 (A), R394.2, R396.1, SW321.3 (C)
- new net: D304.2 (A), R365.1
- new net: R392.1, SW319.3 (A)
- new net: D311.2 (A), R376.2, R379.1, SW315.2
- new net: R393.1, SW320.3 (A)
- new net: D306.2 (A), R368.2, R371.1, SW313.3 (C)
- new net: D301.2 (A), R361.2, R362.1, SW311.2
- new net: R366.1, SW311.3 (A)
- new net: D316.2 (A), R387.2, R390.1, SW320.2
- new net: D309.2 (A), R374.1
- new net: D313.2 (A), R378.2, R381.1, SW317.2
- new net: R384.1, SW317.3 (A)
- new net: D308.2 (A), R373.1
- new net: D305.2 (A), R367.2, R370.1, SW312.3 (C)
- new net: R391.1, SW318.3 (A)
- new net: D310.2 (A), R375.1
- new net: D319.2 (A), R398.1
- new net: R382.1, SW315.3 (A)
- new net: D303.2 (A), R364.1
- new net: D302.2 (A), R363.1
- new net C3_B0: C331.1, D301.1 (K), R362.2
- new net C3_B0_L: R366.2
- new net C3_B0_LA: R363.2
- new net C3_B0_LB: R364.2
- new net C3_B0_LC: R365.2
- new net C3_B1: C332.1, D305.1 (K), R370.2
- new net C3_B10: C341.1, D317.1 (K), R396.2
- new net C3_B10_L: R398.2
- new net C3_B11: C342.1, D318.1 (K), R397.2
- new net C3_B11_L: R399.2
- new net C3_B1_L: R373.2
- new net C3_B2: C333.1, D306.1 (K), R371.2
- new net C3_B2_L: R374.2
- new net C3_B3: C334.1, D307.1 (K), R372.2
- new net C3_B3_L: R375.2
- new net C3_B4: C335.1, D311.1 (K), R379.2
- new net C3_B4_L: R382.2
- new net C3_B5: C336.1, D312.1 (K), R380.2
- new net C3_B5_L: R383.2
- new net C3_B6: C337.1, D313.1 (K), R381.2
- new net C3_B6_L: R384.2
- new net C3_B7: C338.1, D314.1 (K), R388.2
- new net C3_B7_L: R391.2
- new net C3_B8: C339.1, D315.1 (K), R389.2
- new net C3_B8_L: R392.2
- new net C3_B9: C340.1, D316.1 (K), R390.2
- new net C3_B9_L: R393.2

Commit message: pcb controls
Parts:
- C341, C342, D317, D318, R394, R395, R396, R397, R398, R399: now not fitted
- D302, D303, D304, D308, D309, D310, SW312, SW313, SW314: LCSC manual -> dnp
- D319, D320, SW321, SW322: LCSC manual -> dnp; now not fitted
- SW311, SW315, SW316, SW317, SW318, SW319, SW320: footprint My Footprints:CFPB-1CC-4W6 -> My Footprints:CFPB-1CC-4W6_LOWPROF; LCSC manual -> dnp
Changed lines of the file:
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@@
 		(exclude_from_sim no)
 		(in_bom yes)
-		(on_board yes)
+		(on_board no)
 		(in_pos_files yes)
-		(dnp no)
+		(dnp yes)
 		(fields_autoplaced yes)
 		(property "Reference" "D320"
@@
 			)
 		)
-		(property "LCSC" "manual"
+		(property "LCSC" "dnp"
 			(at 175.26 262.89 0)
 			(hide yes)
@@
 		(exclude_from_sim no)
 		(in_bom yes)
-		(on_board yes)
+		(on_board no)
 		(in_pos_files yes)
-		(dnp no)
+		(dnp yes)
 		(property "Reference" "D318"
 			(at 191.516 237.236 0)
@@
 		(exclude_from_sim no)
 		(in_bom yes)
-		(on_board yes)
+		(on_board no)
 		(in_pos_files yes)
-		(dnp no)
+		(dnp yes)
 		(fields_autoplaced yes)
 		(property "Reference" "#PWR0495"
@@
 		(exclude_from_sim no)
 		(in_bom yes)
-		(on_board yes)
+		(on_board no)
 		(in_pos_files yes)
-		(dnp no)
+		(dnp yes)
 		(property "Reference" "R399"
 			(at 185.42 265.43 90)
@@
 			)
 		)
-		(property "Footprint" "My Footprints:CFPB-1CC-4W6"
+		(property "Footprint" "My Footprints:CFPB-1CC-4W6_LOWPROF"
 			(at 107.95 148.59 0)
 			(hide yes)
@@
 			)
 		)
-		(property "LCSC" "manual"
+		(property "LCSC" "dnp"
 			(at 107.95 156.21 0)
 			(hide yes)
@@
 		(exclude_from_sim no)
 		(in_bom yes)
-		(on_board yes)
+		(on_board no)
 		(in_pos_files yes)
-		(dnp no)
+		(dnp yes)
 		(fields_autoplaced yes)
 		(property "Reference" "SW321"
@@
 			)
 		)
-		(property "LCSC" "manual"
+		(property "LCSC" "dnp"
 			(at 107.95 245.11 0)
 			(hide yes)
@@
 		(exclude_from_sim no)
 		(in_bom yes)
-		(on_board yes)
+		(on_board no)
 		(in_pos_files yes)
-		(dnp no)
+		(dnp yes)
 		(property "Reference" "R397"
 			(at 188.976 252.222 90)
@@
 			)
 		)
-		(property "Footprint" "My Footprints:CFPB-1CC-4W6"
+		(property "Footprint" "My Footprints:CFPB-1CC-4W6_LOWPROF"
 			(at 44.45 45.72 0)
 			(hide yes)
@@
 			)
 		)
-		(property "LCSC" "manual"
+		(property "LCSC" "dnp"
 			(at 44.45 53.34 0)
 			(hide yes)
@@
 			)
 		)
-		(property "Footprint" "My Footprints:CFPB-1CC-4W6"
+		(property "Footprint" "My Footprints:CFPB-1CC-4W6_LOWPROF"
 			(at 107.95 199.39 0)
 			(hide yes)
@@
 			)
 		)
-		(property "LCSC" "manual"
+		(property "LCSC" "dnp"
 			(at 107.95 207.01 0)
 			(hide yes)
@@
 			)
 		)
-		(property "Footprint" "My Footprints:CFPB-1CC-4W6"
+		(property "Footprint" "My Footprints:CFPB-1CC-4W6_LOWPROF"
 			(at 171.45 148.59 0)
 			(hide yes)
@@
 			)
 		)
-		(property "LCSC" "manual"
+		(property "LCSC" "dnp"
 			(at 171.45 156.21 0)
 			(hide yes)
@@
 		(exclude_from_sim no)
 		(in_bom yes)
-		(on_board yes)
+		(on_board no)
 		(in_pos_files yes)
-		(dnp no)
+		(dnp yes)
 		(property "Reference" "R396"
 			(at 125.476 252.222 90)
@@
 			)
 		)
-		(property "LCSC" "manual"
+		(property "LCSC" "dnp"
 			(at 48.26 109.22 0)
 			(hide yes)
@@
 		(exclude_from_sim no)
 		(in_bom yes)
-		(on_board yes)
+		(on_board no)
 		(in_pos_files yes)
-		(dnp no)
+		(dnp yes)
 		(fields_autoplaced yes)
 		(property "Reference" "C341"
@@
 		(exclude_from_sim no)
 		(in_bom yes)
-		(on_board yes)
+		(on_board no)
 		(in_pos_files yes)
-		(dnp no)
+		(dnp yes)
 		(property "Reference" "R395"
 			(at 179.324 235.458 0)
@@
 		(exclude_from_sim no)
 		(in_bom yes)
-		(on_board yes)
+		(on_board no)
 		(in_pos_files yes)
-		(dnp no)
+		(dnp yes)
 		(fields_autoplaced yes)
 		(property "Reference" "#PWR0494"
@@
 			)
 		)
-		(property "LCSC" "manual"
+		(property "LCSC" "dnp"
 			(at 107.95 91.44 0)
 			(hide yes)
@@
 		(exclude_from_sim no)
 		(in_bom yes)
-		(on_board yes)
+		(on_board no)
 		(in_pos_files yes)
-		(dnp no)
+		(dnp yes)
 		(fields_autoplaced yes)
 		(property "Reference" "#PWR0490"
@@
 			)
 		)
-		(property "Footprint" "My Footprints:CFPB-1CC-4W6"
+		(property "Footprint" "My Footprints:CFPB-1CC-4W6_LOWPROF"
 			(at 44.45 199.39 0)
 			(hide yes)
@@
 			)
 		)
-		(property "LCSC" "manual"
+		(property "LCSC" "dnp"
 			(at 44.45 207.01 0)
 			(hide yes)
@@
 		(exclude_from_sim no)
 		(in_bom yes)
-		(on_board yes)
+		(on_board no)
 		(in_pos_files yes)
-		(dnp no)
+		(dnp yes)
 		(fields_autoplaced yes)
 		(property "Reference" "SW322"
@@
 			)
 		)
-		(property "LCSC" "manual"
+		(property "LCSC" "dnp"
 			(at 171.45 245.11 0)
 			(hide yes)
@@
 			)
 		)
-		(property "LCSC" "manual"
+		(property "LCSC" "dnp"
 			(at 175.26 109.22 0)
 			(hide yes)
@@
 		(exclude_from_sim no)
 		(in_bom yes)
-		(on_board yes)
+		(on_board no)
 		(in_pos_files yes)
-		(dnp no)
+		(dnp yes)
 		(fields_autoplaced yes)
 		(property "Reference" "D319"
@@
 			)
 		)
-		(property "LCSC" "manual"
+		(property "LCSC" "dnp"
 			(at 111.76 262.89 0)
 			(hide yes)
@@
 			)
 		)
-		(property "Footprint" "My Footprints:CFPB-1CC-4W6"
+		(property "Footprint" "My Footprints:CFPB-1CC-4W6_LOWPROF"
 			(at 171.45 199.39 0)
 			(hide yes)
@@
 			)
 		)
-		(property "LCSC" "manual"
+		(property "LCSC" "dnp"
 			(at 171.45 207.01 0)
 			(hide yes)
@@
 			)
 		)
-		(property "LCSC" "manual"
+		(property "LCSC" "dnp"
 			(at 171.45 91.44 0)
 			(hide yes)
@@
 		(exclude_from_sim no)
 		(in_bom yes)
-		(on_board yes)
+		(on_board no)
 		(in_pos_files yes)
-		(dnp no)
+		(dnp yes)
 		(fields_autoplaced yes)
 		(property "Reference" "#PWR0493"
@@
 		(exclude_from_sim no)
 		(in_bom yes)
-		(on_board yes)
+		(on_board no)
 		(in_pos_files yes)
-		(dnp no)
+		(dnp yes)
 		(fields_autoplaced yes)
 		(property "Reference" "#PWR0496"
@@
 		(exclude_from_sim no)
 		(in_bom yes)
-		(on_board yes)
+		(on_board no)
 		(in_pos_files yes)
-		(dnp no)
+		(dnp yes)
 		(fields_autoplaced yes)
 		(property "Reference" "C342"
@@
 			)
 		)
-		(property "LCSC" "manual"
+		(property "LCSC" "dnp"
 			(at 156.21 48.26 0)
 			(hide yes)
@@
 		(exclude_from_sim no)
 		(in_bom yes)
-		(on_board yes)
+		(on_board no)
 		(in_pos_files yes)
-		(dnp no)
+		(dnp yes)
 		(property "Reference" "D317"
 			(at 128.016 237.236 0)
@@
 		(exclude_from_sim no)
 		(in_bom yes)
-		(on_board yes)
+		(on_board no)
 		(in_pos_files yes)
-		(dnp no)
+		(dnp yes)
 		(fields_autoplaced yes)
 		(property "Reference" "#PWR0491"
@@
 			)
 		)
-		(property "LCSC" "manual"
+		(property "LCSC" "dnp"
 			(at 114.3 48.26 0)
 			(hide yes)
@@
 			)
 		)
-		(property "Footprint" "My Footprints:CFPB-1CC-4W6"
+		(property "Footprint" "My Footprints:CFPB-1CC-4W6_LOWPROF"
 			(at 44.45 148.59 0)
 			(hide yes)
@@
 			)
 		)
-		(property "LCSC" "manual"
+		(property "LCSC" "dnp"
 			(at 44.45 156.21 0)
 			(hide yes)
@@
 		(exclude_from_sim no)
 		(in_bom yes)
-		(on_board yes)
+		(on_board no)
 		(in_pos_files yes)
-		(dnp no)
+		(dnp yes)
 		(fields_autoplaced yes)
 		(property "Reference" "#PWR0489"
@@
 		(exclude_from_sim no)
 		(in_bom yes)
-		(on_board yes)
+		(on_board no)
 		(in_pos_files yes)
-		(dnp no)
+		(dnp yes)
 		(property "Reference" "R398"
 			(at 121.92 265.43 90)
@@
 		(exclude_from_sim no)
 		(in_bom yes)
-		(on_board yes)
+		(on_board no)
 		(in_pos_files yes)
-		(dnp no)
+		(dnp yes)
 		(property "Reference" "R394"
 			(at 115.824 235.458 0)
@@
 		(exclude_from_sim no)
 		(in_bom yes)
-		(on_board yes)
+		(on_board no)
 		(in_pos_files yes)
-		(dnp no)
+		(dnp yes)
 		(fields_autoplaced yes)
 		(property "Reference" "#PWR0492"
@@
 			)
 		)
-		(property "LCSC" "manual"
+		(property "LCSC" "dnp"
 			(at 111.76 109.22 0)
 			(hide yes)
@@
 			)
 		)
-		(property "LCSC" "manual"
+		(property "LCSC" "dnp"
 			(at 196.85 48.26 0)
 			(hide yes)
@@
 			)
 		)
-		(property "LCSC" "manual"
+		(property "LCSC" "dnp"
 			(at 44.45 91.44 0)
 			(hide yes)

Commit message: ctrls board rev 0 done & sent to fab
Parts:
- R363, R364, R365, R373, R374, R375: value 330 -> 6.8k; LCSC C23138 -> C23212
- R366, R382, R383, R384, R391, R392, R393, R398, R399: value 330 -> 470; LCSC C23138 -> C25241
Changed lines of the file:
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@@
 			)
 		)
-		(property "Value" "330"
+		(property "Value" "470"
 			(at 180.086 265.43 90)
 			(show_name no)
@@
 			)
 		)
-		(property "LCSC" "C23138"
+		(property "LCSC" "C25241"
 			(at 182.88 262.89 90)
 			(hide yes)
@@
 			)
 		)
-		(property "Value" "330"
+		(property "Value" "6.8k"
 			(at 201.676 50.8 90)
 			(show_name no)
@@
 			)
 		)
-		(property "LCSC" "C23138"
+		(property "LCSC" "C23212"
 			(at 204.47 48.26 90)
 			(hide yes)
@@
 			)
 		)
-		(property "Value" "330"
+		(property "Value" "470"
 			(at 117.856 209.55 90)
 			(show_name no)
@@
 			)
 		)
-		(property "LCSC" "C23138"
+		(property "LCSC" "C25241"
 			(at 120.65 207.01 90)
 			(hide yes)
@@
 			)
 		)
-		(property "Value" "330"
+		(property "Value" "470"
 			(at 181.356 209.55 90)
 			(show_name no)
@@
 			)
 		)
-		(property "LCSC" "C23138"
+		(property "LCSC" "C25241"
 			(at 184.15 207.01 90)
 			(hide yes)
@@
 			)
 		)
-		(property "Value" "330"
+		(property "Value" "6.8k"
 			(at 116.586 111.76 90)
 			(show_name no)
@@
 			)
 		)
-		(property "LCSC" "C23138"
+		(property "LCSC" "C23212"
 			(at 119.38 109.22 90)
 			(hide yes)
@@
 			)
 		)
-		(property "Value" "330"
+		(property "Value" "470"
 			(at 54.356 55.88 90)
 			(show_name no)
@@
 			)
 		)
-		(property "LCSC" "C23138"
+		(property "LCSC" "C25241"
 			(at 57.15 53.34 90)
 			(hide yes)
@@
 			)
 		)
-		(property "Value" "330"
+		(property "Value" "470"
 			(at 54.356 158.75 90)
 			(show_name no)
@@
 			)
 		)
-		(property "LCSC" "C23138"
+		(property "LCSC" "C25241"
 			(at 57.15 156.21 90)
 			(hide yes)
@@
 			)
 		)
-		(property "Value" "330"
+		(property "Value" "6.8k"
 			(at 161.036 50.8 90)
 			(show_name no)
@@
 			)
 		)
-		(property "LCSC" "C23138"
+		(property "LCSC" "C23212"
 			(at 163.83 48.26 90)
 			(hide yes)
@@
 			)
 		)
-		(property "Value" "330"
+		(property "Value" "6.8k"
 			(at 53.086 111.76 90)
 			(show_name no)
@@
 			)
 		)
-		(property "LCSC" "C23138"
+		(property "LCSC" "C23212"
 			(at 55.88 109.22 90)
 			(hide yes)
@@
 			)
 		)
-		(property "Value" "330"
+		(property "Value" "470"
 			(at 54.356 209.55 90)
 			(show_name no)
@@
 			)
 		)
-		(property "LCSC" "C23138"
+		(property "LCSC" "C25241"
 			(at 57.15 207.01 90)
 			(hide yes)
@@
 			)
 		)
-		(property "Value" "330"
+		(property "Value" "6.8k"
 			(at 119.126 50.8 90)
 			(show_name no)
@@
 			)
 		)
-		(property "LCSC" "C23138"
+		(property "LCSC" "C23212"
 			(at 121.92 48.26 90)
 			(hide yes)
@@
 			)
 		)
-		(property "Value" "330"
+		(property "Value" "470"
 			(at 181.356 158.75 90)
 			(show_name no)
@@
 			)
 		)
-		(property "LCSC" "C23138"
+		(property "LCSC" "C25241"
 			(at 184.15 156.21 90)
 			(hide yes)
@@
 			)
 		)
-		(property "Value" "330"
+		(property "Value" "470"
 			(at 116.586 265.43 90)
 			(show_name no)
@@
 			)
 		)
-		(property "LCSC" "C23138"
+		(property "LCSC" "C25241"
 			(at 119.38 262.89 90)
 			(hide yes)
@@
 			)
 		)
-		(property "Value" "330"
+		(property "Value" "470"
 			(at 117.856 158.75 90)
 			(show_name no)
@@
 			)
 		)
-		(property "LCSC" "C23138"
+		(property "LCSC" "C25241"
 			(at 120.65 156.21 90)
 			(hide yes)
@@
 			)
 		)
-		(property "Value" "330"
+		(property "Value" "6.8k"
 			(at 180.086 111.76 90)
 			(show_name no)
@@
 			)
 		)
-		(property "LCSC" "C23138"
+		(property "LCSC" "C23212"
 			(at 182.88 109.22 90)
 			(hide yes)
