File: PCB_CAD/BUCKET_DAC/CV_DAC.kicad_pcb (KiCad board)
At the start: 4 copper layers, 108 x 77 mm, 222 parts, among them J1 Channel_0_CV_Out1, J10 I2C2, J11 I2C3, J12 I2C4, J13 POWER_IN, J14 LDAC, J2 Channel_0_CV_Out2, J3 Channel_1_CV_Out1, J4 Channel_1_CV_Out2, J5 Channel_2_CV_Out1, J6 Channel_2_CV_Out2, J7 Channel_3_CV_Out1, J8 Channel_3_CV_Out2, J9 I2C1, U1 MCP4728, U10 MCP4728, U11 MCP4728, U12 MCP4728, U13 MCP4728, U14 MCP4728, U15 MCP4728, U16 MCP4728, U17 MCP4728, U18 MCP4728, U19 MCP4728, U2 MCP4728, U20 MCP4728, U3 MCP4728, U4 MCP4728, U5 MCP4728, U6 MCP4728, U7 MCP4728, U8 MCP4728, U9 MCP4728

Commit message: analog design ugh
Parts:
- added R81: 4.7k, Resistor_THT:R_Axial_DIN0207_L6.3mm_D2.5mm_P2.54mm_Vertical, F.Cu at (144.5, 95.2)
- added R82: 4.7k, Resistor_THT:R_Axial_DIN0207_L6.3mm_D2.5mm_P2.54mm_Vertical, F.Cu at (148.1, 95.2)
- added R83: 4.7k, Resistor_THT:R_Axial_DIN0207_L6.3mm_D2.5mm_P2.54mm_Vertical, F.Cu at (156.0, 96.5)
- added R84: 4.7k, Resistor_THT:R_Axial_DIN0207_L6.3mm_D2.5mm_P2.54mm_Vertical, F.Cu at (175.6, 85.7)
- added R85: 4.7k, Resistor_THT:R_Axial_DIN0207_L6.3mm_D2.5mm_P2.54mm_Vertical, F.Cu at (165.0, 88.8)
- added REF**: LayerMarker_4_6.35x2.54mm_TextH1mm_P1.27mm_BottomMirrored, Symbol:LayerMarker_4_6.35x2.54mm_TextH1mm_P1.27mm_BottomMirrored, F.Cu at (190.4, 124.4)
Routing:
- net LDAC2_CHAN0: track 118.9 -> 125.6 mm
- net LDAC0_CHAN0: track 140.8 -> 146.2 mm
- net LDAC1_CHAN0: track 128.2 -> 133.1 mm
- net LDAC3_CHAN0: track 117.0 -> 121.7 mm
- net LDAC4_CHAN0: track 139.8 -> 144.1 mm
- net GND: vias 355 -> 351
Other:
- board text added: "CV DAC BOARD"
- board text added: "DIGILOG"
- board text added: "REV 0"
