File: PCB_CAD/BUCKET_DAC/CV_DAC.kicad_sch (KiCad schematic)
At the start: 14 parts, among them J10 I2C2, J11 I2C3, J12 I2C4, J13 POWER_IN, J14 LDAC, J9 I2C1

Commit message: analog design ugh
Parts:
- added R81, R82, R83, R84, R85: 4.7k, Resistor_THT:R_Axial_DIN0207_L6.3mm_D2.5mm_P2.54mm_Vertical, symbol Device:R_Small_US
Connections:
- net GND: now also R81.2, R82.2, R83.2, R84.2, R85.2
- net LDAC0_CHAN0: now also R81.1
- net LDAC1_CHAN0: now also R82.1
- net LDAC2_CHAN0: now also R83.1
- net LDAC3_CHAN0: now also R84.1
- net LDAC4_CHAN0: now also R85.1
