File: PCB_CAD/Analog/EQ/EQ.kicad_sch (KiCad schematic)
At the start: 4 parts, among them U1 OPA4197, U2 SSM2164, U4 ADG1436, U5 OPA1679

Commit message: analog design ugh
Parts:
- removed U1: OPA4197, Package_SO:SOIC-14_3.9x8.7mm_P1.27mm, symbol Amplifier_Operational:OPA4197xD
- removed U2: SSM2164, 4ms_Package_SOIC:SOIC-16_3.9x9.9mm_Pitch1.27mm, symbol PCM_4ms_IC:SSM2164
- removed U4: ADG1436, ADG1436:TSSOP16, symbol My Symbols:ADG1436
- removed U5: OPA1679, symbol Amplifier_Operational:OPA1679
Other:
- added sheet LMF (lmf.kicad_sch)

Commit message: cad, pcb, designing the eq circuits yay, writing and documenting analog design, started the report aaaahhh i finna end it all jk
Other:
- added sheet HF (hf.kicad_sch)
- added sheet HMF (hmf.kicad_sch)
- added sheet LF (lf.kicad_sch)
Changed lines of the file:
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@@
 		(rev "0")
 		(company "EECE CAPSTONE")
+		(comment 2 "control voltage scaler/buffers. Includes temp. compensation")
 		(comment 3 "S.E.D.")
 	)
 	(sheet
-		(at 48.26 39.37)
-		(size 86.36 95.25)
+		(at 161.29 36.83)
+		(size 46.99 39.37)
 		(exclude_from_sim no)
 		(in_bom yes)
@@
 			(color 0 0 0 0)
 		)
-		(property "Sheetname" "LMF"
-			(at 52.324 48.514 0)
+		(property "Sheetname" "HF"
+			(at 165.608 46.736 0)
 			(show_name no)
 			(do_not_autoplace no)
@@
 			)
 		)
-		(property "Sheetfile" "lmf.kicad_sch"
-			(at 48.26 135.2046 0)
+		(property "Sheetfile" "hf.kicad_sch"
+			(at 161.29 76.7846 0)
 			(show_name no)
 			(do_not_autoplace no)
@@
 				)
 			)
+		)
+	)
+	(sheet
+		(at 160.02 143.51)
+		(size 52.07 45.72)
+		(exclude_from_sim no)
+		(in_bom yes)
+		(on_board yes)
+		(dnp no)
+		(stroke
+			(width 0.1524)
+			(type solid)
+		)
+		(fill
+			(color 0 0 0 0)
+		)
+		(property "Sheetname" "LMF"
+			(at 164.084 152.654 0)
+			(show_name no)
+			(do_not_autoplace no)
+			(effects
+				(font
+					(size 3.81 3.81)
+					(thickness 0.762)
+					(bold yes)
+				)
+				(justify left bottom)
+			)
+		)
+		(property "Sheetfile" "lmf.kicad_sch"
+			(at 174.752 180.34 0)
+			(show_name no)
+			(do_not_autoplace no)
+			(effects
+				(font
+					(size 1.27 1.27)
+				)
+				(justify left top)
+			)
+		)
+		(instances
+			(project "EQ"
+				(path "/a379ffa5-dfb1-4f56-af77-387c7dfe3dba"
+					(page "4")
+				)
+			)
+		)
+	)
+	(sheet
+		(at 158.75 86.36)
+		(size 53.34 50.8)
+		(exclude_from_sim no)
+		(in_bom yes)
+		(on_board yes)
+		(dnp no)
+		(stroke
+			(width 0.1524)
+			(type solid)
+		)
+		(fill
+			(color 0 0 0 0)
+		)
+		(property "Sheetname" "HMF"
+			(at 161.036 94.488 0)
+			(show_name no)
+			(do_not_autoplace no)
+			(effects
+				(font
+					(size 3.81 3.81)
+					(thickness 0.762)
+					(bold yes)
+				)
+				(justify left bottom)
+			)
+		)
+		(property "Sheetfile" "hmf.kicad_sch"
+			(at 170.18 127.254 0)
+			(show_name no)
+			(do_not_autoplace no)
+			(effects
+				(font
+					(size 1.27 1.27)
+				)
+				(justify left top)
+			)
+		)
+		(instances
+			(project "EQ"
+				(path "/a379ffa5-dfb1-4f56-af77-387c7dfe3dba"
+					(page "3")
+				)
+			)
+		)
+	)
+	(sheet
+		(at 163.83 205.74)
+		(size 46.99 45.72)
+		(exclude_from_sim no)
+		(in_bom yes)
+		(on_board yes)
+		(dnp no)
+		(stroke
+			(width 0.1524)
+			(type solid)
+		)
+		(fill
+			(color 0 0 0 0)
+		)
+		(property "Sheetname" "LF"
+			(at 165.354 215.392 0)
+			(show_name no)
+			(do_not_autoplace no)
+			(effects
+				(font
+					(size 3.81 3.81)
+					(thickness 0.762)
+					(bold yes)
+				)
+				(justify left bottom)
+			)
+		)
+		(property "Sheetfile" "lf.kicad_sch"
+			(at 163.83 252.0446 0)
+			(show_name no)
+			(do_not_autoplace no)
+			(effects
+				(font
+					(size 1.27 1.27)
+				)
+				(justify left top)
+			)
+		)
+		(instances
+			(project "EQ"
+				(path "/a379ffa5-dfb1-4f56-af77-387c7dfe3dba"
+					(page "5")
+				)
+			)

Commit message: first version of eq circuit finished phew
Other:
- removed sheet HF
- removed sheet LF
- added sheet LF_HF (lf_hf.kicad_sch)
Changed lines of the file:
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@@
-	)
-	(sheet
-		(at 161.29 36.83)
-		(size 46.99 39.37)
-		(exclude_from_sim no)
-		(in_bom yes)
-		(on_board yes)
-		(dnp no)
-		(stroke
-			(width 0.1524)
-			(type solid)
-		)
-		(fill
-			(color 0 0 0 0)
-		)
-		(property "Sheetname" "HF"
-			(at 165.608 46.736 0)
-			(show_name no)
-			(do_not_autoplace no)
-			(effects
-				(font
-					(size 3.81 3.81)
-					(thickness 0.762)
-					(bold yes)
-				)
-				(justify left bottom)
-			)
-		)
-		(property "Sheetfile" "hf.kicad_sch"
-			(at 161.29 76.7846 0)
-			(show_name no)
-			(do_not_autoplace no)
-			(effects
-				(font
-					(size 1.27 1.27)
-				)
-				(justify left top)
-			)
-		)
-		(instances
-			(project "EQ"
-				(path "/a379ffa5-dfb1-4f56-af77-387c7dfe3dba"
-					(page "2")
-				)
-			)
-		)
 	)
 	(sheet
@@
 	)
 	(sheet
-		(at 163.83 205.74)
-		(size 46.99 45.72)
+		(at 156.21 20.32)
+		(size 83.82 57.15)
 		(exclude_from_sim no)
 		(in_bom yes)
@@
 			(color 0 0 0 0)
 		)
-		(property "Sheetname" "LF"
-			(at 165.354 215.392 0)
+		(property "Sheetname" "LF_HF"
+			(at 162.56 32.258 0)
 			(show_name no)
 			(do_not_autoplace no)
@@
 			)
 		)
-		(property "Sheetfile" "lf.kicad_sch"
-			(at 163.83 252.0446 0)
+		(property "Sheetfile" "lf_hf.kicad_sch"
+			(at 156.21 78.0546 0)
 			(show_name no)
 			(do_not_autoplace no)
@@
 			(project "EQ"
 				(path "/a379ffa5-dfb1-4f56-af77-387c7dfe3dba"
-					(page "5")
+					(page "2")
 				)
 			)
