File: PCB_CAD/Analog/EQ/hmf.kicad_sch (KiCad schematic)
At the start: 66 parts, among them U10 OPA1679, U11 OPA4197, U6 OPA1678, U8 SSI2164, U9 AS2180

Commit message: first version of eq circuit finished phew
Parts:
- removed U6: OPA1678, Package_SO:SOIC-8_3.9x4.9mm_P1.27mm, symbol Amplifier_Operational:OPA2197xD
- added R140: 22k, Resistor_SMD:R_0603_1608Metric, symbol Device:R_US
- added U14: OPA1679, Package_SO:SOIC-14_3.9x8.7mm_P1.27mm, symbol Amplifier_Operational:OPA1679
- U10: footprint (none) -> Package_SO:SOIC-14_3.9x8.7mm_P1.27mm
Connections:
- net +15V: now also R140.1
- net GND: now also U14.5 (+)
- net HMF_OUT: now also U14.7
- net at C109.1, R116.1, R139.1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: now also U14.6 (-)
- net at U8.1: now also R140.2
- no-connect marks 2 -> 1
