File: PCB_CAD/Analog/EQ/lmf.kicad_sch (KiCad schematic)
At the start: 76 parts, among them U1 OPA4197, U2 SSI2164, U3 AS2180, U4 ADG1436, U5 OPA1679, U6 OPA1678, U7 ADR5041

Commit message: cad, pcb, designing the eq circuits yay, writing and documenting analog design, started the report aaaahhh i finna end it all jk
Parts:
- removed unit 2 of U6
- added R40: 2.2k, Resistor_SMD:R_0603_1608Metric, symbol Device:R_US
- added R41: 120k, Resistor_SMD:R_0603_1608Metric, symbol Device:R_US
- R21, R27: value 97.6k -> 140k
- R22, R28: value 124k -> 88.7k
- R24, R25: value 47.5k -> 34.0k
- R30, R31: value 42.2k -> 30.1k
- R33: value 90.9k -> 130k
- R34: value 133k -> 95.3k
- R36, R37: value 30.9k -> 22.1k
Connections:
- net REF_N2V5 is gone; now on net -2V5: U1.13 (-), U1.14
- net GND: now also R41.2; no longer U4.9 (IN2)
- net HMF_OUT: now reaches U4.10 (S2A)
- net HMF_V: now reaches U4.11 (D2)
- net HMF_IN: now reaches U4.12 (S2B)
- new net: R40.1, R41.1, U4.9 (IN2)
- new net HMF_CUT_LCV: R40.2
- no-connect marks 5 -> 2
Other:
- title: Channel EQ Circuit: LMF -> Channel EQ Circuit

Commit message: first version of eq circuit finished phew
Parts:
- removed U6: OPA1678, Package_SO:SOIC-8_3.9x4.9mm_P1.27mm, symbol Amplifier_Operational:OPA2197xD
- added R42: 22k, Resistor_SMD:R_0603_1608Metric, symbol Device:R_US
- added U6: OPA1679, Package_SO:SOIC-14_3.9x8.7mm_P1.27mm, symbol Amplifier_Operational:OPA1679
- U5: footprint (none) -> Package_SO:SOIC-14_3.9x8.7mm_P1.27mm
Connections:
- net +15V: now also R42.1, U6.4 (V+)
- net -15V: now also U6.11 (V-)
- net GND: now also U6.3 (+)
- net LMF_OUT: now also U6.1
- net at U2.1: now also R42.2
- net at C9.1, R16.1, R39.1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: now also U6.2 (-)
- no-connect marks 2 -> 1
