File: PCB_CAD/BUCKET_FADER/buttons.kicad_sch (KiCad schematic)
At the start: 56 parts, among them SW1 C0_B10, SW2 C0_B11, SW3 C0_B10, SW4 C0_B11, SW5 C0_B10, SW6 C0_B11, SW7 C0_B10, SW8 C0_B11

Commit message: fader board design done
Parts:
- R10, R11, R12, R21, R22, R23, R24, R9: LCSC C25819 -> C25600
- R17, R18, R19, R20, R29, R30, R31, R32: LCSC C25241 -> C23212
Changed lines of the file:
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@@
 			)
 		)
-		(property "LCSC" "C25241"
+		(property "LCSC" "C23212"
 			(at 176.53 137.16 90)
 			(hide yes)
@@
 			)
 		)
-		(property "LCSC" "C25819"
+		(property "LCSC" "C25600"
 			(at 186.69 46.99 0)
 			(hide yes)
@@
 			)
 		)
-		(property "LCSC" "C25241"
+		(property "LCSC" "C23212"
 			(at 176.53 72.39 90)
 			(hide yes)
@@
 			)
 		)
-		(property "LCSC" "C25819"
+		(property "LCSC" "C25600"
 			(at 250.19 46.99 0)
 			(hide yes)
@@
 			)
 		)
-		(property "LCSC" "C25241"
+		(property "LCSC" "C23212"
 			(at 240.03 72.39 90)
 			(hide yes)
@@
 			)
 		)
-		(property "LCSC" "C25819"
+		(property "LCSC" "C25600"
 			(at 250.19 111.76 0)
 			(hide yes)
@@
 			)
 		)
-		(property "LCSC" "C25241"
+		(property "LCSC" "C23212"
 			(at 240.03 137.16 90)
 			(hide yes)
@@
 			)
 		)
-		(property "LCSC" "C25241"
+		(property "LCSC" "C23212"
 			(at 101.6 72.39 90)
 			(hide yes)
@@
 			)
 		)
-		(property "LCSC" "C25241"
+		(property "LCSC" "C23212"
 			(at 38.1 72.39 90)
 			(hide yes)
@@
 			)
 		)
-		(property "LCSC" "C25819"
+		(property "LCSC" "C25600"
 			(at 111.76 111.76 0)
 			(hide yes)
@@
 			)
 		)
-		(property "LCSC" "C25819"
+		(property "LCSC" "C25600"
 			(at 48.26 111.76 0)
 			(hide yes)
@@
 			)
 		)
-		(property "LCSC" "C25819"
+		(property "LCSC" "C25600"
 			(at 111.76 46.99 0)
 			(hide yes)
@@
 			)
 		)
-		(property "LCSC" "C25241"
+		(property "LCSC" "C23212"
 			(at 38.1 137.16 90)
 			(hide yes)
@@
 			)
 		)
-		(property "LCSC" "C25241"
+		(property "LCSC" "C23212"
 			(at 101.6 137.16 90)
 			(hide yes)
@@
 			)
 		)
-		(property "LCSC" "C25819"
+		(property "LCSC" "C25600"
 			(at 186.69 111.76 0)
 			(hide yes)
@@
 			)
 		)
-		(property "LCSC" "C25819"
+		(property "LCSC" "C25600"
 			(at 48.26 46.99 0)
 			(hide yes)
