File: PCB_CAD/Bucket/Analog/PAN_FADER/PAN_FADER.kicad_sch (KiCad schematic)
At the start: 99 parts, among them J1 COMP_CV, J2 CV_FROM_DAC, J3 POWER, J4 AUD_OUT, J5 TO_INSERT_MATRIX, J6 AUD_IN, U1 THAT2180A, U2 OPA1679, U3 OPA1637, U5 THAT2180A, U6 OPA2197xD, U7 OPA1637, U8 ADR5041, U9 ADG1436

Commit message: getting ready to upgrade mx file
Other:
- moved on the sheet: H1, H2, H3
Changed lines of the file:
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@@
 	(symbol
 		(lib_id "Auxiliary_Items:MountingScrew")
-		(at 53.34 233.68 0)
+		(at 50.8 238.76 0)
 		(unit 1)
 		(body_style 1)
@@
 		(fields_autoplaced yes)
 		(property "Reference" "H1"
-			(at 55.88 233.0449 0)
+			(at 53.34 238.1249 0)
 			(show_name no)
 			(do_not_autoplace no)
@@
 		)
 		(property "Value" "MountingHole_Pad"
-			(at 55.88 233.6799 0)
+			(at 53.34 238.7599 0)
 			(hide yes)
 			(show_name no)
@@
 		)
 		(property "Footprint" "MountingHole:MountingHole_2.2mm_M2"
-			(at 53.34 233.68 0)
+			(at 50.8 238.76 0)
 			(hide yes)
 			(show_name no)
@@
 		)
 		(property "Datasheet" ""
-			(at 53.34 233.68 0)
+			(at 50.8 238.76 0)
 			(hide yes)
 			(show_name no)
@@
 		)
 		(property "Description" "Mounting screw"
-			(at 53.34 233.68 0)
+			(at 50.8 238.76 0)
 			(hide yes)
 			(show_name no)
@@
 	(symbol
 		(lib_id "Auxiliary_Items:MountingScrew")
-		(at 53.34 219.71 0)
+		(at 50.8 224.79 0)
 		(unit 1)
 		(body_style 1)
@@
 		(fields_autoplaced yes)
 		(property "Reference" "H2"
-			(at 55.88 219.0749 0)
+			(at 53.34 224.1549 0)
 			(show_name no)
 			(do_not_autoplace no)
@@
 		)
 		(property "Value" "MountingHole_Pad"
-			(at 55.88 219.7099 0)
+			(at 53.34 224.7899 0)
 			(hide yes)
 			(show_name no)
@@
 		)
 		(property "Footprint" "MountingHole:MountingHole_2.2mm_M2"
-			(at 53.34 219.71 0)
+			(at 50.8 224.79 0)
 			(hide yes)
 			(show_name no)
@@
 		)
 		(property "Datasheet" ""
-			(at 53.34 219.71 0)
+			(at 50.8 224.79 0)
 			(hide yes)
 			(show_name no)
@@
 		)
 		(property "Description" "Mounting screw"
-			(at 53.34 219.71 0)
+			(at 50.8 224.79 0)
 			(hide yes)
 			(show_name no)
@@
 	(symbol
 		(lib_id "Auxiliary_Items:MountingScrew")
-		(at 45.72 227.33 0)
+		(at 43.18 232.41 0)
 		(unit 1)
 		(body_style 1)
@@
 		(fields_autoplaced yes)
 		(property "Reference" "H3"
-			(at 48.26 226.6949 0)
+			(at 45.72 231.7749 0)
 			(show_name no)
 			(do_not_autoplace no)
@@
 		)
 		(property "Value" "MountingHole_Pad"
-			(at 48.26 227.3299 0)
+			(at 45.72 232.4099 0)
 			(hide yes)
 			(show_name no)
@@
 		)
 		(property "Footprint" "MountingHole:MountingHole_2.2mm_M2"
-			(at 45.72 227.33 0)
+			(at 43.18 232.41 0)
 			(hide yes)
 			(show_name no)
@@
 		)
 		(property "Datasheet" ""
-			(at 45.72 227.33 0)
+			(at 43.18 232.41 0)
 			(hide yes)
 			(show_name no)
@@
 		)
 		(property "Description" "Mounting screw"
-			(at 45.72 227.33 0)
-			(hide yes)
-			(show_name no)
+			(at 43.18 232.41 0)
+			(hide yes)
+			(show_name no)
