File: PCB_CAD/Bucket/BUCKET_FADER/BUCKET_FADER.kicad_pcb (KiCad board)
At the start: 4 copper layers, 146 x 103 mm, 123 parts, among them J1 POW, J2 F0_MCU, J3 F1_MCU, J4 F0_BTN, J5 F1_BTN, J6 F2_BTN, J7 F3_BTN, J8 F2_MCU, J9 F3_MCU, SW1 C0_B10, SW2 C0_B11, SW3 C0_B10, SW4 C0_B11, SW5 C0_B10, SW6 C0_B11, SW7 C0_B10, SW8 C0_B11, U1 AT42QT1011-M, U2 AT42QT1011-M, U3 AT42QT1011-M, U4 AT42QT1011-M, U5 DRV8871DDA, U6 DRV8871DDA, U7 DRV8871DDA, U8 DRV8871DDA

Commit message: pcb
Other:
- board text added: "3v3 F_Pos GND F_Touch F_MA F_MB"
- board text added: "BUCKET FADER BOARD"
