File: PCB_CAD/Bucket/BUCKET_FADER/BUCKET_FADER.kicad_sch (KiCad schematic)
At the start: 67 parts, among them J1 POW, J2 F0_MCU, J3 F1_MCU, J4 F0_BTN, J5 F1_BTN, J6 F2_BTN, J7 F3_BTN, J8 F2_MCU, J9 F3_MCU, U1 AT42QT1011-M, U2 AT42QT1011-M, U3 AT42QT1011-M, U4 AT42QT1011-M, U5 DRV8871DDA, U6 DRV8871DDA, U7 DRV8871DDA, U8 DRV8871DDA

Commit message: pcb
Parts:
- H1, H2, H3, H4, H5, H6, H7, H8: LCSC (none) -> dnp
- U1, U2, U3, U4: LCSC (none) -> C2652045
- U5, U6, U7, U8: LCSC (none) -> C75864
Changed lines of the file:
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@@
 			)
 		)
+		(property "LCSC" "dnp"
+			(at 330.2 190.5 0)
+			(hide yes)
+			(show_name no)
+			(do_not_autoplace no)
+			(effects
+				(font
+					(size 1.27 1.27)
+				)
+			)
+		)
 		(instances
 			(project "BUCKET_FADER"
@@
 			)
 		)
+		(property "LCSC" "dnp"
+			(at 345.44 201.93 0)
+			(hide yes)
+			(show_name no)
+			(do_not_autoplace no)
+			(effects
+				(font
+					(size 1.27 1.27)
+				)
+			)
+		)
 		(instances
 			(project "BUCKET_FADER"
@@
 			)
 		)
+		(property "LCSC" "C2652045"
+			(at 158.75 102.87 0)
+			(hide yes)
+			(show_name no)
+			(do_not_autoplace no)
+			(effects
+				(font
+					(size 1.27 1.27)
+				)
+			)
+		)
 		(pin "2"
 		)
@@
 			)
 		)
+		(property "LCSC" "C75864"
+			(at 93.98 149.86 0)
+			(hide yes)
+			(show_name no)
+			(do_not_autoplace no)
+			(effects
+				(font
+					(size 1.27 1.27)
+				)
+			)
+		)
 		(pin "1"
 		)
@@
 			)
 		)
+		(property "LCSC" "dnp"
+			(at 335.28 190.5 0)
+			(hide yes)
+			(show_name no)
+			(do_not_autoplace no)
+			(effects
+				(font
+					(size 1.27 1.27)
+				)
+			)
+		)
 		(instances
 			(project "BUCKET_FADER"
@@
 			)
 		)
+		(property "LCSC" "dnp"
+			(at 335.28 201.93 0)
+			(hide yes)
+			(show_name no)
+			(do_not_autoplace no)
+			(effects
+				(font
+					(size 1.27 1.27)
+				)
+			)
+		)
 		(instances
 			(project "BUCKET_FADER"
@@
 			)
 		)
+		(property "LCSC" "dnp"
+			(at 330.2 201.93 0)
+			(hide yes)
+			(show_name no)
+			(do_not_autoplace no)
+			(effects
+				(font
+					(size 1.27 1.27)
+				)
+			)
+		)
 		(instances
 			(project "BUCKET_FADER"
@@
 			)
 		)
+		(property "LCSC" "C75864"
+			(at 284.48 149.86 0)
+			(hide yes)
+			(show_name no)
+			(do_not_autoplace no)
+			(effects
+				(font
+					(size 1.27 1.27)
+				)
+			)
+		)
 		(pin "1"
 		)
@@
 			)
 		)
+		(property "LCSC" "C2652045"
+			(at 222.25 102.87 0)
+			(hide yes)
+			(show_name no)
+			(do_not_autoplace no)
+			(effects
+				(font
+					(size 1.27 1.27)
+				)
+			)
+		)
 		(pin "2"
 		)
@@
 			)
 		)
+		(property "LCSC" "C2652045"
+			(at 95.25 102.87 0)
+			(hide yes)
+			(show_name no)
+			(do_not_autoplace no)
+			(effects
+				(font
+					(size 1.27 1.27)
+				)
+			)
+		)
 		(pin "2"
 		)
@@
 			)
 		)
+		(property "LCSC" "C75864"
+			(at 157.48 149.86 0)
+			(hide yes)
+			(show_name no)
+			(do_not_autoplace no)
+			(effects
+				(font
+					(size 1.27 1.27)
+				)
+			)
+		)
 		(pin "1"
 		)
@@
 			)
 		)
+		(property "LCSC" "dnp"
+			(at 345.44 190.5 0)
+			(hide yes)
+			(show_name no)
+			(do_not_autoplace no)
+			(effects
+				(font
+					(size 1.27 1.27)
+				)
+			)
+		)
 		(instances
 			(project "BUCKET_FADER"
@@
 			)
 		)
+		(property "LCSC" "C2652045"
+			(at 285.75 102.87 0)
+			(hide yes)
+			(show_name no)
+			(do_not_autoplace no)
+			(effects
+				(font
+					(size 1.27 1.27)
+				)
+			)
+		)
 		(pin "2"
 		)
@@
 			)
 		)
+		(property "LCSC" "dnp"
+			(at 340.36 201.93 0)
+			(hide yes)
+			(show_name no)
+			(do_not_autoplace no)
+			(effects
+				(font
+					(size 1.27 1.27)
+				)
+			)
+		)
 		(instances
 			(project "BUCKET_FADER"
@@
 			)
 		)
+		(property "LCSC" "dnp"
+			(at 340.36 190.5 0)
+			(hide yes)
+			(show_name no)
+			(do_not_autoplace no)
+			(effects
+				(font
+					(size 1.27 1.27)
+				)
+			)
+		)
 		(instances
 			(project "BUCKET_FADER"
@@
 			(at 220.98 149.86 0)
 			(hide yes)
+			(show_name no)
+			(do_not_autoplace no)
+			(effects
+				(font
+					(size 1.27 1.27)
+				)
+			)
+		)
+		(property "LCSC" "C75864"
+			(at 220.98 149.86 0)
+			(hide yes)
