File: PCB_CAD/Bucket/Analog/EQ/EQ.kicad_pcb (KiCad board)
At the start: 2 copper layers, 36 x 150 mm, 0 parts

Commit message: input analog board pcb
Parts:
- added C1: 4.7p, Capacitor_SMD:C_0603_1608Metric, F.Cu at (161.1, 69.9)
- added C10: 2.2n, Capacitor_SMD:C_0805_2012Metric, F.Cu at (180.2, 112.6)
- added C101: 4.7p, Capacitor_SMD:C_0603_1608Metric, F.Cu at (161.1, 118.0)
- added C102: 1.2n, Capacitor_SMD:C_1206_3216Metric, F.Cu at (190.8, 118.5)
- added C103: 1.2n, Capacitor_SMD:C_1206_3216Metric, F.Cu at (190.8, 121.8)
- added C104: 1200p, Capacitor_SMD:C_1206_3216Metric, F.Cu at (190.8, 125.2)
- added C105: 1200p, Capacitor_SMD:C_1206_3216Metric, F.Cu at (190.8, 128.5)
- added C106: 1200p, Capacitor_SMD:C_1206_3216Metric, F.Cu at (190.8, 131.9)
- added C107: 1200p, Capacitor_SMD:C_1206_3216Metric, F.Cu at (190.8, 135.2)
- added C108: 10u, Capacitor_SMD:CP_Elec_6.3x5.4_Nichicon, F.Cu at (190.5, 145.2)
- added C109: 22p, Capacitor_SMD:C_0603_1608Metric, F.Cu at (161.1, 120.6)
- added C11: 100n, Capacitor_SMD:C_0603_1608Metric, F.Cu at (161.1, 80.0)
- added C110: 2.2n, Capacitor_SMD:C_0805_2012Metric, F.Cu at (161.3, 153.8)
- added C111: 100n, Capacitor_SMD:C_0603_1608Metric, F.Cu at (161.1, 123.1)
- added C112: 100n, Capacitor_SMD:C_0603_1608Metric, F.Cu at (161.1, 125.6)
- added C113: 100n, Capacitor_SMD:C_0603_1608Metric, F.Cu at (161.1, 128.1)
- added C114: 100n, Capacitor_SMD:C_0603_1608Metric, F.Cu at (161.1, 130.6)
- added C117: 100n, Capacitor_SMD:C_0603_1608Metric, F.Cu at (161.1, 133.1)
- added C12: 100n, Capacitor_SMD:C_0603_1608Metric, F.Cu at (161.1, 82.5)
- added C120: 22n, Capacitor_THT:C_Rect_L7.2mm_W2.5mm_P5.00mm, F.Cu at (181.1, 118.8)
- added C121: 22n, Capacitor_THT:C_Rect_L7.2mm_W2.5mm_P5.00mm, F.Cu at (181.1, 122.9)
- added C122: 22n, Capacitor_THT:C_Rect_L7.2mm_W2.5mm_P5.00mm, F.Cu at (181.1, 126.9)
- added C123: 22n, Capacitor_THT:C_Rect_L7.2mm_W2.5mm_P5.00mm, F.Cu at (181.1, 131.0)
- added C124: 22n, Capacitor_THT:C_Rect_L7.2mm_W2.5mm_P5.00mm, F.Cu at (181.1, 135.0)
- added C125: 22n, Capacitor_THT:C_Rect_L7.2mm_W2.5mm_P5.00mm, F.Cu at (181.1, 139.1)
- added C127: 100n, Capacitor_SMD:C_0603_1608Metric, F.Cu at (161.1, 135.6)
- added C128: 100n, Capacitor_SMD:C_0603_1608Metric, F.Cu at (161.1, 138.1)
- added C13: 100n, Capacitor_SMD:C_0603_1608Metric, F.Cu at (161.1, 85.0)
- added C14: 100n, Capacitor_SMD:C_0603_1608Metric, F.Cu at (161.1, 87.5)
- added C15: 100n, Capacitor_SMD:C_0603_1608Metric, F.Cu at (161.1, 90.0)
- added C16: 100n, Capacitor_SMD:C_0603_1608Metric, F.Cu at (161.1, 92.5)
- added C17: 100n, Capacitor_SMD:C_0603_1608Metric, F.Cu at (161.1, 95.0)
- added C18: 100n, Capacitor_SMD:C_0603_1608Metric, F.Cu at (165.1, 69.9)
- added C19: 100n, Capacitor_SMD:C_0603_1608Metric, F.Cu at (165.1, 72.4)
- added C2: 3.3n, Capacitor_SMD:C_0603_1608Metric, F.Cu at (161.1, 72.4)
- added C20: 22n, Capacitor_THT:C_Rect_L7.2mm_W2.5mm_P5.00mm, F.Cu at (185.1, 70.7)
- added C201: 22n, Capacitor_THT:C_Rect_L7.2mm_W2.5mm_P5.00mm, F.Cu at (108.0, 70.7)
- added C202: 22n, Capacitor_THT:C_Rect_L7.2mm_W2.5mm_P5.00mm, F.Cu at (108.0, 74.8)
- added C203: 22n, Capacitor_THT:C_Rect_L7.2mm_W2.5mm_P5.00mm, F.Cu at (108.0, 78.8)
- added C204: 22n, Capacitor_THT:C_Rect_L7.2mm_W2.5mm_P5.00mm, F.Cu at (108.0, 82.8)
- added C205: 22n, Capacitor_THT:C_Rect_L7.2mm_W2.5mm_P5.00mm, F.Cu at (108.0, 86.9)
- added C206: 22n, Capacitor_THT:C_Rect_L7.2mm_W2.5mm_P5.00mm, F.Cu at (108.0, 91.0)
- added C207: 22n, Capacitor_THT:C_Rect_L7.2mm_W2.5mm_P5.00mm, F.Cu at (108.0, 95.0)
- added C208: 22n, Capacitor_THT:C_Rect_L7.2mm_W2.5mm_P5.00mm, F.Cu at (108.0, 99.0)
- added C209: 4.7p, Capacitor_SMD:C_0603_1608Metric, F.Cu at (116.9, 69.9)
- added C21: 22n, Capacitor_THT:C_Rect_L7.2mm_W2.5mm_P5.00mm, F.Cu at (185.1, 74.8)
- added C210: 1200p, Capacitor_SMD:C_1206_3216Metric, F.Cu at (151.9, 86.7)
- added C211: 15n, Capacitor_THT:C_Rect_L7.2mm_W2.5mm_P5.00mm, F.Cu at (108.0, 103.1)
- added C212: 1200p, Capacitor_SMD:C_1206_3216Metric, F.Cu at (151.9, 90.0)
- added C213: 15n, Capacitor_THT:C_Rect_L7.2mm_W2.5mm_P5.00mm, F.Cu at (108.0, 107.2)
- added C214: 4.7p, Capacitor_SMD:C_0603_1608Metric, F.Cu at (116.9, 72.4)
- added C215: 1200p, Capacitor_SMD:C_1206_3216Metric, F.Cu at (151.9, 93.3)
- added C216: 390p, Capacitor_SMD:C_0603_1608Metric, F.Cu at (116.9, 75.0)
- added C217: 1200p, Capacitor_SMD:C_1206_3216Metric, F.Cu at (151.9, 96.7)
- added C218: 390p, Capacitor_SMD:C_0603_1608Metric, F.Cu at (116.9, 77.5)
- added C219: 2.2n, Capacitor_SMD:C_0805_2012Metric, F.Cu at (126.2, 115.7)
- added C22: 22n, Capacitor_THT:C_Rect_L7.2mm_W2.5mm_P5.00mm, F.Cu at (185.1, 78.8)
- added C220: 22p, Capacitor_SMD:C_0603_1608Metric, F.Cu at (116.9, 80.0)
- added C221: 10u, Capacitor_SMD:CP_Elec_6.3x5.4_Nichicon, F.Cu at (148.2, 72.8)
- added C222: 2.2n, Capacitor_SMD:C_0805_2012Metric, F.Cu at (126.2, 118.7)
- added C223: 47p, Capacitor_SMD:C_0603_1608Metric, F.Cu at (116.9, 82.5)
- added C224: 10u, Capacitor_SMD:CP_Elec_6.3x5.4_Nichicon, F.Cu at (148.2, 80.9)
- added C225: 100n, Capacitor_SMD:C_0603_1608Metric, F.Cu at (116.9, 85.0)
- added C226: 100n, Capacitor_SMD:C_0603_1608Metric, F.Cu at (116.9, 87.5)
- added C227: 100n, Capacitor_SMD:C_0603_1608Metric, F.Cu at (116.9, 90.0)
- added C228: 100n, Capacitor_SMD:C_0603_1608Metric, F.Cu at (116.9, 92.5)
- added C229: 100n, Capacitor_SMD:C_0603_1608Metric, F.Cu at (116.9, 95.0)
- added C23: 22n, Capacitor_THT:C_Rect_L7.2mm_W2.5mm_P5.00mm, F.Cu at (185.1, 82.8)
- added C230: 100n, Capacitor_SMD:C_0603_1608Metric, F.Cu at (116.9, 97.5)
- added C231: 100n, Capacitor_SMD:C_0603_1608Metric, F.Cu at (116.9, 100.0)
- added C232: 100n, Capacitor_SMD:C_0603_1608Metric, F.Cu at (116.9, 102.6)
- added C233: 100n, Capacitor_SMD:C_0603_1608Metric, F.Cu at (120.9, 69.9)
- added C234: 100n, Capacitor_SMD:C_0603_1608Metric, F.Cu at (120.9, 72.4)
- added C235: 100n, Capacitor_SMD:C_0603_1608Metric, F.Cu at (120.9, 75.0)
- added C236: 100n, Capacitor_SMD:C_0603_1608Metric, F.Cu at (120.9, 77.5)
- added C24: 22n, Capacitor_THT:C_Rect_L7.2mm_W2.5mm_P5.00mm, F.Cu at (185.1, 86.9)
- added C25: 22n, Capacitor_THT:C_Rect_L7.2mm_W2.5mm_P5.00mm, F.Cu at (185.1, 91.0)
- added C26: 100n, Capacitor_SMD:C_0603_1608Metric, F.Cu at (165.1, 75.0)
- added C27: 100n, Capacitor_SMD:C_0603_1608Metric, F.Cu at (165.1, 77.5)
- added C28: 100n, Capacitor_SMD:C_0603_1608Metric, F.Cu at (165.1, 80.0)
- added C3: 3.3n, Capacitor_SMD:C_0603_1608Metric, F.Cu at (161.1, 75.0)
- added C4: 1200p, Capacitor_SMD:C_1206_3216Metric, F.Cu at (187.3, 98.0)
- added C5: 1200p, Capacitor_SMD:C_1206_3216Metric, F.Cu at (187.3, 101.3)
- added C6: 1200p, Capacitor_SMD:C_1206_3216Metric, F.Cu at (187.3, 104.7)
- added C7: 1200p, Capacitor_SMD:C_1206_3216Metric, F.Cu at (187.3, 108.0)
- added C8: 10u, Capacitor_SMD:CP_Elec_6.3x5.4_Nichicon, F.Cu at (164.3, 110.7)
- added C9: 22p, Capacitor_SMD:C_0603_1608Metric, F.Cu at (161.1, 77.5)
- added R1: 20k, Resistor_SMD:R_0603_1608Metric, F.Cu at (165.1, 82.5)
- added R10: 220, Resistor_SMD:R_0603_1608Metric, F.Cu at (169.2, 77.5)
- added R101: 20k, Resistor_SMD:R_0603_1608Metric, F.Cu at (161.1, 140.6)
- added R102: 10k, Resistor_SMD:R_0603_1608Metric, F.Cu at (165.1, 118.0)
- added R103: 20k, Resistor_SMD:R_0603_1608Metric, F.Cu at (165.1, 120.6)
- added R104: 20k, Resistor_SMD:R_0603_1608Metric, F.Cu at (165.1, 123.1)
- added R105: 20k, Resistor_SMD:R_0603_1608Metric, F.Cu at (165.1, 125.6)
- added R106: 10k, Resistor_SMD:R_0603_1608Metric, F.Cu at (165.1, 128.1)
- added R107: 10k, Resistor_SMD:R_0603_1608Metric, F.Cu at (165.1, 130.6)
- added R108: 20k, Resistor_SMD:R_0603_1608Metric, F.Cu at (165.1, 133.1)
- added R109: 220, Resistor_SMD:R_0603_1608Metric, F.Cu at (165.1, 135.6)
- added R11: 220, Resistor_SMD:R_0603_1608Metric, F.Cu at (169.2, 80.0)
- added R110: 220, Resistor_SMD:R_0603_1608Metric, F.Cu at (165.1, 138.1)
- added R111: 220, Resistor_SMD:R_0603_1608Metric, F.Cu at (165.1, 140.6)
- added R112: 220, Resistor_SMD:R_0603_1608Metric, F.Cu at (169.2, 118.0)
- added R113: 10k, Resistor_SMD:R_0603_1608Metric, F.Cu at (169.2, 120.6)
- added R114: 5.1k, Resistor_SMD:R_0603_1608Metric, F.Cu at (169.2, 123.1)
- added R116: 20k, Resistor_SMD:R_0603_1608Metric, F.Cu at (169.2, 125.6)
- added R117: 100, Resistor_SMD:R_0603_1608Metric, F.Cu at (169.2, 128.1)
- added R12: 220, Resistor_SMD:R_0603_1608Metric, F.Cu at (169.2, 82.5)
- added R120: 100k, Resistor_SMD:R_0603_1608Metric, F.Cu at (169.2, 130.6)
- added R121: 130k, Resistor_SMD:R_0603_1608Metric, F.Cu at (169.2, 133.1)
- added R122: 88.7k, Resistor_SMD:R_0603_1608Metric, F.Cu at (169.2, 135.6)
- added R123: 20k, Resistor_SMD:R_0603_1608Metric, F.Cu at (169.2, 138.1)
- added R124: 20k, Resistor_SMD:R_0603_1608Metric, F.Cu at (169.2, 140.6)
- added R125: 20k, Resistor_SMD:R_0603_1608Metric, F.Cu at (173.2, 118.0)
- added R126: 100k, Resistor_SMD:R_0603_1608Metric, F.Cu at (173.2, 120.6)
- added R127: 130k, Resistor_SMD:R_0603_1608Metric, F.Cu at (173.2, 123.1)
- added R128: 88.7k, Resistor_SMD:R_0603_1608Metric, F.Cu at (173.2, 125.6)
- added R129: 20k, Resistor_SMD:R_0603_1608Metric, F.Cu at (173.2, 128.1)
- added R13: 10k, Resistor_SMD:R_0603_1608Metric, F.Cu at (169.2, 85.0)
- added R130: 30.1k, Resistor_SMD:R_0603_1608Metric, F.Cu at (173.2, 130.6)
- added R131: 30.1k, Resistor_SMD:R_0603_1608Metric, F.Cu at (173.2, 133.1)
- added R132: 100k, Resistor_SMD:R_0603_1608Metric, F.Cu at (173.2, 135.6)
- added R133: 130k, Resistor_SMD:R_0603_1608Metric, F.Cu at (173.2, 138.1)
- added R134: 95.3k, Resistor_SMD:R_0603_1608Metric, F.Cu at (173.2, 140.6)
- added R135: 20k, Resistor_SMD:R_0603_1608Metric, F.Cu at (177.2, 118.0)
- added R136: 22.1k, Resistor_SMD:R_0603_1608Metric, F.Cu at (177.2, 120.6)
- added R137: 22.1k, Resistor_SMD:R_0603_1608Metric, F.Cu at (177.2, 123.1)
- added R139: 20k, Resistor_SMD:R_0603_1608Metric, F.Cu at (177.2, 125.6)
- added R14: 5.1k, Resistor_SMD:R_0603_1608Metric, F.Cu at (169.2, 87.5)
- added R140: 22k, Resistor_SMD:R_0603_1608Metric, F.Cu at (177.2, 128.1)
- added R141: 10k, Resistor_SMD:R_0603_1608Metric, F.Cu at (177.2, 130.6)
- added R142: 10k, Resistor_SMD:R_0603_1608Metric, F.Cu at (177.2, 133.1)
- added R143: 14.0k, Resistor_SMD:R_0603_1608Metric, F.Cu at (177.2, 135.6)
- added R144: 14.0k, Resistor_SMD:R_0603_1608Metric, F.Cu at (177.2, 138.1)
- added R16: 20k, Resistor_SMD:R_0603_1608Metric, F.Cu at (169.2, 90.0)
- added R17: 100, Resistor_SMD:R_0603_1608Metric, F.Cu at (169.2, 92.5)
- added R18: 10k, Resistor_SMD:R_0603_1608Metric, F.Cu at (169.2, 95.0)
- added R19: 100k, Resistor_SMD:R_0603_1608Metric, F.Cu at (173.2, 69.9)
- added R2: 10k, Resistor_SMD:R_0603_1608Metric, F.Cu at (165.1, 85.0)
- added R20: 100k, Resistor_SMD:R_0603_1608Metric, F.Cu at (173.2, 72.4)
- added R201: 20k, Resistor_SMD:R_0603_1608Metric, F.Cu at (120.9, 80.0)
- added R202: 130k, Resistor_SMD:R_0603_1608Metric, F.Cu at (120.9, 82.5)
- added R203: 88.7k, Resistor_SMD:R_0603_1608Metric, F.Cu at (120.9, 85.0)
- added R204: 100k, Resistor_SMD:R_0603_1608Metric, F.Cu at (120.9, 87.5)
- added R205: 20k, Resistor_SMD:R_0603_1608Metric, F.Cu at (120.9, 90.0)
- added R206: 20k, Resistor_SMD:R_0603_1608Metric, F.Cu at (120.9, 92.5)
- added R207: 100k, Resistor_SMD:R_0603_1608Metric, F.Cu at (120.9, 95.0)
- added R208: 130k, Resistor_SMD:R_0603_1608Metric, F.Cu at (120.9, 97.5)
- added R209: 95.3k, Resistor_SMD:R_0603_1608Metric, F.Cu at (120.9, 100.0)
- added R21: 130k, Resistor_SMD:R_0603_1608Metric, F.Cu at (173.2, 75.0)
- added R210: 20k, Resistor_SMD:R_0603_1608Metric, F.Cu at (120.9, 102.6)
- added R211: 22.1k, Resistor_SMD:R_0603_1608Metric, F.Cu at (124.9, 69.9)
- added R212: 22.1k, Resistor_SMD:R_0603_1608Metric, F.Cu at (124.9, 72.4)
- added R213: 20k, Resistor_SMD:R_0603_1608Metric, F.Cu at (124.9, 75.0)
- added R214: 130k, Resistor_SMD:R_0603_1608Metric, F.Cu at (124.9, 77.5)
- added R215: 88.7k, Resistor_SMD:R_0603_1608Metric, F.Cu at (124.9, 80.0)
- added R216: 100k, Resistor_SMD:R_0603_1608Metric, F.Cu at (124.9, 82.5)
- added R217: 20k, Resistor_SMD:R_0603_1608Metric, F.Cu at (124.9, 85.0)
- added R218: 20k, Resistor_SMD:R_0603_1608Metric, F.Cu at (124.9, 87.5)
- added R219: 100k, Resistor_SMD:R_0603_1608Metric, F.Cu at (124.9, 90.0)
- added R22: 88.7k, Resistor_SMD:R_0603_1608Metric, F.Cu at (173.2, 77.5)
- added R220: 130k, Resistor_SMD:R_0603_1608Metric, F.Cu at (124.9, 92.5)
- added R221: 95.3k, Resistor_SMD:R_0603_1608Metric, F.Cu at (124.9, 95.0)
- added R222: 20k, Resistor_SMD:R_0603_1608Metric, F.Cu at (124.9, 97.5)
- added R223: 22.1k, Resistor_SMD:R_0603_1608Metric, F.Cu at (124.9, 100.0)
- added R224: 22.1k, Resistor_SMD:R_0603_1608Metric, F.Cu at (124.9, 102.6)
- added R225: 20k, Resistor_SMD:R_0603_1608Metric, F.Cu at (128.9, 69.9)
- added R226: 20k, Resistor_SMD:R_0603_1608Metric, F.Cu at (128.9, 72.4)
- added R227: 20k, Resistor_SMD:R_0603_1608Metric, F.Cu at (128.9, 75.0)
- added R228: 220, Resistor_SMD:R_0603_1608Metric, F.Cu at (128.9, 77.5)
- added R229: 20k, Resistor_SMD:R_0603_1608Metric, F.Cu at (128.9, 80.0)
- added R23: 20k, Resistor_SMD:R_0603_1608Metric, F.Cu at (173.2, 80.0)
- added R230: 220, Resistor_SMD:R_0603_1608Metric, F.Cu at (128.9, 82.5)
- added R231: 10k, Resistor_SMD:R_0603_1608Metric, F.Cu at (128.9, 85.0)
- added R232: 10k, Resistor_SMD:R_0603_1608Metric, F.Cu at (128.9, 87.5)
- added R233: 14.0k, Resistor_SMD:R_0603_1608Metric, F.Cu at (128.9, 90.0)
- added R234: 20k, Resistor_SMD:R_0603_1608Metric, F.Cu at (128.9, 92.5)
- added R235: 20k, Resistor_SMD:R_0603_1608Metric, F.Cu at (128.9, 95.0)
- added R236: 20k, Resistor_SMD:R_0603_1608Metric, F.Cu at (128.9, 97.5)
- added R237: 20k, Resistor_SMD:R_0603_1608Metric, F.Cu at (128.9, 100.0)
- added R238: 220, Resistor_SMD:R_0603_1608Metric, F.Cu at (128.9, 102.6)
- added R239: 20k, Resistor_SMD:R_0603_1608Metric, F.Cu at (132.9, 69.9)
- added R24: 20k, Resistor_SMD:R_0603_1608Metric, F.Cu at (173.2, 82.5)
- added R240: 220, Resistor_SMD:R_0603_1608Metric, F.Cu at (132.9, 72.4)
- added R241: 10k, Resistor_SMD:R_0603_1608Metric, F.Cu at (132.9, 75.0)
- added R242: 10k, Resistor_SMD:R_0603_1608Metric, F.Cu at (132.9, 77.5)
- added R243: 14.0k, Resistor_SMD:R_0603_1608Metric, F.Cu at (132.9, 80.0)
- added R244: 20k, Resistor_SMD:R_0603_1608Metric, F.Cu at (132.9, 82.5)
- added R245: 5.1k, Resistor_SMD:R_0603_1608Metric, F.Cu at (132.9, 85.0)
- added R246: 20k, Resistor_SMD:R_0603_1608Metric, F.Cu at (132.9, 87.5)
- added R247: 20k, Resistor_SMD:R_0603_1608Metric, F.Cu at (132.9, 90.0)
- added R248: 100, Resistor_SMD:R_0603_1608Metric, F.Cu at (132.9, 92.5)
- added R249: 46.4k, Resistor_SMD:R_0603_1608Metric, F.Cu at (132.9, 95.0)
- added R25: 20k, Resistor_SMD:R_0603_1608Metric, F.Cu at (173.2, 85.0)
- added R250: 20k, Resistor_SMD:R_0603_1608Metric, F.Cu at (132.9, 97.5)
- added R251: 5.1k, Resistor_SMD:R_0603_1608Metric, F.Cu at (132.9, 100.0)
- added R252: 20k, Resistor_SMD:R_0603_1608Metric, F.Cu at (132.9, 102.6)
- added R253: 20k, Resistor_SMD:R_0603_1608Metric, F.Cu at (136.9, 69.9)
- added R254: 100, Resistor_SMD:R_0603_1608Metric, F.Cu at (136.9, 72.4)
- added R255: 46.4k, Resistor_SMD:R_0603_1608Metric, F.Cu at (136.9, 75.0)
- added R256: 20k, Resistor_SMD:R_0603_1608Metric, F.Cu at (136.9, 77.5)
- added R257: 10k, Resistor_SMD:R_0603_1608Metric, F.Cu at (136.9, 80.0)
- added R258: 100k, Resistor_SMD:R_0603_1608Metric, F.Cu at (136.9, 82.5)
- added R259: 10k, Resistor_SMD:R_0603_1608Metric, F.Cu at (136.9, 85.0)
- added R26: 100k, Resistor_SMD:R_0603_1608Metric, F.Cu at (173.2, 87.5)
- added R260: 100k, Resistor_SMD:R_0603_1608Metric, F.Cu at (136.9, 87.5)
- added R261: 10k, Resistor_SMD:R_0603_1608Metric, F.Cu at (136.9, 90.0)
- added R262: 100k, Resistor_SMD:R_0603_1608Metric, F.Cu at (136.9, 92.5)
- added R263: 10k, Resistor_SMD:R_0603_1608Metric, F.Cu at (136.9, 95.0)
- added R264: 100k, Resistor_SMD:R_0603_1608Metric, F.Cu at (136.9, 97.5)
- added R265: 22k, Resistor_SMD:R_0603_1608Metric, F.Cu at (136.9, 100.0)
- added R266: 10k, Resistor_SMD:R_0603_1608Metric, F.Cu at (136.9, 102.6)
- added R267: 10k, Resistor_SMD:R_0603_1608Metric, F.Cu at (140.9, 69.9)
- added R268: 14.0k, Resistor_SMD:R_0603_1608Metric, F.Cu at (140.9, 72.4)
- added R269: 14.0k, Resistor_SMD:R_0603_1608Metric, F.Cu at (140.9, 75.0)
- added R27: 130k, Resistor_SMD:R_0603_1608Metric, F.Cu at (173.2, 90.0)
- added R270: 14.0k, Resistor_SMD:R_0603_1608Metric, F.Cu at (140.9, 77.5)
- added R271: 14.0k, Resistor_SMD:R_0603_1608Metric, F.Cu at (140.9, 80.0)
- added R272: 20k, Resistor_SMD:R_0603_1608Metric, F.Cu at (140.9, 82.5)
- added R273: 20k, Resistor_SMD:R_0603_1608Metric, F.Cu at (140.9, 85.0)
- added R274: 20k, Resistor_SMD:R_0603_1608Metric, F.Cu at (140.9, 87.5)
- added R275: 20k, Resistor_SMD:R_0603_1608Metric, F.Cu at (140.9, 90.0)
- added R28: 88.7k, Resistor_SMD:R_0603_1608Metric, F.Cu at (173.2, 92.5)
- added R29: 20k, Resistor_SMD:R_0603_1608Metric, F.Cu at (173.2, 95.0)
- added R3: 20k, Resistor_SMD:R_0603_1608Metric, F.Cu at (165.1, 87.5)
- added R30: 30.1k, Resistor_SMD:R_0603_1608Metric, F.Cu at (177.2, 69.9)
- added R31: 30.1k, Resistor_SMD:R_0603_1608Metric, F.Cu at (177.2, 72.4)
- added R32: 100k, Resistor_SMD:R_0603_1608Metric, F.Cu at (177.2, 75.0)
- added R33: 130k, Resistor_SMD:R_0603_1608Metric, F.Cu at (177.2, 77.5)
- added R34: 95.3k, Resistor_SMD:R_0603_1608Metric, F.Cu at (177.2, 80.0)
- added R35: 20k, Resistor_SMD:R_0603_1608Metric, F.Cu at (177.2, 82.5)
- added R36: 22.1k, Resistor_SMD:R_0603_1608Metric, F.Cu at (177.2, 85.0)
- added R37: 22.1k, Resistor_SMD:R_0603_1608Metric, F.Cu at (177.2, 87.5)
- added R38: 46.4k, Resistor_SMD:R_0603_1608Metric, F.Cu at (177.2, 90.0)
- added R39: 20k, Resistor_SMD:R_0603_1608Metric, F.Cu at (177.2, 92.5)
- added R4: 20k, Resistor_SMD:R_0603_1608Metric, F.Cu at (165.1, 90.0)
- added R40: 10k, Resistor_SMD:R_0603_1608Metric, F.Cu at (177.2, 95.0)
- added R41: 100k, Resistor_SMD:R_0603_1608Metric, F.Cu at (181.2, 69.9)
- added R42: 22k, Resistor_SMD:R_0603_1608Metric, F.Cu at (181.2, 72.4)
- added R43: 10k, Resistor_SMD:R_0603_1608Metric, F.Cu at (181.2, 75.0)
- added R44: 10k, Resistor_SMD:R_0603_1608Metric, F.Cu at (181.2, 77.5)
- added R45: 14.0k, Resistor_SMD:R_0603_1608Metric, F.Cu at (181.2, 80.0)
- added R46: 14.0k, Resistor_SMD:R_0603_1608Metric, F.Cu at (181.2, 82.5)
- added R47: 20k, Resistor_SMD:R_0603_1608Metric, F.Cu at (181.2, 85.0)
- added R48: 20k, Resistor_SMD:R_0603_1608Metric, F.Cu at (181.2, 87.5)
- added R5: 20k, Resistor_SMD:R_0603_1608Metric, F.Cu at (165.1, 92.5)
- added R6: 10k, Resistor_SMD:R_0603_1608Metric, F.Cu at (165.1, 95.0)
- added R7: 10k, Resistor_SMD:R_0603_1608Metric, F.Cu at (169.2, 69.9)
- added R8: 20k, Resistor_SMD:R_0603_1608Metric, F.Cu at (169.2, 72.4)
- added R9: 220, Resistor_SMD:R_0603_1608Metric, F.Cu at (169.2, 75.0)
- added TH1: NTC 47k, Resistor_THT:R_Axial_DIN0207_L6.3mm_D2.5mm_P2.54mm_Vertical, F.Cu at (192.2, 98.3)
- added TH101: NTC 47k, Resistor_THT:R_Axial_DIN0207_L6.3mm_D2.5mm_P2.54mm_Vertical, F.Cu at (181.2, 143.1)
- added TH102: NTC 47k, Resistor_THT:R_Axial_DIN0207_L6.3mm_D2.5mm_P2.54mm_Vertical, F.Cu at (181.2, 147.2)
- added TH103: NTC 47k, Resistor_THT:R_Axial_DIN0207_L6.3mm_D2.5mm_P2.54mm_Vertical, F.Cu at (181.2, 151.2)
- added TH2: NTC 47k, Resistor_THT:R_Axial_DIN0207_L6.3mm_D2.5mm_P2.54mm_Vertical, F.Cu at (192.2, 102.4)
- added TH201: NTC 47k, Resistor_THT:R_Axial_DIN0207_L6.3mm_D2.5mm_P2.54mm_Vertical, F.Cu at (145.0, 87.0)
- added TH202: NTC 47k, Resistor_THT:R_Axial_DIN0207_L6.3mm_D2.5mm_P2.54mm_Vertical, F.Cu at (145.0, 91.0)
- added TH203: NTC 47k, Resistor_THT:R_Axial_DIN0207_L6.3mm_D2.5mm_P2.54mm_Vertical, F.Cu at (145.0, 95.1)
- added TH204: NTC 47k, Resistor_THT:R_Axial_DIN0207_L6.3mm_D2.5mm_P2.54mm_Vertical, F.Cu at (145.0, 99.2)
- added TH3: NTC 47k, Resistor_THT:R_Axial_DIN0207_L6.3mm_D2.5mm_P2.54mm_Vertical, F.Cu at (192.2, 106.4)
- added U1: OPA4197, Package_SO:SOIC-14_3.9x8.7mm_P1.27mm, F.Cu at (163.3, 101.5)
- added U10: OPA1679, Package_SO:SOIC-14_3.9x8.7mm_P1.27mm, F.Cu at (163.3, 147.2)
- added U11: OPA4197, Package_SO:SOIC-14_3.9x8.7mm_P1.27mm, F.Cu at (171.8, 147.2)
- added U13: AS2180, Package_SO:SOIC-8-1EP_3.9x4.9mm_P1.27mm_EP2.29x3mm_ThermalVias, F.Cu at (152.9, 107.2)
- added U14: OPA1679, Package_SO:SOIC-14_3.9x8.7mm_P1.27mm, F.Cu at (119.1, 109.1)
- added U15: OPA1679, Package_SO:SOIC-14_3.9x8.7mm_P1.27mm, F.Cu at (127.5, 109.1)
- added U16: OPA1679, Package_SO:SOIC-14_3.9x8.7mm_P1.27mm, F.Cu at (136.0, 109.1)
- added U17: OPA4197, Package_SO:SOIC-14_3.9x8.7mm_P1.27mm, F.Cu at (144.4, 109.1)
- added U18: ADG1434, Package_SO:TSSOP-20_4.4x6.5mm_P0.65mm, F.Cu at (119.6, 118.2)
- added U19: AS2180, Package_SO:SOIC-8-1EP_3.9x4.9mm_P1.27mm_EP2.29x3mm_ThermalVias, F.Cu at (152.9, 113.8)
- added U3: AS2180, Package_SO:SOIC-8-1EP_3.9x4.9mm_P1.27mm_EP2.29x3mm_ThermalVias, F.Cu at (173.8, 110.0)
- added U5: OPA1679, Package_SO:SOIC-14_3.9x8.7mm_P1.27mm, F.Cu at (171.8, 101.5)
- added U6: OPA1679, Package_SO:SOIC-14_3.9x8.7mm_P1.27mm, F.Cu at (180.2, 101.5)
- added U7: ADR5041, Package_TO_SOT_SMD:SOT-23, F.Cu at (180.5, 108.9)
- added U9: AS2180, Package_SO:SOIC-8-1EP_3.9x4.9mm_P1.27mm_EP2.29x3mm_ThermalVias, F.Cu at (189.5, 152.6)
Other:
- board size 36 x 150 mm -> 36 x 180 mm
