File: PCB_CAD/Bucket/Analog/EQ/hmf.kicad_sch (KiCad schematic)
At the start: 67 parts, among them U10 OPA1679, U11 OPA4197, U14 OPA1679, U8 SSI2164, U9 AS2180

Commit message: getting ready to upgrade mx file
Parts:
- C120, C121, C122, C123, C124, C125: footprint Capacitor_SMD:C_0603_1608Metric -> Capacitor_THT:C_Rect_L7.2mm_W2.5mm_P5.00mm
Other:
- note removed: "Spare Op-Amp"
- moved on the sheet: C117, U11D
Changed lines of the file:
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@@
 		)
 	)
-	(rectangle
-		(start 41.91 179.07)
-		(end 127 220.98)
-		(stroke
-			(width 0)
-			(type default)
-		)
-		(fill
-			(type none)
-		)
-	)
 	(text "State Variable Filter - Voltage Controlled"
 		(exclude_from_sim no)
@@
 		)
 	)
-	(text "Spare Op-Amp"
-		(exclude_from_sim no)
-		(at 83.058 186.944 0)
-		(effects
-			(font
-				(size 3.81 3.81)
-				(thickness 0.762)
-				(bold yes)
-			)
-		)
-	)
 	(text "CV Buffers\n"
 		(exclude_from_sim no)
@@
 	(wire
 		(pts
-			(xy 107.95 210.82) (xy 87.63 210.82)
+			(xy 224.79 266.7) (xy 204.47 266.7)
 		)
 		(stroke
@@
 	(wire
 		(pts
-			(xy 90.17 200.66) (xy 85.09 200.66)
+			(xy 207.01 256.54) (xy 201.93 256.54)
 		)
 		(stroke
@@
 	(wire
 		(pts
-			(xy 87.63 210.82) (xy 87.63 205.74)
+			(xy 204.47 266.7) (xy 204.47 261.62)
 		)
 		(stroke
@@
 	(wire
 		(pts
-			(xy 105.41 203.2) (xy 107.95 203.2)
+			(xy 222.25 259.08) (xy 224.79 259.08)
 		)
 		(stroke
@@
 	(wire
 		(pts
-			(xy 87.63 205.74) (xy 90.17 205.74)
+			(xy 204.47 261.62) (xy 207.01 261.62)
 		)
 		(stroke
@@
 	(wire
 		(pts
-			(xy 107.95 203.2) (xy 107.95 210.82)
+			(xy 224.79 259.08) (xy 224.79 266.7)
 		)
 		(stroke
@@
 			)
 		)
-		(property "Footprint" "Capacitor_SMD:C_0603_1608Metric"
+		(property "Footprint" "Capacitor_THT:C_Rect_L7.2mm_W2.5mm_P5.00mm"
 			(at 111.76 69.85 0)
 			(hide yes)
@@
 			)
 		)
-		(property "Footprint" "Capacitor_SMD:C_0603_1608Metric"
+		(property "Footprint" "Capacitor_THT:C_Rect_L7.2mm_W2.5mm_P5.00mm"
 			(at 85.09 146.05 0)
 			(hide yes)
@@
 			)
 		)
-		(property "Footprint" "Capacitor_SMD:C_0603_1608Metric"
+		(property "Footprint" "Capacitor_THT:C_Rect_L7.2mm_W2.5mm_P5.00mm"
 			(at 111.76 107.95 0)
 			(hide yes)
@@
 			)
 		)
-		(property "Footprint" "Capacitor_SMD:C_0603_1608Metric"
+		(property "Footprint" "Capacitor_THT:C_Rect_L7.2mm_W2.5mm_P5.00mm"
 			(at 85.09 106.68 0)
 			(hide yes)
@@
 	(symbol
 		(lib_id "power:+16.6V")
-		(at 209.55 259.08 0)
+		(at 167.64 259.08 0)
 		(unit 1)
 		(body_style 1)
@@
 		(dnp no)
 		(property "Reference" "#PWR0215"
-			(at 209.55 262.89 0)
+			(at 167.64 262.89 0)
 			(hide yes)
 			(show_name no)
@@
 		)
 		(property "Value" "+15V"
-			(at 209.55 255.524 0)
+			(at 167.64 255.524 0)
 			(show_name no)
 			(do_not_autoplace no)
@@
 		)
 		(property "Footprint" ""
-			(at 209.55 259.08 0)
+			(at 167.64 259.08 0)
 			(hide yes)
 			(show_name no)
@@
 		)
 		(property "Datasheet" ""
-			(at 209.55 259.08 0)
+			(at 167.64 259.08 0)
 			(hide yes)
 			(show_name no)
@@
 		)
 		(property "Description" "Power symbol creates a global label with name \"+15V\""
-			(at 209.55 259.08 0)
+			(at 167.64 259.08 0)
 			(hide yes)
 			(show_name no)
@@
 	(symbol
 		(lib_id "Amplifier_Operational:OPA4197xD")
-		(at 97.79 203.2 0)
+		(at 214.63 259.08 0)
 		(unit 4)
 		(body_style 1)
@@
 		(dnp no)
 		(property "Reference" "U11"
-			(at 99.06 193.04 0)
+			(at 215.9 248.92 0)
 			(show_name no)
 			(do_not_autoplace no)
@@
 		)
 		(property "Value" "OPA4197"
-			(at 99.06 195.58 0)
+			(at 215.9 251.46 0)
 			(show_name no)
 			(do_not_autoplace no)
@@
 		)
 		(property "Footprint" "Package_SO:SOIC-14_3.9x8.7mm_P1.27mm"
-			(at 97.79 203.2 0)
+			(at 214.63 259.08 0)
 			(hide yes)
 			(show_name no)
@@
 		)
 		(property "Datasheet" "http://www.ti.com/lit/ds/symlink/opa4197.pdf"
-			(at 97.79 203.2 0)
+			(at 214.63 259.08 0)
 			(hide yes)
 			(show_name no)
@@
 		)
 		(property "Description" "Quad 36V, Precision, Rail-to-Rail Input/Output, Low Offset Voltage, Operational Amplifier, SOIC-14"
-			(at 97.79 203.2 0)
+			(at 214.63 259.08 0)
 			(hide yes)
 			(show_name no)
@@
 		)
 		(property "LCSC" "C2058532"
-			(at 97.79 203.2 0)
+			(at 214.63 259.08 0)
 			(hide yes)
 			(show_name no)
@@
 			)
 		)
-		(property "Footprint" "Capacitor_SMD:C_0603_1608Metric"
+		(property "Footprint" "Capacitor_THT:C_Rect_L7.2mm_W2.5mm_P5.00mm"
 			(at 111.76 147.32 0)
 			(hide yes)
@@
 			)
 		)
-		(property "Footprint" "Capacitor_SMD:C_0603_1608Metric"
+		(property "Footprint" "Capacitor_THT:C_Rect_L7.2mm_W2.5mm_P5.00mm"
 			(at 85.09 68.58 0)
 			(hide yes)
@@
 	(symbol
 		(lib_id "Device:C")
-		(at 209.55 262.89 0)
+		(at 167.64 262.89 0)
 		(unit 1)
 		(body_style 1)
@@
 		(dnp no)
 		(property "Reference" "C117"
-			(at 212.598 261.62 0)
+			(at 170.688 261.62 0)
 			(show_name no)
 			(do_not_autoplace no)
@@
 		)
 		(property "Value" "100n"
-			(at 212.598 264.16 0)
+			(at 170.688 264.16 0)
 			(show_name no)
 			(do_not_autoplace no)
@@
 		)
 		(property "Footprint" "Capacitor_SMD:C_0603_1608Metric"
-			(at 209.55 262.89 0)
+			(at 167.64 262.89 0)
 			(hide yes)
 			(show_name no)
@@
 		)
 		(property "Datasheet" ""
-			(at 209.55 262.89 0)
+			(at 167.64 262.89 0)
 			(hide yes)
 			(show_name no)
@@
 		)
 		(property "Description" "Unpolarized capacitor"
-			(at 209.55 262.89 0)
+			(at 167.64 262.89 0)
 			(hide yes)
 			(show_name no)
@@
 		)
 		(property "LCSC" "C1591"
-			(at 209.55 262.89 0)
+			(at 167.64 262.89 0)
 			(hide yes)
 			(show_name no)
@@
 	(symbol
 		(lib_id "power:GND")
-		(at 209.55 266.7 0)
+		(at 167.64 266.7 0)
 		(unit 1)
 		(body_style 1)
@@
 		(dnp no)
 		(property "Reference" "#PWR0224"
-			(at 209.55 273.05 0)
+			(at 167.64 273.05 0)
 			(hide yes)
 			(show_name no)
@@
 		)
 		(property "Value" "GND"
-			(at 209.55 271.78 0)
+			(at 167.64 271.78 0)
 			(hide yes)
 			(show_name no)
@@
 		)
 		(property "Footprint" ""
-			(at 209.55 266.7 0)
+			(at 167.64 266.7 0)
 			(hide yes)
 			(show_name no)
@@
 		)
 		(property "Datasheet" ""
-			(at 209.55 266.7 0)
+			(at 167.64 266.7 0)
 			(hide yes)
 			(show_name no)
@@
 		)
 		(property "Description" "Power symbol creates a global label with name \"GND\" , ground"
-			(at 209.55 266.7 0)
+			(at 167.64 266.7 0)
 			(hide yes)
 			(show_name no)
@@
 	(symbol
 		(lib_id "power:GND")
-		(at 85.09 200.66 0)
+		(at 201.93 256.54 0)
 		(unit 1)
 		(body_style 1)
@@
 		(dnp no)
 		(property "Reference" "#PWR0248"
-			(at 85.09 207.01 0)
+			(at 201.93 262.89 0)
 			(hide yes)
 			(show_name no)
@@
 		)
 		(property "Value" "GND"
-			(at 85.09 205.74 0)
+			(at 201.93 261.62 0)
 			(hide yes)
 			(show_name no)
@@
 		)
 		(property "Footprint" ""
-			(at 85.09 200.66 0)
+			(at 201.93 256.54 0)
 			(hide yes)
 			(show_name no)
@@
 		)
 		(property "Datasheet" ""
-			(at 85.09 200.66 0)
+			(at 201.93 256.54 0)
 			(hide yes)
 			(show_name no)
@@
 		)
 		(property "Description" "Power symbol creates a global label with name \"GND\" , ground"
-			(at 85.09 200.66 0)
+			(at 201.93 256.54 0)
 			(hide yes)
 			(show_name no)

Commit message: input analog board pcb
Parts:
- added R141, R142: 10k, Resistor_SMD:R_0603_1608Metric, symbol Device:R_US
- added R143, R144: 14.0k, Resistor_SMD:R_0603_1608Metric, symbol Device:R_US
- C101: LCSC (none) -> C282071
- C102, C103, C104, C105, C106, C107: footprint Capacitor_SMD:C_0603_1608Metric -> Capacitor_SMD:C_1206_3216Metric; LCSC (none) -> C527278
- C109: LCSC (none) -> C105620
- C110: footprint Capacitor_SMD:C_0603_1608Metric -> Capacitor_SMD:C_0805_2012Metric; LCSC (none) -> C107103
- C120, C121, C122, C123, C124, C125, TH101, TH102, TH103, U8, U9: LCSC (none) -> dnp
- R121, R127: value 140k -> 130k
- R124, R125: value 34.0k -> 20k; Note 1% -> 0.1% thin film
- U10, U14: LCSC (none) -> C2057264
Connections:
- net HMF_F_CV: now also R143.2; no longer R124.2
- net at R128.2, R129.1, TH102.1: now also R142.2; no longer R127.2
- net at R122.2, R123.1, TH101.1: now also R141.2; no longer R121.2
- net at C121.1, U11.2 (-): now also R144.2; no longer R125.2
- new net: R124.2, R143.1
- new net: R127.2, R142.1
- new net: R121.2, R141.1
- new net: R125.2, R144.1
Other:
- moved on the sheet: R121, R124, R125, R127
