File: PCB_CAD/Bucket/Analog/EQ/lf_hf.kicad_sch (KiCad schematic)
At the start: 113 parts, among them U12 SSI2164, U13 AS2180, U14 OPA1679, U15 OPA1679, U16 OPA1679, U17 OPA4197, U18 ADG1434, U19 AS2180

Commit message: getting ready to upgrade mx file
Parts:
- C201, C202, C203, C204, C205, C206, C207, C208: footprint Capacitor_SMD:C_0603_1608Metric -> Capacitor_THT:C_Rect_L7.2mm_W2.5mm_P5.00mm
Other:
- note added: "Boost/Cut, Shelf/Bell Sel"
- note removed: "Boost/Cut + Shelf/Bell Select"
- note removed: "Power Supply Decoupling"
- moved on the sheet: C201, C202, C203, C204, C205, C206, C207, C208, C209, C210, C211, C212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

Commit message: input analog board pcb
Parts:
- added R266, R267: 10k, Resistor_SMD:R_0603_1608Metric, symbol Device:R_US
- added R268, R269, R270, R271: 14.0k, Resistor_SMD:R_0603_1608Metric, symbol Device:R_US
- added R272, R273, R274, R275: 20k, Resistor_SMD:R_0603_1608Metric, symbol Device:R_US
- C201, C202, C203, C204, C205, C206, C207, C208, TH201, TH202, TH203, TH204, U12, U13, U19: LCSC (none) -> dnp
- C209, C214: LCSC (none) -> C282071
- C210, C212, C215, C217: footprint Capacitor_SMD:C_0603_1608Metric -> Capacitor_SMD:C_1206_3216Metric; LCSC (none) -> C527278
- C211, C213: footprint Capacitor_SMD:C_0603_1608Metric -> Capacitor_THT:C_Rect_L7.2mm_W2.5mm_P5.00mm; LCSC (none) -> dnp
- C216, C218: LCSC (none) -> C107050
- C219, C222: footprint Capacitor_SMD:C_0603_1608Metric -> Capacitor_SMD:C_0805_2012Metric; LCSC (none) -> C107103
- C220: LCSC (none) -> C105620
- C223: LCSC (none) -> C105622
- R201, R205, R213, R217: value 34.0k -> 20k; Note 1% -> 0.1% thin film
- R202, R214: value 140k -> 130k
- R250, R256: value 20.0k -> 20k
- R257, R259, R261, R263: value 2.2k -> 10k; Note (none) -> 0.1% thin film
- R258, R260, R262, R264: value 120k -> 100k
- U14, U15, U16: LCSC (none) -> C2057264
- U18: LCSC (none) -> C408906
Connections:
- net GND: now also R272.2, R273.2, R274.2, R275.2; no longer R258.2, R260.2, R262.2, R264.2
- net HF_F_CV: now also R270.2; no longer R213.2
- net LF_F_CV: now also R268.2; no longer R201.2
- net at R203.2, R206.1, TH201.1: now also R266.2; no longer R202.2
- net at R215.2, R218.1, TH203.1: now also R267.2; no longer R214.2
- net at C202.1, U17.2 (-): now also R269.2; no longer R205.2
- net at C206.1, U17.9 (-): now also R271.2; no longer R217.2
- new net: R264.2, R275.1
- new net: R214.2, R267.1
- new net: R213.2, R270.1
- new net: R202.2, R266.1
- new net: R258.2, R272.1
- new net: R205.2, R269.1
- new net: R262.2, R274.1
- new net: R260.2, R273.1
- new net: R201.2, R268.1
- new net: R217.2, R271.1
Other:
- moved on the sheet: R201, R202, R205, R213, R214, R217
