File: PCB_CAD/Bucket/Analog/INPUT/INPUT.kicad_pcb (KiCad board)
At the start: 4 copper layers, 36 x 100 mm, 95 parts, among them K1 G6K-2F-Y DC12, Q1 2N7002, Q2 2N7002, U1 INA849, U2 AQY210EHAX, U3 INA137, U4 OPA1679, U5 ADG1434, U6 AS2180, U7 OPA4197, U8 ADR5041

Commit message: pcb
Parts:
- added C33: 47u 63V, Capacitor_SMD:CP_Elec_6.3x7.7, F.Cu at (130.7, -13.9)
- added J1: Logic_CV, Connector_PinHeader_2.54mm:PinHeader_1x08_P2.54mm_Vertical, F.Cu at (100.4, -15.2)
- added J2: CV, Connector_PinHeader_2.54mm:PinHeader_1x02_P2.54mm_Vertical, F.Cu at (105.0, -15.2)
- added J3: AUDIO_IO, Connector_PinHeader_2.54mm:PinHeader_1x10_P2.54mm_Vertical, F.Cu at (56.8, 145.5)
- added J4: POWER, Connector_PinHeader_2.54mm:PinHeader_1x04_P2.54mm_Vertical, F.Cu at (117.0, -16.2)
- moved C17 274.8 mm to (401.9, 66.6)
- moved C18 274.8 mm to (401.9, 70.7)
- moved R39 274.8 mm to (411.6, 40.7)
- moved R40 274.8 mm to (411.6, 43.2)
- moved R41 274.8 mm to (411.6, 45.8)
- moved R42 274.8 mm to (411.6, 48.3)
- moved R44 274.8 mm to (411.6, 53.3)
- moved TH1 274.8 mm to (391.6, 82.9)
- moved R43 274.8 mm to (411.6, 50.8)
- moved C13 262.3 mm to (376.8, 8.40)
- moved C16 262.3 mm to (376.8, 11.4)
- moved U7 259.8 mm to (394.0, 57.2)
- moved R38 257.5 mm to (392.1, 25.5)
- moved U6 257.5 mm to (385.9, 10.5)
- moved C14 256.7 mm to (366.6, 19.9)
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
Commit message: working on softwareee
Parts:
- J1, J2, J3, J4: moved to B.Cu
- moved R42 355.0 mm to (58.5, 85.0), turned to -90 degrees
- moved R43 352.9 mm to (60.3, 84.7), turned to -90 degrees
- moved R44 351.4 mm to (61.6, 84.7), turned to 90 degrees
- moved R39 351.0 mm to (61.8, 69.3), turned to 90 degrees
- moved R40 348.9 mm to (63.7, 69.3), turned to 90 degrees
- moved R41 345.7 mm to (66.7, 68.7), turned to 90 degrees
- moved C17 344.8 mm to (57.4, 81.7), turned to 90 degrees
- moved C18 333.4 mm to (68.7, 82.1), turned to 180 degrees
- moved R35 331.9 mm to (56.2, 85.1), turned to -90 degrees
- moved U7 324.5 mm to (70.0, 74.7), turned to 90 degrees
- moved R38 323.1 mm to (75.4, 89.6), turned to -90 degrees
- moved C14 318.0 mm to (56.2, 89.0), turned to -90 degrees
- moved R37 317.1 mm to (70.3, 84.7)
- moved R33 314.4 mm to (75.3, 86.3), turned to 90 degrees
- moved C16 313.7 mm to (73.0, 89.9), turned to 90 degrees
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Routing:
- added copper zone on B.Cu, net GND
- added copper zone on F.Cu, net GND
- added copper zone on In1.Cu, net GND
- added copper zone on In2.Cu, net GND
Other:
- board size 36 x 100 mm -> 36 x 95 mm

Commit message: input analog board pcb
Parts:
- added H1: MountingScrew, MountingHole:MountingHole_2.2mm_M2, F.Cu at (54.0, 60.5)
- added H2: MountingScrew, MountingHole:MountingHole_2.2mm_M2, F.Cu at (61.0, 142.2)
- added H3: MountingScrew, MountingHole:MountingHole_2.2mm_M2, F.Cu at (78.7, 97.2)
- added JP1: LINE_ONLY, Jumper:SolderJumper-2_P1.3mm_Open_TrianglePad1.0x1.5mm, F.Cu at (62.1, 91.9)
- added REF**: LayerMarker_4_6.35x2.54mm_TextH1mm_P1.27mm_LowerMirrored, Symbol:LayerMarker_4_6.35x2.54mm_TextH1mm_P1.27mm_LowerMirrored, F.Cu at (64.2, 59.5)
- R1, R2: footprint Resistor_SMD:R_0603_1608Metric -> Resistor_SMD:R_2010_5025Metric
- U1: footprint Package_SO:MSOP-8-1EP_3x3mm_P0.65mm_EP1.68x1.88mm_ThermalVias -> Package_SO:MSOP-8_3x3mm_P0.65mm
- U3, U6: footprint Package_SO:SOIC-8-1EP_3.9x4.9mm_P1.27mm_EP2.29x3mm_ThermalVias -> Package_SO:SOIC-8_3.9x4.9mm_P1.27mm
- moved C6 37.8 mm to (56.5, 132.7), turned to -90 degrees
- moved R13 36.9 mm to (57.0, 88.7), turned to 90 degrees
- moved C22 36.8 mm to (66.9, 124.7), turned to 0 degrees
- moved C7 36.1 mm to (56.5, 129.3), turned to -90 degrees
- moved R5 36.1 mm to (83.4, 110.0), turned to 0 degrees
- moved C14 35.5 mm to (77.9, 60.9), turned to 180 degrees
- moved Q2 34.1 mm to (53.5, 87.4), turned to 90 degrees
- moved R3 32.9 mm to (83.5, 112.5), turned to 180 degrees
- moved R35 32.2 mm to (80.5, 64.0), turned to 90 degrees
- moved R4 32.2 mm to (77.7, 111.0)
- moved R38 31.8 mm to (54.5, 113.5), turned to 0 degrees
- moved C23 31.7 mm to (58.8, 129.4), turned to -90 degrees
- moved U2 31.1 mm to (62.5, 82.0)
- moved U3 30.9 mm to (61.3, 124.9)
- moved R15 29.4 mm to (54.0, 81.0), turned to 180 degrees
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Routing:
- net -15V: track 0.00 -> 221.7 mm, vias 0 -> 7
- net +15V: track 0.00 -> 177.9 mm, vias 0 -> 9
- net /P48_BUS: track 0.00 -> 77.3 mm, vias 0 -> 2
- net /GAIN_CV: track 0.00 -> 57.6 mm, vias 0 -> 2
- net /TO_VCA: track 0.00 -> 52.7 mm, vias 0 -> 2
- net INPUT_OUT: track 0.00 -> 46.5 mm, vias 0 -> 4
- net /LINE_OUT: track 0.00 -> 44.5 mm, vias 0 -> 4
- net Net-(C3--): track 0.00 -> 43.3 mm, vias 0 -> 2
- net Net-(C11-Pad2): track 0.00 -> 41.9 mm, vias 0 -> 2
- net Net-(R40-Pad2): track 0.00 -> 37.9 mm, vias 0 -> 2
- net /MIC_OUT: track 0.00 -> 37.2 mm, vias 0 -> 4
- net +48V: track 0.00 -> 34.2 mm
- net Net-(C4--): track 0.00 -> 31.2 mm, vias 0 -> 2
- net Net-(U7A--): track 0.00 -> 29.8 mm, vias 0 -> 2
- net PHASE_LCV: track 0.00 -> 29.3 mm
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Other:
- board text added: "+48 +15 GND -15"
- board text added: "48V SWITCH MIC SWITCH LINE SWITCH HI-Z SWITCH PHASE FLIP HPF IN PAD IN GND"
- board text added: "AUDIO I/O"
- board text added: "AUDIO OUT GND GND HI-Z IN GND LINE IN - LINE IN + GND MIC IN - MIC IN +"
- board text added: "CV"
- board text added: "Channel INPUT Card"
- board text added: "DIGILOG"
- board text added: "IN GAIN GND"
- board text added: "LINE ONLY"
- board text added: "POWER"
- board text added: "REV 0 2026 RoHS"
- board text added: "SWITCH CV"
- board text added: "Skylar Evelyn Denno"
