File: PCB_CAD/Bucket/Analog/INPUT/INPUT.kicad_sch (KiCad schematic)
At the start: 95 parts, among them K1 G6K-2F-Y DC12, Q1 2N7002, Q2 2N7002, U1 INA849, U2 AQY210EHAX, U3 INA137, U4 OPA1679, U5 ADG1434, U6 AS2180, U7 OPA4197, U8 ADR5041

Commit message: getting ready to upgrade mx file
Parts:
- C1, C2: value 470p 100V C0G -> 470p C0G; footprint Capacitor_SMD:C_0805_2012Metric -> Capacitor_SMD:C_0603_1608Metric; LCSC (none) -> C326973
- C10, C15: LCSC (none) -> C105620
- C11, C12, C9: value 100n C0G -> 100n FILM; footprint Capacitor_SMD:C_1206_3216Metric -> Capacitor_SMD:C_1812_4532Metric; LCSC (none) -> C569829
- C13, C16: footprint Capacitor_SMD:CP_Elec_6.3x5.4_Nichicon -> Capacitor_SMD:C_0805_2012Metric; LCSC (none) -> C1713
- C14: value 2.2n C0G -> 2.2n FILM; LCSC (none) -> C178417
- C17, C18: value 22n C0G -> 22n FILM; footprint Capacitor_SMD:C_0603_1608Metric -> Capacitor_THT:C_Rect_L7.2mm_W2.5mm_P5.00mm; LCSC (none) -> _DNP_
- C19, C20, C21, C22, C23, C24, C25, C26, C27, C28, C29, C30: LCSC (none) -> C1590
- C3, C4: footprint Capacitor_SMD:CP_Elec_8x10 -> Capacitor_SMD:CP_Elec_6.3x7.7; LCSC (none) -> C48971005
- C31, C32: LCSC (none) -> C21397
- C5: footprint Capacitor_SMD:CP_Elec_10x10 -> Capacitor_SMD:CP_Elec_10x10.5; LCSC (none) -> C51953411
- C6, C7: LCSC (none) -> C326973
- C8: LCSC (none) -> C14665
- D1, D2, D3, D4: LCSC (none) -> C2481
- D5: LCSC (none) -> C2099
- D6: LCSC (none) -> C145516
- K1: LCSC (none) -> C397194
- Q1, Q2: LCSC (none) -> C8545
- R1, R2: footprint Resistor_SMD:R_2010_5025Metric -> Resistor_SMD:R_0603_1608Metric; LCSC (none) -> C861538
- R10: LCSC (none) -> C351654
- R11, R13, R38, R39: LCSC (none) -> C122538
- R12: LCSC (none) -> C351650
- R14, R35: LCSC (none) -> C122970
- R15: LCSC (none) -> C25654
- R16: LCSC (none) -> C110776
- R17, R20: LCSC (none) -> C234360
- R18, R19: value 10k -> 10k 0.1%; LCSC (none) -> C95204
- R21, R22: LCSC (none) -> C95204
- R23: LCSC (none) -> C861102
- R24: LCSC (none) -> C667077
- R25, R26, R27, R28: LCSC (none) -> C309092
- R29, R30, R31, R32: LCSC (none) -> C136959
- R3, R4: LCSC (none) -> C137732
- R33, R36: LCSC (none) -> C190611
- R34: LCSC (none) -> C122969
- R37: LCSC (none) -> C218045
- R40: LCSC (none) -> C217893
- R41: footprint Resistor_SMD:R_0603_1608Metric -> Resistor_SMD:R_0402_1005Metric; LCSC (none) -> C852585
- R42: LCSC (none) -> C861369
- R43, R44: footprint Resistor_SMD:R_0603_1608Metric -> Resistor_SMD:R_0402_1005Metric; LCSC (none) -> C705633
- R45: footprint Resistor_SMD:R_0603_1608Metric -> Resistor_SMD:R_0402_1005Metric; LCSC (none) -> C36157922
- R5: LCSC (none) -> C318130
- R6, R7: LCSC (none) -> C217691
- R8: footprint Resistor_SMD:R_0603_1608Metric -> Resistor_SMD:R_0402_1005Metric; LCSC (none) -> C852867
- R9: LCSC (none) -> C861514
- TH1, U6: LCSC (none) -> _DNP_
- U1: footprint Package_SO:SOIC-8_3.9x4.9mm_P1.27mm -> Package_SO:MSOP-8-1EP_3x3mm_P0.65mm_EP1.68x1.88mm_ThermalVias; LCSC (none) -> C4370731
- U2: LCSC (none) -> C24728
- U3: footprint Package_SO:SOIC-8_3.9x4.9mm_P1.27mm -> Package_SO:SOIC-8-1EP_3.9x4.9mm_P1.27mm_EP2.29x3mm_ThermalVias; LCSC (none) -> C2652878
- U4: footprint Package_SO:SOIC-14_3.9x8.7mm_P1.27mm -> Package_SO:TSSOP-14_4.4x5mm_P0.65mm; LCSC (none) -> C2057264
- U5: LCSC (none) -> C408906
- U7: LCSC (none) -> C2058532
- U8: LCSC (none) -> C2686108
Other:
- moved on the sheet: C1, C11, C12, C13, C14, C15, C16, C17, C18, C19, C2, C20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

Commit message: pcb
Parts:
- added C33: 47u 63V, Capacitor_SMD:CP_Elec_6.3x7.7, symbol Device:C_Polarized
- added J1: Logic_CV, Connector_PinHeader_2.54mm:PinHeader_1x08_P2.54mm_Vertical, symbol PCM_4ms_Connector:Conn_01x08
- added J2: CV, Connector_PinHeader_2.54mm:PinHeader_1x02_P2.54mm_Vertical, symbol PCM_4ms_Connector:Conn_01x02
- added J3: AUDIO_IO, Connector_PinHeader_2.54mm:PinHeader_1x10_P2.54mm_Vertical, symbol Connector_Generic:Conn_01x10
- added J4: POWER, Connector_PinHeader_2.54mm:PinHeader_1x04_P2.54mm_Vertical, symbol Connector_Generic:Conn_01x04
Connections:
- net +15V: now also J4.2 (Pin_2)
- net +48V: now also C33.1 (+), J4.1 (Pin_1)
- net -15V: now also J4.4 (Pin_4)
- net CV_IN_GAIN: now also J2.1 (Pin_1)
- net GND: now also C33.2 (-), J1.8 (Pin_8), J2.2 (Pin_2), J3.3 (Pin_3), J3.6 (Pin_6), J3.8 (Pin_8), J3.9 (Pin_9), J4.3 (Pin_3)
- net HIZ_IN: now also J3.7 (Pin_7)
- net HIZ_SEL_LCV: now also J1.4 (Pin_4)
- net HPF_LCV: now also J1.6 (Pin_6)
- net INPUT_OUT: now also J3.10 (Pin_10)
- net LINE_COLD: now also J3.5 (Pin_5)
- net LINE_HOT: now also J3.4 (Pin_4)
- net LINE_SEL_LCV: now also J1.3 (Pin_3)
- net MIC_COLD: now also J3.2 (Pin_2)
- net MIC_HOT: now also J3.1 (Pin_1)
- net MIC_SEL_LCV: now also J1.2 (Pin_2)
- net P48_LCV: now also J1.1 (Pin_1)
- net PAD_LCV: now also J1.7 (Pin_7)
- net PHASE_LCV: now also J1.5 (Pin_5)

Commit message: input analog board pcb
Parts:
- added H1, H2, H3: MountingScrew, MountingHole:MountingHole_2.2mm_M2, symbol Auxiliary_Items:MountingScrew
- added JP1: LINE_ONLY, Jumper:SolderJumper-2_P1.3mm_Open_TrianglePad1.0x1.5mm, symbol Jumper:SolderJumper_2_Open
- R1, R2: footprint Resistor_SMD:R_0603_1608Metric -> Resistor_SMD:R_2010_5025Metric; LCSC C861538 -> C54102447
- U1: footprint Package_SO:MSOP-8-1EP_3x3mm_P0.65mm_EP1.68x1.88mm_ThermalVias -> Package_SO:MSOP-8_3x3mm_P0.65mm
- U3, U6: footprint Package_SO:SOIC-8-1EP_3.9x4.9mm_P1.27mm_EP2.29x3mm_ThermalVias -> Package_SO:SOIC-8_3.9x4.9mm_P1.27mm
Connections:
- net LINE_OUT: now also JP1.2 (B)
- net TO_VCA: now also JP1.1 (A)
