File: PCB_CAD/Bucket/BUCKET_ROUTING/BUCKET_ROUTING.kicad_pcb (KiCad board)
At the start: 4 copper layers, 146 x 435 mm, 42 parts, among them J1 POWER, J10 MIX_BUS, J11 POWER, J12 CV, J13 AUD_IN, J14 INSERT, J15 MIX_BUS, J16 POWER, J17 CV, J18 AUD_IN, J19 INSERT, J2 CV, J20 MIX_BUS, J3 AUD_IN, J4 INSERT, J5 MIX_BUS, J6 POWER, J7 CV, J8 AUD_IN, J9 INSERT, P1 POWER

Commit message: input analog board pcb
Parts:
- removed H1, H19, H2, H20, H21, H3, H4, H5, H6: MountingScrew, MountingHole:MountingHole_3.2mm_M3
- moved H11 8.54 mm to (60.7, 425.5)
- moved H14 8.54 mm to (97.2, 425.5)
- moved H17 8.54 mm to (133.5, 425.5)
- moved H8 8.54 mm to (24.4, 425.5)
- moved J1 8.54 mm to (44.9, 352.5)
- moved J11 8.54 mm to (117.8, 352.5)
- moved J12 8.54 mm to (106.0, 379.5)
- moved J13 8.54 mm to (113.3, 419.0)
- moved J14 8.54 mm to (113.5, 428.5)
- moved J16 8.54 mm to (154.1, 352.5)
- moved J17 8.54 mm to (142.3, 379.5)
- moved J18 8.54 mm to (149.6, 419.0)
- moved J19 8.54 mm to (149.8, 428.5)
- moved J2 8.54 mm to (33.1, 379.5)
- moved J3 8.54 mm to (40.4, 419.0)
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