File: PCB_CAD/Bucket/BUCKET_ROUTING/BUCKET_ROUTING.kicad_sch (KiCad schematic)
At the start: 42 parts, among them J1 POWER, J10 MIX_BUS, J11 POWER, J12 CV, J13 AUD_IN, J14 INSERT, J15 MIX_BUS, J16 POWER, J17 CV, J18 AUD_IN, J19 INSERT, J2 CV, J20 MIX_BUS, J3 AUD_IN, J4 INSERT, J5 MIX_BUS, J6 POWER, J7 CV, J8 AUD_IN, J9 INSERT, P1 POWER

Commit message: input analog board pcb
Parts:
- removed H1, H19, H2, H20, H21, H3, H4, H5, H6: MountingScrew, MountingHole:MountingHole_3.2mm_M3, symbol Auxiliary_Items:MountingScrew
- added H19, H20, H21: MountingHole, MountingHole:MountingHole_2.2mm_M2, symbol Mechanical:MountingHole
- added J21: LOGIC_CV, Connector_PinSocket_2.54mm:PinSocket_1x08_P2.54mm_Vertical, symbol Connector_Generic:Conn_01x08
- added J22: AUDIO, Connector_PinSocket_2.54mm:PinSocket_1x08_P2.54mm_Vertical, symbol Connector_Generic:Conn_01x10
- added J23: POWER, Connector_PinSocket_2.54mm:PinSocket_1x03_P2.54mm_Vertical, symbol Connector_Generic:Conn_01x04
- added J24: CV, Connector_PinSocket_2.54mm:PinSocket_1x03_P2.54mm_Vertical, symbol Connector_Generic:Conn_01x02
Other:
- moved on the sheet: J1, J10, J11, J12, J13, J14, J15, J16, J17, J18, J19, J2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
