File: PCB_CAD/01 Analog/INPUT/INPUT.kicad_pcb (KiCad board)
At the start: 4 copper layers, 36 x 95 mm, 105 parts, among them J1 Logic_CV, J2 CV, J3 AUDIO_IO, J4 POWER, K1 G6K-2F-Y DC12, Q1 2N7002, Q2 2N7002, U1 INA849, U2 AQY210EHAX, U3 INA137, U4 OPA1679, U5 ADG1434, U6 AS2180, U7 OPA4197, U8 ADR5041

Commit message: input board done
Parts:
- C13, C16: footprint Capacitor_SMD:C_0805_2012Metric -> Capacitor_SMD:CP_Elec_6.3x5.4_Nichicon
- R40: value 237k 0.1% -> 182k 0.1%
- R41: value 196k 0.1% -> 301k 0.1%
- R43: value 44.2k 0.1% -> 67.3k 0.1%
- U6: footprint Package_SO:SOIC-8_3.9x4.9mm_P1.27mm -> Connector_PinHeader_2.54mm:PinHeader_1x08_P2.54mm_Vertical
- moved H3 23.2 mm to (73.6, 74.6)
- moved C8 17.6 mm to (72.3, 108.3), turned to 180 degrees
- moved C9 11.6 mm to (73.7, 111.2), turned to 180 degrees
- moved U6 11.5 mm to (80.8, 60.3), turned to 0 degrees
- moved R17 10.6 mm to (69.2, 111.7)
- moved C13 9.97 mm to (73.2, 62.1), turned to 90 degrees
- moved R16 8.59 mm to (58.3, 115.1), turned to 0 degrees
- moved REF** 8.08 mm to (56.9, 62.9)
- moved C33 6.74 mm to (65.8, 62.1)
- moved R33 6.38 mm to (77.9, 61.6), turned to 90 degrees
- moved C28 6.17 mm to (77.2, 74.1), turned to 90 degrees
- moved R34 6.15 mm to (77.3, 70.0), turned to 90 degrees
- moved C14 6.00 mm to (83.8, 60.8), turned to 90 degrees
- moved D6 5.63 mm to (62.7, 116.8)
- moved C16 4.91 mm to (79.6, 97.6), turned to 90 degrees
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Routing:
- net /TO_VCA: track 52.7 -> 42.1 mm
- net HIZ_IN: track 3.26 -> 11.0 mm
- net GND: track 26.7 -> 20.0 mm, vias 46 -> 170
- net Net-(C8-Pad1): track 15.8 -> 22.2 mm, vias 0 -> 2
- net Net-(D6-K1A2): track 27.0 -> 22.4 mm, vias 2 -> 3
- net -15V: track 221.7 -> 225.0 mm, vias 7 -> 8
- net INPUT_OUT: track 46.5 -> 43.3 mm
- net Net-(C13-Pad2): track 3.09 -> 5.91 mm
- net Net-(U4D-+): track 22.7 -> 20.1 mm, vias 0 -> 2
- net Net-(C11-Pad2): track 41.9 -> 39.8 mm, vias 2 -> 4
- net +48V: track 34.2 -> 36.1 mm
- net Net-(C14-Pad1): track 3.15 -> 1.58 mm
- net Net-(U6--): track 3.88 -> 2.34 mm
- net Net-(U6-V-): track 4.69 -> 3.17 mm
- net Net-(C15-Pad2): track 6.72 -> 8.17 mm
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Other:
- board text added: "1"
- board text added: "2180"

Commit message: input board fr done
Parts:
- C1, C2: value 470p C0G -> 470p C0G 100V
- R10: footprint Resistor_SMD:R_0603_1608Metric -> Resistor_SMD:R_1206_3216Metric
- R14: value 100 -> 330; footprint Resistor_SMD:R_0603_1608Metric -> Resistor_SMD:R_1206_3216Metric
- R41: footprint Resistor_SMD:R_0402_1005Metric -> Resistor_SMD:R_0603_1608Metric
- R43: value 67.3k 0.1% -> 66.5k 0.1%
- moved R14 0.22 mm to (60.4, 64.3), turned to -90 degrees
Routing:
- net Net-(R14-Pad1): track 21.2 -> 23.3 mm
- net Net-(R40-Pad2): track 39.2 -> 37.3 mm
- net GND: track 20.0 -> 18.6 mm, vias 170 -> 171
- net Net-(C17-Pad1): track 25.9 -> 27.2 mm
- net /P48_BUS: track 77.3 -> 76.3 mm
- net +15V: track 178.8 -> 178.1 mm
- net CV_IN_GAIN: track 9.73 -> 10.3 mm
