File: PCB_CAD/01 Analog/INPUT/INPUT.kicad_sch (KiCad schematic)
At the start: 104 parts, among them J1 Logic_CV, J2 CV, J3 AUDIO_IO, J4 POWER, K1 G6K-2F-Y DC12, Q1 2N7002, Q2 2N7002, U1 INA849, U2 AQY210EHAX, U3 INA137, U4 OPA1679, U5 ADG1434, U6 AS2180, U7 OPA4197, U8 ADR5041

Commit message: more pcb work, fmc timing optimizations for displays, display driver tools
Parts:
- R40: value 237k 0.1% -> 182k 0.1%
- R41: value 196k 0.1% -> 301k 0.1%
- R43: value 44.2k 0.1% -> 67.3k 0.1%
Other:
- note added: "DAC 0 V = mute (-79 dB), 2.0475 V (code 4095) = +28 dB, 26 mdB/LSB. Drift +/-0.035 dB, 10-45 C. MFB fc 133 Hz."
- note removed: "DAC 0 V = mute (-79 dB), 4.095 V = +28 dB, 26 mdB/LSB. Drift +/-0.035 dB, 10-45 C. MFB fc 164 Hz."
Changed lines of the file:
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@@
 		)
 	)
-	(text "DAC 0 V = mute (-79 dB), 4.095 V = +28 dB, 26 mdB/LSB.\nDrift +/-0.035 dB, 10-45 C. MFB fc 164 Hz."
+	(text "DAC 0 V = mute (-79 dB), 2.0475 V (code 4095) = +28 dB, 26 mdB/LSB.\nDrift +/-0.035 dB, 10-45 C. MFB fc 133 Hz."
 		(exclude_from_sim no)
 		(at 131.318 188.214 0)
@@
 			)
 		)
-		(property "Value" "237k 0.1%"
+		(property "Value" "182k 0.1%"
 			(at 158.75 175.26 90)
 			(show_name no)
@@
 			)
 		)
-		(property "Value" "44.2k 0.1%"
+		(property "Value" "67.3k 0.1%"
 			(at 190.754 166.116 0)
 			(show_name no)
@@
 			)
 		)
-		(property "Value" "196k 0.1%"
+		(property "Value" "301k 0.1%"
 			(at 175.26 170.18 0)
 			(show_name no)

Commit message: input board done
Parts:
- C13, C16: footprint Capacitor_SMD:C_0805_2012Metric -> Capacitor_SMD:CP_Elec_6.3x5.4_Nichicon; LCSC C1713 -> C340735
- H1, H2, H3, J1, J2, J3, J4, JP1: LCSC (none) -> _DNP_
- R40: LCSC C217893 -> C861170
- R41: LCSC C852585 -> C2936623
- R43: LCSC C705633 -> C851084
- U6: footprint Package_SO:SOIC-8_3.9x4.9mm_P1.27mm -> Connector_PinHeader_2.54mm:PinHeader_1x08_P2.54mm_Vertical
Changed lines of the file:
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@@
 			)
 		)
+		(property "LCSC" "_DNP_"
+			(at 400.05 115.57 0)
+			(hide yes)
+			(show_name no)
+			(do_not_autoplace no)
+			(effects
+				(font
+					(size 1.27 1.27)
+				)
+			)
+		)
 		(pin "4"
 		)
@@
 			)
 		)
-		(property "Footprint" "Capacitor_SMD:C_0805_2012Metric"
+		(property "Footprint" "Capacitor_SMD:CP_Elec_6.3x5.4_Nichicon"
 			(at 337.82 151.13 0)
 			(hide yes)
@@
 			)
 		)
-		(property "LCSC" "C1713"
+		(property "LCSC" "C340735"
 			(at 337.82 151.13 90)
 			(hide yes)
@@
 			)
 		)
-		(property "Footprint" "Capacitor_SMD:C_0805_2012Metric"
+		(property "Footprint" "Capacitor_SMD:CP_Elec_6.3x5.4_Nichicon"
 			(at 259.08 148.59 0)
 			(hide yes)
@@
 			)
 		)
-		(property "LCSC" "C1713"
+		(property "LCSC" "C340735"
 			(at 259.08 148.59 90)
 			(hide yes)
@@
 			)
 		)
+		(property "LCSC" "_DNP_"
+			(at 400.05 64.77 0)
+			(hide yes)
+			(show_name no)
+			(do_not_autoplace no)
+			(effects
+				(font
+					(size 1.27 1.27)
+				)
+			)
+		)
 		(pin "4"
 		)
@@
 			)
 		)
-		(property "LCSC" "C217893"
+		(property "LCSC" "C861170"
 			(at 158.75 172.72 90)
 			(hide yes)
@@
 			)
 		)
+		(property "LCSC" "_DNP_"
+			(at 400.05 146.05 0)
+			(hide yes)
+			(show_name no)
+			(do_not_autoplace no)
+			(effects
+				(font
+					(size 1.27 1.27)
+				)
+			)
+		)
 		(pin "4"
 		)
@@
 			)
 		)
-		(property "LCSC" "C705633"
+		(property "LCSC" "C851084"
 			(at 191.77 168.91 0)
 			(hide yes)
@@
 			)
 		)
+		(property "LCSC" "_DNP_"
+			(at 182.88 254 0)
+			(hide yes)
+			(show_name no)
+			(do_not_autoplace no)
+			(effects
+				(font
+					(size 1.27 1.27)
+				)
+			)
+		)
 		(instances
 			(project "INPUT"
@@
 			)
 		)
-		(property "Footprint" "Package_SO:SOIC-8_3.9x4.9mm_P1.27mm"
+		(property "Footprint" "Connector_PinHeader_2.54mm:PinHeader_1x08_P2.54mm_Vertical"
 			(at 283.21 148.59 0)
 			(hide yes)
@@
 			)
 		)
+		(property "LCSC" "_DNP_"
+			(at 176.53 254 0)
+			(hide yes)
+			(show_name no)
+			(do_not_autoplace no)
+			(effects
+				(font
+					(size 1.27 1.27)
+				)
+			)
+		)
 		(instances
 			(project "INPUT"
@@
 			)
 		)
+		(property "LCSC" "_DNP_"
+			(at 400.05 90.17 0)
+			(hide yes)
+			(show_name no)
+			(do_not_autoplace no)
+			(effects
+				(font
+					(size 1.27 1.27)
+				)
+			)
+		)
 		(pin "2"
 		)
@@
 			)
 		)
+		(property "LCSC" "_DNP_"
+			(at 381 31.75 90)
+			(hide yes)
+			(show_name no)
+			(do_not_autoplace no)
+			(effects
+				(font
+					(size 1.27 1.27)
+				)
+			)
+		)
 		(pin "1"
 		)
@@
 			)
 		)
-		(property "LCSC" "C852585"
+		(property "LCSC" "C2936623"
 			(at 177.8 168.91 0)
 			(hide yes)
@@
 			(at 189.23 254 0)
 			(hide yes)
+			(show_name no)
+			(do_not_autoplace no)
+			(effects
+				(font
+					(size 1.27 1.27)
+				)
+			)
+		)
+		(property "LCSC" "_DNP_"
+			(at 189.23 254 0)
+			(hide yes)

Commit message: input board fr done
Parts:
- C1, C2: value 470p C0G -> 470p C0G 100V
- R10: footprint Resistor_SMD:R_0603_1608Metric -> Resistor_SMD:R_1206_3216Metric; LCSC C351654 -> C17930
- R14: value 100 -> 330; footprint Resistor_SMD:R_0603_1608Metric -> Resistor_SMD:R_1206_3216Metric; LCSC C122970 -> C17930
- R41: footprint Resistor_SMD:R_0402_1005Metric -> Resistor_SMD:R_0603_1608Metric; LCSC C2936623 -> C861309
- R43: value 67.3k 0.1% -> 66.5k 0.1%
Changed lines of the file:
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@@
 			)
 		)
-		(property "Value" "470p C0G"
+		(property "Value" "470p C0G 100V"
 			(at 264.16 78.74 0)
 			(show_name no)
@@
 			)
 		)
-		(property "Value" "100"
+		(property "Value" "330"
 			(at 85.09 227.33 90)
 			(show_name no)
@@
 			)
 		)
-		(property "Footprint" "Resistor_SMD:R_0603_1608Metric"
+		(property "Footprint" "Resistor_SMD:R_1206_3216Metric"
 			(at 85.09 224.79 0)
 			(hide yes)
@@
 			)
 		)
-		(property "LCSC" "C122970"
+		(property "LCSC" "C17930"
 			(at 85.09 224.79 90)
 			(hide yes)
@@
 			)
 		)
-		(property "Value" "470p C0G"
+		(property "Value" "470p C0G 100V"
 			(at 264.16 53.34 0)
 			(show_name no)
@@
 			)
 		)
-		(property "Footprint" "Resistor_SMD:R_0603_1608Metric"
+		(property "Footprint" "Resistor_SMD:R_1206_3216Metric"
 			(at 60.96 38.1 0)
 			(hide yes)
@@
 			)
 		)
-		(property "LCSC" "C351654"
+		(property "LCSC" "C17930"
 			(at 60.96 38.1 0)
 			(hide yes)
@@
 			)
 		)
-		(property "Value" "67.3k 0.1%"
+		(property "Value" "66.5k 0.1%"
 			(at 190.754 166.116 0)
 			(show_name no)
@@
 			)
 		)
-		(property "Footprint" "Resistor_SMD:R_0402_1005Metric"
+		(property "Footprint" "Resistor_SMD:R_0603_1608Metric"
 			(at 177.8 168.91 0)
 			(hide yes)
@@
 			)
 		)
-		(property "LCSC" "C2936623"
+		(property "LCSC" "C861309"
 			(at 177.8 168.91 0)
 			(hide yes)
