File: PCB_CAD/02 Bucket/BUCKET_CONTROLS/encoders_debounce_1.kicad_sch (KiCad schematic)
At the start: 100 parts, among them SW101 C1_K0, SW102 C1_K1, SW103 C1_K2, SW104 C1_K3, SW105 C1_K4, SW106 C1_K5, SW107 C1_K6, SW108 C1_K7, SW109 C1_K8, SW110 C1_K9

Commit message: pcbs omg when does it end
Parts:
- SW101, SW102, SW103, SW104, SW105, SW106, SW107, SW108, SW109, SW110: footprint My Footprints:EC11_miniboard_castellated -> My Footprints:EC11J0924411; symbol My Symbols:EC11_Rotary_Encoder_Board -> My Symbols:EC11_Rotary_Encoder
Connections:
- net GND: now also SW101.C (Pin_2), SW101.D (Pin_4), SW102.C (Pin_2), SW102.D (Pin_4), SW103.C (Pin_2), SW103.D (Pin_4), SW104.C (Pin_2), SW104.D (Pin_4), SW105.C (Pin_2), SW105.D (Pin_4), SW106.C (Pin_2), SW106.D (Pin_4), SW107.C (Pin_2), SW107.D (Pin_4), SW108.C (Pin_2), SW108.D (Pin_4), SW109.C (Pin_2), SW109.D (Pin_4), SW110.C (Pin_2), SW110.D (Pin_4)
Changed lines of the file:
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@@
 	)
 	(symbol
-		(lib_id "My Symbols:EC11_Rotary_Encoder_Board")
+		(lib_id "My Symbols:EC11_Rotary_Encoder")
 		(at 81.28 147.32 180)
 		(unit 1)
@@
 			)
 		)
-		(property "Footprint" "My Footprints:EC11_miniboard_castellated"
+		(property "Footprint" "My Footprints:EC11J0924411"
 			(at 81.28 147.32 0)
 			(hide yes)
@@
 		(pin "B"
 		)
+		(pin "C"
+		)
+		(pin "D"
+		)
 		(instances
 			(project "bucket_controls"
@@
 	)
 	(symbol
-		(lib_id "My Symbols:EC11_Rotary_Encoder_Board")
+		(lib_id "My Symbols:EC11_Rotary_Encoder")
 		(at 81.28 45.72 180)
 		(unit 1)
@@
 			)
 		)
-		(property "Footprint" "My Footprints:EC11_miniboard_castellated"
+		(property "Footprint" "My Footprints:EC11J0924411"
 			(at 81.28 45.72 0)
 			(hide yes)
@@
 		(pin "B"
 		)
+		(pin "C"
+		)
+		(pin "D"
+		)
 		(instances
 			(project "bucket_controls"
@@
 	)
 	(symbol
-		(lib_id "My Symbols:EC11_Rotary_Encoder_Board")
+		(lib_id "My Symbols:EC11_Rotary_Encoder")
 		(at 81.28 96.52 180)
 		(unit 1)
@@
 			)
 		)
-		(property "Footprint" "My Footprints:EC11_miniboard_castellated"
+		(property "Footprint" "My Footprints:EC11J0924411"
 			(at 81.28 96.52 0)
 			(hide yes)
@@
 		(pin "B"
 		)
+		(pin "C"
+		)
+		(pin "D"
+		)
 		(instances
 			(project "bucket_controls"
@@
 	)
 	(symbol
-		(lib_id "My Symbols:EC11_Rotary_Encoder_Board")
+		(lib_id "My Symbols:EC11_Rotary_Encoder")
 		(at 201.93 147.32 180)
 		(unit 1)
@@
 			)
 		)
-		(property "Footprint" "My Footprints:EC11_miniboard_castellated"
+		(property "Footprint" "My Footprints:EC11J0924411"
 			(at 201.93 147.32 0)
 			(hide yes)
@@
 		(pin "B"
 		)
+		(pin "C"
+		)
+		(pin "D"
+		)
 		(instances
 			(project "bucket_controls"
@@
 	)
 	(symbol
-		(lib_id "My Symbols:EC11_Rotary_Encoder_Board")
+		(lib_id "My Symbols:EC11_Rotary_Encoder")
 		(at 201.93 96.52 180)
 		(unit 1)
@@
 			)
 		)
-		(property "Footprint" "My Footprints:EC11_miniboard_castellated"
+		(property "Footprint" "My Footprints:EC11J0924411"
 			(at 201.93 96.52 0)
 			(hide yes)
@@
 		(pin "B"
 		)
+		(pin "D"
+		)
+		(pin "C"
+		)
 		(instances
 			(project "bucket_controls"
@@
 	)
 	(symbol
-		(lib_id "My Symbols:EC11_Rotary_Encoder_Board")
+		(lib_id "My Symbols:EC11_Rotary_Encoder")
 		(at 201.93 248.92 180)
 		(unit 1)
@@
 			)
 		)
-		(property "Footprint" "My Footprints:EC11_miniboard_castellated"
+		(property "Footprint" "My Footprints:EC11J0924411"
 			(at 201.93 248.92 0)
 			(hide yes)
@@
 		(pin "B"
 		)
+		(pin "C"
+		)
+		(pin "D"
+		)
 		(instances
 			(project "bucket_controls"
@@
 	)
 	(symbol
-		(lib_id "My Symbols:EC11_Rotary_Encoder_Board")
+		(lib_id "My Symbols:EC11_Rotary_Encoder")
 		(at 201.93 45.72 180)
 		(unit 1)
@@
 			)
 		)
-		(property "Footprint" "My Footprints:EC11_miniboard_castellated"
+		(property "Footprint" "My Footprints:EC11J0924411"
 			(at 201.93 45.72 0)
 			(hide yes)
@@
 		(pin "B"
 		)
+		(pin "D"
+		)
+		(pin "C"
+		)
 		(instances
 			(project "bucket_controls"
@@
 	)
 	(symbol
-		(lib_id "My Symbols:EC11_Rotary_Encoder_Board")
+		(lib_id "My Symbols:EC11_Rotary_Encoder")
 		(at 81.28 198.12 180)
 		(unit 1)
@@
 			)
 		)
-		(property "Footprint" "My Footprints:EC11_miniboard_castellated"
+		(property "Footprint" "My Footprints:EC11J0924411"
 			(at 81.28 198.12 0)
 			(hide yes)
@@
 		(pin "B"
 		)
+		(pin "C"
+		)
+		(pin "D"
+		)
 		(instances
 			(project "bucket_controls"
@@
 	)
 	(symbol
-		(lib_id "My Symbols:EC11_Rotary_Encoder_Board")
+		(lib_id "My Symbols:EC11_Rotary_Encoder")
 		(at 201.93 198.12 180)
 		(unit 1)
@@
 			)
 		)
-		(property "Footprint" "My Footprints:EC11_miniboard_castellated"
+		(property "Footprint" "My Footprints:EC11J0924411"
 			(at 201.93 198.12 0)
 			(hide yes)
@@
 		(pin "B"
 		)
+		(pin "D"
+		)
+		(pin "C"
+		)
 		(instances
 			(project "bucket_controls"
@@
 	)
 	(symbol
-		(lib_id "My Symbols:EC11_Rotary_Encoder_Board")
+		(lib_id "My Symbols:EC11_Rotary_Encoder")
 		(at 81.28 248.92 180)
 		(unit 1)
@@
 			)
 		)
-		(property "Footprint" "My Footprints:EC11_miniboard_castellated"
+		(property "Footprint" "My Footprints:EC11J0924411"
 			(at 81.28 248.92 0)
 			(hide yes)
@@
 		(pin "B"
 		)
+		(pin "C"
+		)
+		(pin "D"
+		)
 		(instances
