File: PCB_CAD/01 Analog/COMP/COMP.kicad_sch (KiCad schematic)
At the start: 27 parts, among them U1 OPA4197, U2 ADR5041

Commit message: more pcb work, fmc timing optimizations for displays, display driver tools
Parts:
- R7: value 78.7k 0.1% -> 48.7k 0.1%
Other:
- note added: "ADC (ENV_ADC), sample >= 20 kHz: level_dBu = 20 log10( V / 0.2421 ) DAC (GR_DAC), output buffer ON: V = (0.2685 + 0.0061 x G_dB) / 0.2053 G = -40...+20 dB (cut and make-up), 0 dB = 1.308 V VREF+: R7 = 78.7k x VREF/3.3, R5 = 22.1k x VREF/3.3(3.0 V: R7 71.5k, R5 20.0k)"
- note added: "COMP_CV = 0.2685 - 0.2053 x GR_DAC (DAC FS 2.048 V, 6.1 mV/dB) DAC 0.119 V = -40 dB, 1.308 V = 0 dB, 1.902 V = +20 dB; 16.8 mdB/LSB. DAC 0 V (reset, R11) = -44 dB: a failure always cuts, never boosts. MFB: 8.0 kHz, Q 0.72."
- note removed: "ADC (ENV_ADC), sample >= 20 kHz: level_dBu = 20 log10( V / 0.2421 ) DAC (GR_DAC), output buffer ON: V = (0.2685 + 0.0061 x G_dB) / 0.1271 G = -40...+20 dB (cut and make-up), 0 dB = 2.113 V VREF+: R7 = 78.7k x VREF/3.3, R5 = 22.1k x VREF/3.3(3.0 V: R7 71.5k, R5 20.0k)"
- note removed: "COMP_CV = 0.2685 - 0.1271 x GR_DAC (VREF+ = 3.3 V, 6.1 mV/dB) DAC 0.193 V = -40 dB, 2.113 V = 0 dB, 3.073 V = +20 dB; 16.8 mdB/LSB. DAC 0 V (reset, R11) = -44 dB: a failure always cuts, never boosts. MFB: 8.0 kHz, Q 0.74."
Changed lines of the file:
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@@
 		)
 	)
-	(text "ADC (ENV_ADC), sample >= 20 kHz:\n  level_dBu = 20 log10( V / 0.2421 )\n\nDAC (GR_DAC), output buffer ON:\n  V = (0.2685 + 0.0061 x G_dB) / 0.1271\n  G = -40...+20 dB (cut and make-up), 0 dB = 2.113 V\n\nVREF+: R7 = 78.7k x VREF/3.3, R5\n  = 22.1k x VREF/3.3(3.0 V: R7 71.5k, R5 20.0k)"
+	(text "ADC (ENV_ADC), sample >= 20 kHz:\n  level_dBu = 20 log10( V / 0.2421 )\n\nDAC (GR_DAC), output buffer ON:\n  V = (0.2685 + 0.0061 x G_dB) / 0.2053\n  G = -40...+20 dB (cut and make-up), 0 dB = 1.308 V\n\nVREF+: R7 = 78.7k x VREF/3.3, R5\n  = 22.1k x VREF/3.3(3.0 V: R7 71.5k, R5 20.0k)"
 		(exclude_from_sim no)
 		(at 213.36 27.94 0)
@@
 		)
 	)
-	(text "COMP_CV = 0.2685 - 0.1271 x GR_DAC  (VREF+ = 3.3 V, 6.1 mV/dB)\nDAC 0.193 V = -40 dB, 2.113 V = 0 dB, 3.073 V = +20 dB; 16.8 mdB/LSB.\nDAC 0 V (reset, R11) = -44 dB: a failure always cuts, never boosts.\nMFB: 8.0 kHz, Q 0.74."
+	(text "COMP_CV = 0.2685 - 0.2053 x GR_DAC  (DAC FS 2.048 V, 6.1 mV/dB)\nDAC 0.119 V = -40 dB, 1.308 V = 0 dB, 1.902 V = +20 dB; 16.8 mdB/LSB.\nDAC 0 V (reset, R11) = -44 dB: a failure always cuts, never boosts.\nMFB: 8.0 kHz, Q 0.72."
 		(exclude_from_sim no)
 		(at 34.29 143.51 0)
@@
 			)
 		)
-		(property "Value" "78.7k 0.1%"
+		(property "Value" "48.7k 0.1%"
 			(at 56.896 132.588 90)
 			(show_name no)

Commit message: so much pcb analog stuff ugh
Parts:
- added H1, H2: MountingScrew, MountingHole:MountingHole_2.2mm_M2, symbol Auxiliary_Items:MountingScrew
- added J1: POWER, Connector_PinHeader_2.54mm:PinHeader_1x04_P2.54mm_Vertical, symbol Connector_Generic:Conn_01x04
- added J2: CV_IO, Connector_PinHeader_2.54mm:PinHeader_1x04_P2.54mm_Vertical, symbol Connector_Generic:Conn_01x04
- added J3: ENV, Connector_PinHeader_2.54mm:PinHeader_1x04_P2.54mm_Vertical, symbol Connector_Generic:Conn_01x04
- C1: LCSC (none) -> C50254
- C10, C9: LCSC (none) -> C9807
- C2: footprint Capacitor_SMD:C_0805_2012Metric -> Capacitor_THT:C_Rect_L10.0mm_W2.5mm_P7.50mm_MKS4; LCSC (none) -> dnp
- C3: LCSC (none) -> C106210
- C4: LCSC (none) -> C107048
- C5: LCSC (none) -> C527067
- C6, C7, C8: LCSC (none) -> C1590
- D1: LCSC (none) -> C2500
- D2: LCSC (none) -> C12765
- R1, R11, R2, R3: LCSC (none) -> C122538
- R10, R9: LCSC (none) -> C95204
- R12: LCSC (none) -> C122970
- R13: LCSC (none) -> C23080
- R4: LCSC (none) -> C311894
- R5: LCSC (none) -> C137768
- R6: LCSC (none) -> C21190
- R7: LCSC (none) -> C667111
- R8: LCSC (none) -> C705799
- U1: LCSC (none) -> C2058532
- U2: LCSC (none) -> C659594
Connections:
- net +15V: now also J1.1 (Pin_1)
- net +3V3: now also J1.4 (Pin_4)
- net -15V: now also J1.3 (Pin_3)
- net COMP_CV: now also J2.3 (Pin_3)
- net DET_IN: now also J3.1 (Pin_1)
- net ENV_ADC: now also J3.3 (Pin_3)
- net GND: now also J1.2 (Pin_2), J2.2 (Pin_2), J2.4 (Pin_4), J3.2 (Pin_2), J3.4 (Pin_4)
- net GR_DAC: now also J2.1 (Pin_1)
