File: PCB_CAD/01 Analog/EQ/EQ.kicad_pcb (KiCad board)
At the start: 2 copper layers, 36 x 180 mm, 274 parts, among them U1 OPA4197, U10 OPA1679, U11 OPA4197, U13 AS2180, U14 OPA1679, U15 OPA1679, U16 OPA1679, U17 OPA4197, U18 ADG1434, U19 AS2180, U3 AS2180, U5 OPA1679, U6 OPA1679, U7 ADR5041, U9 AS2180

Commit message: more pcb work, fmc timing optimizations for displays, display driver tools
Parts:
- added H1: MountingScrew, MountingHole:MountingHole_2.2mm_M2, F.Cu at (115.0, 151.6)
- added H2: MountingScrew, MountingHole:MountingHole_2.2mm_M2, F.Cu at (115.0, 157.5)
- added H3: MountingScrew, MountingHole:MountingHole_2.2mm_M2, F.Cu at (115.0, 163.4)
- added H4: MountingScrew, MountingHole:MountingHole_2.2mm_M2, F.Cu at (115.0, 169.4)
- added J1: AUDIO, Connector_PinHeader_2.54mm:PinHeader_1x04_P2.54mm_Vertical, B.Cu at (136.0, 164.8)
- added J2: CV, Connector_PinHeader_2.54mm:PinHeader_2x10_P2.54mm_Vertical, B.Cu at (153.4, 164.8)
- added J3: LOGIC_CV, Connector_PinHeader_2.54mm:PinHeader_1x08_P2.54mm_Vertical, B.Cu at (140.3, 164.8)
- added J4: POWER, Connector_PinHeader_2.54mm:PinHeader_1x03_P2.54mm_Vertical, B.Cu at (135.7, 177.0)
- R121, R127, R133, R202, R208, R21, R214, R220, R27, R33: value 130k -> 88.7k
- R122, R128, R203, R215, R22, R28: value 88.7k -> 130k
- R130, R30: value 30.1k -> 43.7k
- R134, R209, R221, R34: value 95.3k -> 130k
- R136, R211, R223, R36: value 22.1k -> 30.5k
- R141, R142, R266, R267, R43, R44: value 10k -> 14.0k
- R143, R268, R270, R45: value 14.0k -> 29.4k
- U13, U19, U3, U9: footprint Package_SO:SOIC-8-1EP_3.9x4.9mm_P1.27mm_EP2.29x3mm_ThermalVias -> Package_SO:SOIC-8_3.9x4.9mm_P1.27mm
- moved C205 30.6 mm to (101.0, 57.1)
- moved C209 30.6 mm to (109.9, 40.2)
- moved C223 30.6 mm to (109.9, 52.7)
- moved C227 30.6 mm to (109.9, 60.3)
- moved C233 30.6 mm to (113.9, 40.2)
- moved R202 30.6 mm to (113.9, 52.7)
- moved R205 30.6 mm to (113.9, 60.3)
- moved R211 30.6 mm to (117.9, 40.2)
- moved R216 30.6 mm to (117.9, 52.7)
- moved R219 30.6 mm to (117.9, 60.3)
- moved R225 30.6 mm to (121.9, 40.2)
- moved R230 30.6 mm to (121.9, 52.7)
- moved R233 30.6 mm to (121.9, 60.3)
- moved R239 30.6 mm to (125.9, 40.2)
- moved R244 30.6 mm to (125.9, 52.7)
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Connections:
- net /LF_HF/HF_OUT renamed /EQ_OUT
- C9 pad 2: /LMF/LMF_OUT -> HMF_IN
- R16 pad 2: /LMF/LMF_OUT -> HMF_IN
- R18 pad 2: /LMF/LMF_CUT_LCV -> /LMF_CUT_LCV
- R253 pad 2: /LF_HF/HF_IN -> HMF_OUT
- R39 pad 2: /LMF/LMF_IN -> /LF_HF/LF_OUT
- R40 pad 2: /LMF/HMF_CUT_LCV -> /HMF_CUT_LCV
- U18 pad 7: /LF_HF/HF_IN -> HMF_OUT
- U6 pad 1: /LMF/LMF_OUT -> HMF_IN
Routing:
- added copper zone on B.Cu, net GND
- added copper zone on F.Cu, net GND
- added copper zone on In1.Cu, net GND
- added copper zone on In2.Cu, net GND
Other:
- board size 36 x 180 mm -> 36 x 200 mm
- copper layers 2 -> 4

Commit message: input board done
Parts:
- added C237: 100n, Capacitor_SMD:C_0603_1608Metric, F.Cu at (154.7, 46.6)
- added C238: 100n, Capacitor_SMD:C_0603_1608Metric, F.Cu at (154.7, 49.1)
- J2: value CV -> LF_HF_CV; footprint Connector_PinHeader_2.54mm:PinHeader_2x10_P2.54mm_Vertical -> Connector_PinHeader_2.54mm:PinHeader_1x08_P2.54mm_Vertical
- U13, U19, U3, U9: footprint Package_SO:SOIC-8_3.9x4.9mm_P1.27mm -> Connector_PinHeader_2.54mm:PinHeader_1x08_P2.54mm_Vertical
- moved J2 70.3 mm to (113.5, 106.8)
Connections:
- J2 pad 2: CV_IN_LF_F -> CV_IN_LF_G
- J2 pad 3: CV_IN_LF_G -> GND
- J2 pad 4: GND -> CV_IN_LF_F
- J2 pad 6: CV_IN_LMF_F -> CV_IN_HF_G
- J2 pad 7: CV_IN_LMF_Q -> GND
- J2 pad 8: GND -> CV_IN_HF_F
- U14 pad 11: (no net) -> -15V
- U14 pad 4: (no net) -> +15V

Commit message: pcbs omg when does it end
Parts:
- removed C15, C16: 100n, Capacitor_SMD:C_0603_1608Metric
- removed U6: OPA1679, Package_SO:SOIC-14_3.9x8.7mm_P1.27mm
- added J5: HMF_CV, Connector_PinHeader_2.54mm:PinHeader_1x06_P2.54mm_Vertical, B.Cu at (53.5, 105.4)
- added J6: LMF_CV, Connector_PinHeader_2.54mm:PinHeader_1x06_P2.54mm_Vertical, B.Cu at (53.5, 74.9)
- added R145: 14.0k, Resistor_SMD:R_0603_1608Metric, F.Cu at (56.4, 114.0)
- added R146: 10k, Resistor_SMD:R_0603_1608Metric, F.Cu at (84.3, 135.3)
- added R276: 10k, Resistor_SMD:R_0603_1608Metric, F.Cu at (56.4, 195.8)
- added R277: 10k, Resistor_SMD:R_0603_1608Metric, F.Cu at (58.9, 181.6)
- added R49: 14.0k, Resistor_SMD:R_0603_1608Metric, F.Cu at (84.3, 60.7)
- added R50: 10k, Resistor_SMD:R_0603_1608Metric, F.Cu at (84.3, 131.8)
- added U12: SSI2164, Package_SO:SOIC-16_3.9x9.9mm_P1.27mm, F.Cu at (68.6, 213.4)
- added U2: SSI2164, Package_SO:SOIC-16_3.9x9.9mm_P1.27mm, F.Cu at (64.8, 62.2)
- added U4: ADG1436, Package_SO:TSSOP-16_4.4x5mm_P0.65mm, F.Cu at (59.7, 148.0)
- added U8: SSI2164, Package_SO:SOIC-16_3.9x9.9mm_P1.27mm, F.Cu at (64.8, 97.8)
- C11, C111, C112, C113, C114, C117, C12, C127, C128, C13, C14, C17, C18, C19, C225, C226, C227, C228, C229, C230, C231, C232, C233, C234, C235, C236, C237, C238, C27, C28: moved to B.Cu
- R117, R17, R248, R254: value 100 -> 220
- R130, R30: value 43.7k -> 29.4k
- R131, R31: value 30.1k -> 29.4k
- R136, R211, R223, R36: value 30.5k -> 20k
- R137, R212, R224, R37: value 22.1k -> 20k
- moved R239 191.2 mm to (74.1, 224.2), turned to 90 degrees
- moved R240 189.5 mm to (71.6, 224.2), turned to -90 degrees
- moved R213 183.7 mm to (76.7, 224.2), turned to -90 degrees
- moved R241 182.3 mm to (76.7, 220.7), turned to -90 degrees
- moved R226 181.6 mm to (51.3, 210.0), turned to 90 degrees
- moved R215 180.8 mm to (69.0, 224.2), turned to 90 degrees
- moved R242 179.2 mm to (79.2, 220.7), turned to 90 degrees
- moved C216 179.1 mm to (74.1, 220.7), turned to -90 degrees
- moved R227 178.3 mm to (53.8, 210.0), turned to 90 degrees
- moved R231 177.9 mm to (66.5, 224.2), turned to 90 degrees
- moved C233 177.8 mm to (73.7, 213.4)
- moved C209 176.3 mm to (51.3, 206.5), turned to -90 degrees
- moved R232 173.3 mm to (53.8, 217.1), turned to -90 degrees
- moved R216 173.1 mm to (53.8, 213.6), turned to -90 degrees
- moved R228 169.9 mm to (61.4, 206.5), turned to 90 degrees
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Connections:
- U14 pad 1: (no net) -> HMF_IN
- U14 pad 2: (no net) -> Net-(U6A--)
- U14 pad 3: (no net) -> GND
Other:
- board size 36 x 200 mm -> 36 x 180 mm

Commit message: so much pcb analog stuff ugh
Parts:
- added REF**: LayerMarker_4_6.35x2.54mm_TextH1mm_P1.27mm_LowerMirrored, Symbol:LayerMarker_4_6.35x2.54mm_TextH1mm_P1.27mm_LowerMirrored, F.Cu at (141.8, 93.4)
- moved H2 176.8 mm to (52.9, 227.2), turned to 180 degrees
- moved H1 176.7 mm to (82.9, 227.2), turned to 180 degrees
- moved H4 176.4 mm to (52.9, 53.2), turned to 180 degrees
- moved H3 176.4 mm to (82.9, 53.2), turned to 180 degrees
- moved C217 175.5 mm to (65.6, 52.4), turned to 0 degrees
- moved R5 174.0 mm to (77.0, 226.6), turned to 90 degrees
- moved C3 173.9 mm to (59.3, 226.6), turned to -90 degrees
- moved R10 173.6 mm to (74.5, 226.6), turned to -90 degrees
- moved R3 173.5 mm to (61.8, 226.6), turned to -90 degrees
- moved C213 173.3 mm to (78.8, 54.1), turned to 180 degrees
- moved C1 173.2 mm to (64.3, 226.6), turned to -90 degrees
- moved C5 173.2 mm to (70.7, 226.6), turned to 180 degrees
- moved R4 173.1 mm to (66.9, 226.6), turned to -90 degrees
- moved R270 169.8 mm to (56.7, 55.9), turned to -90 degrees
- moved R213 169.2 mm to (59.3, 55.9), turned to 90 degrees
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Other:
- board text added: "1"
- board text added: "2180"
- board text added: "48V SWITCH MIC SWITCH LINE SWITCH HI-Z SWITCH PHASE FLIP HPF IN PAD IN GND"
- board text added: "Channel EQ Card"
- board text added: "DIGILOG"
- board text added: "REV 0 2026 RoHS"
- board text added: "SWITCH CV"
- board text added: "Skylar Evelyn Denno"
