File: PCB_CAD/01 Analog/EQ/lf_hf.kicad_sch (KiCad schematic)
At the start: 123 parts, among them U12 SSI2164, U13 AS2180, U14 OPA1679, U15 OPA1679, U16 OPA1679, U17 OPA4197, U18 ADG1434, U19 AS2180

Commit message: more pcb work, fmc timing optimizations for displays, display driver tools
Parts:
- R202, R208, R214, R220: value 130k -> 88.7k
- R203, R215: value 88.7k -> 130k
- R209, R221: value 95.3k -> 130k
- R211, R223: value 22.1k -> 30.5k; Note 1% -> 0.1% thin film
- R266, R267: value 10k -> 14.0k
- R268, R270: value 14.0k -> 29.4k
- U13, U19: footprint Package_SO:SOIC-8-1EP_3.9x4.9mm_P1.27mm_EP2.29x3mm_ThermalVias -> Package_SO:SOIC-8_3.9x4.9mm_P1.27mm
Changed lines of the file:
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@@
 		)
 	)
-	(label "HF_IN"
-		(at 283.21 171.45 180)
-		(effects
-			(font
-				(size 1.27 1.27)
-			)
-			(justify right bottom)
-		)
-	)
 	(label "HF_G_CV"
 		(at 236.22 251.46 0)
@@
 		)
 	)
-	(label "LF_IN"
-		(at 345.44 53.34 180)
-		(effects
-			(font
-				(size 1.27 1.27)
-			)
-			(justify right bottom)
-		)
-	)
 	(label "LF_NBP"
 		(at 86.36 80.01 180)
@@
 		)
 	)
-	(label "HF_CUT_LCV"
-		(at 389.89 66.04 0)
-		(effects
-			(font
-				(size 1.27 1.27)
-			)
-			(justify left bottom)
-		)
-	)
 	(label "HF_NBP"
 		(at 345.44 88.9 180)
@@
 		)
 	)
-	(label "HF_OUT"
-		(at 311.15 138.43 0)
-		(effects
-			(font
-				(size 1.27 1.27)
-			)
-			(justify left bottom)
-		)
-	)
-	(label "HF_OUT"
-		(at 345.44 63.5 180)
-		(effects
-			(font
-				(size 1.27 1.27)
-			)
-			(justify right bottom)
-		)
-	)
-	(label "HF_MODE_LCV"
-		(at 389.89 91.44 0)
-		(effects
-			(font
-				(size 1.27 1.27)
-			)
-			(justify left bottom)
-		)
-	)
-	(label "LF_MODE_LCV"
-		(at 389.89 78.74 0)
-		(effects
-			(font
-				(size 1.27 1.27)
-			)
-			(justify left bottom)
-		)
-	)
-	(label "LF_OUT"
-		(at 345.44 50.8 180)
-		(effects
-			(font
-				(size 1.27 1.27)
-			)
-			(justify right bottom)
-		)
-	)
 	(label "LF_V"
 		(at 29.21 52.07 180)
@@
 		)
 	)
-	(label "LF_OUT"
-		(at 313.69 54.61 0)
-		(effects
-			(font
-				(size 1.27 1.27)
-			)
-			(justify left bottom)
-		)
-	)
 	(label "LF_F_CV"
 		(at 148.59 62.23 0)
@@
 		)
 	)
-	(label "LF_IN"
-		(at 285.75 87.63 180)
-		(effects
-			(font
-				(size 1.27 1.27)
-			)
-			(justify right bottom)
-		)
-	)
-	(label "HF_IN"
-		(at 345.44 66.04 180)
-		(effects
-			(font
-				(size 1.27 1.27)
-			)
-			(justify right bottom)
-		)
-	)
 	(label "HF_V"
 		(at 29.21 137.16 180)
@@
 		)
 	)
-	(label "LF_CUT_LCV"
-		(at 389.89 53.34 0)
-		(effects
-			(font
-				(size 1.27 1.27)
-			)
-			(justify left bottom)
-		)
-	)
 	(label "LF_F_CV"
 		(at 125.73 215.9 0)
@@
 		)
 	)
+	(hierarchical_label "HF_IN"
+		(shape input)
+		(at 283.21 171.45 180)
+		(effects
+			(font
+				(size 1.27 1.27)
+			)
+			(justify right)
+		)
+	)
+	(hierarchical_label "LF_IN"
+		(shape input)
+		(at 345.44 53.34 180)
+		(effects
+			(font
+				(size 1.27 1.27)
+			)
+			(justify right)
+		)
+	)
+	(hierarchical_label "HF_CUT_LCV"
+		(shape input)
+		(at 389.89 66.04 0)
+		(effects
+			(font
+				(size 1.27 1.27)
+			)
+			(justify left)
+		)
+	)
+	(hierarchical_label "HF_OUT"
+		(shape output)
+		(at 311.15 138.43 0)
+		(effects
+			(font
+				(size 1.27 1.27)
+			)
+			(justify left)
+		)
+	)
+	(hierarchical_label "HF_OUT"
+		(shape output)
+		(at 345.44 63.5 180)
+		(effects
+			(font
+				(size 1.27 1.27)
+			)
+			(justify right)
+		)
+	)
+	(hierarchical_label "HF_MODE_LCV"
+		(shape input)
+		(at 389.89 91.44 0)
+		(effects
+			(font
+				(size 1.27 1.27)
+			)
+			(justify left)
+		)
+	)
+	(hierarchical_label "LF_MODE_LCV"
+		(shape input)
+		(at 389.89 78.74 0)
+		(effects
+			(font
+				(size 1.27 1.27)
+			)
+			(justify left)
+		)
+	)
+	(hierarchical_label "LF_OUT"
+		(shape output)
+		(at 345.44 50.8 180)
+		(effects
+			(font
+				(size 1.27 1.27)
+			)
+			(justify right)
+		)
+	)
+	(hierarchical_label "LF_OUT"
+		(shape output)
+		(at 313.69 54.61 0)
+		(effects
+			(font
+				(size 1.27 1.27)
+			)
+			(justify left)
+		)
+	)
+	(hierarchical_label "LF_IN"
+		(shape input)
+		(at 285.75 87.63 180)
+		(effects
+			(font
+				(size 1.27 1.27)
+			)
+			(justify right)
+		)
+	)
+	(hierarchical_label "HF_IN"
+		(shape input)
+		(at 345.44 66.04 180)
+		(effects
+			(font
+				(size 1.27 1.27)
+			)
+			(justify right)
+		)
+	)
+	(hierarchical_label "LF_CUT_LCV"
+		(shape input)
+		(at 389.89 53.34 0)
+		(effects
+			(font
+				(size 1.27 1.27)
+			)
+			(justify left)
+		)
+	)
 	(symbol
 		(lib_id "power:GND")
@@
 			)
 		)
-		(property "Value" "10k"
+		(property "Value" "14.0k"
 			(at 172.72 220.98 0)
 			(show_name no)
@@
 			)
 		)
-		(property "Value" "130k"
+		(property "Value" "88.7k"
 			(at 49.53 223.52 0)
 			(show_name no)
@@
 			)
 		)
-		(property "Value" "130k"
+		(property "Value" "88.7k"
 			(at 160.02 220.98 0)
 			(show_name no)
@@
 			)
 		)
-		(property "Value" "95.3k"
+		(property "Value" "130k"
 			(at 59.69 251.46 0)
 			(show_name no)
@@
 			)
 		)
-		(property "Value" "130k"
+		(property "Value" "88.7k"
 			(at 166.37 256.794 90)
 			(show_name no)
@@
 			)
 		)
-		(property "Value" "10k"
+		(property "Value" "14.0k"
 			(at 62.23 223.52 0)
 			(show_name no)
@@
 			)
 		)
-		(property "Footprint" "Package_SO:SOIC-8-1EP_3.9x4.9mm_P1.27mm_EP2.29x3mm_ThermalVias"
+		(property "Footprint" "Package_SO:SOIC-8_3.9x4.9mm_P1.27mm"
 			(at 260.35 57.15 0)
 			(hide yes)
@@
 			)
 		)
-		(property "Value" "14.0k"
+		(property "Value" "29.4k"
 			(at 107.95 203.2 0)
 			(show_name no)
@@
 			)
 		)
-		(property "Footprint" "Package_SO:SOIC-8-1EP_3.9x4.9mm_P1.27mm_EP2.29x3mm_ThermalVias"
+		(property "Footprint" "Package_SO:SOIC-8_3.9x4.9mm_P1.27mm"
 			(at 257.81 140.97 0)
 			(hide yes)
@@
 			)
 		)
-		(property "Value" "88.7k"
+		(property "Value" "130k"
 			(at 170.18 210.82 0)
 			(show_name no)
@@
 			)
 		)
-		(property "Value" "22.1k"
+		(property "Value" "30.5k"
 			(at 101.6 246.634 90)
 			(show_name no)
@@
 			)
 		)
-		(property "Note" "1%"
+		(property "Note" "0.1% thin film"
 			(at 101.6 243.84 0)
 			(hide yes)
@@
 			)
 		)
-		(property "Value" "14.0k"
+		(property "Value" "29.4k"
 			(at 218.44 200.66 0)
 			(show_name no)
@@
 			)
 		)
-		(property "Value" "130k"
+		(property "Value" "88.7k"
 			(at 55.88 259.334 90)
 			(show_name no)
@@
 			)
 		)
-		(property "Value" "95.3k"
+		(property "Value" "130k"
 			(at 170.18 248.92 0)
 			(show_name no)
@@
 			)
 		)
-		(property "Value" "22.1k"
+		(property "Value" "30.5k"
 			(at 212.09 244.094 90)
 			(show_name no)
@@
 			)
 		)
-		(property "Note" "1%"
+		(property "Note" "0.1% thin film"
 			(at 212.09 241.3 0)
 			(hide yes)
@@
 			)
 		)
-		(property "Value" "88.7k"
+		(property "Value" "130k"
 			(at 59.69 213.36 0)
 			(show_name no)

Commit message: input board done
Parts:
- added C237, C238: 100n, Capacitor_SMD:C_0603_1608Metric, symbol Device:C
- added unit 5 of U14
- U13, U19: footprint Package_SO:SOIC-8_3.9x4.9mm_P1.27mm -> Connector_PinHeader_2.54mm:PinHeader_1x08_P2.54mm_Vertical
Connections:
- net +15V: now also C237.1, U14.4 (V+)
- net -15V: now also C238.1, U14.11 (V-)
- net GND: now also C237.2, C238.2

Commit message: pcbs omg when does it end
Parts:
- added R276, R277: 10k, Resistor_SMD:R_0603_1608Metric, symbol Device:R_US
- R211, R223: value 30.5k -> 20k
- R212, R224: value 22.1k -> 20k; Note 1% -> 0.1% thin film
- R248, R254: value 100 -> 220
- U12: footprint 4ms_Package_SOIC:SOIC-16_3.9x9.9mm_Pitch1.27mm -> Package_SO:SOIC-16_3.9x9.9mm_P1.27mm
Connections:
- net HF_G_CV: now also R277.2; no longer R223.2
- net LF_G_CV: now also R276.2; no longer R211.2
- new net: R223.2, R277.1
- new net: R211.2, R276.1
Other:
- moved on the sheet: R211, R223

Commit message: even more pcbs we're slowly getting there lmaoi
Parts:
- U12: footprint Package_SO:SOIC-16_3.9x9.9mm_P1.27mm -> My Footprints:SSI2164_breakout
Changed lines of the file:
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@@
 			)
 		)
-		(property "Footprint" "Package_SO:SOIC-16_3.9x9.9mm_P1.27mm"
+		(property "Footprint" "My Footprints:SSI2164_breakout"
 			(at 353.06 140.97 0)
 			(hide yes)
@@
 			)
 		)
-		(property "Footprint" "Package_SO:SOIC-16_3.9x9.9mm_P1.27mm"
+		(property "Footprint" "My Footprints:SSI2164_breakout"
 			(at 152.4 44.45 0)
 			(hide yes)
@@
 			)
 		)
-		(property "Footprint" "Package_SO:SOIC-16_3.9x9.9mm_P1.27mm"
+		(property "Footprint" "My Footprints:SSI2164_breakout"
 			(at 88.9 129.54 0)
 			(hide yes)
@@
 			)
 		)
-		(property "Footprint" "Package_SO:SOIC-16_3.9x9.9mm_P1.27mm"
+		(property "Footprint" "My Footprints:SSI2164_breakout"
 			(at 88.9 44.45 0)
 			(hide yes)
@@
 			)
 		)
-		(property "Footprint" "Package_SO:SOIC-16_3.9x9.9mm_P1.27mm"
+		(property "Footprint" "My Footprints:SSI2164_breakout"
 			(at 152.4 129.54 0)
 			(hide yes)
