File: PCB_CAD/02 Bucket/BUCKET_ROUTING/BUCKET_ROUTING.kicad_pcb (KiCad board)
At the start: 4 copper layers, 146 x 435 mm, 33 parts, among them J1 POWER, J10 MIX_BUS, J11 POWER, J12 CV, J13 AUD_IN, J14 INSERT, J15 MIX_BUS, J16 POWER, J17 CV, J18 AUD_IN, J19 INSERT, J2 CV, J20 MIX_BUS, J3 AUD_IN, J4 INSERT, J5 MIX_BUS, J6 POWER, J7 CV, J8 AUD_IN, J9 INSERT, P1 POWER

Commit message: so much pcb analog stuff ugh
Parts:
- added H19: MountingHole, MountingHole:MountingHole_2.2mm_M2, F.Cu at (24.4, 44.5)
- added H20: MountingHole, MountingHole:MountingHole_2.2mm_M2, F.Cu at (31.4, 126.2)
- added H21: MountingHole, MountingHole:MountingHole_2.2mm_M2, F.Cu at (44.0, 58.6)
- added H22: MountingHole, MountingHole:MountingHole_2.2mm_M2, F.Cu at (53.4, 306.5)
- added H23: MountingHole, MountingHole:MountingHole_2.2mm_M2, F.Cu at (23.4, 306.5)
- added H24: MountingHole, MountingHole:MountingHole_2.2mm_M2, F.Cu at (53.4, 132.5)
- added H25: MountingHole, MountingHole:MountingHole_2.2mm_M2, F.Cu at (23.4, 132.5)
- added H26: MountingHole, MountingHole:MountingHole_2.2mm_M2, F.Cu at (37.1, 313.0)
- added H27: MountingHole, MountingHole:MountingHole_2.2mm_M2, F.Cu at (29.2, 334.3)
- added H28: MountingHole, MountingHole:MountingHole_2.2mm_M2, F.Cu at (60.7, 44.5)
- added H29: MountingHole, MountingHole:MountingHole_2.2mm_M2, F.Cu at (67.7, 126.2)
- added H30: MountingHole, MountingHole:MountingHole_2.2mm_M2, F.Cu at (80.3, 58.6)
- added H31: MountingHole, MountingHole:MountingHole_2.2mm_M2, F.Cu at (89.7, 306.5)
- added H32: MountingHole, MountingHole:MountingHole_2.2mm_M2, F.Cu at (59.7, 306.5)
- added H33: MountingHole, MountingHole:MountingHole_2.2mm_M2, F.Cu at (89.7, 132.5)
- added H34: MountingHole, MountingHole:MountingHole_2.2mm_M2, F.Cu at (59.7, 132.5)
- added H35: MountingHole, MountingHole:MountingHole_2.2mm_M2, F.Cu at (73.5, 313.0)
- added H36: MountingHole, MountingHole:MountingHole_2.2mm_M2, F.Cu at (65.6, 334.3)
- added H37: MountingHole, MountingHole:MountingHole_2.2mm_M2, F.Cu at (97.2, 44.5)
- added H38: MountingHole, MountingHole:MountingHole_2.2mm_M2, F.Cu at (104.2, 126.2)
- added H39: MountingHole, MountingHole:MountingHole_2.2mm_M2, F.Cu at (116.8, 58.6)
- added H40: MountingHole, MountingHole:MountingHole_2.2mm_M2, F.Cu at (126.2, 306.5)
- added H41: MountingHole, MountingHole:MountingHole_2.2mm_M2, F.Cu at (96.2, 306.5)
- added H42: MountingHole, MountingHole:MountingHole_2.2mm_M2, F.Cu at (126.2, 132.5)
- added H43: MountingHole, MountingHole:MountingHole_2.2mm_M2, F.Cu at (96.2, 132.5)
- added H44: MountingHole, MountingHole:MountingHole_2.2mm_M2, F.Cu at (110.0, 313.0)
- added H45: MountingHole, MountingHole:MountingHole_2.2mm_M2, F.Cu at (102.1, 334.3)
- added H46: MountingHole, MountingHole:MountingHole_2.2mm_M2, F.Cu at (133.5, 44.5)
- added H47: MountingHole, MountingHole:MountingHole_2.2mm_M2, F.Cu at (140.5, 126.2)
- added H48: MountingHole, MountingHole:MountingHole_2.2mm_M2, F.Cu at (153.1, 58.6)
- added H49: MountingHole, MountingHole:MountingHole_2.2mm_M2, F.Cu at (162.5, 306.5)
- added H50: MountingHole, MountingHole:MountingHole_2.2mm_M2, F.Cu at (132.5, 306.5)
- added H51: MountingHole, MountingHole:MountingHole_2.2mm_M2, F.Cu at (162.5, 132.5)
- added H52: MountingHole, MountingHole:MountingHole_2.2mm_M2, F.Cu at (132.5, 132.5)
- added H53: MountingHole, MountingHole:MountingHole_2.2mm_M2, F.Cu at (146.2, 313.0)
- added H54: MountingHole, MountingHole:MountingHole_2.2mm_M2, F.Cu at (138.4, 334.3)
- added J21: CH1_IN_LOGIC, Connector_PinSocket_2.54mm:PinSocket_1x08_P2.54mm_Vertical, F.Cu at (23.5, 76.1)
- added J22: CH1_IN_AUDIO, Connector_PinSocket_2.54mm:PinSocket_1x10_P2.54mm_Vertical, F.Cu at (23.5, 123.6)
- added J23: CH1_IN_POWER, Connector_PinSocket_2.54mm:PinSocket_1x04_P2.54mm_Vertical, F.Cu at (45.4, 37.1)
- added J24: CH1_IN_CV, Connector_PinSocket_2.54mm:PinSocket_1x02_P2.54mm_Vertical, F.Cu at (41.5, 65.6)
- added J25: CH1_EQ_AUDIO, Connector_PinSocket_2.54mm:PinSocket_1x04_P2.54mm_Vertical, F.Cu at (52.9, 191.9)
- added J26: CH1_EQ_LF_HF_CV, Connector_PinSocket_2.54mm:PinSocket_1x08_P2.54mm_Vertical, F.Cu at (52.9, 172.8)
- added J27: CH1_EQ_LOGIC, Connector_PinSocket_2.54mm:PinSocket_1x08_P2.54mm_Vertical, F.Cu at (52.9, 216.0)
- added J28: CH1_EQ_POWER, Connector_PinSocket_2.54mm:PinSocket_1x03_P2.54mm_Vertical, F.Cu at (52.9, 266.8)
- added J29: CH1_EQ_HMF_CV, Connector_PinSocket_2.54mm:PinSocket_1x06_P2.54mm_Vertical, F.Cu at (52.9, 254.1)
- added J30: CH1_EQ_LMF_CV, Connector_PinSocket_2.54mm:PinSocket_1x06_P2.54mm_Vertical, F.Cu at (52.9, 284.6)
- added J31: CH1_COMP_POWER, Connector_PinSocket_2.54mm:PinSocket_1x04_P2.54mm_Vertical, F.Cu at (23.0, 324.1)
- added J32: CH1_COMP_CV_IO, Connector_PinSocket_2.54mm:PinSocket_1x04_P2.54mm_Vertical, F.Cu at (23.0, 335.6)
- added J33: CH1_COMP_ENV, Connector_PinSocket_2.54mm:PinSocket_1x04_P2.54mm_Vertical, F.Cu at (23.0, 312.7)
- added J34: CH2_IN_LOGIC, Connector_PinSocket_2.54mm:PinSocket_1x08_P2.54mm_Vertical, F.Cu at (59.9, 76.1)
- added J35: CH2_IN_CV, Connector_PinSocket_2.54mm:PinSocket_1x02_P2.54mm_Vertical, F.Cu at (77.9, 65.6)
- added J36: CH2_IN_AUDIO, Connector_PinSocket_2.54mm:PinSocket_1x10_P2.54mm_Vertical, F.Cu at (59.9, 123.6)
- added J37: CH2_IN_POWER, Connector_PinSocket_2.54mm:PinSocket_1x04_P2.54mm_Vertical, F.Cu at (81.7, 37.1)
- added J38: CH2_EQ_AUDIO, Connector_PinSocket_2.54mm:PinSocket_1x04_P2.54mm_Vertical, F.Cu at (89.2, 191.9)
- added J39: CH2_EQ_LF_HF_CV, Connector_PinSocket_2.54mm:PinSocket_1x08_P2.54mm_Vertical, F.Cu at (89.2, 172.8)
- added J40: CH2_EQ_LOGIC, Connector_PinSocket_2.54mm:PinSocket_1x08_P2.54mm_Vertical, F.Cu at (89.2, 216.0)
- added J41: CH2_EQ_POWER, Connector_PinSocket_2.54mm:PinSocket_1x03_P2.54mm_Vertical, F.Cu at (89.2, 266.8)
- added J42: CH2_EQ_HMF_CV, Connector_PinSocket_2.54mm:PinSocket_1x06_P2.54mm_Vertical, F.Cu at (89.2, 254.1)
- added J43: CH2_EQ_LMF_CV, Connector_PinSocket_2.54mm:PinSocket_1x06_P2.54mm_Vertical, F.Cu at (89.2, 284.6)
- added J44: CH2_COMP_POWER, Connector_PinSocket_2.54mm:PinSocket_1x04_P2.54mm_Vertical, F.Cu at (59.3, 324.1)
- added J45: CH2_COMP_CV_IO, Connector_PinSocket_2.54mm:PinSocket_1x04_P2.54mm_Vertical, F.Cu at (59.3, 335.6)
- added J46: CH2_COMP_ENV, Connector_PinSocket_2.54mm:PinSocket_1x04_P2.54mm_Vertical, F.Cu at (59.3, 312.7)
- added J47: CH3_IN_LOGIC, Connector_PinSocket_2.54mm:PinSocket_1x08_P2.54mm_Vertical, F.Cu at (96.4, 76.1)
- added J48: CH3_IN_CV, Connector_PinSocket_2.54mm:PinSocket_1x02_P2.54mm_Vertical, F.Cu at (114.4, 65.6)
- added J49: CH3_IN_AUDIO, Connector_PinSocket_2.54mm:PinSocket_1x10_P2.54mm_Vertical, F.Cu at (96.4, 123.6)
- added J50: CH3_IN_POWER, Connector_PinSocket_2.54mm:PinSocket_1x04_P2.54mm_Vertical, F.Cu at (118.2, 37.1)
- added J51: CH3_EQ_AUDIO, Connector_PinSocket_2.54mm:PinSocket_1x04_P2.54mm_Vertical, F.Cu at (125.7, 191.9)
- added J52: CH3_EQ_LF_HF_CV, Connector_PinSocket_2.54mm:PinSocket_1x08_P2.54mm_Vertical, F.Cu at (125.7, 172.8)
- added J53: CH3_EQ_LOGIC, Connector_PinSocket_2.54mm:PinSocket_1x08_P2.54mm_Vertical, F.Cu at (125.7, 216.0)
- added J54: CH3_EQ_POWER, Connector_PinSocket_2.54mm:PinSocket_1x03_P2.54mm_Vertical, F.Cu at (125.7, 266.8)
- added J55: CH3_EQ_HMF_CV, Connector_PinSocket_2.54mm:PinSocket_1x06_P2.54mm_Vertical, F.Cu at (125.7, 254.1)
- added J56: CH3_EQ_LMF_CV, Connector_PinSocket_2.54mm:PinSocket_1x06_P2.54mm_Vertical, F.Cu at (125.7, 284.6)
- added J57: CH3_COMP_POWER, Connector_PinSocket_2.54mm:PinSocket_1x04_P2.54mm_Vertical, F.Cu at (95.8, 324.1)
- added J58: CH3_COMP_CV_IO, Connector_PinSocket_2.54mm:PinSocket_1x04_P2.54mm_Vertical, F.Cu at (95.8, 335.6)
- added J59: CH3_COMP_ENV, Connector_PinSocket_2.54mm:PinSocket_1x04_P2.54mm_Vertical, F.Cu at (95.8, 312.7)
- added J60: CH4_IN_LOGIC, Connector_PinSocket_2.54mm:PinSocket_1x08_P2.54mm_Vertical, F.Cu at (132.7, 76.1)
- added J61: CH4_IN_CV, Connector_PinSocket_2.54mm:PinSocket_1x02_P2.54mm_Vertical, F.Cu at (150.7, 65.6)
- added J62: CH4_IN_AUDIO, Connector_PinSocket_2.54mm:PinSocket_1x10_P2.54mm_Vertical, F.Cu at (132.7, 123.6)
- added J63: CH4_IN_POWER, Connector_PinSocket_2.54mm:PinSocket_1x04_P2.54mm_Vertical, F.Cu at (154.5, 37.1)
- added J64: CH4_EQ_AUDIO, Connector_PinSocket_2.54mm:PinSocket_1x04_P2.54mm_Vertical, F.Cu at (162.0, 191.9)
- added J65: CH4_EQ_LF_HF_CV, Connector_PinSocket_2.54mm:PinSocket_1x08_P2.54mm_Vertical, F.Cu at (162.0, 172.8)
- added J66: CH4_EQ_LOGIC, Connector_PinSocket_2.54mm:PinSocket_1x08_P2.54mm_Vertical, F.Cu at (162.0, 216.0)
- added J67: CH4_EQ_POWER, Connector_PinSocket_2.54mm:PinSocket_1x03_P2.54mm_Vertical, F.Cu at (162.0, 266.8)
- added J68: CH4_EQ_HMF_CV, Connector_PinSocket_2.54mm:PinSocket_1x06_P2.54mm_Vertical, F.Cu at (162.0, 254.1)
- added J69: CH4_EQ_LMF_CV, Connector_PinSocket_2.54mm:PinSocket_1x06_P2.54mm_Vertical, F.Cu at (162.0, 284.6)
- added J70: CH4_COMP_POWER, Connector_PinSocket_2.54mm:PinSocket_1x04_P2.54mm_Vertical, F.Cu at (132.1, 324.1)
- added J71: CH4_COMP_CV_IO, Connector_PinSocket_2.54mm:PinSocket_1x04_P2.54mm_Vertical, F.Cu at (132.1, 335.6)
- added J72: CH4_COMP_ENV, Connector_PinSocket_2.54mm:PinSocket_1x04_P2.54mm_Vertical, F.Cu at (132.1, 312.7)
- added J73: BUS_A_MIX_AUX, Connector_IDC:IDC-Header_2x12_P2.54mm_Vertical, F.Cu at (26.0, 29.3)
- added J74: BUS_B_MIX_AUX, Connector_IDC:IDC-Header_2x12_P2.54mm_Vertical, F.Cu at (132.0, 29.3)
- added P2: PWR_IN_+48V, Connector_Samtec_HPM_THT:Samtec_HPM-03-05-x-S_Straight_1x03_Pitch5.08mm, F.Cu at (100.0, 27.0)
- added P3: PWR_IN_+3V3, Connector_PinSocket_2.54mm:PinSocket_1x02_P2.54mm_Vertical, F.Cu at (116.0, 27.0)
- J1: value POWER -> CH1_PF_POWER
- J10: value MIX_BUS -> CH2_PF_MIX_BUS
- J11: value POWER -> CH3_PF_POWER
- J12: value CV -> CH3_PF_CV
- J13: value AUD_IN -> CH3_PF_AUD_IN
- J14: value INSERT -> CH3_PF_INSERT
- J15: value MIX_BUS -> CH3_PF_MIX_BUS
- J16: value POWER -> CH4_PF_POWER
- J17: value CV -> CH4_PF_CV
- J18: value AUD_IN -> CH4_PF_AUD_IN
- J19: value INSERT -> CH4_PF_INSERT
- J2: value CV -> CH1_PF_CV
- J20: value MIX_BUS -> CH4_PF_MIX_BUS
- J3: value AUD_IN -> CH1_PF_AUD_IN
- J4: value INSERT -> CH1_PF_INSERT
- J5: value MIX_BUS -> CH1_PF_MIX_BUS
- J6: value POWER -> CH2_PF_POWER
- J7: value CV -> CH2_PF_CV
- J8: value AUD_IN -> CH2_PF_AUD_IN
- J9: value INSERT -> CH2_PF_INSERT
- P1: value POWER -> PWR_IN_+-15V
- moved H10 2.00 mm to (76.7, 350.1)
- moved H11 2.00 mm to (60.7, 423.5)
- moved H12 2.00 mm to (88.4, 448.3)
- moved H13 2.00 mm to (113.2, 350.1)
- moved H14 2.00 mm to (97.2, 423.5)
- moved H15 2.00 mm to (124.9, 448.3)
- moved H16 2.00 mm to (149.5, 350.1)
- moved H17 2.00 mm to (133.5, 423.5)
- moved H18 2.00 mm to (161.2, 448.3)
- moved H7 2.00 mm to (40.3, 350.1)
- moved H8 2.00 mm to (24.4, 423.5)
- moved H9 2.00 mm to (52.0, 448.3)
- moved J1 2.00 mm to (44.9, 350.5)
- moved J10 2.00 mm to (64.7, 448.5)
- moved J11 2.00 mm to (117.8, 350.5)
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Connections:
- J1 pad 1: unconnected-(J1-Pin_1-Pad1) -> +15V
- J1 pad 2: unconnected-(J1-Pin_2-Pad2) -> GND
- J1 pad 3: unconnected-(J1-Pin_3-Pad3) -> -15V
- J10 pad 1: unconnected-(J10-Pin_1-Pad1) -> /MIX_L+
- J10 pad 2: unconnected-(J10-Pin_2-Pad2) -> GND
- J10 pad 3: unconnected-(J10-Pin_3-Pad3) -> /MIX_L-
- J10 pad 4: unconnected-(J10-Pin_4-Pad4) -> GND
- J10 pad 5: unconnected-(J10-Pin_5-Pad5) -> GND
- J10 pad 6: unconnected-(J10-Pin_6-Pad6) -> /MIX_R+
- J10 pad 7: unconnected-(J10-Pin_7-Pad7) -> GND
- J10 pad 8: unconnected-(J10-Pin_8-Pad8) -> /MIX_R-
- J11 pad 1: unconnected-(J11-Pin_1-Pad1) -> +15V
- J11 pad 2: unconnected-(J11-Pin_2-Pad2) -> GND
- J11 pad 3: unconnected-(J11-Pin_3-Pad3) -> -15V
- J12 pad 1: unconnected-(J12-Pin_1-Pad1) -> /CH3_PAN_L_CV
- J12 pad 2: unconnected-(J12-Pin_2-Pad2) -> /CH3_PAN_R_CV
- J12 pad 3: unconnected-(J12-Pin_3-Pad3) -> /CH3_INS_PRE_LCV
- J12 pad 4: unconnected-(J12-Pin_4-Pad4) -> /CH3_INSERT_LCV
- J12 pad 5: unconnected-(J12-Pin_5-Pad5) -> GND
- J13 pad 1: unconnected-(J13-Pin_1-Pad1) -> /CH3_EQ_OUT
- J13 pad 2: unconnected-(J13-Pin_2-Pad2) -> /CH3_INPUT_OUT
- J13 pad 3: unconnected-(J13-Pin_3-Pad3) -> GND
- J14 pad 1: unconnected-(J14-Pin_1-Pad1) -> /CH3_INS_RTN
- J14 pad 2: unconnected-(J14-Pin_2-Pad2) -> /CH3_INS_SEND
- J14 pad 3: unconnected-(J14-Pin_3-Pad3) -> GND
- J15 pad 1: unconnected-(J15-Pin_1-Pad1) -> /MIX_L+
- J15 pad 2: unconnected-(J15-Pin_2-Pad2) -> GND
- J15 pad 3: unconnected-(J15-Pin_3-Pad3) -> /MIX_L-
- J15 pad 4: unconnected-(J15-Pin_4-Pad4) -> GND
- J15 pad 5: unconnected-(J15-Pin_5-Pad5) -> GND
- J15 pad 6: unconnected-(J15-Pin_6-Pad6) -> /MIX_R+
- J15 pad 7: unconnected-(J15-Pin_7-Pad7) -> GND
- J15 pad 8: unconnected-(J15-Pin_8-Pad8) -> /MIX_R-
- J16 pad 1: unconnected-(J16-Pin_1-Pad1) -> +15V
- J16 pad 2: unconnected-(J16-Pin_2-Pad2) -> GND
- J16 pad 3: unconnected-(J16-Pin_3-Pad3) -> -15V
- J17 pad 1: unconnected-(J17-Pin_1-Pad1) -> /CH4_PAN_L_CV
- J17 pad 2: unconnected-(J17-Pin_2-Pad2) -> /CH4_PAN_R_CV
- J17 pad 3: unconnected-(J17-Pin_3-Pad3) -> /CH4_INS_PRE_LCV
- J17 pad 4: unconnected-(J17-Pin_4-Pad4) -> /CH4_INSERT_LCV
- J17 pad 5: unconnected-(J17-Pin_5-Pad5) -> GND
- J18 pad 1: unconnected-(J18-Pin_1-Pad1) -> /CH4_EQ_OUT
- J18 pad 2: unconnected-(J18-Pin_2-Pad2) -> /CH4_INPUT_OUT
- J18 pad 3: unconnected-(J18-Pin_3-Pad3) -> GND
- J19 pad 1: unconnected-(J19-Pin_1-Pad1) -> /CH4_INS_RTN
- J19 pad 2: unconnected-(J19-Pin_2-Pad2) -> /CH4_INS_SEND
- J19 pad 3: unconnected-(J19-Pin_3-Pad3) -> GND
- J2 pad 1: unconnected-(J2-Pin_1-Pad1) -> /CH1_PAN_L_CV
- J2 pad 2: unconnected-(J2-Pin_2-Pad2) -> /CH1_PAN_R_CV
- J2 pad 3: unconnected-(J2-Pin_3-Pad3) -> /CH1_INS_PRE_LCV
- J2 pad 4: unconnected-(J2-Pin_4-Pad4) -> /CH1_INSERT_LCV
- J2 pad 5: unconnected-(J2-Pin_5-Pad5) -> GND
- J20 pad 1: unconnected-(J20-Pin_1-Pad1) -> /MIX_L+
- J20 pad 2: unconnected-(J20-Pin_2-Pad2) -> GND
- J20 pad 3: unconnected-(J20-Pin_3-Pad3) -> /MIX_L-
- J20 pad 4: unconnected-(J20-Pin_4-Pad4) -> GND
- J20 pad 5: unconnected-(J20-Pin_5-Pad5) -> GND
- J20 pad 6: unconnected-(J20-Pin_6-Pad6) -> /MIX_R+
- J20 pad 7: unconnected-(J20-Pin_7-Pad7) -> GND
- J20 pad 8: unconnected-(J20-Pin_8-Pad8) -> /MIX_R-
- J3 pad 1: unconnected-(J3-Pin_1-Pad1) -> /CH1_EQ_OUT
- J3 pad 2: unconnected-(J3-Pin_2-Pad2) -> /CH1_INPUT_OUT
- J3 pad 3: unconnected-(J3-Pin_3-Pad3) -> GND
- J4 pad 1: unconnected-(J4-Pin_1-Pad1) -> /CH1_INS_RTN
- J4 pad 2: unconnected-(J4-Pin_2-Pad2) -> /CH1_INS_SEND
- J4 pad 3: unconnected-(J4-Pin_3-Pad3) -> GND
- J5 pad 1: unconnected-(J5-Pin_1-Pad1) -> /MIX_L+
- J5 pad 2: unconnected-(J5-Pin_2-Pad2) -> GND
- J5 pad 3: unconnected-(J5-Pin_3-Pad3) -> /MIX_L-
- J5 pad 4: unconnected-(J5-Pin_4-Pad4) -> GND
- J5 pad 5: unconnected-(J5-Pin_5-Pad5) -> GND
- J5 pad 6: unconnected-(J5-Pin_6-Pad6) -> /MIX_R+
- J5 pad 7: unconnected-(J5-Pin_7-Pad7) -> GND
- J5 pad 8: unconnected-(J5-Pin_8-Pad8) -> /MIX_R-
- J6 pad 1: unconnected-(J6-Pin_1-Pad1) -> +15V
- J6 pad 2: unconnected-(J6-Pin_2-Pad2) -> GND
- J6 pad 3: unconnected-(J6-Pin_3-Pad3) -> -15V
- J7 pad 1: unconnected-(J7-Pin_1-Pad1) -> /CH2_PAN_L_CV
- J7 pad 2: unconnected-(J7-Pin_2-Pad2) -> /CH2_PAN_R_CV
- J7 pad 3: unconnected-(J7-Pin_3-Pad3) -> /CH2_INS_PRE_LCV
- J7 pad 4: unconnected-(J7-Pin_4-Pad4) -> /CH2_INSERT_LCV
- J7 pad 5: unconnected-(J7-Pin_5-Pad5) -> GND
- J8 pad 1: unconnected-(J8-Pin_1-Pad1) -> /CH2_EQ_OUT
- J8 pad 2: unconnected-(J8-Pin_2-Pad2) -> /CH2_INPUT_OUT
- J8 pad 3: unconnected-(J8-Pin_3-Pad3) -> GND
- J9 pad 1: unconnected-(J9-Pin_1-Pad1) -> /CH2_INS_RTN
- J9 pad 2: unconnected-(J9-Pin_2-Pad2) -> /CH2_INS_SEND
- J9 pad 3: unconnected-(J9-Pin_3-Pad3) -> GND
- P1 pad 1: +15 -> +15V
- P1 pad 3: -15 -> -15V
Routing:
- added copper zone on B.Cu, net GND
- added copper zone on F.Cu, net GND
- added copper zone on In1.Cu, net GND
- added copper zone on In2.Cu, net GND
- removed copper zone on B.Cu, net (none)
- removed copper zone on F.Cu, net (none)
- removed copper zone on In1.Cu, net (none)
- removed copper zone on In2.Cu, net (none)
Other:
- board size 146 x 435 mm -> 146 x 433 mm
- board text added: "CH 1"
- board text added: "CH 2"
- board text added: "CH 3"
- board text added: "CH 4"
- board text added: "COMP"
- board text added: "EQ"
- board text added: "INPUT"
- board text added: "MIX+AUX BUS"

Commit message: even more pcbs we're slowly getting there lmaoi
Parts:
- removed J25: CH1_EQ_AUDIO, Connector_PinSocket_2.54mm:PinSocket_1x04_P2.54mm_Vertical
- removed J26: CH1_EQ_LF_HF_CV, Connector_PinSocket_2.54mm:PinSocket_1x08_P2.54mm_Vertical
- removed J27: CH1_EQ_LOGIC, Connector_PinSocket_2.54mm:PinSocket_1x08_P2.54mm_Vertical
- removed J28: CH1_EQ_POWER, Connector_PinSocket_2.54mm:PinSocket_1x03_P2.54mm_Vertical
- removed J29: CH1_EQ_HMF_CV, Connector_PinSocket_2.54mm:PinSocket_1x06_P2.54mm_Vertical
- removed J30: CH1_EQ_LMF_CV, Connector_PinSocket_2.54mm:PinSocket_1x06_P2.54mm_Vertical
- removed J31: CH1_COMP_POWER, Connector_PinSocket_2.54mm:PinSocket_1x04_P2.54mm_Vertical
- removed J32: CH1_COMP_CV_IO, Connector_PinSocket_2.54mm:PinSocket_1x04_P2.54mm_Vertical
- removed J33: CH1_COMP_ENV, Connector_PinSocket_2.54mm:PinSocket_1x04_P2.54mm_Vertical
- removed J34: CH2_IN_LOGIC, Connector_PinSocket_2.54mm:PinSocket_1x08_P2.54mm_Vertical
- removed J35: CH2_IN_CV, Connector_PinSocket_2.54mm:PinSocket_1x02_P2.54mm_Vertical
- removed J36: CH2_IN_AUDIO, Connector_PinSocket_2.54mm:PinSocket_1x10_P2.54mm_Vertical
- removed J37: CH2_IN_POWER, Connector_PinSocket_2.54mm:PinSocket_1x04_P2.54mm_Vertical
- removed J38: CH2_EQ_AUDIO, Connector_PinSocket_2.54mm:PinSocket_1x04_P2.54mm_Vertical
- removed J39: CH2_EQ_LF_HF_CV, Connector_PinSocket_2.54mm:PinSocket_1x08_P2.54mm_Vertical
- removed J40: CH2_EQ_LOGIC, Connector_PinSocket_2.54mm:PinSocket_1x08_P2.54mm_Vertical
- removed J41: CH2_EQ_POWER, Connector_PinSocket_2.54mm:PinSocket_1x03_P2.54mm_Vertical
- removed J42: CH2_EQ_HMF_CV, Connector_PinSocket_2.54mm:PinSocket_1x06_P2.54mm_Vertical
- removed J43: CH2_EQ_LMF_CV, Connector_PinSocket_2.54mm:PinSocket_1x06_P2.54mm_Vertical
- removed J44: CH2_COMP_POWER, Connector_PinSocket_2.54mm:PinSocket_1x04_P2.54mm_Vertical
- removed J45: CH2_COMP_CV_IO, Connector_PinSocket_2.54mm:PinSocket_1x04_P2.54mm_Vertical
- removed J46: CH2_COMP_ENV, Connector_PinSocket_2.54mm:PinSocket_1x04_P2.54mm_Vertical
- removed J47: CH3_IN_LOGIC, Connector_PinSocket_2.54mm:PinSocket_1x08_P2.54mm_Vertical
- removed J48: CH3_IN_CV, Connector_PinSocket_2.54mm:PinSocket_1x02_P2.54mm_Vertical
- removed J49: CH3_IN_AUDIO, Connector_PinSocket_2.54mm:PinSocket_1x10_P2.54mm_Vertical
- removed J50: CH3_IN_POWER, Connector_PinSocket_2.54mm:PinSocket_1x04_P2.54mm_Vertical
- removed J51: CH3_EQ_AUDIO, Connector_PinSocket_2.54mm:PinSocket_1x04_P2.54mm_Vertical
- removed J52: CH3_EQ_LF_HF_CV, Connector_PinSocket_2.54mm:PinSocket_1x08_P2.54mm_Vertical
- removed J53: CH3_EQ_LOGIC, Connector_PinSocket_2.54mm:PinSocket_1x08_P2.54mm_Vertical
- removed J54: CH3_EQ_POWER, Connector_PinSocket_2.54mm:PinSocket_1x03_P2.54mm_Vertical
- removed J55: CH3_EQ_HMF_CV, Connector_PinSocket_2.54mm:PinSocket_1x06_P2.54mm_Vertical
- removed J56: CH3_EQ_LMF_CV, Connector_PinSocket_2.54mm:PinSocket_1x06_P2.54mm_Vertical
- removed J57: CH3_COMP_POWER, Connector_PinSocket_2.54mm:PinSocket_1x04_P2.54mm_Vertical
- removed J58: CH3_COMP_CV_IO, Connector_PinSocket_2.54mm:PinSocket_1x04_P2.54mm_Vertical
- removed J59: CH3_COMP_ENV, Connector_PinSocket_2.54mm:PinSocket_1x04_P2.54mm_Vertical
- removed J60: CH4_IN_LOGIC, Connector_PinSocket_2.54mm:PinSocket_1x08_P2.54mm_Vertical
- removed J61: CH4_IN_CV, Connector_PinSocket_2.54mm:PinSocket_1x02_P2.54mm_Vertical
- removed J62: CH4_IN_AUDIO, Connector_PinSocket_2.54mm:PinSocket_1x10_P2.54mm_Vertical
- removed J63: CH4_IN_POWER, Connector_PinSocket_2.54mm:PinSocket_1x04_P2.54mm_Vertical
- removed J64: CH4_EQ_AUDIO, Connector_PinSocket_2.54mm:PinSocket_1x04_P2.54mm_Vertical
- removed J65: CH4_EQ_LF_HF_CV, Connector_PinSocket_2.54mm:PinSocket_1x08_P2.54mm_Vertical
- removed J66: CH4_EQ_LOGIC, Connector_PinSocket_2.54mm:PinSocket_1x08_P2.54mm_Vertical
- removed J67: CH4_EQ_POWER, Connector_PinSocket_2.54mm:PinSocket_1x03_P2.54mm_Vertical
- removed J68: CH4_EQ_HMF_CV, Connector_PinSocket_2.54mm:PinSocket_1x06_P2.54mm_Vertical
- removed J69: CH4_EQ_LMF_CV, Connector_PinSocket_2.54mm:PinSocket_1x06_P2.54mm_Vertical
- removed J70: CH4_COMP_POWER, Connector_PinSocket_2.54mm:PinSocket_1x04_P2.54mm_Vertical
- removed J71: CH4_COMP_CV_IO, Connector_PinSocket_2.54mm:PinSocket_1x04_P2.54mm_Vertical
- removed J72: CH4_COMP_ENV, Connector_PinSocket_2.54mm:PinSocket_1x04_P2.54mm_Vertical
- added A1: CH1 INPUT, My Footprints:INPUT_CARD, F.Cu at (20.2, 33.0)
- added A10: CH2 SENDS, My Footprints:SENDS_CARD, F.Cu at (92.8, 326.0)
- added A11: CH3 INPUT, My Footprints:INPUT_CARD, F.Cu at (93.2, 33.0)
- added A12: CH3 EQ, My Footprints:EQ_CARD, B.Cu at (129.2, 146.0)
- added A13: CH3 COMP, My Footprints:COMP_CARD, B.Cu at (129.2, 120.8)
- added A14: CH3 FADER VCA, My Footprints:FADER_VCA_CARD, F.Cu at (129.2, 234.5)
- added A15: CH3 SENDS, My Footprints:SENDS_CARD, F.Cu at (129.2, 326.0)
- added A16: CH4 INPUT, My Footprints:INPUT_CARD, F.Cu at (129.8, 33.0)
- added A17: CH4 EQ, My Footprints:EQ_CARD, B.Cu at (165.8, 146.0)
- added A18: CH4 COMP, My Footprints:COMP_CARD, B.Cu at (165.8, 120.8)
- added A19: CH4 FADER VCA, My Footprints:FADER_VCA_CARD, F.Cu at (165.8, 234.5)
- added A2: CH1 EQ, My Footprints:EQ_CARD, B.Cu at (56.2, 146.0)
- added A20: CH4 SENDS, My Footprints:SENDS_CARD, F.Cu at (165.8, 326.0)
- added A3: CH1 COMP, My Footprints:COMP_CARD, B.Cu at (56.2, 120.8)
- added A4: CH1 FADER VCA, My Footprints:FADER_VCA_CARD, F.Cu at (56.2, 234.5)
- added A5: CH1 SENDS, My Footprints:SENDS_CARD, F.Cu at (56.2, 326.0)
- added A6: CH2 INPUT, My Footprints:INPUT_CARD, F.Cu at (56.8, 33.0)
- added A7: CH2 EQ, My Footprints:EQ_CARD, B.Cu at (92.8, 146.0)
- added A8: CH2 COMP, My Footprints:COMP_CARD, B.Cu at (92.8, 120.8)
- added A9: CH2 FADER VCA, My Footprints:FADER_VCA_CARD, F.Cu at (92.8, 234.5)
- added C1: 100n, Capacitor_SMD:C_0603_1608Metric, F.Cu at (47.0, 137.2)
- added C10: 100n, Capacitor_SMD:C_0603_1608Metric, F.Cu at (156.2, 137.2)
- added C11: 100n, Capacitor_SMD:C_0603_1608Metric, F.Cu at (145.4, 136.5)
- added C12: 100n, Capacitor_SMD:C_0603_1608Metric, F.Cu at (156.2, 139.1)
- added C13: 1u, Capacitor_SMD:C_0603_1608Metric, F.Cu at (36.2, 267.3)
- added C14: 100n, Capacitor_SMD:C_0603_1608Metric, F.Cu at (48.3, 267.3)
- added C15: 100n, Capacitor_SMD:C_0603_1608Metric, F.Cu at (73.0, 267.3)
- added C16: 100n, Capacitor_SMD:C_0603_1608Metric, F.Cu at (85.1, 267.3)
- added C17: 100n, Capacitor_SMD:C_0603_1608Metric, F.Cu at (109.2, 267.3)
- added C18: 100n, Capacitor_SMD:C_0603_1608Metric, F.Cu at (121.3, 267.3)
- added C19: 100n, Capacitor_SMD:C_0603_1608Metric, F.Cu at (146.1, 267.3)
- added C2: 100n, Capacitor_SMD:C_0603_1608Metric, F.Cu at (36.2, 136.5)
- added C20: 100n, Capacitor_SMD:C_0603_1608Metric, F.Cu at (158.1, 267.3)
- added C21: 100n, Capacitor_SMD:C_0603_1608Metric, F.Cu at (36.2, 275.6)
- added C3: 100n, Capacitor_SMD:C_0603_1608Metric, F.Cu at (47.0, 139.1)
- added C4: 100n, Capacitor_SMD:C_0603_1608Metric, F.Cu at (83.2, 137.2)
- added C5: 100n, Capacitor_SMD:C_0603_1608Metric, F.Cu at (72.4, 136.5)
- added C6: 100n, Capacitor_SMD:C_0603_1608Metric, F.Cu at (83.2, 139.1)
- added C7: 100n, Capacitor_SMD:C_0603_1608Metric, F.Cu at (120.0, 137.2)
- added C8: 100n, Capacitor_SMD:C_0603_1608Metric, F.Cu at (109.2, 136.5)
- added C9: 100n, Capacitor_SMD:C_0603_1608Metric, F.Cu at (120.0, 139.1)
- added H1: M3 console standoff, MountingHole:MountingHole_3.2mm_M3, F.Cu at (26.0, 26.5)
- added H2: M3 console standoff, MountingHole:MountingHole_3.2mm_M3, F.Cu at (160.0, 26.5)
- added H3: M3 console standoff, MountingHole:MountingHole_3.2mm_M3, F.Cu at (26.0, 332.0)
- added H4: M3 console standoff, MountingHole:MountingHole_3.2mm_M3, F.Cu at (160.0, 332.0)
- added H55: MountingHole, MountingHole:MountingHole_2.2mm_M2, F.Cu at (162.8, 149.0)
- added H56: MountingHole, MountingHole:MountingHole_2.2mm_M2, F.Cu at (132.8, 149.0)
- added H57: MountingHole, MountingHole:MountingHole_2.2mm_M2, F.Cu at (162.8, 323.0)
- added H58: MountingHole, MountingHole:MountingHole_2.2mm_M2, F.Cu at (132.8, 323.0)
- added H59: MountingHole, MountingHole:MountingHole_2.2mm_M2, F.Cu at (162.7, 129.0)
- added H60: MountingHole, MountingHole:MountingHole_2.2mm_M2, F.Cu at (141.5, 136.8)
- added H61: MountingHole, MountingHole:MountingHole_2.2mm_M2, F.Cu at (134.1, 132.7)
- added H62: MountingHole, MountingHole:MountingHole_2.2mm_M2, F.Cu at (145.8, 230.9)
- added H63: MountingHole, MountingHole:MountingHole_2.2mm_M2, F.Cu at (161.8, 157.5)
- added H64: MountingHole, MountingHole:MountingHole_2.2mm_M2, F.Cu at (147.8, 323.2)
- added H65: MountingHole, MountingHole:MountingHole_2.2mm_M2, F.Cu at (163.0, 237.8)
- added H66: MountingHole, MountingHole:MountingHole_2.2mm_M2, F.Cu at (132.5, 237.8)
- added R1: 100k, Resistor_SMD:R_0603_1608Metric, F.Cu at (36.2, 139.7)
- added R2: 100k, Resistor_SMD:R_0603_1608Metric, F.Cu at (72.4, 139.7)
- added R3: 100k, Resistor_SMD:R_0603_1608Metric, F.Cu at (109.2, 139.7)
- added R4: 100k, Resistor_SMD:R_0603_1608Metric, F.Cu at (145.4, 139.7)
- added R5: 1M, Resistor_SMD:R_0603_1608Metric, F.Cu at (36.2, 277.5)
- added R6: 1k, Resistor_SMD:R_0603_1608Metric, F.Cu at (33.7, 276.2)
- added U1: ADG1412, Package_SO:TSSOP-16_4.4x5mm_P0.65mm, F.Cu at (41.3, 137.8)
- added U10: 74HC595, Package_SO:TSSOP-16_4.4x5mm_P0.65mm, F.Cu at (118.1, 271.8)
- added U11: 74HC595, Package_SO:TSSOP-16_4.4x5mm_P0.65mm, F.Cu at (142.9, 271.8)
- added U12: 74HC595, Package_SO:TSSOP-16_4.4x5mm_P0.65mm, F.Cu at (154.9, 271.8)
- added U2: ADG1412, Package_SO:TSSOP-16_4.4x5mm_P0.65mm, F.Cu at (77.5, 137.8)
- added U3: ADG1412, Package_SO:TSSOP-16_4.4x5mm_P0.65mm, F.Cu at (114.3, 137.8)
- added U4: ADG1412, Package_SO:TSSOP-16_4.4x5mm_P0.65mm, F.Cu at (150.5, 137.8)
- added U5: 74HC595, Package_SO:TSSOP-16_4.4x5mm_P0.65mm, F.Cu at (33.0, 271.8)
- added U6: 74HC595, Package_SO:TSSOP-16_4.4x5mm_P0.65mm, F.Cu at (45.1, 271.8)
- added U7: 74HC595, Package_SO:TSSOP-16_4.4x5mm_P0.65mm, F.Cu at (69.8, 271.8)
- added U8: 74HC595, Package_SO:TSSOP-16_4.4x5mm_P0.65mm, F.Cu at (81.9, 271.8)
- added U9: 74HC595, Package_SO:TSSOP-16_4.4x5mm_P0.65mm, F.Cu at (106.0, 271.8)
- J1: value CH1_PF_POWER -> CH1_DAC_OUT1; footprint Connector_PinSocket_2.54mm:PinSocket_1x03_P2.54mm_Vertical -> Connector_PinSocket_1.27mm:PinSocket_2x10_P1.27mm_Vertical; moved to B.Cu
- J10: value CH2_PF_MIX_BUS -> CH2_COMP_CV_LINK; footprint Connector_PinSocket_2.54mm:PinSocket_1x08_P2.54mm_Vertical -> Connector_PinHeader_2.54mm:PinHeader_1x02_P2.54mm_Vertical
- J11: value CH3_PF_POWER -> CH3_DAC_OUT1; footprint Connector_PinSocket_2.54mm:PinSocket_1x03_P2.54mm_Vertical -> Connector_PinSocket_1.27mm:PinSocket_2x10_P1.27mm_Vertical; moved to B.Cu
- J12: value CH3_PF_CV -> CH3_DAC_OUT2; footprint Connector_PinSocket_2.54mm:PinSocket_1x05_P2.54mm_Vertical -> Connector_PinSocket_1.27mm:PinSocket_2x10_P1.27mm_Vertical; moved to B.Cu
- J13: value CH3_PF_AUD_IN -> CH3_AUDIO_IN; footprint Connector_PinSocket_2.54mm:PinSocket_1x03_P2.54mm_Vertical -> Connector_PinHeader_2.54mm:PinHeader_1x08_P2.54mm_Vertical; moved to B.Cu
- J14: value CH3_PF_INSERT -> CH3_INSERT; footprint Connector_PinSocket_2.54mm:PinSocket_1x03_P2.54mm_Vertical -> Connector_PinHeader_2.54mm:PinHeader_1x04_P2.54mm_Vertical; moved to B.Cu
- J15: value CH3_PF_MIX_BUS -> CH3_COMP_CV_LINK; footprint Connector_PinSocket_2.54mm:PinSocket_1x08_P2.54mm_Vertical -> Connector_PinHeader_2.54mm:PinHeader_1x02_P2.54mm_Vertical
- J16: value CH4_PF_POWER -> CH4_DAC_OUT1; footprint Connector_PinSocket_2.54mm:PinSocket_1x03_P2.54mm_Vertical -> Connector_PinSocket_1.27mm:PinSocket_2x10_P1.27mm_Vertical; moved to B.Cu
- J17: value CH4_PF_CV -> CH4_DAC_OUT2; footprint Connector_PinSocket_2.54mm:PinSocket_1x05_P2.54mm_Vertical -> Connector_PinSocket_1.27mm:PinSocket_2x10_P1.27mm_Vertical; moved to B.Cu
- J18: value CH4_PF_AUD_IN -> CH4_AUDIO_IN; footprint Connector_PinSocket_2.54mm:PinSocket_1x03_P2.54mm_Vertical -> Connector_PinHeader_2.54mm:PinHeader_1x08_P2.54mm_Vertical; moved to B.Cu
- J19: value CH4_PF_INSERT -> CH4_INSERT; footprint Connector_PinSocket_2.54mm:PinSocket_1x03_P2.54mm_Vertical -> Connector_PinHeader_2.54mm:PinHeader_1x04_P2.54mm_Vertical; moved to B.Cu
- J2: value CH1_PF_CV -> CH1_DAC_OUT2; footprint Connector_PinSocket_2.54mm:PinSocket_1x05_P2.54mm_Vertical -> Connector_PinSocket_1.27mm:PinSocket_2x10_P1.27mm_Vertical; moved to B.Cu
- J20: value CH4_PF_MIX_BUS -> CH4_COMP_CV_LINK; footprint Connector_PinSocket_2.54mm:PinSocket_1x08_P2.54mm_Vertical -> Connector_PinHeader_2.54mm:PinHeader_1x02_P2.54mm_Vertical
- J21: value CH1_IN_LOGIC -> SPI_A; footprint Connector_PinSocket_2.54mm:PinSocket_1x08_P2.54mm_Vertical -> Connector_IDC:IDC-Header_2x05_P2.54mm_Vertical; moved to B.Cu
- J22: value CH1_IN_AUDIO -> SPI_B; footprint Connector_PinSocket_2.54mm:PinSocket_1x10_P2.54mm_Vertical -> Connector_IDC:IDC-Header_2x05_P2.54mm_Vertical; moved to B.Cu
- J23: value CH1_IN_POWER -> ENV_TO_CONTROLLER; footprint Connector_PinSocket_2.54mm:PinSocket_1x04_P2.54mm_Vertical -> Connector_PinHeader_2.54mm:PinHeader_1x08_P2.54mm_Vertical; moved to B.Cu
- J24: value CH1_IN_CV -> SHIFTREG_IN; footprint Connector_PinSocket_2.54mm:PinSocket_1x02_P2.54mm_Vertical -> Connector_PinHeader_2.54mm:PinHeader_1x08_P2.54mm_Vertical; moved to B.Cu
- J3: value CH1_PF_AUD_IN -> CH1_AUDIO_IN; footprint Connector_PinSocket_2.54mm:PinSocket_1x03_P2.54mm_Vertical -> Connector_PinHeader_2.54mm:PinHeader_1x08_P2.54mm_Vertical; moved to B.Cu
- J4: value CH1_PF_INSERT -> CH1_INSERT; footprint Connector_PinSocket_2.54mm:PinSocket_1x03_P2.54mm_Vertical -> Connector_PinHeader_2.54mm:PinHeader_1x04_P2.54mm_Vertical; moved to B.Cu
- J5: value CH1_PF_MIX_BUS -> CH1_COMP_CV_LINK; footprint Connector_PinSocket_2.54mm:PinSocket_1x08_P2.54mm_Vertical -> Connector_PinHeader_2.54mm:PinHeader_1x02_P2.54mm_Vertical
- J6: value CH2_PF_POWER -> CH2_DAC_OUT1; footprint Connector_PinSocket_2.54mm:PinSocket_1x03_P2.54mm_Vertical -> Connector_PinSocket_1.27mm:PinSocket_2x10_P1.27mm_Vertical; moved to B.Cu
- J7: value CH2_PF_CV -> CH2_DAC_OUT2; footprint Connector_PinSocket_2.54mm:PinSocket_1x05_P2.54mm_Vertical -> Connector_PinSocket_1.27mm:PinSocket_2x10_P1.27mm_Vertical; moved to B.Cu
- J8: value CH2_PF_AUD_IN -> CH2_AUDIO_IN; footprint Connector_PinSocket_2.54mm:PinSocket_1x03_P2.54mm_Vertical -> Connector_PinHeader_2.54mm:PinHeader_1x08_P2.54mm_Vertical; moved to B.Cu
- J9: value CH2_PF_INSERT -> CH2_INSERT; footprint Connector_PinSocket_2.54mm:PinSocket_1x03_P2.54mm_Vertical -> Connector_PinHeader_2.54mm:PinHeader_1x04_P2.54mm_Vertical; moved to B.Cu
- moved H8 366.4 mm to (43.9, 57.6)
- moved J8 347.3 mm to (66.7, 69.8), turned to 0 degrees
- moved J3 347.3 mm to (30.5, 69.8), turned to 0 degrees
- moved J18 347.3 mm to (139.7, 69.8), turned to 0 degrees
- moved J13 347.3 mm to (103.5, 69.8), turned to 0 degrees
- moved J17 337.5 mm to (147.3, 40.0), turned to 0 degrees
- moved J7 337.5 mm to (74.3, 40.0), turned to 0 degrees
- moved J12 337.5 mm to (110.5, 40.0), turned to 0 degrees
- moved J2 337.5 mm to (37.5, 40.0), turned to 0 degrees
- moved J9 330.7 mm to (66.7, 95.9), turned to 0 degrees
- moved J4 330.7 mm to (30.5, 95.9), turned to 0 degrees
- moved J19 330.7 mm to (139.7, 95.9), turned to 0 degrees
- moved J14 330.7 mm to (103.5, 95.9), turned to 0 degrees
- moved H15 325.0 mm to (32.0, 136.8)
- moved H9 323.7 mm to (31.2, 125.2)
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Connections:
- J1 pad 1: +15V -> GND
- J1 pad 2: GND -> /CH1_CV_HMF_G
- J1 pad 3: -15V -> /CH1_CV_HF_G
- J10 pad 1: /MIX_L+ -> /CH2_COMP_CV
- J11 pad 1: +15V -> GND
- J11 pad 2: GND -> /CH3_CV_HMF_G
- J11 pad 3: -15V -> /CH3_CV_HF_G
- J12 pad 1: /CH3_PAN_L_CV -> GND
- J12 pad 2: /CH3_PAN_R_CV -> /CH3_CV_SEND2_L
- J12 pad 3: /CH3_INS_PRE_LCV -> /CH3_CV_HMF_Q
- J12 pad 4: /CH3_INSERT_LCV -> GND
- J13 pad 1: /CH3_EQ_OUT -> /CH3_MIC_HOT
- J13 pad 2: /CH3_INPUT_OUT -> /CH3_MIC_COLD
- J14 pad 1: /CH3_INS_RTN -> /CH3_INS_SEND
- J14 pad 2: /CH3_INS_SEND -> GND
- J14 pad 3: GND -> /CH3_INS_RTN
- J15 pad 1: /MIX_L+ -> /CH3_COMP_CV
- J16 pad 1: +15V -> GND
- J16 pad 2: GND -> /CH4_CV_HMF_G
- J16 pad 3: -15V -> /CH4_CV_HF_G
- J17 pad 1: /CH4_PAN_L_CV -> GND
- J17 pad 2: /CH4_PAN_R_CV -> /CH4_CV_SEND2_L
- J17 pad 3: /CH4_INS_PRE_LCV -> /CH4_CV_HMF_Q
- J17 pad 4: /CH4_INSERT_LCV -> GND
- J18 pad 1: /CH4_EQ_OUT -> /CH4_MIC_HOT
- J18 pad 2: /CH4_INPUT_OUT -> /CH4_MIC_COLD
- J19 pad 1: /CH4_INS_RTN -> /CH4_INS_SEND
- J19 pad 2: /CH4_INS_SEND -> GND
- J19 pad 3: GND -> /CH4_INS_RTN
- J2 pad 1: /CH1_PAN_L_CV -> GND
- J2 pad 2: /CH1_PAN_R_CV -> /CH1_CV_SEND2_L
- J2 pad 3: /CH1_INS_PRE_LCV -> /CH1_CV_HMF_Q
- J2 pad 4: /CH1_INSERT_LCV -> GND
- J20 pad 1: /MIX_L+ -> /CH4_COMP_CV
- J21 pad 1: /CH1_P48_LCV -> /SPI_SCK
- J21 pad 2: /CH1_MIC_SEL_LCV -> GND
- J21 pad 3: /CH1_LINE_SEL_LCV -> /SPI_MOSI
- J21 pad 4: /CH1_HIZ_SEL_LCV -> GND
- J21 pad 5: /CH1_PHASE_LCV -> /SPI_MISO
- J21 pad 6: /CH1_HPF_LCV -> GND
- J21 pad 7: /CH1_PAD_LCV -> /SPI_CS
- J22 pad 1: /CH1_MIC_HOT -> /SPI_SCK
- J22 pad 10: /CH1_INPUT_OUT -> GND
- J22 pad 2: /CH1_MIC_COLD -> GND
- J22 pad 3: GND -> /SPI_MOSI
- J22 pad 4: /CH1_LINE_HOT -> GND
- J22 pad 5: /CH1_LINE_COLD -> /SPI_MISO
- J22 pad 7: /CH1_HIZ_IN -> /SPI_CS
- J22 pad 9: GND -> unconnected-(J22-Pin_9-Pad9)
- J23 pad 1: +48V -> /CH1_ENV_ADC
- J23 pad 2: +15V -> GND
- J23 pad 3: GND -> /CH2_ENV_ADC
- J23 pad 4: -15V -> GND
- J24 pad 1: /CH1_GAIN_CV -> /LOGIC SHIFT REGISTERS/SR_DAT
- J3 pad 1: /CH1_EQ_OUT -> /CH1_MIC_HOT
- J3 pad 2: /CH1_INPUT_OUT -> /CH1_MIC_COLD
- J4 pad 1: /CH1_INS_RTN -> /CH1_INS_SEND
- J4 pad 2: /CH1_INS_SEND -> GND
- J4 pad 3: GND -> /CH1_INS_RTN
- J5 pad 1: /MIX_L+ -> /CH1_COMP_CV
- J6 pad 1: +15V -> GND
- J6 pad 2: GND -> /CH2_CV_HMF_G
- J6 pad 3: -15V -> /CH2_CV_HF_G
- J7 pad 1: /CH2_PAN_L_CV -> GND
- J7 pad 2: /CH2_PAN_R_CV -> /CH2_CV_SEND2_L
- J7 pad 3: /CH2_INS_PRE_LCV -> /CH2_CV_HMF_Q
- J7 pad 4: /CH2_INSERT_LCV -> GND
- J73 pad 22: (no net) -> unconnected-(J73-Pin_22-Pad22)
- J73 pad 23: (no net) -> unconnected-(J73-Pin_23-Pad23)
- J74 pad 22: (no net) -> unconnected-(J74-Pin_22-Pad22)
- J74 pad 23: (no net) -> unconnected-(J74-Pin_23-Pad23)
- J8 pad 1: /CH2_EQ_OUT -> /CH2_MIC_HOT
- J8 pad 2: /CH2_INPUT_OUT -> /CH2_MIC_COLD
- J9 pad 1: /CH2_INS_RTN -> /CH2_INS_SEND
- J9 pad 2: /CH2_INS_SEND -> GND
- J9 pad 3: GND -> /CH2_INS_RTN
- P2 pad 3: (no net) -> unconnected-(P2-Pin_3-Pad3)
Other:
- board size 146 x 433 mm -> 146 x 318 mm
- board text removed: "COMP"
- board text removed: "EQ"
- board text removed: "FADER VCA"
- board text removed: "INPUT"
