File: PCB_CAD/01 Analog/SENDS/SENDS.kicad_pcb (KiCad board)
At the start: 4 copper layers, 36 x 80 mm, 0 parts

Commit message: even more pcbs we're slowly getting there lmaoi
Parts:
- added C1: 22p C0G, Capacitor_SMD:C_0603_1608Metric, F.Cu at (62.6, 113.2)
- added C10: 47p C0G, Capacitor_SMD:C_0603_1608Metric, F.Cu at (73.4, 83.8)
- added C11: 10u, Capacitor_SMD:CP_Elec_6.3x5.4_Nichicon, F.Cu at (78.8, 71.7)
- added C12: 1200p C0G, Capacitor_SMD:C_0603_1608Metric, F.Cu at (81.3, 81.2)
- added C13: 47p C0G, Capacitor_SMD:C_0603_1608Metric, F.Cu at (73.4, 80.2)
- added C14: 10u, Capacitor_SMD:CP_Elec_6.3x5.4_Nichicon, F.Cu at (57.2, 105.0)
- added C15: 1200p C0G, Capacitor_SMD:C_0603_1608Metric, F.Cu at (57.1, 118.0)
- added C16: 47p C0G, Capacitor_SMD:C_0603_1608Metric, F.Cu at (62.6, 116.7)
- added C17: 10u, Capacitor_SMD:CP_Elec_6.3x5.4_Nichicon, F.Cu at (64.4, 105.0)
- added C18: 1200p C0G, Capacitor_SMD:C_0603_1608Metric, F.Cu at (69.8, 108.5)
- added C19: 47p C0G, Capacitor_SMD:C_0603_1608Metric, F.Cu at (73.4, 116.7)
- added C2: 10u, Capacitor_SMD:CP_Elec_6.3x5.4_Nichicon, F.Cu at (57.2, 71.7)
- added C20: 10u, Capacitor_SMD:CP_Elec_6.3x5.4_Nichicon, F.Cu at (78.8, 105.0)
- added C21: 2.2n C0G, Capacitor_SMD:C_0603_1608Metric, F.Cu at (78.7, 118.0)
- added C22: 100p C0G, Capacitor_SMD:C_0603_1608Metric, F.Cu at (73.4, 113.2)
- added C23: 6.8n C0G, Capacitor_SMD:C_0603_1608Metric, F.Cu at (57.7, 56.7)
- added C24: 1.2n C0G, Capacitor_SMD:C_0603_1608Metric, F.Cu at (62.8, 56.7)
- added C25: 6.8n C0G, Capacitor_SMD:C_0603_1608Metric, F.Cu at (57.7, 63.1)
- added C26: 1.2n C0G, Capacitor_SMD:C_0603_1608Metric, F.Cu at (62.8, 63.1)
- added C27: 6.8n C0G, Capacitor_SMD:C_0603_1608Metric, F.Cu at (78.3, 63.1)
- added C28: 1.2n C0G, Capacitor_SMD:C_0603_1608Metric, F.Cu at (73.2, 63.1)
- added C29: 6.8n C0G, Capacitor_SMD:C_0603_1608Metric, F.Cu at (78.3, 56.7)
- added C3: 1200p C0G, Capacitor_SMD:C_0603_1608Metric, F.Cu at (57.1, 84.3)
- added C30: 1.2n C0G, Capacitor_SMD:C_0603_1608Metric, F.Cu at (73.2, 56.7)
- added C31: 6.8n C0G, Capacitor_SMD:C_0603_1608Metric, F.Cu at (57.7, 90.3)
- added C32: 1.2n C0G, Capacitor_SMD:C_0603_1608Metric, F.Cu at (62.8, 90.3)
- added C33: 6.8n C0G, Capacitor_SMD:C_0603_1608Metric, F.Cu at (57.7, 96.7)
- added C34: 1.2n C0G, Capacitor_SMD:C_0603_1608Metric, F.Cu at (62.8, 96.7)
- added C35: 6.8n C0G, Capacitor_SMD:C_0603_1608Metric, F.Cu at (78.3, 96.7)
- added C36: 1.2n C0G, Capacitor_SMD:C_0603_1608Metric, F.Cu at (73.2, 96.7)
- added C37: 100n, Capacitor_SMD:C_0603_1608Metric, F.Cu at (78.7, 90.0)
- added C38: 100n, Capacitor_SMD:C_0603_1608Metric, F.Cu at (78.7, 79.9)
- added C39: 100n, Capacitor_SMD:C_0603_1608Metric, F.Cu at (73.7, 60.2)
- added C4: 47p C0G, Capacitor_SMD:C_0603_1608Metric, F.Cu at (62.6, 80.2)
- added C40: 100n, Capacitor_SMD:C_0603_1608Metric, F.Cu at (71.8, 110.4)
- added C41: 100n, Capacitor_SMD:C_0603_1608Metric, F.Cu at (74.3, 93.2)
- added C42: 100n, Capacitor_SMD:C_0603_1608Metric, F.Cu at (66.0, 85.6)
- added C43: 100n, Capacitor_SMD:C_0603_1608Metric, F.Cu at (69.8, 85.6)
- added C44: 100n, Capacitor_SMD:C_0603_1608Metric, F.Cu at (66.0, 118.6)
- added C45: 100n, Capacitor_SMD:C_0603_1608Metric, F.Cu at (69.8, 118.6)
- added C46: 100n, Capacitor_SMD:C_0603_1608Metric, F.Cu at (62.2, 60.2)
- added C47: 100n, Capacitor_SMD:C_0603_1608Metric, F.Cu at (76.0, 59.9)
- added C48: 100n, Capacitor_SMD:C_0603_1608Metric, F.Cu at (62.2, 93.2)
- added C49: 100n, Capacitor_SMD:C_0603_1608Metric, F.Cu at (73.7, 90.0)
- added C5: 10u, Capacitor_SMD:CP_Elec_6.3x5.4_Nichicon, F.Cu at (64.4, 71.7)
- added C50: 22u 25V, Capacitor_SMD:C_1210_3225Metric, F.Cu at (76.6, 134.0)
- added C51: 22u 25V, Capacitor_SMD:C_1210_3225Metric, F.Cu at (76.6, 128.9)
- added C6: 1200p C0G, Capacitor_SMD:C_0603_1608Metric, F.Cu at (69.2, 87.5)
- added C7: 47p C0G, Capacitor_SMD:C_0603_1608Metric, F.Cu at (62.6, 83.8)
- added C8: 10u, Capacitor_SMD:CP_Elec_6.3x5.4_Nichicon, F.Cu at (71.6, 71.7)
- added C9: 1200p C0G, Capacitor_SMD:C_0603_1608Metric, F.Cu at (57.1, 60.2)
- added H1: MountingScrew, MountingHole:MountingHole_2.2mm_M2, F.Cu at (68.0, 52.8)
- added H2: MountingScrew, MountingHole:MountingHole_2.2mm_M2, F.Cu at (52.8, 138.2)
- added H3: MountingScrew, MountingHole:MountingHole_2.2mm_M2, F.Cu at (83.2, 138.2)
- added J1: POWER, Connector_PinHeader_2.54mm:PinHeader_1x03_P2.54mm_Vertical, B.Cu at (72.5, 134.0)
- added J2: CV_IN, Connector_PinHeader_2.54mm:PinHeader_2x07_P2.54mm_Vertical, B.Cu at (65.0, 138.8)
- added J3: AUDIO_IO, Connector_PinHeader_2.54mm:PinHeader_2x08_P2.54mm_Vertical, B.Cu at (57.5, 138.8)
- added R1: 20k 0.1%, Resistor_SMD:R_0603_1608Metric, F.Cu at (61.3, 110.8)
- added R10: 10k, Resistor_SMD:R_0603_1608Metric, F.Cu at (61.3, 86.2)
- added R11: 20k 0.1%, Resistor_SMD:R_0603_1608Metric, F.Cu at (68.6, 65.9)
- added R12: 220, Resistor_SMD:R_0603_1608Metric, F.Cu at (65.4, 65.9)
- added R13: 20k 0.1%, Resistor_SMD:R_0603_1608Metric, F.Cu at (75.9, 83.8)
- added R14: 10k, Resistor_SMD:R_0603_1608Metric, F.Cu at (74.7, 86.2)
- added R15: 20k 0.1%, Resistor_SMD:R_0603_1608Metric, F.Cu at (78.1, 77.3)
- added R16: 220, Resistor_SMD:R_0603_1608Metric, F.Cu at (81.3, 78.0)
- added R17: 20k 0.1%, Resistor_SMD:R_0603_1608Metric, F.Cu at (75.9, 80.2)
- added R18: 10k, Resistor_SMD:R_0603_1608Metric, F.Cu at (74.7, 77.8)
- added R19: 20k 0.1%, Resistor_SMD:R_0603_1608Metric, F.Cu at (57.1, 111.6)
- added R2: 20k 0.1%, Resistor_SMD:R_0603_1608Metric, F.Cu at (60.1, 113.2)
- added R20: 220, Resistor_SMD:R_0603_1608Metric, F.Cu at (57.1, 114.8)
- added R21: 20k 0.1%, Resistor_SMD:R_0603_1608Metric, F.Cu at (60.1, 116.7)
- added R22: 10k, Resistor_SMD:R_0603_1608Metric, F.Cu at (61.3, 119.2)
- added R23: 20k 0.1%, Resistor_SMD:R_0603_1608Metric, F.Cu at (66.0, 111.0)
- added R24: 220, Resistor_SMD:R_0603_1608Metric, F.Cu at (69.2, 111.0)
- added R25: 20k 0.1%, Resistor_SMD:R_0603_1608Metric, F.Cu at (75.9, 116.7)
- added R26: 10k, Resistor_SMD:R_0603_1608Metric, F.Cu at (74.7, 119.2)
- added R27: 10k 0.1%, Resistor_SMD:R_0603_1608Metric, F.Cu at (78.7, 111.6)
- added R28: 110, Resistor_SMD:R_0603_1608Metric, F.Cu at (78.7, 114.8)
- added R29: 10k 0.1%, Resistor_SMD:R_0603_1608Metric, F.Cu at (75.9, 113.2)
- added R3: 20k 0.1%, Resistor_SMD:R_0603_1608Metric, F.Cu at (57.1, 78.0)
- added R30: 10k, Resistor_SMD:R_0603_1608Metric, F.Cu at (74.7, 110.8)
- added R31: 100k, Resistor_SMD:R_0603_1608Metric, F.Cu at (52.6, 56.7)
- added R32: 200k 0.1%, Resistor_SMD:R_0603_1608Metric, F.Cu at (54.5, 54.1)
- added R33: 274k 0.1%, Resistor_SMD:R_0603_1608Metric, F.Cu at (55.2, 56.7)
- added R34: 42.2k 0.1%, Resistor_SMD:R_0603_1608Metric, F.Cu at (58.0, 54.1)
- added R35: 357k 0.1%, Resistor_SMD:R_0603_1608Metric, F.Cu at (61.5, 54.1)
- added R36: 78.7k 0.1%, Resistor_SMD:R_0603_1608Metric, F.Cu at (60.3, 56.7)
- added R37: 100k, Resistor_SMD:R_0603_1608Metric, F.Cu at (52.6, 63.1)
- added R38: 200k 0.1%, Resistor_SMD:R_0603_1608Metric, F.Cu at (54.5, 65.7)
- added R39: 274k 0.1%, Resistor_SMD:R_0603_1608Metric, F.Cu at (55.2, 63.1)
- added R4: 220, Resistor_SMD:R_0603_1608Metric, F.Cu at (57.1, 81.2)
- added R40: 42.2k 0.1%, Resistor_SMD:R_0603_1608Metric, F.Cu at (58.0, 65.7)
- added R41: 357k 0.1%, Resistor_SMD:R_0603_1608Metric, F.Cu at (61.5, 65.7)
- added R42: 78.7k 0.1%, Resistor_SMD:R_0603_1608Metric, F.Cu at (60.3, 63.1)
- added R43: 100k, Resistor_SMD:R_0603_1608Metric, F.Cu at (83.4, 63.1)
- added R44: 200k 0.1%, Resistor_SMD:R_0603_1608Metric, F.Cu at (81.5, 65.7)
- added R45: 274k 0.1%, Resistor_SMD:R_0603_1608Metric, F.Cu at (80.8, 63.1)
- added R46: 42.2k 0.1%, Resistor_SMD:R_0603_1608Metric, F.Cu at (78.0, 65.7)
- added R47: 357k 0.1%, Resistor_SMD:R_0603_1608Metric, F.Cu at (74.5, 65.7)
- added R48: 78.7k 0.1%, Resistor_SMD:R_0603_1608Metric, F.Cu at (75.7, 63.1)
- added R49: 100k, Resistor_SMD:R_0603_1608Metric, F.Cu at (83.4, 56.7)
- added R5: 20k 0.1%, Resistor_SMD:R_0603_1608Metric, F.Cu at (60.1, 80.2)
- added R50: 200k 0.1%, Resistor_SMD:R_0603_1608Metric, F.Cu at (81.5, 54.1)
- added R51: 274k 0.1%, Resistor_SMD:R_0603_1608Metric, F.Cu at (80.8, 56.7)
- added R52: 42.2k 0.1%, Resistor_SMD:R_0603_1608Metric, F.Cu at (78.0, 54.1)
- added R53: 357k 0.1%, Resistor_SMD:R_0603_1608Metric, F.Cu at (74.5, 54.1)
- added R54: 78.7k 0.1%, Resistor_SMD:R_0603_1608Metric, F.Cu at (75.7, 56.7)
- added R55: 100k, Resistor_SMD:R_0603_1608Metric, F.Cu at (52.6, 90.3)
- added R56: 200k 0.1%, Resistor_SMD:R_0603_1608Metric, F.Cu at (54.5, 87.8)
- added R57: 274k 0.1%, Resistor_SMD:R_0603_1608Metric, F.Cu at (55.2, 90.3)
- added R58: 42.2k 0.1%, Resistor_SMD:R_0603_1608Metric, F.Cu at (58.0, 87.8)
- added R59: 357k 0.1%, Resistor_SMD:R_0603_1608Metric, F.Cu at (61.5, 87.8)
- added R6: 10k, Resistor_SMD:R_0603_1608Metric, F.Cu at (61.3, 77.8)
- added R60: 78.7k 0.1%, Resistor_SMD:R_0603_1608Metric, F.Cu at (60.3, 90.3)
- added R61: 100k, Resistor_SMD:R_0603_1608Metric, F.Cu at (52.6, 96.7)
- added R62: 200k 0.1%, Resistor_SMD:R_0603_1608Metric, F.Cu at (54.5, 99.2)
- added R63: 274k 0.1%, Resistor_SMD:R_0603_1608Metric, F.Cu at (55.2, 96.7)
- added R64: 42.2k 0.1%, Resistor_SMD:R_0603_1608Metric, F.Cu at (58.0, 99.2)
- added R65: 357k 0.1%, Resistor_SMD:R_0603_1608Metric, F.Cu at (61.5, 99.2)
- added R66: 78.7k 0.1%, Resistor_SMD:R_0603_1608Metric, F.Cu at (60.3, 96.7)
- added R67: 100k, Resistor_SMD:R_0603_1608Metric, F.Cu at (83.4, 96.7)
- added R68: 200k 0.1%, Resistor_SMD:R_0603_1608Metric, F.Cu at (81.5, 99.2)
- added R69: 274k 0.1%, Resistor_SMD:R_0603_1608Metric, F.Cu at (80.8, 96.7)
- added R7: 20k 0.1%, Resistor_SMD:R_0603_1608Metric, F.Cu at (65.4, 77.3)
- added R70: 42.2k 0.1%, Resistor_SMD:R_0603_1608Metric, F.Cu at (78.0, 99.2)
- added R71: 357k 0.1%, Resistor_SMD:R_0603_1608Metric, F.Cu at (74.5, 99.2)
- added R72: 78.7k 0.1%, Resistor_SMD:R_0603_1608Metric, F.Cu at (75.7, 96.7)
- added R73: 56.2k, Resistor_SMD:R_0603_1608Metric, F.Cu at (77.5, 92.6)
- added R74: 22k, Resistor_SMD:R_0603_1608Metric, F.Cu at (54.6, 79.9)
- added R75: 22k, Resistor_SMD:R_0603_1608Metric, F.Cu at (54.6, 112.9)
- added R8: 220, Resistor_SMD:R_0603_1608Metric, F.Cu at (68.6, 77.3)
- added R9: 20k 0.1%, Resistor_SMD:R_0603_1608Metric, F.Cu at (60.1, 83.8)
- added TH1: NTC 47k, PCM_Resistor_THT_AKL:R_Axial_DIN0207_L6.3mm_D2.5mm_P2.54mm_Vertical, B.Cu at (52.1, 71.0)
- added TH2: NTC 47k, PCM_Resistor_THT_AKL:R_Axial_DIN0207_L6.3mm_D2.5mm_P2.54mm_Vertical, B.Cu at (52.1, 74.2)
- added TH3: NTC 47k, PCM_Resistor_THT_AKL:R_Axial_DIN0207_L6.3mm_D2.5mm_P2.54mm_Vertical, B.Cu at (83.8, 71.0)
- added TH4: NTC 47k, PCM_Resistor_THT_AKL:R_Axial_DIN0207_L6.3mm_D2.5mm_P2.54mm_Vertical, B.Cu at (83.8, 74.2)
- added TH5: NTC 47k, PCM_Resistor_THT_AKL:R_Axial_DIN0207_L6.3mm_D2.5mm_P2.54mm_Vertical, B.Cu at (52.1, 104.0)
- added TH6: NTC 47k, PCM_Resistor_THT_AKL:R_Axial_DIN0207_L6.3mm_D2.5mm_P2.54mm_Vertical, B.Cu at (52.1, 107.2)
- added TH7: NTC 47k, PCM_Resistor_THT_AKL:R_Axial_DIN0207_L6.3mm_D2.5mm_P2.54mm_Vertical, B.Cu at (83.8, 104.0)
- added U1: SSI2164, My Footprints:SSI2164_breakout, B.Cu at (61.6, 79.8)
- added U2: SSI2164, My Footprints:SSI2164_breakout, B.Cu at (61.6, 113.1)
- added U3: OPA1679, Package_SO:TSSOP-14_4.4x5mm_P0.65mm, F.Cu at (68.0, 82.0)
- added U4: OPA1679, Package_SO:TSSOP-14_4.4x5mm_P0.65mm, F.Cu at (68.0, 115.0)
- added U5: OPA4197, Package_SO:SOIC-14_3.9x8.7mm_P1.27mm, F.Cu at (68.0, 59.9)
- added U6: OPA4197, Package_SO:SOIC-14_3.9x8.7mm_P1.27mm, F.Cu at (68.0, 93.5)
- added U7: ADR5041, Package_TO_SOT_SMD:SOT-23, F.Cu at (76.2, 89.4)
Routing:
- added copper zone on B.Cu, net GND
- added copper zone on F.Cu, net GND
- added copper zone on In1.Cu, net GND
- added copper zone on In2.Cu, net GND
Other:
- board size 36 x 80 mm -> 36 x 91 mm
- board text added: "+15V GND -15V"
- board text added: "Channel SENDS Card"
- board text added: "DIGILOG"
- board text added: "POWER"
- board text added: "Skylar Evelyn Denno"

Commit message: sends pcb done guhhh
Parts:
- added REF**: LayerMarker_4_6.35x2.54mm_TextH1mm_P1.27mm_BottomMirrored, Symbol:LayerMarker_4_6.35x2.54mm_TextH1mm_P1.27mm_BottomMirrored, F.Cu at (50.9, 79.8)
- moved R50 87.1 mm to (54.4, 136.9), turned to 0 degrees
- moved R32 87.1 mm to (81.5, 136.9), turned to 180 degrees
- moved H1 85.5 mm to (67.8, 138.2), turned to 180 degrees
- moved R52 85.1 mm to (58.0, 136.9), turned to 0 degrees
- moved R34 85.1 mm to (78.0, 136.9), turned to 180 degrees
- moved R53 83.8 mm to (61.5, 136.9), turned to 180 degrees
- moved R35 83.7 mm to (74.4, 136.9), turned to 0 degrees
- moved R49 83.5 mm to (52.6, 134.3), turned to 90 degrees
- moved R31 83.4 mm to (83.3, 134.3), turned to 90 degrees
- moved R51 81.7 mm to (55.1, 134.3), turned to -90 degrees
- moved R33 81.7 mm to (80.8, 134.3), turned to -90 degrees
- moved C29 80.3 mm to (57.7, 134.3), turned to 90 degrees
- moved C23 80.3 mm to (78.2, 134.3), turned to 90 degrees
- moved R54 79.1 mm to (60.2, 134.3), turned to 90 degrees
- moved R36 79.1 mm to (75.7, 134.3), turned to 90 degrees
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Routing:
- net +15V: track 0.00 -> 165.2 mm, vias 0 -> 9
- net -2V5: track 0.00 -> 133.1 mm, vias 0 -> 7
- net -15V: track 0.00 -> 124.1 mm, vias 0 -> 7
- net /VCA_DRV: track 0.00 -> 107.0 mm, vias 0 -> 5
- net CV_SEND1_L: track 0.00 -> 68.5 mm, vias 0 -> 1
- net CV_SEND1_R: track 0.00 -> 55.9 mm, vias 0 -> 2
- net /VC3L: track 0.00 -> 48.1 mm, vias 0 -> 5
- net CV_SEND3_R: track 0.00 -> 46.4 mm, vias 0 -> 1
- net CV_SEND3_L: track 0.00 -> 45.4 mm, vias 0 -> 2
- net /VC4: track 0.00 -> 40.6 mm, vias 0 -> 1
- net Net-(C33-Pad1): track 0.00 -> 39.2 mm
- net Net-(R62-Pad2): track 0.00 -> 38.0 mm
- net Net-(C29-Pad1): track 0.00 -> 37.1 mm, vias 0 -> 1
- net Net-(C31-Pad1): track 0.00 -> 36.0 mm, vias 0 -> 1
- net Net-(R56-Pad2): track 0.00 -> 35.4 mm, vias 0 -> 1
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Other:
- board size 36 x 91 mm -> 36 x 86 mm
- board text added: "REV 0, 2026"
- board text added: "RoHS"

Commit message: finished sends board fr this time ordered
Routing:
- net SEND4: track 14.9 -> 14.2 mm
Other:
- board text added: "AUDIO I/O"
- board text added: "AUD_IN SEND2_R SEND4 SEND2_L SEND3_R SEND1_R SEND3_L SEND1_L"
- board text added: "CTRL Vs"
- board text added: "CV1_L"
- board text added: "CV3_L CV1_R CV3_R CV2_L CV4 CV2_R"
